Commit message: just got error for jointName = ...  Says to use ==

File: body10.urdf (robot description, URDF)
Before this commit: robot robot, 9 links, 8 joints
Joints:
- joint Torso_BackLeg: origin xyz=0 -0.5 1 rpy=0 0 0 -> xyz=0 9.5 1 rpy=0 0 0
- joint Torso_FrontLeg: origin xyz=0 0.5 1 rpy=0 0 0 -> xyz=0 10.5 1 rpy=0 0 0
- joint Torso_LeftLeg: origin xyz=-0.5 0 1 rpy=0 0 0 -> xyz=-0.5 10 1 rpy=0 0 0
- joint Torso_RightLeg: origin xyz=0.5 0 1 rpy=0 0 0 -> xyz=0.5 10 1 rpy=0 0 0

File: body5.urdf (robot description, URDF)
Before this commit: robot robot, 9 links, 8 joints
Joints:
- joint Torso_BackLeg: origin xyz=0 -0.5 1 rpy=0 0 0 -> xyz=0 4.5 1 rpy=0 0 0
- joint Torso_FrontLeg: origin xyz=0 0.5 1 rpy=0 0 0 -> xyz=0 5.5 1 rpy=0 0 0
- joint Torso_LeftLeg: origin xyz=-0.5 0 1 rpy=0 0 0 -> xyz=-0.5 5 1 rpy=0 0 0
- joint Torso_RightLeg: origin xyz=0.5 0 1 rpy=0 0 0 -> xyz=0.5 5 1 rpy=0 0 0
