Commit message: Changed obstacles, changed bot positions

File: body0-12.urdf (robot description, URDF)
Before this commit: robot robot, 9 links, 8 joints
Joints:
- joint Torso_BackLeg: origin xyz=4 -4.5 1 rpy=0 0 0 -> xyz=0 -12.5 1 rpy=0 0 0
- joint Torso_FrontLeg: origin xyz=4 -3.5 1 rpy=0 0 0 -> xyz=0 -11.5 1 rpy=0 0 0
- joint Torso_LeftLeg: origin xyz=3.5 -4 1 rpy=0 0 0 -> xyz=-0.5 -12 1 rpy=0 0 0
- joint Torso_RightLeg: origin xyz=4.5 -4 1 rpy=0 0 0 -> xyz=0.5 -12 1 rpy=0 0 0

File: body0-20.urdf (robot description, URDF)
Before this commit: robot robot, 9 links, 8 joints
Joints:
- joint Torso_BackLeg: origin xyz=-8 -0.5 1 rpy=0 0 0 -> xyz=0 -20.5 1 rpy=0 0 0
- joint Torso_FrontLeg: origin xyz=-8 0.5 1 rpy=0 0 0 -> xyz=0 -19.5 1 rpy=0 0 0
- joint Torso_LeftLeg: origin xyz=-8.5 0 1 rpy=0 0 0 -> xyz=-0.5 -20 1 rpy=0 0 0
- joint Torso_RightLeg: origin xyz=-7.5 0 1 rpy=0 0 0 -> xyz=0.5 -20 1 rpy=0 0 0

File: body0-28.urdf (robot description, URDF)
Before this commit: robot robot, 9 links, 8 joints
Joints:
- joint Torso_BackLeg: origin xyz=-4 3.5 1 rpy=0 0 0 -> xyz=0 -28.5 1 rpy=0 0 0
- joint Torso_FrontLeg: origin xyz=-4 4.5 1 rpy=0 0 0 -> xyz=0 -27.5 1 rpy=0 0 0
- joint Torso_LeftLeg: origin xyz=-4.5 4 1 rpy=0 0 0 -> xyz=-0.5 -28 1 rpy=0 0 0
- joint Torso_RightLeg: origin xyz=-3.5 4 1 rpy=0 0 0 -> xyz=0.5 -28 1 rpy=0 0 0

File: body0-36.urdf (robot description, URDF)
Before this commit: robot robot, 9 links, 8 joints
Joints:
- joint Torso_BackLeg: origin xyz=0 -0.5 1 rpy=0 0 0 -> xyz=0 -36.5 1 rpy=0 0 0
- joint Torso_FrontLeg: origin xyz=0 0.5 1 rpy=0 0 0 -> xyz=0 -35.5 1 rpy=0 0 0
- joint Torso_LeftLeg: origin xyz=-0.5 0 1 rpy=0 0 0 -> xyz=-0.5 -36 1 rpy=0 0 0
- joint Torso_RightLeg: origin xyz=0.5 0 1 rpy=0 0 0 -> xyz=0.5 -36 1 rpy=0 0 0

File: body0-4.urdf (robot description, URDF)
Before this commit: robot robot, 9 links, 8 joints
Joints:
- joint Torso_BackLeg: origin xyz=4 -0.5 1 rpy=0 0 0 -> xyz=0 -4.5 1 rpy=0 0 0
- joint Torso_FrontLeg: origin xyz=4 0.5 1 rpy=0 0 0 -> xyz=0 -3.5 1 rpy=0 0 0
- joint Torso_LeftLeg: origin xyz=3.5 0 1 rpy=0 0 0 -> xyz=-0.5 -4 1 rpy=0 0 0
- joint Torso_RightLeg: origin xyz=4.5 0 1 rpy=0 0 0 -> xyz=0.5 -4 1 rpy=0 0 0

File: body012.urdf (robot description, URDF)
Before this commit: robot robot, 9 links, 8 joints
Joints:
- joint Torso_BackLeg: origin xyz=-4 -4.5 1 rpy=0 0 0 -> xyz=0 11.5 1 rpy=0 0 0
- joint Torso_FrontLeg: origin xyz=-4 -3.5 1 rpy=0 0 0 -> xyz=0 12.5 1 rpy=0 0 0
- joint Torso_LeftLeg: origin xyz=-4.5 -4 1 rpy=0 0 0 -> xyz=-0.5 12 1 rpy=0 0 0
- joint Torso_RightLeg: origin xyz=-3.5 -4 1 rpy=0 0 0 -> xyz=0.5 12 1 rpy=0 0 0

File: body020.urdf (robot description, URDF)
Before this commit: robot robot, 9 links, 8 joints
Joints:
- joint Torso_BackLeg: origin xyz=0 -8.5 1 rpy=0 0 0 -> xyz=0 19.5 1 rpy=0 0 0
- joint Torso_FrontLeg: origin xyz=0 -7.5 1 rpy=0 0 0 -> xyz=0 20.5 1 rpy=0 0 0
- joint Torso_LeftLeg: origin xyz=-0.5 -8 1 rpy=0 0 0 -> xyz=-0.5 20 1 rpy=0 0 0
- joint Torso_RightLeg: origin xyz=0.5 -8 1 rpy=0 0 0 -> xyz=0.5 20 1 rpy=0 0 0

File: body028.urdf (robot description, URDF)
Before this commit: robot robot, 9 links, 8 joints
Joints:
- joint Torso_BackLeg: origin xyz=4 3.5 1 rpy=0 0 0 -> xyz=0 27.5 1 rpy=0 0 0
- joint Torso_FrontLeg: origin xyz=4 4.5 1 rpy=0 0 0 -> xyz=0 28.5 1 rpy=0 0 0
- joint Torso_LeftLeg: origin xyz=3.5 4 1 rpy=0 0 0 -> xyz=-0.5 28 1 rpy=0 0 0
- joint Torso_RightLeg: origin xyz=4.5 4 1 rpy=0 0 0 -> xyz=0.5 28 1 rpy=0 0 0

File: body036.urdf (robot description, URDF)
Before this commit: robot robot, 9 links, 8 joints
Joints:
- joint Torso_BackLeg: origin xyz=0 7.5 1 rpy=0 0 0 -> xyz=0 35.5 1 rpy=0 0 0
- joint Torso_FrontLeg: origin xyz=0 8.5 1 rpy=0 0 0 -> xyz=0 36.5 1 rpy=0 0 0
- joint Torso_LeftLeg: origin xyz=-0.5 8 1 rpy=0 0 0 -> xyz=-0.5 36 1 rpy=0 0 0
- joint Torso_RightLeg: origin xyz=0.5 8 1 rpy=0 0 0 -> xyz=0.5 36 1 rpy=0 0 0

File: body04.urdf (robot description, URDF)
Before this commit: robot robot, 9 links, 8 joints
Joints:
- joint Torso_BackLeg: origin xyz=0 -0.5 1 rpy=0 0 0 -> xyz=0 3.5 1 rpy=0 0 0
- joint Torso_FrontLeg: origin xyz=0 0.5 1 rpy=0 0 0 -> xyz=0 4.5 1 rpy=0 0 0
- joint Torso_LeftLeg: origin xyz=-0.5 0 1 rpy=0 0 0 -> xyz=-0.5 4 1 rpy=0 0 0
- joint Torso_RightLeg: origin xyz=0.5 0 1 rpy=0 0 0 -> xyz=0.5 4 1 rpy=0 0 0
