Commit message: quadruped robot

File: body.urdf (robot description, URDF)
Before this commit: robot robot, 3 links, 2 joints
Links:
- added link BackLowerLeg, mass 1; collision box size=0.2 0.2 1; visual box size=0.2 0.2 1
- added link FrontLowerLeg, mass 1; collision box size=0.2 0.2 1; visual box size=0.2 0.2 1
- added link LeftLeg, mass 1; collision box size=1 0.2 0.2; visual box size=1 0.2 0.2
- added link LeftLowerLeg, mass 1; collision box size=0.2 0.2 1; visual box size=0.2 0.2 1
- added link RightLeg, mass 1; collision box size=1 0.2 0.2; visual box size=1 0.2 0.2
- added link RightLowerLeg, mass 1; collision box size=0.2 0.2 1; visual box size=0.2 0.2 1
- link BackLeg: geometry collision box size=0.2 1 0.2; visual box size=0.2 1 0.2
- link FrontLeg: geometry collision box size=0.2 1 0.2; visual box size=0.2 1 0.2
Joints:
- added joint BackLeg_BackLowerLeg: type revolute, parent BackLeg, child BackLowerLeg, origin xyz=0 -1 0 rpy=0 0 0, axis 1 0 1, limit lower=-3.14159 upper=3.14159 effort=0.0 velocity=0.0
- added joint FrontLeg_FrontLowerLeg: type revolute, parent FrontLeg, child FrontLowerLeg, origin xyz=0 1 0 rpy=0 0 0, axis 1 0 1, limit lower=-3.14159 upper=3.14159 effort=0.0 velocity=0.0
- added joint LeftLeg_LeftLowerLeg: type revolute, parent LeftLeg, child LeftLowerLeg, origin xyz=-1 0 0 rpy=0 0 0, axis 0 1 1, limit lower=-3.14159 upper=3.14159 effort=0.0 velocity=0.0
- added joint RightLeg_RightLowerLeg: type revolute, parent RightLeg, child RightLowerLeg, origin xyz=1 0 0 rpy=0 0 0, axis 0 1 1, limit lower=-3.14159 upper=3.14159 effort=0.0 velocity=0.0
- added joint Torso_LeftLeg: type revolute, parent Torso, child LeftLeg, origin xyz=-0.5 0 1 rpy=0 0 0, axis 0 1 1, limit lower=-3.14159 upper=3.14159 effort=0.0 velocity=0.0
- added joint Torso_RightLeg: type revolute, parent Torso, child RightLeg, origin xyz=0.5 0 1 rpy=0 0 0, axis 0 1 1, limit lower=-3.14159 upper=3.14159 effort=0.0 velocity=0.0
- joint Torso_BackLeg: axis 0 1 0 -> 1 0 1; origin xyz=1 0 1 rpy=0 0 0 -> xyz=0 -0.5 1 rpy=0 0 0
- joint Torso_FrontLeg: axis 0 1 0 -> 1 0 1; origin xyz=2 0 1 rpy=0 0 0 -> xyz=0 0.5 1 rpy=0 0 0

Commit message: step 15 quadruped

File: body.urdf (robot description, URDF)
Before this commit: robot robot, 3 links, 2 joints
Joints:
- joint Torso_FrontLeg: origin xyz=2 0 1 rpy=0 0 0 -> xyz=0 0.5 1 rpy=0 0 0

Commit message: step 22 quadruped

File: body.urdf (robot description, URDF)
Before this commit: robot robot, 3 links, 2 joints
Links:
- link BackLeg: geometry collision box size=0.2 1 0.2; visual box size=0.2 1 0.2
- link FrontLeg: geometry collision box size=0.2 1 0.2; visual box size=0.2 1 0.2
Joints:
- joint Torso_BackLeg: origin xyz=1 0 1 rpy=0 0 0 -> xyz=0 -0.5 1 rpy=0 0 0

Commit message: step 37 quadruped

File: body.urdf (robot description, URDF)
Before this commit: robot robot, 3 links, 2 joints
Links:
- added link LeftLeg, mass 1; collision box size=1 0.2 0.2; visual box size=1 0.2 0.2
Joints:
- added joint Torso_LeftLeg: type revolute, parent Torso, child LeftLeg, origin xyz=-0.5 0 1 rpy=0 0 0, axis 1 0 0, limit lower=-3.14159 upper=3.14159 effort=0.0 velocity=0.0

Commit message: Added position and size of all upper legs. Still need to edit Generate_Brain() accordingly

File: body.urdf (robot description, URDF)
Before this commit: robot robot, 4 links, 3 joints
Links:
- added link RightLeg, mass 1; collision box size=1 0.2 0.2; visual box size=1 0.2 0.2
Joints:
- added joint Torso_RightLeg: type revolute, parent Torso, child RightLeg, origin xyz=-0.5 0 1 rpy=0 0 0, axis 0 1 0, limit lower=-3.14159 upper=3.14159 effort=0.0 velocity=0.0
- joint Torso_LeftLeg: axis 1 0 0 -> 0 1 0

Commit message: Added BackLowerLeg quadruped

File: body.urdf (robot description, URDF)
Before this commit: robot robot, 5 links, 4 joints
Joints:
- joint Torso_RightLeg: origin xyz=-0.5 0 1 rpy=0 0 0 -> xyz=0.5 0 1 rpy=0 0 0

Commit message: changed joint type from revolute to fixed in solution.py

File: body.urdf (robot description, URDF)
Before this commit: robot robot, 9 links, 8 joints
Joints:
- joint BackLeg_BackLowerLeg: type revolute -> fixed
- joint FrontLeg_FrontLowerLeg: type revolute -> fixed
- joint LeftLeg_LeftLowerLeg: type revolute -> fixed
- joint RightLeg_RightLowerLeg: type revolute -> fixed
- joint Torso_FrontLeg: type revolute -> fixed
- joint Torso_LeftLeg: type revolute -> fixed
- joint Torso_RightLeg: type revolute -> fixed

Commit message: sphere bot

File: body.urdf (robot description, URDF)
Before this commit: robot robot, 9 links, 8 joints
Links:
- link BackLeg: geometry collision sphere radius=0.5; visual sphere radius=0.5
- link BackLowerLeg: geometry collision sphere radius=0.5; visual sphere radius=0.5
- link FrontLeg: geometry collision sphere radius=0.5; visual sphere radius=0.5
- link FrontLowerLeg: geometry collision sphere radius=0.5; visual sphere radius=0.5
- link LeftLeg: geometry collision sphere radius=0.5; visual sphere radius=0.5
- link LeftLowerLeg: geometry collision sphere radius=0.5; visual sphere radius=0.5
- link RightLeg: geometry collision sphere radius=0.5; visual sphere radius=0.5
- link RightLowerLeg: geometry collision sphere radius=0.5; visual sphere radius=0.5

Commit message: Edited solution.py to create doublesphere

File: body.urdf (robot description, URDF)
Before this commit: robot robot, 9 links, 8 joints
Links:
- removed link BackLeg
- removed link BackLowerLeg
- removed link FrontLeg
- removed link FrontLowerLeg
- removed link LeftLeg
- removed link LeftLowerLeg
- removed link RightLowerLeg
- link RightLeg: geometry collision sphere radius=0.8; visual sphere radius=0.8
Joints:
- removed joint BackLeg_BackLowerLeg
- removed joint FrontLeg_FrontLowerLeg
- removed joint LeftLeg_LeftLowerLeg
- removed joint RightLeg_RightLowerLeg
- removed joint Torso_BackLeg
- removed joint Torso_FrontLeg
- removed joint Torso_LeftLeg
- joint Torso_RightLeg: type revolute -> fixed

Commit message: small spheres, offset force

File: body.urdf (robot description, URDF)
Before this commit: robot robot, 2 links, 1 joints
Links:
- added link RightLeg2, mass 1; collision sphere radius=0.5; visual sphere radius=0.5
- link RightLeg: geometry collision sphere radius=0.5; visual sphere radius=0.5
- link Torso: geometry collision sphere radius=0.5; visual sphere radius=0.5
Joints:
- added joint RightLeg_RightLeg2: type fixed, parent RightLeg, child RightLeg2, origin xyz=1.5 0 1 rpy=0 0 0, axis 0 1 0, limit lower=-3.14159 upper=3.14159 effort=0.0 velocity=0.0

Commit message: large spheres, offset force

File: body.urdf (robot description, URDF)
Before this commit: robot robot, 3 links, 2 joints
Links:
- link RightLeg: geometry collision sphere radius=1.5; visual sphere radius=1.5
- link RightLeg2: geometry collision sphere radius=1.5; visual sphere radius=1.5
- link Torso: geometry collision sphere radius=1.5; visual sphere radius=1.5

Commit message: one leg on each side

File: body.urdf (robot description, URDF)
Before this commit: robot robot, 9 links, 8 joints
Links:
- removed link LeftLeg
- removed link LeftLowerLeg
- removed link RightLeg
- removed link RightLowerLeg
Joints:
- removed joint LeftLeg_LeftLowerLeg
- removed joint RightLeg_RightLowerLeg
- removed joint Torso_LeftLeg
- removed joint Torso_RightLeg

Commit message: here's a messed up hexapod

File: body.urdf (robot description, URDF)
Before this commit: robot robot, 5 links, 4 joints
Links:
- removed link BackLeg
- removed link BackLowerLeg
- removed link FrontLeg
- removed link FrontLowerLeg
- added link BackLeg0, mass 1; collision box size=0.2 1 0.2; visual box size=0.2 1 0.2
- added link BackLeg1, mass 1; collision box size=0.2 1 0.2; visual box size=0.2 1 0.2
- added link BackLeg2, mass 1; collision box size=0.2 1 0.2; visual box size=0.2 1 0.2
- added link BackLowerLeg0, mass 1; collision box size=0.2 0.2 1; visual box size=0.2 0.2 1
- added link BackLowerLeg1, mass 1; collision box size=0.2 0.2 1; visual box size=0.2 0.2 1
- added link BackLowerLeg2, mass 1; collision box size=0.2 0.2 1; visual box size=0.2 0.2 1
- added link FrontLeg0, mass 1; collision box size=0.2 1 0.2; visual box size=0.2 1 0.2
- added link FrontLeg1, mass 1; collision box size=0.2 1 0.2; visual box size=0.2 1 0.2
- added link FrontLeg2, mass 1; collision box size=0.2 1 0.2; visual box size=0.2 1 0.2
- added link FrontLowerLeg0, mass 1; collision box size=0.2 0.2 1; visual box size=0.2 0.2 1
- added link FrontLowerLeg1, mass 1; collision box size=0.2 0.2 1; visual box size=0.2 0.2 1
- added link FrontLowerLeg2, mass 1; collision box size=0.2 0.2 1; visual box size=0.2 0.2 1
Joints:
- removed joint BackLeg_BackLowerLeg
- removed joint FrontLeg_FrontLowerLeg
- removed joint Torso_BackLeg
- removed joint Torso_FrontLeg
- added joint BackLeg0_BackLowerLeg0: type revolute, parent BackLeg0, child BackLowerLeg0, origin xyz=0 -1 0 rpy=0 0 0, axis 1 0 0, limit lower=-3.14159 upper=3.14159 effort=0.0 velocity=0.0
- added joint BackLeg1_BackLowerLeg1: type revolute, parent BackLeg1, child BackLowerLeg1, origin xyz=0 -1 0 rpy=0 0 0, axis 1 0 0, limit lower=-3.14159 upper=3.14159 effort=0.0 velocity=0.0
- added joint BackLeg2_BackLowerLeg2: type revolute, parent BackLeg2, child BackLowerLeg2, origin xyz=0 -1 0 rpy=0 0 0, axis 1 0 0, limit lower=-3.14159 upper=3.14159 effort=0.0 velocity=0.0
- added joint FrontLeg0_FrontLowerLeg0: type revolute, parent FrontLeg0, child FrontLowerLeg0, origin xyz=0 1 0 rpy=0 0 0, axis 1 0 0, limit lower=-3.14159 upper=3.14159 effort=0.0 velocity=0.0
- added joint FrontLeg1_FrontLowerLeg1: type revolute, parent FrontLeg1, child FrontLowerLeg1, origin xyz=0 1 0 rpy=0 0 0, axis 1 0 0, limit lower=-3.14159 upper=3.14159 effort=0.0 velocity=0.0
- added joint FrontLeg2_FrontLowerLeg2: type revolute, parent FrontLeg2, child FrontLowerLeg2, origin xyz=0 1 0 rpy=0 0 0, axis 1 0 0, limit lower=-3.14159 upper=3.14159 effort=0.0 velocity=0.0
- added joint Torso_BackLeg0: type revolute, parent Torso, child BackLeg0, origin xyz=-0.4 -0.5 1 rpy=0 0 0, axis 1 0 0, limit lower=-3.14159 upper=3.14159 effort=0.0 velocity=0.0
- added joint Torso_BackLeg1: type revolute, parent Torso, child BackLeg1, origin xyz=0 -0.5 1 rpy=0 0 0, axis 1 0 0, limit lower=-3.14159 upper=3.14159 effort=0.0 velocity=0.0
- added joint Torso_BackLeg2: type revolute, parent Torso, child BackLeg2, origin xyz=0.4 -0.5 1 rpy=0 0 0, axis 1 0 0, limit lower=-3.14159 upper=3.14159 effort=0.0 velocity=0.0
- added joint Torso_FrontLeg0: type revolute, parent Torso, child FrontLeg0, origin xyz=-0.4 0.5 1 rpy=0 0 0, axis 1 0 0, limit lower=-3.14159 upper=3.14159 effort=0.0 velocity=0.0
- added joint Torso_FrontLeg1: type revolute, parent Torso, child FrontLeg1, origin xyz=0 0.5 1 rpy=0 0 0, axis 1 0 0, limit lower=-3.14159 upper=3.14159 effort=0.0 velocity=0.0
- added joint Torso_FrontLeg2: type revolute, parent Torso, child FrontLeg2, origin xyz=0.4 0.5 1 rpy=0 0 0, axis 1 0 0, limit lower=-3.14159 upper=3.14159 effort=0.0 velocity=0.0

Commit message: Here's a hexapod. Try messing with the arrangement and joints

File: body.urdf (robot description, URDF)
Before this commit: robot robot, 13 links, 12 joints
Joints:
- joint Torso_BackLeg0: axis 1 0 0 -> 0 0 1; origin xyz=-0.4 -0.5 1 rpy=0 0 0 -> xyz=-0.2 -0.5 1 rpy=0 0 0
- joint Torso_BackLeg1: axis 1 0 0 -> 0 0 1
- joint Torso_BackLeg2: axis 1 0 0 -> 0 0 1; origin xyz=0.4 -0.5 1 rpy=0 0 0 -> xyz=0.2 -0.5 1 rpy=0 0 0
- joint Torso_FrontLeg0: axis 1 0 0 -> 0 0 1; origin xyz=-0.4 0.5 1 rpy=0 0 0 -> xyz=-0.2 0.5 1 rpy=0 0 0
- joint Torso_FrontLeg1: axis 1 0 0 -> 0 0 1
- joint Torso_FrontLeg2: axis 1 0 0 -> 0 0 1; origin xyz=0.4 0.5 1 rpy=0 0 0 -> xyz=0.2 0.5 1 rpy=0 0 0; type revolute -> spherical

Commit message: Hexapod version 2.0

File: body.urdf (robot description, URDF)
Before this commit: robot robot, 13 links, 12 joints
Links:
- removed link BackLeg0
- removed link BackLeg1
- removed link BackLeg2
- removed link BackLowerLeg0
- removed link BackLowerLeg1
- removed link BackLowerLeg2
- removed link FrontLeg0
- removed link FrontLeg1
- removed link FrontLeg2
- removed link FrontLowerLeg0
- removed link FrontLowerLeg1
- removed link FrontLowerLeg2
- added link BackLeg, mass 1; collision box size=0.2 1 0.2; visual box size=0.2 1 0.2
- added link BackLowerLeg, mass 1; collision box size=0.2 0.2 1; visual box size=0.2 0.2 1
- added link FrontLeg, mass 1; collision box size=0.2 1 0.2; visual box size=0.2 1 0.2
- added link FrontLowerLeg, mass 1; collision box size=0.2 0.2 1; visual box size=0.2 0.2 1
- added link LeftLeg1, mass 1; collision box size=1 0.2 0.2; visual box size=1 0.2 0.2
- added link LeftLeg2, mass 1; collision box size=1 0.2 0.2; visual box size=1 0.2 0.2
- added link LeftLowerLeg1, mass 1; collision box size=0.2 0.2 1; visual box size=0.2 0.2 1
- added link LeftLowerLeg2, mass 1; collision box size=0.2 0.2 1; visual box size=0.2 0.2 1
- added link RightLeg1, mass 1; collision box size=1 0.2 0.2; visual box size=1 0.2 0.2
- added link RightLeg2, mass 1; collision box size=1 0.2 0.2; visual box size=1 0.2 0.2
- added link RightLowerLeg1, mass 1; collision box size=0.2 0.2 1; visual box size=0.2 0.2 1
- added link RightLowerLeg2, mass 1; collision box size=0.2 0.2 1; visual box size=0.2 0.2 1
Joints:
- removed joint BackLeg0_BackLowerLeg0
- removed joint BackLeg1_BackLowerLeg1
- removed joint BackLeg2_BackLowerLeg2
- removed joint FrontLeg0_FrontLowerLeg0
- removed joint FrontLeg1_FrontLowerLeg1
- removed joint FrontLeg2_FrontLowerLeg2
- removed joint Torso_BackLeg0
- removed joint Torso_BackLeg1
- removed joint Torso_BackLeg2
- removed joint Torso_FrontLeg0
- removed joint Torso_FrontLeg1
- removed joint Torso_FrontLeg2
- added joint BackLeg_BackLowerLeg: type revolute, parent BackLeg, child BackLowerLeg, origin xyz=0 -1 0 rpy=0 0 0, axis 1 0 0, limit lower=-3.14159 upper=3.14159 effort=0.0 velocity=0.0
- added joint FrontLeg_FrontLowerLeg: type revolute, parent FrontLeg, child FrontLowerLeg, origin xyz=0 1 0 rpy=0 0 0, axis 1 0 0, limit lower=-3.14159 upper=3.14159 effort=0.0 velocity=0.0
- added joint LeftLeg1_LeftLowerLeg1: type revolute, parent LeftLeg1, child LeftLowerLeg1, origin xyz=-1 0 0 rpy=0 0 0, axis 0 1 0, limit lower=-3.14159 upper=3.14159 effort=0.0 velocity=0.0
- added joint LeftLeg2_LeftLowerLeg2: type revolute, parent LeftLeg2, child LeftLowerLeg2, origin xyz=-1 0 0 rpy=0 0 0, axis 0 1 0, limit lower=-3.14159 upper=3.14159 effort=0.0 velocity=0.0
- added joint RightLeg1_RightLowerLeg1: type revolute, parent RightLeg1, child RightLowerLeg1, origin xyz=1 0 0 rpy=0 0 0, axis 0 1 0, limit lower=-3.14159 upper=3.14159 effort=0.0 velocity=0.0
- added joint RightLeg2_RightLowerLeg2: type revolute, parent RightLeg2, child RightLowerLeg2, origin xyz=1 0 0 rpy=0 0 0, axis 0 1 0, limit lower=-3.14159 upper=3.14159 effort=0.0 velocity=0.0
- added joint Torso_BackLeg: type revolute, parent Torso, child BackLeg, origin xyz=0 -0.5 1 rpy=0 0 0, axis 0 0 1, limit lower=-3.14159 upper=3.14159 effort=0.0 velocity=0.0
- added joint Torso_FrontLeg: type revolute, parent Torso, child FrontLeg, origin xyz=0 0.5 1 rpy=0 0 0, axis 0 0 1, limit lower=-3.14159 upper=3.14159 effort=0.0 velocity=0.0
- added joint Torso_LeftLeg1: type revolute, parent Torso, child LeftLeg1, origin xyz=-0.5 -0.2 1 rpy=0 0 0, axis 0 1 0, limit lower=-3.14159 upper=3.14159 effort=0.0 velocity=0.0
- added joint Torso_LeftLeg2: type revolute, parent Torso, child LeftLeg2, origin xyz=-0.5 0.2 1 rpy=0 0 0, axis 0 1 0, limit lower=-3.14159 upper=3.14159 effort=0.0 velocity=0.0
- added joint Torso_RightLeg1: type revolute, parent Torso, child RightLeg1, origin xyz=0.5 -0.2 1 rpy=0 0 0, axis 0 1 0, limit lower=-3.14159 upper=3.14159 effort=0.0 velocity=0.0
- added joint Torso_RightLeg2: type revolute, parent Torso, child RightLeg2, origin xyz=0.5 0.2 1 rpy=0 0 0, axis 0 1 0, limit lower=-3.14159 upper=3.14159 effort=0.0 velocity=0.0

Commit message: Here's a hexapod that walks well.

File: body.urdf (robot description, URDF)
Before this commit: robot robot, 13 links, 12 joints
Joints:
- joint Torso_BackLeg: axis 0 0 1 -> 0 1 0
- joint Torso_FrontLeg: axis 0 0 1 -> 0 1 0

Commit message: hexapod with 3 forwards and 3 backwards

File: body.urdf (robot description, URDF)
Before this commit: robot robot, 13 links, 12 joints
Links:
- removed link BackLeg
- removed link BackLowerLeg
- removed link FrontLeg
- removed link FrontLowerLeg
- added link LeftLeg0, mass 1; collision box size=1 0.2 0.2; visual box size=1 0.2 0.2
- added link LeftLowerLeg0, mass 1; collision box size=0.2 0.2 1; visual box size=0.2 0.2 1
- added link RightLeg0, mass 1; collision box size=1 0.2 0.2; visual box size=1 0.2 0.2
- added link RightLowerLeg0, mass 1; collision box size=0.2 0.2 1; visual box size=0.2 0.2 1
Joints:
- removed joint BackLeg_BackLowerLeg
- removed joint FrontLeg_FrontLowerLeg
- removed joint Torso_BackLeg
- removed joint Torso_FrontLeg
- added joint LeftLeg0_LeftLowerLeg0: type fixed, parent LeftLeg0, child LeftLowerLeg0, origin xyz=-1 0 0 rpy=0 0 0, axis 0 1 0, limit lower=-3.14159 upper=3.14159 effort=0.0 velocity=0.0
- added joint RightLeg0_RightLowerLeg0: type fixed, parent RightLeg0, child RightLowerLeg0, origin xyz=1 0 0 rpy=0 0 0, axis 0 1 0, limit lower=-3.14159 upper=3.14159 effort=0.0 velocity=0.0
- added joint Torso_LeftLeg0: type fixed, parent Torso, child LeftLeg0, origin xyz=-0.5 -0.2 1 rpy=0 0 0, axis 0 1 0, limit lower=-3.14159 upper=3.14159 effort=0.0 velocity=0.0
- added joint Torso_RightLeg0: type fixed, parent Torso, child RightLeg0, origin xyz=0.5 -0.2 1 rpy=0 0 0, axis 0 1 0, limit lower=-3.14159 upper=3.14159 effort=0.0 velocity=0.0
- joint LeftLeg1_LeftLowerLeg1: type revolute -> fixed
- joint LeftLeg2_LeftLowerLeg2: type revolute -> fixed
- joint RightLeg1_RightLowerLeg1: type revolute -> fixed
- joint Torso_LeftLeg1: origin xyz=-0.5 -0.2 1 rpy=0 0 0 -> xyz=-0.5 0 1 rpy=0 0 0; type revolute -> fixed
- joint Torso_LeftLeg2: type revolute -> fixed
- joint Torso_RightLeg1: origin xyz=0.5 -0.2 1 rpy=0 0 0 -> xyz=0.5 0 1 rpy=0 0 0; type revolute -> fixed
- joint Torso_RightLeg2: type revolute -> fixed

Commit message: quadruped with surrounding legs

File: body.urdf (robot description, URDF)
Before this commit: robot robot, 13 links, 12 joints
Links:
- removed link LeftLeg1
- removed link LeftLeg2
- removed link LeftLowerLeg1
- removed link LeftLowerLeg2
- removed link RightLeg1
- removed link RightLeg2
- removed link RightLowerLeg1
- removed link RightLowerLeg2
- added link LeftLeg, mass 1; collision box size=1 0.2 0.2; visual box size=1 0.2 0.2
- added link LeftLowerLeg, mass 1; collision box size=0.2 0.2 1; visual box size=0.2 0.2 1
- added link RightLeg, mass 1; collision box size=1 0.2 0.2; visual box size=1 0.2 0.2
- added link RightLowerLeg, mass 1; collision box size=0.2 0.2 1; visual box size=0.2 0.2 1
Joints:
- removed joint LeftLeg1_LeftLowerLeg1
- removed joint LeftLeg2_LeftLowerLeg2
- removed joint RightLeg1_RightLowerLeg1
- removed joint RightLeg2_RightLowerLeg2
- removed joint Torso_LeftLeg1
- removed joint Torso_LeftLeg2
- removed joint Torso_RightLeg1
- removed joint Torso_RightLeg2
- added joint LeftLeg_LeftLowerLeg: type revolute, parent LeftLeg, child LeftLowerLeg, origin xyz=-1 0 0 rpy=0 0 0, axis 0 1 0, limit lower=-3.14159 upper=3.14159 effort=0.0 velocity=0.0
- added joint RightLeg_RightLowerLeg: type revolute, parent RightLeg, child RightLowerLeg, origin xyz=1 0 0 rpy=0 0 0, axis 0 1 0, limit lower=-3.14159 upper=3.14159 effort=0.0 velocity=0.0
- added joint Torso_LeftLeg: type revolute, parent Torso, child LeftLeg, origin xyz=-0.5 0 1 rpy=0 0 0, axis 0 1 0, limit lower=-3.14159 upper=3.14159 effort=0.0 velocity=0.0
- added joint Torso_RightLeg: type revolute, parent Torso, child RightLeg, origin xyz=0.5 0 1 rpy=0 0 0, axis 0 1 0, limit lower=-3.14159 upper=3.14159 effort=0.0 velocity=0.0

Commit message: quadruped with 2 legs forward, 2 legs backwards relative to motion

File: body.urdf (robot description, URDF)
Before this commit: robot robot, 13 links, 12 joints
Links:
- removed link BackLeg
- removed link BackLowerLeg
- removed link FrontLeg
- removed link FrontLowerLeg
Joints:
- removed joint BackLeg_BackLowerLeg
- removed joint FrontLeg_FrontLowerLeg
- removed joint Torso_BackLeg
- removed joint Torso_FrontLeg

Commit message: elongated sphere shape. Rough design.

File: body.urdf (robot description, URDF)
Before this commit: robot robot, 3 links, 2 joints
Links:
- added link RightLeg3, mass 1; collision sphere radius=1.5; visual sphere radius=1.5
- added link RightLeg4, mass 1; collision sphere radius=1.5; visual sphere radius=1.5
- added link RightLeg5, mass 1; collision sphere radius=1.5; visual sphere radius=1.5
- added link RightLeg6, mass 1; collision sphere radius=1.5; visual sphere radius=1.5
- added link RightLeg7, mass 1; collision sphere radius=1.5; visual sphere radius=1.5
- added link RightLeg8, mass 1; collision sphere radius=1.5; visual sphere radius=1.5
Joints:
- added joint RightLeg2_RightLeg3: type fixed, parent RightLeg2, child RightLeg3, origin xyz=1 0 0 rpy=0 0 0, axis 0 1 0, limit lower=-3.14159 upper=3.14159 effort=0.0 velocity=0.0
- added joint RightLeg3_RightLeg4: type fixed, parent RightLeg3, child RightLeg4, origin xyz=1 0 0 rpy=0 0 0, axis 0 1 0, limit lower=-3.14159 upper=3.14159 effort=0.0 velocity=0.0
- added joint RightLeg4_RightLeg5: type fixed, parent RightLeg4, child RightLeg5, origin xyz=1 0 0 rpy=0 0 0, axis 0 1 0, limit lower=-3.14159 upper=3.14159 effort=0.0 velocity=0.0
- added joint RightLeg5_RightLeg6: type fixed, parent RightLeg5, child RightLeg6, origin xyz=1 0 0 rpy=0 0 0, axis 0 1 0, limit lower=-3.14159 upper=3.14159 effort=0.0 velocity=0.0
- added joint RightLeg6_RightLeg7: type fixed, parent RightLeg6, child RightLeg7, origin xyz=1 0 0 rpy=0 0 0, axis 0 1 0, limit lower=-3.14159 upper=3.14159 effort=0.0 velocity=0.0
- added joint RightLeg7_RightLeg8: type fixed, parent RightLeg7, child RightLeg8, origin xyz=1 0 0 rpy=0 0 0, axis 0 1 0, limit lower=-3.14159 upper=3.14159 effort=0.0 velocity=0.0

Commit message: elongated sphere shape.

File: body.urdf (robot description, URDF)
Before this commit: robot robot, 9 links, 8 joints
Joints:
- joint RightLeg_RightLeg2: origin xyz=1.5 0 1 rpy=0 0 0 -> xyz=1 0 1 rpy=0 0 0
- joint Torso_RightLeg: origin xyz=0.5 0 1 rpy=0 0 0 -> xyz=0 0 1 rpy=0 0 0
