Commit message: each sphere centered on upstream joint

File: body.urdf (robot description, URDF)
Before this commit: robot robot, 9 links, 8 joints
Links:
- removed link RightLeg6
- removed link RightLeg7
- removed link RightLeg8
- link RightLeg: geometry collision sphere radius=1; visual sphere radius=1
- link RightLeg2: geometry collision sphere radius=1; visual sphere radius=1
- link RightLeg3: geometry collision sphere radius=1; visual sphere radius=1
- link RightLeg4: geometry collision sphere radius=1; visual sphere radius=1
- link Torso: geometry collision sphere radius=1; visual sphere radius=1
Joints:
- removed joint RightLeg5_RightLeg6
- removed joint RightLeg6_RightLeg7
- removed joint RightLeg7_RightLeg8
- joint RightLeg2_RightLeg3: origin xyz=1 0 0 rpy=0 0 0 -> xyz=0 0 1 rpy=0 0 0
- joint RightLeg3_RightLeg4: origin xyz=1 0 0 rpy=0 0 0 -> xyz=0 1 0 rpy=0 0 0
- joint RightLeg_RightLeg2: origin xyz=1 0 1 rpy=0 0 0 -> xyz=0 0 1 rpy=0 0 0
- joint Torso_RightLeg: origin xyz=0 0 1 rpy=0 0 0 -> xyz=1 0 1 rpy=0 0 0

Commit message: Irregular conformation of spheres with irregularly distributed forces

File: body.urdf (robot description, URDF)
Before this commit: robot robot, 6 links, 5 joints
Links:
- link RightLeg5: geometry collision sphere radius=1; visual sphere radius=1

Commit message: Here's triped1. It's working.

File: body.urdf (robot description, URDF)
Before this commit: robot robot, 9 links, 8 joints
Links:
- removed link BackLeg
- removed link BackLowerLeg
Joints:
- removed joint BackLeg_BackLowerLeg
- removed joint Torso_BackLeg

Commit message: Here is triped2 body.

File: body.urdf (robot description, URDF)
Before this commit: robot robot, 13 links, 12 joints
Links:
- removed link LeftLeg0
- removed link LeftLeg2
- removed link LeftLowerLeg0
- removed link LeftLowerLeg2
- removed link RightLeg1
- removed link RightLowerLeg1
Joints:
- removed joint LeftLeg0_LeftLowerLeg0
- removed joint LeftLeg2_LeftLowerLeg2
- removed joint RightLeg1_RightLowerLeg1
- removed joint Torso_LeftLeg0
- removed joint Torso_LeftLeg2
- removed joint Torso_RightLeg1
- joint RightLeg2_RightLowerLeg2: type revolute -> fixed

Commit message: Here's triped2. It's working, and it's fast.

File: body.urdf (robot description, URDF)
Before this commit: robot robot, 7 links, 6 joints
Joints:
- joint LeftLeg1_LeftLowerLeg1: type fixed -> revolute
- joint RightLeg0_RightLowerLeg0: type fixed -> revolute
- joint RightLeg2_RightLowerLeg2: type fixed -> revolute
- joint Torso_LeftLeg1: type fixed -> revolute
- joint Torso_RightLeg0: type fixed -> revolute
- joint Torso_RightLeg2: type fixed -> revolute

Commit message: Here's pentapod1. It's working.

File: body.urdf (robot description, URDF)
Before this commit: robot robot, 13 links, 12 joints
Links:
- removed link RightLeg2
- removed link RightLowerLeg2
Joints:
- removed joint RightLeg2_RightLowerLeg2
- removed joint Torso_RightLeg2
- joint Torso_RightLeg1: origin xyz=0.5 -0.2 1 rpy=0 0 0 -> xyz=0.5 0 1 rpy=0 0 0

Commit message: Here's pentapod2. Just the body.

File: body.urdf (robot description, URDF)
Before this commit: robot robot, 13 links, 12 joints
Links:
- removed link RightLeg1
- removed link RightLowerLeg1
Joints:
- removed joint RightLeg1_RightLowerLeg1
- removed joint Torso_RightLeg1
- joint RightLeg2_RightLowerLeg2: type revolute -> fixed

Commit message: Working dish sim, no neural network

File: body.urdf (robot description, URDF)
Before this commit: robot robot, 3 links, 2 joints
Links:
- removed link BackLeg
- removed link FrontLeg
- added link RightLeg, mass 1; collision sphere radius=1; visual sphere radius=1
- added link RightLeg2, mass 1; collision sphere radius=1; visual sphere radius=1
- added link RightLeg3, mass 1; collision sphere radius=1; visual sphere radius=1
- added link RightLeg4, mass 1; collision sphere radius=1; visual sphere radius=1
- added link RightLeg5, mass 1; collision sphere radius=1; visual sphere radius=1
- link Torso: geometry collision sphere radius=1; visual sphere radius=1
Joints:
- removed joint Torso_BackLeg
- removed joint Torso_FrontLeg
- added joint RightLeg2_RightLeg3: type fixed, parent RightLeg2, child RightLeg3, origin xyz=0 0 1 rpy=0 0 0, axis 0 1 0, limit lower=-3.14159 upper=3.14159 effort=0.0 velocity=0.0
- added joint RightLeg3_RightLeg4: type fixed, parent RightLeg3, child RightLeg4, origin xyz=0 1 0 rpy=0 0 0, axis 0 1 0, limit lower=-3.14159 upper=3.14159 effort=0.0 velocity=0.0
- added joint RightLeg4_RightLeg5: type fixed, parent RightLeg4, child RightLeg5, origin xyz=1 0 0 rpy=0 0 0, axis 0 1 0, limit lower=-3.14159 upper=3.14159 effort=0.0 velocity=0.0
- added joint RightLeg_RightLeg2: type fixed, parent RightLeg, child RightLeg2, origin xyz=0 0 1 rpy=0 0 0, axis 0 1 0, limit lower=-3.14159 upper=3.14159 effort=0.0 velocity=0.0
- added joint Torso_RightLeg: type fixed, parent Torso, child RightLeg, origin xyz=1 0 1 rpy=0 0 0, axis 0 1 0, limit lower=-3.14159 upper=3.14159 effort=0.0 velocity=0.0

Commit message: IRREGULAR2

File: body.urdf (robot description, URDF)
Before this commit: robot robot, 6 links, 5 joints
Links:
- added link RightLeg6, mass 1; collision sphere radius=1; visual sphere radius=1
Joints:
- added joint RightLeg5_RightLeg6: type fixed, parent RightLeg5, child RightLeg6, origin xyz=0 0 1 rpy=0 0 0, axis 0 1 0, limit lower=-3.14159 upper=3.14159 effort=0.0 velocity=0.0

Commit message: irregular3

File: body.urdf (robot description, URDF)
Before this commit: robot robot, 7 links, 6 joints
Links:
- added link RightLeg7, mass 1; collision sphere radius=1; visual sphere radius=1
- added link RightLeg8, mass 1; collision sphere radius=1; visual sphere radius=1
Joints:
- added joint RightLeg6_RightLeg7: type fixed, parent RightLeg6, child RightLeg7, origin xyz=0 1 0 rpy=0 0 0, axis 0 1 0, limit lower=-3.14159 upper=3.14159 effort=0.0 velocity=0.0
- added joint RightLeg7_RightLeg8: type fixed, parent RightLeg7, child RightLeg8, origin xyz=1 0 0 rpy=0 0 0, axis 0 1 0, limit lower=-3.14159 upper=3.14159 effort=0.0 velocity=0.0

Commit message: irregular4

File: body.urdf (robot description, URDF)
Before this commit: robot robot, 9 links, 8 joints
Links:
- added link RightLeg10, mass 1; collision sphere radius=1; visual sphere radius=1
- added link RightLeg11, mass 1; collision sphere radius=1; visual sphere radius=1
- added link RightLeg12, mass 1; collision sphere radius=1; visual sphere radius=1
- added link RightLeg13, mass 1; collision sphere radius=1; visual sphere radius=1
- added link RightLeg9, mass 1; collision sphere radius=1; visual sphere radius=1
Joints:
- added joint RightLeg10_RightLeg11: type fixed, parent RightLeg10, child RightLeg11, origin xyz=1 0 0 rpy=0 0 0, axis 0 1 0, limit lower=-3.14159 upper=3.14159 effort=0.0 velocity=0.0
- added joint RightLeg11_RightLeg12: type fixed, parent RightLeg11, child RightLeg12, origin xyz=0 1 0 rpy=0 0 0, axis 0 1 0, limit lower=-3.14159 upper=3.14159 effort=0.0 velocity=0.0
- added joint RightLeg12_RightLeg13: type fixed, parent RightLeg12, child RightLeg13, origin xyz=0 1 0 rpy=0 0 0, axis 0 1 0, limit lower=-3.14159 upper=3.14159 effort=0.0 velocity=0.0
- added joint RightLeg8_RightLeg9: type fixed, parent RightLeg8, child RightLeg9, origin xyz=0 0 1 rpy=0 0 0, axis 0 1 0, limit lower=-3.14159 upper=3.14159 effort=0.0 velocity=0.0
- added joint RightLeg9_RightLeg10: type fixed, parent RightLeg9, child RightLeg10, origin xyz=0 1 0 rpy=0 0 0, axis 0 1 0, limit lower=-3.14159 upper=3.14159 effort=0.0 velocity=0.0

Commit message: print final xCoordinate

File: body.urdf (robot description, URDF)
Before this commit: robot robot, 11 links, 10 joints
Joints:
- joint LeftLeg0_LeftLowerLeg0: type fixed -> revolute
- joint LeftLeg1_LeftLowerLeg1: type fixed -> revolute
- joint LeftLeg2_LeftLowerLeg2: type fixed -> revolute
- joint RightLeg0_RightLowerLeg0: type fixed -> revolute
- joint RightLeg2_RightLowerLeg2: type fixed -> revolute
- joint Torso_LeftLeg0: type fixed -> revolute
- joint Torso_LeftLeg1: type fixed -> revolute
- joint Torso_LeftLeg2: type fixed -> revolute
- joint Torso_RightLeg0: type fixed -> revolute
- joint Torso_RightLeg2: type fixed -> revolute

Commit message: irregular with 22 spheres

File: body.urdf (robot description, URDF)
Before this commit: robot robot, 14 links, 13 joints
Links:
- added link RightLeg14, mass 1; collision sphere radius=1; visual sphere radius=1
- added link RightLeg15, mass 1; collision sphere radius=1; visual sphere radius=1
- added link RightLeg16, mass 1; collision sphere radius=1; visual sphere radius=1
- added link RightLeg17, mass 1; collision sphere radius=1; visual sphere radius=1
- added link RightLeg18, mass 1; collision sphere radius=1; visual sphere radius=1
- added link RightLeg19, mass 1; collision sphere radius=1; visual sphere radius=1
- added link RightLeg20, mass 1; collision sphere radius=1; visual sphere radius=1
- added link RightLeg21, mass 1; collision sphere radius=1; visual sphere radius=1
- added link RightLeg22, mass 1; collision sphere radius=1; visual sphere radius=1
Joints:
- added joint RightLeg13_RightLeg14: type fixed, parent RightLeg13, child RightLeg14, origin xyz=0 1 0 rpy=0 0 0, axis 0 1 0, limit lower=-3.14159 upper=3.14159 effort=0.0 velocity=0.0
- added joint RightLeg14_RightLeg15: type fixed, parent RightLeg14, child RightLeg15, origin xyz=0 0 1 rpy=0 0 0, axis 0 1 0, limit lower=-3.14159 upper=3.14159 effort=0.0 velocity=0.0
- added joint RightLeg15_RightLeg16: type fixed, parent RightLeg15, child RightLeg16, origin xyz=0 0 1 rpy=0 0 0, axis 0 1 0, limit lower=-3.14159 upper=3.14159 effort=0.0 velocity=0.0
- added joint RightLeg16_RightLeg17: type fixed, parent RightLeg16, child RightLeg17, origin xyz=0 1 0 rpy=0 0 0, axis 0 1 0, limit lower=-3.14159 upper=3.14159 effort=0.0 velocity=0.0
- added joint RightLeg17_RightLeg18: type fixed, parent RightLeg17, child RightLeg18, origin xyz=1 0 0 rpy=0 0 0, axis 0 1 0, limit lower=-3.14159 upper=3.14159 effort=0.0 velocity=0.0
- added joint RightLeg18_RightLeg19: type fixed, parent RightLeg18, child RightLeg19, origin xyz=0 1 0 rpy=0 0 0, axis 0 1 0, limit lower=-3.14159 upper=3.14159 effort=0.0 velocity=0.0
- added joint RightLeg19_RightLeg20: type fixed, parent RightLeg19, child RightLeg20, origin xyz=0 1 0 rpy=0 0 0, axis 0 1 0, limit lower=-3.14159 upper=3.14159 effort=0.0 velocity=0.0
- added joint RightLeg20_RightLeg21: type fixed, parent RightLeg20, child RightLeg21, origin xyz=0 0 1 rpy=0 0 0, axis 0 1 0, limit lower=-3.14159 upper=3.14159 effort=0.0 velocity=0.0
- added joint RightLeg21_RightLeg22: type fixed, parent RightLeg21, child RightLeg22, origin xyz=1 0 0 rpy=0 0 0, axis 0 1 0, limit lower=-3.14159 upper=3.14159 effort=0.0 velocity=0.0

Commit message: good constants settings. Set at 13 spheres.

File: body.urdf (robot description, URDF)
Before this commit: robot robot, 23 links, 22 joints
Links:
- removed link RightLeg13
- removed link RightLeg14
- removed link RightLeg15
- removed link RightLeg16
- removed link RightLeg17
- removed link RightLeg18
- removed link RightLeg19
- removed link RightLeg20
- removed link RightLeg21
- removed link RightLeg22
Joints:
- removed joint RightLeg12_RightLeg13
- removed joint RightLeg13_RightLeg14
- removed joint RightLeg14_RightLeg15
- removed joint RightLeg15_RightLeg16
- removed joint RightLeg16_RightLeg17
- removed joint RightLeg17_RightLeg18
- removed joint RightLeg18_RightLeg19
- removed joint RightLeg19_RightLeg20
- removed joint RightLeg20_RightLeg21
- removed joint RightLeg21_RightLeg22

Commit message: codebase for hexapod2 data collection for fitness curve

File: body.urdf (robot description, URDF)
Before this commit: robot robot, 13 links, 12 joints
Joints:
- joint LeftLeg0_LeftLowerLeg0: type fixed -> revolute
- joint LeftLeg1_LeftLowerLeg1: type fixed -> revolute
- joint LeftLeg2_LeftLowerLeg2: type fixed -> revolute
- joint RightLeg0_RightLowerLeg0: type fixed -> revolute
- joint RightLeg1_RightLowerLeg1: type fixed -> revolute
- joint Torso_LeftLeg0: type fixed -> revolute
- joint Torso_LeftLeg1: type fixed -> revolute
- joint Torso_LeftLeg2: type fixed -> revolute
- joint Torso_RightLeg0: type fixed -> revolute
- joint Torso_RightLeg1: type fixed -> revolute
- joint Torso_RightLeg2: type fixed -> revolute

Commit message: Simulation generating. X and Y coordinates being written

File: body.urdf (robot description, URDF)
Before this commit: robot robot, 13 links, 12 joints
Links:
- removed link RightLeg10
- removed link RightLeg11
- removed link RightLeg12
Joints:
- removed joint RightLeg10_RightLeg11
- removed joint RightLeg11_RightLeg12
- removed joint RightLeg9_RightLeg10

Commit message: 7 Spheres reversed circular motion during simulation

File: body.urdf (robot description, URDF)
Before this commit: robot robot, 10 links, 9 joints
Links:
- removed link RightLeg7
- removed link RightLeg8
- removed link RightLeg9
Joints:
- removed joint RightLeg6_RightLeg7
- removed joint RightLeg7_RightLeg8
- removed joint RightLeg8_RightLeg9

Commit message: done with trajectory graphs

File: body.urdf (robot description, URDF)
Before this commit: robot robot, 7 links, 6 joints
Links:
- removed link RightLeg4
- removed link RightLeg5
- removed link RightLeg6
Joints:
- removed joint RightLeg3_RightLeg4
- removed joint RightLeg4_RightLeg5
- removed joint RightLeg5_RightLeg6

Commit message: robot with customizable initial y position

File: body.urdf (robot description, URDF)
Before this commit: robot robot, 9 links, 8 joints
Joints:
- joint Torso_BackLeg: origin xyz=0 -0.5 1 rpy=0 0 0 -> xyz=0 2.5 1 rpy=0 0 0
- joint Torso_FrontLeg: origin xyz=0 0.5 1 rpy=0 0 0 -> xyz=0 3.5 1 rpy=0 0 0
- joint Torso_LeftLeg: origin xyz=-0.5 0 1 rpy=0 0 0 -> xyz=-0.5 3 1 rpy=0 0 0
- joint Torso_RightLeg: origin xyz=0.5 0 1 rpy=0 0 0 -> xyz=0.5 3 1 rpy=0 0 0

Commit message: touch sensor issue persists x2

File: body.urdf (robot description, URDF)
Before this commit: robot robot, 9 links, 8 joints
Links:
- added link Box, mass 1; collision box size=1 1 1; visual box size=1 1 1

Commit message: empty and obstacles, same fitness

File: body.urdf (robot description, URDF)
Before this commit: robot robot, 3 links, 2 joints
Joints:
- joint Torso_BackLeg: origin xyz=1 0 1 rpy=0 0 0 -> xyz=-0.5 0 1.0 rpy=0 0 0
- joint Torso_FrontLeg: origin xyz=2 0 1 rpy=0 0 0 -> xyz=0.5 0 1.0 rpy=0 0 0

Commit message: cleaning up...

File: body.urdf (robot description, URDF)
Before this commit: robot robot, 10 links, 8 joints
Links:
- removed link Box
Joints:
- joint BackLeg_BackLowerLeg: axis 1 0 0 -> 1 0 1
- joint FrontLeg_FrontLowerLeg: axis 1 0 0 -> 1 0 1
- joint LeftLeg_LeftLowerLeg: axis 0 1 0 -> 0 1 1
- joint RightLeg_RightLowerLeg: axis 0 1 0 -> 0 1 1
- joint Torso_BackLeg: axis 1 0 0 -> 1 0 1
- joint Torso_FrontLeg: axis 1 0 0 -> 1 0 1
- joint Torso_LeftLeg: axis 0 1 0 -> 0 1 1
- joint Torso_RightLeg: axis 0 1 0 -> 0 1 1
