Commit message: collected case3 with weightsFiles

File: bodyFiles/body0-1010.urdf (robot description, URDF)
Before this commit: robot robot, 9 links, 8 joints
Links:
- link BackLeg: geometry collision box size=0.2 0.9220852996555571 0.2; visual box size=0.2 0.9220852996555571 0.2
- link BackLowerLeg: geometry collision box size=0.2 0.2 1.1245765721402559; visual box size=0.2 0.2 1.1245765721402559
- link FrontLeg: geometry collision box size=0.2 0.8407882028193432 0.2; visual box size=0.2 0.8407882028193432 0.2
- link FrontLowerLeg: geometry collision box size=0.2 0.2 0.946165282118653; visual box size=0.2 0.2 0.946165282118653
- link LeftLeg: geometry collision box size=1.025487895197134 0.2 0.2; visual box size=1.025487895197134 0.2 0.2
- link LeftLowerLeg: geometry collision box size=0.2 0.2 1.049611990765326; visual box size=0.2 0.2 1.049611990765326
- link RightLeg: geometry collision box size=1.288473352944602 0.2 0.2; visual box size=1.288473352944602 0.2 0.2
- link RightLowerLeg: geometry collision box size=0.2 0.2 0.882821800308789; visual box size=0.2 0.2 0.882821800308789
Joints:
- joint BackLeg_BackLowerLeg: origin xyz=0 -1.4090852278780965 0 rpy=0 0 0 -> xyz=0 -0.9220852996555571 0 rpy=0 0 0
- joint FrontLeg_FrontLowerLeg: origin xyz=0 0.9607894874261254 0 rpy=0 0 0 -> xyz=0 0.8407882028193432 0 rpy=0 0 0
- joint LeftLeg_LeftLowerLeg: origin xyz=-1.0464030274848133 0 0 rpy=0 0 0 -> xyz=-1.025487895197134 0 0 rpy=0 0 0
- joint RightLeg_RightLowerLeg: origin xyz=1.3141739622597255 0 0 rpy=0 0 0 -> xyz=1.288473352944602 0 0 rpy=0 0 0
- joint Torso_BackLeg: origin xyz=0 -10.5 1.4090852278780965 rpy=0 0 0 -> xyz=0 -10.5 1.288473352944602 rpy=0 0 0
- joint Torso_FrontLeg: origin xyz=0 -9.5 1.4090852278780965 rpy=0 0 0 -> xyz=0 -9.5 1.288473352944602 rpy=0 0 0
- joint Torso_LeftLeg: origin xyz=-0.5 -10 1.4090852278780965 rpy=0 0 0 -> xyz=-0.5 -10 1.288473352944602 rpy=0 0 0
- joint Torso_RightLeg: origin xyz=0.5 -10 1.4090852278780965 rpy=0 0 0 -> xyz=0.5 -10 1.288473352944602 rpy=0 0 0

File: bodyFiles/body0-101034.urdf (robot description, URDF)
Before this commit: robot robot, 9 links, 8 joints
Links:
- link BackLeg: geometry collision box size=0.2 1.2121639302740672 0.2; visual box size=0.2 1.2121639302740672 0.2
- link BackLowerLeg: geometry collision box size=0.2 0.2 1.4784620830875828; visual box size=0.2 0.2 1.4784620830875828
- link FrontLeg: geometry collision box size=0.2 0.6059559934242897 0.2; visual box size=0.2 0.6059559934242897 0.2
- link FrontLowerLeg: geometry collision box size=0.2 0.2 1.217664671045292; visual box size=0.2 0.2 1.217664671045292
- link LeftLeg: geometry collision box size=1.179365430834113 0.2 0.2; visual box size=1.179365430834113 0.2 0.2
- link LeftLowerLeg: geometry collision box size=0.2 0.2 0.971088230039384; visual box size=0.2 0.2 0.971088230039384
- link RightLeg: geometry collision box size=1.1013902890178153 0.2 0.2; visual box size=1.1013902890178153 0.2 0.2
- link RightLowerLeg: geometry collision box size=0.2 0.2 0.9367734242461674; visual box size=0.2 0.2 0.9367734242461674
Joints:
- joint BackLeg_BackLowerLeg: origin xyz=0 -0.5923778854220229 0 rpy=0 0 0 -> xyz=0 -1.2121639302740672 0 rpy=0 0 0
- joint FrontLeg_FrontLowerLeg: origin xyz=0 1.4220381086240987 0 rpy=0 0 0 -> xyz=0 0.6059559934242897 0 rpy=0 0 0
- joint LeftLeg_LeftLowerLeg: origin xyz=-0.5985178371821482 0 0 rpy=0 0 0 -> xyz=-1.179365430834113 0 0 rpy=0 0 0
- joint RightLeg_RightLowerLeg: origin xyz=0.7599267928344847 0 0 rpy=0 0 0 -> xyz=1.1013902890178153 0 0 rpy=0 0 0
- joint Torso_BackLeg: origin xyz=0 -10.5 1.4957065423903753 rpy=0 0 0 -> xyz=0 -10.5 1.4784620830875828 rpy=0 0 0
- joint Torso_FrontLeg: origin xyz=0 -9.5 1.4957065423903753 rpy=0 0 0 -> xyz=0 -9.5 1.4784620830875828 rpy=0 0 0
- joint Torso_LeftLeg: origin xyz=-0.5 -10 1.4957065423903753 rpy=0 0 0 -> xyz=-0.5 -10 1.4784620830875828 rpy=0 0 0
- joint Torso_RightLeg: origin xyz=0.5 -10 1.4957065423903753 rpy=0 0 0 -> xyz=0.5 -10 1.4784620830875828 rpy=0 0 0

File: bodyFiles/body0-10104.urdf (robot description, URDF)
Before this commit: robot robot, 9 links, 8 joints
Links:
- link BackLeg: geometry collision box size=0.2 1.0721545735055709 0.2; visual box size=0.2 1.0721545735055709 0.2
- link BackLowerLeg: geometry collision box size=0.2 0.2 1.3366922788169435; visual box size=0.2 0.2 1.3366922788169435
- link FrontLeg: geometry collision box size=0.2 1.1368756145736665 0.2; visual box size=0.2 1.1368756145736665 0.2
- link FrontLowerLeg: geometry collision box size=0.2 0.2 1.0237443778373936; visual box size=0.2 0.2 1.0237443778373936
- link LeftLeg: geometry collision box size=0.6711257136467211 0.2 0.2; visual box size=0.6711257136467211 0.2 0.2
- link LeftLowerLeg: geometry collision box size=0.2 0.2 0.8227359875420476; visual box size=0.2 0.2 0.8227359875420476
- link RightLeg: geometry collision box size=0.8638017792838052 0.2 0.2; visual box size=0.8638017792838052 0.2 0.2
- link RightLowerLeg: geometry collision box size=0.2 0.2 0.7075216837056069; visual box size=0.2 0.2 0.7075216837056069
Joints:
- joint BackLeg_BackLowerLeg: origin xyz=0 -0.5397208110596992 0 rpy=0 0 0 -> xyz=0 -1.0721545735055709 0 rpy=0 0 0
- joint FrontLeg_FrontLowerLeg: origin xyz=0 0.6047284848980241 0 rpy=0 0 0 -> xyz=0 1.1368756145736665 0 rpy=0 0 0
- joint LeftLeg_LeftLowerLeg: origin xyz=-1.3936995986964509 0 0 rpy=0 0 0 -> xyz=-0.6711257136467211 0 0 rpy=0 0 0
- joint RightLeg_RightLowerLeg: origin xyz=0.69259729102041 0 0 rpy=0 0 0 -> xyz=0.8638017792838052 0 0 rpy=0 0 0
- joint Torso_BackLeg: origin xyz=0 -10.5 1.3936995986964509 rpy=0 0 0 -> xyz=0 -10.5 1.3366922788169435 rpy=0 0 0
- joint Torso_FrontLeg: origin xyz=0 -9.5 1.3936995986964509 rpy=0 0 0 -> xyz=0 -9.5 1.3366922788169435 rpy=0 0 0
- joint Torso_LeftLeg: origin xyz=-0.5 -10 1.3936995986964509 rpy=0 0 0 -> xyz=-0.5 -10 1.3366922788169435 rpy=0 0 0
- joint Torso_RightLeg: origin xyz=0.5 -10 1.3936995986964509 rpy=0 0 0 -> xyz=0.5 -10 1.3366922788169435 rpy=0 0 0

File: bodyFiles/body0-101065.urdf (robot description, URDF)
Before this commit: robot robot, 9 links, 8 joints
Links:
- link BackLeg: geometry collision box size=0.2 1.2014125987006175 0.2; visual box size=0.2 1.2014125987006175 0.2
- link BackLowerLeg: geometry collision box size=0.2 0.2 0.9487882272285714; visual box size=0.2 0.2 0.9487882272285714
- link FrontLeg: geometry collision box size=0.2 1.3564532170111852 0.2; visual box size=0.2 1.3564532170111852 0.2
- link FrontLowerLeg: geometry collision box size=0.2 0.2 0.8871036827098103; visual box size=0.2 0.2 0.8871036827098103
- link LeftLeg: geometry collision box size=1.1087719306563486 0.2 0.2; visual box size=1.1087719306563486 0.2 0.2
- link LeftLowerLeg: geometry collision box size=0.2 0.2 1.0246539284896468; visual box size=0.2 0.2 1.0246539284896468
- link RightLeg: geometry collision box size=1.0009863054677388 0.2 0.2; visual box size=1.0009863054677388 0.2 0.2
- link RightLowerLeg: geometry collision box size=0.2 0.2 1.2286543019756284; visual box size=0.2 0.2 1.2286543019756284
Joints:
- joint BackLeg_BackLowerLeg: origin xyz=0 -0.5128842321711606 0 rpy=0 0 0 -> xyz=0 -1.2014125987006175 0 rpy=0 0 0
- joint FrontLeg_FrontLowerLeg: origin xyz=0 1.1280303355430767 0 rpy=0 0 0 -> xyz=0 1.3564532170111852 0 rpy=0 0 0
- joint LeftLeg_LeftLowerLeg: origin xyz=-1.1534798057734803 0 0 rpy=0 0 0 -> xyz=-1.1087719306563486 0 0 rpy=0 0 0
- joint RightLeg_RightLowerLeg: origin xyz=1.286705025156039 0 0 rpy=0 0 0 -> xyz=1.0009863054677388 0 0 rpy=0 0 0
- joint Torso_BackLeg: origin xyz=0 -10.5 1.4891646916608474 rpy=0 0 0 -> xyz=0 -10.5 1.3564532170111852 rpy=0 0 0
- joint Torso_FrontLeg: origin xyz=0 -9.5 1.4891646916608474 rpy=0 0 0 -> xyz=0 -9.5 1.3564532170111852 rpy=0 0 0
- joint Torso_LeftLeg: origin xyz=-0.5 -10 1.4891646916608474 rpy=0 0 0 -> xyz=-0.5 -10 1.3564532170111852 rpy=0 0 0
- joint Torso_RightLeg: origin xyz=0.5 -10 1.4891646916608474 rpy=0 0 0 -> xyz=0.5 -10 1.3564532170111852 rpy=0 0 0

File: bodyFiles/body0-10137.urdf (robot description, URDF)
Before this commit: robot robot, 9 links, 8 joints
Links:
- link BackLeg: geometry collision box size=0.2 0.5594391134313723 0.2; visual box size=0.2 0.5594391134313723 0.2
- link BackLowerLeg: geometry collision box size=0.2 0.2 1.445220661331586; visual box size=0.2 0.2 1.445220661331586
- link FrontLeg: geometry collision box size=0.2 1.0702214467159612 0.2; visual box size=0.2 1.0702214467159612 0.2
- link FrontLowerLeg: geometry collision box size=0.2 0.2 0.6875286270712239; visual box size=0.2 0.2 0.6875286270712239
- link LeftLeg: geometry collision box size=1.0258866049401933 0.2 0.2; visual box size=1.0258866049401933 0.2 0.2
- link LeftLowerLeg: geometry collision box size=0.2 0.2 1.3473355448288817; visual box size=0.2 0.2 1.3473355448288817
- link RightLeg: geometry collision box size=1.3526570170962389 0.2 0.2; visual box size=1.3526570170962389 0.2 0.2
- link RightLowerLeg: geometry collision box size=0.2 0.2 0.681581902101156; visual box size=0.2 0.2 0.681581902101156
Joints:
- joint BackLeg_BackLowerLeg: origin xyz=0 -1.4721250780708013 0 rpy=0 0 0 -> xyz=0 -0.5594391134313723 0 rpy=0 0 0
- joint FrontLeg_FrontLowerLeg: origin xyz=0 1.0055909513291912 0 rpy=0 0 0 -> xyz=0 1.0702214467159612 0 rpy=0 0 0
- joint LeftLeg_LeftLowerLeg: origin xyz=-0.6423330482956809 0 0 rpy=0 0 0 -> xyz=-1.0258866049401933 0 0 rpy=0 0 0
- joint RightLeg_RightLowerLeg: origin xyz=1.4545113997002583 0 0 rpy=0 0 0 -> xyz=1.3526570170962389 0 0 rpy=0 0 0
- joint Torso_BackLeg: origin xyz=0 -10.5 1.4973523409786937 rpy=0 0 0 -> xyz=0 -10.5 1.445220661331586 rpy=0 0 0
- joint Torso_FrontLeg: origin xyz=0 -9.5 1.4973523409786937 rpy=0 0 0 -> xyz=0 -9.5 1.445220661331586 rpy=0 0 0
- joint Torso_LeftLeg: origin xyz=-0.5 -10 1.4973523409786937 rpy=0 0 0 -> xyz=-0.5 -10 1.445220661331586 rpy=0 0 0
- joint Torso_RightLeg: origin xyz=0.5 -10 1.4973523409786937 rpy=0 0 0 -> xyz=0.5 -10 1.445220661331586 rpy=0 0 0

File: bodyFiles/body0-10168.urdf (robot description, URDF)
Before this commit: robot robot, 9 links, 8 joints
Links:
- link BackLeg: geometry collision box size=0.2 0.9416800575213753 0.2; visual box size=0.2 0.9416800575213753 0.2
- link BackLowerLeg: geometry collision box size=0.2 0.2 0.8958877605180859; visual box size=0.2 0.2 0.8958877605180859
- link FrontLeg: geometry collision box size=0.2 1.0921333390596577 0.2; visual box size=0.2 1.0921333390596577 0.2
- link FrontLowerLeg: geometry collision box size=0.2 0.2 1.4310011010000352; visual box size=0.2 0.2 1.4310011010000352
- link LeftLeg: geometry collision box size=0.995672951487715 0.2 0.2; visual box size=0.995672951487715 0.2 0.2
- link LeftLowerLeg: geometry collision box size=0.2 0.2 1.1608982034687818; visual box size=0.2 0.2 1.1608982034687818
- link RightLeg: geometry collision box size=0.7323130582972708 0.2 0.2; visual box size=0.7323130582972708 0.2 0.2
- link RightLowerLeg: geometry collision box size=0.2 0.2 0.8399138770242728; visual box size=0.2 0.2 0.8399138770242728
Joints:
- joint BackLeg_BackLowerLeg: origin xyz=0 -0.8957992395330023 0 rpy=0 0 0 -> xyz=0 -0.9416800575213753 0 rpy=0 0 0
- joint FrontLeg_FrontLowerLeg: origin xyz=0 0.6213552899976392 0 rpy=0 0 0 -> xyz=0 1.0921333390596577 0 rpy=0 0 0
- joint LeftLeg_LeftLowerLeg: origin xyz=-0.8750656020765538 0 0 rpy=0 0 0 -> xyz=-0.995672951487715 0 0 rpy=0 0 0
- joint RightLeg_RightLowerLeg: origin xyz=0.7330579563271648 0 0 rpy=0 0 0 -> xyz=0.7323130582972708 0 0 rpy=0 0 0
- joint Torso_BackLeg: origin xyz=0 -10.5 1.3772509060821092 rpy=0 0 0 -> xyz=0 -10.5 1.4310011010000352 rpy=0 0 0
- joint Torso_FrontLeg: origin xyz=0 -9.5 1.3772509060821092 rpy=0 0 0 -> xyz=0 -9.5 1.4310011010000352 rpy=0 0 0
- joint Torso_LeftLeg: origin xyz=-0.5 -10 1.3772509060821092 rpy=0 0 0 -> xyz=-0.5 -10 1.4310011010000352 rpy=0 0 0
- joint Torso_RightLeg: origin xyz=0.5 -10 1.3772509060821092 rpy=0 0 0 -> xyz=0.5 -10 1.4310011010000352 rpy=0 0 0

File: bodyFiles/body0-10205.urdf (robot description, URDF)
Before this commit: robot robot, 9 links, 8 joints
Links:
- link BackLeg: geometry collision box size=0.2 1.0531876928403774 0.2; visual box size=0.2 1.0531876928403774 0.2
- link BackLowerLeg: geometry collision box size=0.2 0.2 1.3854644206679805; visual box size=0.2 0.2 1.3854644206679805
- link FrontLeg: geometry collision box size=0.2 0.7243964375335676 0.2; visual box size=0.2 0.7243964375335676 0.2
- link FrontLowerLeg: geometry collision box size=0.2 0.2 0.8013610990154632; visual box size=0.2 0.2 0.8013610990154632
- link LeftLeg: geometry collision box size=1.418683228986751 0.2 0.2; visual box size=1.418683228986751 0.2 0.2
- link LeftLowerLeg: geometry collision box size=0.2 0.2 0.9625551305724173; visual box size=0.2 0.2 0.9625551305724173
- link RightLeg: geometry collision box size=0.7067867675623617 0.2 0.2; visual box size=0.7067867675623617 0.2 0.2
- link RightLowerLeg: geometry collision box size=0.2 0.2 0.9210663934555833; visual box size=0.2 0.2 0.9210663934555833
Joints:
- joint BackLeg_BackLowerLeg: origin xyz=0 -1.0152702177774107 0 rpy=0 0 0 -> xyz=0 -1.0531876928403774 0 rpy=0 0 0
- joint FrontLeg_FrontLowerLeg: origin xyz=0 1.1818595440357793 0 rpy=0 0 0 -> xyz=0 0.7243964375335676 0 rpy=0 0 0
- joint LeftLeg_LeftLowerLeg: origin xyz=-1.1109999044337173 0 0 rpy=0 0 0 -> xyz=-1.418683228986751 0 0 rpy=0 0 0
- joint RightLeg_RightLowerLeg: origin xyz=0.6586882960173703 0 0 rpy=0 0 0 -> xyz=0.7067867675623617 0 0 rpy=0 0 0
- joint Torso_BackLeg: origin xyz=0 -10.5 1.4419235970029254 rpy=0 0 0 -> xyz=0 -10.5 1.418683228986751 rpy=0 0 0
- joint Torso_FrontLeg: origin xyz=0 -9.5 1.4419235970029254 rpy=0 0 0 -> xyz=0 -9.5 1.418683228986751 rpy=0 0 0
- joint Torso_LeftLeg: origin xyz=-0.5 -10 1.4419235970029254 rpy=0 0 0 -> xyz=-0.5 -10 1.418683228986751 rpy=0 0 0
- joint Torso_RightLeg: origin xyz=0.5 -10 1.4419235970029254 rpy=0 0 0 -> xyz=0.5 -10 1.418683228986751 rpy=0 0 0

File: bodyFiles/body0-10238.urdf (robot description, URDF)
Before this commit: robot robot, 9 links, 8 joints
Links:
- link BackLeg: geometry collision box size=0.2 0.8327554538610643 0.2; visual box size=0.2 0.8327554538610643 0.2
- link BackLowerLeg: geometry collision box size=0.2 0.2 1.2044278043597811; visual box size=0.2 0.2 1.2044278043597811
- link FrontLeg: geometry collision box size=0.2 1.3021422239376534 0.2; visual box size=0.2 1.3021422239376534 0.2
- link FrontLowerLeg: geometry collision box size=0.2 0.2 0.7752448218869075; visual box size=0.2 0.2 0.7752448218869075
- link LeftLeg: geometry collision box size=1.0901289197527808 0.2 0.2; visual box size=1.0901289197527808 0.2 0.2
- link LeftLowerLeg: geometry collision box size=0.2 0.2 0.6152279341066635; visual box size=0.2 0.2 0.6152279341066635
- link RightLeg: geometry collision box size=0.5322753933926542 0.2 0.2; visual box size=0.5322753933926542 0.2 0.2
- link RightLowerLeg: geometry collision box size=0.2 0.2 0.8634277020237884; visual box size=0.2 0.2 0.8634277020237884
Joints:
- joint BackLeg_BackLowerLeg: origin xyz=0 -1.308238766062125 0 rpy=0 0 0 -> xyz=0 -0.8327554538610643 0 rpy=0 0 0
- joint FrontLeg_FrontLowerLeg: origin xyz=0 0.5100555829531151 0 rpy=0 0 0 -> xyz=0 1.3021422239376534 0 rpy=0 0 0
- joint LeftLeg_LeftLowerLeg: origin xyz=-1.2821848322522111 0 0 rpy=0 0 0 -> xyz=-1.0901289197527808 0 0 rpy=0 0 0
- joint RightLeg_RightLowerLeg: origin xyz=0.5462528743233537 0 0 rpy=0 0 0 -> xyz=0.5322753933926542 0 0 rpy=0 0 0
- joint Torso_BackLeg: origin xyz=0 -10.5 1.3355874681841438 rpy=0 0 0 -> xyz=0 -10.5 1.3021422239376534 rpy=0 0 0
- joint Torso_FrontLeg: origin xyz=0 -9.5 1.3355874681841438 rpy=0 0 0 -> xyz=0 -9.5 1.3021422239376534 rpy=0 0 0
- joint Torso_LeftLeg: origin xyz=-0.5 -10 1.3355874681841438 rpy=0 0 0 -> xyz=-0.5 -10 1.3021422239376534 rpy=0 0 0
- joint Torso_RightLeg: origin xyz=0.5 -10 1.3355874681841438 rpy=0 0 0 -> xyz=0.5 -10 1.3021422239376534 rpy=0 0 0

File: bodyFiles/body0-10270.urdf (robot description, URDF)
Before this commit: robot robot, 9 links, 8 joints
Links:
- link BackLeg: geometry collision box size=0.2 0.9598225911765685 0.2; visual box size=0.2 0.9598225911765685 0.2
- link BackLowerLeg: geometry collision box size=0.2 0.2 1.4982976268262127; visual box size=0.2 0.2 1.4982976268262127
- link FrontLeg: geometry collision box size=0.2 1.421458590887183 0.2; visual box size=0.2 1.421458590887183 0.2
- link FrontLowerLeg: geometry collision box size=0.2 0.2 1.3000340692813954; visual box size=0.2 0.2 1.3000340692813954
- link LeftLeg: geometry collision box size=0.9243773444531971 0.2 0.2; visual box size=0.9243773444531971 0.2 0.2
- link LeftLowerLeg: geometry collision box size=0.2 0.2 1.052473554848718; visual box size=0.2 0.2 1.052473554848718
- link RightLeg: geometry collision box size=0.9839797557019082 0.2 0.2; visual box size=0.9839797557019082 0.2 0.2
- link RightLowerLeg: geometry collision box size=0.2 0.2 0.8664118033690609; visual box size=0.2 0.2 0.8664118033690609
Joints:
- joint BackLeg_BackLowerLeg: origin xyz=0 -1.332736161975493 0 rpy=0 0 0 -> xyz=0 -0.9598225911765685 0 rpy=0 0 0
- joint FrontLeg_FrontLowerLeg: origin xyz=0 1.373898456266606 0 rpy=0 0 0 -> xyz=0 1.421458590887183 0 rpy=0 0 0
- joint LeftLeg_LeftLowerLeg: origin xyz=-0.5382098941602057 0 0 rpy=0 0 0 -> xyz=-0.9243773444531971 0 0 rpy=0 0 0
- joint RightLeg_RightLowerLeg: origin xyz=0.8993537410944455 0 0 rpy=0 0 0 -> xyz=0.9839797557019082 0 0 rpy=0 0 0
- joint Torso_BackLeg: origin xyz=0 -10.5 1.4114263014231248 rpy=0 0 0 -> xyz=0 -10.5 1.4982976268262127 rpy=0 0 0
- joint Torso_FrontLeg: origin xyz=0 -9.5 1.4114263014231248 rpy=0 0 0 -> xyz=0 -9.5 1.4982976268262127 rpy=0 0 0
- joint Torso_LeftLeg: origin xyz=-0.5 -10 1.4114263014231248 rpy=0 0 0 -> xyz=-0.5 -10 1.4982976268262127 rpy=0 0 0
- joint Torso_RightLeg: origin xyz=0.5 -10 1.4114263014231248 rpy=0 0 0 -> xyz=0.5 -10 1.4982976268262127 rpy=0 0 0

File: bodyFiles/body0-10294.urdf (robot description, URDF)
Before this commit: robot robot, 9 links, 8 joints
Links:
- link BackLeg: geometry collision box size=0.2 1.0938102148376432 0.2; visual box size=0.2 1.0938102148376432 0.2
- link BackLowerLeg: geometry collision box size=0.2 0.2 1.4395090305125509; visual box size=0.2 0.2 1.4395090305125509
- link FrontLeg: geometry collision box size=0.2 1.2477759250932796 0.2; visual box size=0.2 1.2477759250932796 0.2
- link FrontLowerLeg: geometry collision box size=0.2 0.2 0.7820528232300652; visual box size=0.2 0.2 0.7820528232300652
- link LeftLeg: geometry collision box size=1.38056233673465 0.2 0.2; visual box size=1.38056233673465 0.2 0.2
- link LeftLowerLeg: geometry collision box size=0.2 0.2 1.2017270905596567; visual box size=0.2 0.2 1.2017270905596567
- link RightLeg: geometry collision box size=0.5356045092106064 0.2 0.2; visual box size=0.5356045092106064 0.2 0.2
- link RightLowerLeg: geometry collision box size=0.2 0.2 0.6888598103492242; visual box size=0.2 0.2 0.6888598103492242
Joints:
- joint BackLeg_BackLowerLeg: origin xyz=0 -0.8300346621759594 0 rpy=0 0 0 -> xyz=0 -1.0938102148376432 0 rpy=0 0 0
- joint FrontLeg_FrontLowerLeg: origin xyz=0 1.0281112088199822 0 rpy=0 0 0 -> xyz=0 1.2477759250932796 0 rpy=0 0 0
- joint LeftLeg_LeftLowerLeg: origin xyz=-0.9000379161471664 0 0 rpy=0 0 0 -> xyz=-1.38056233673465 0 0 rpy=0 0 0
- joint RightLeg_RightLowerLeg: origin xyz=1.2277469816650475 0 0 rpy=0 0 0 -> xyz=0.5356045092106064 0 0 rpy=0 0 0
- joint Torso_BackLeg: origin xyz=0 -10.5 1.2277469816650475 rpy=0 0 0 -> xyz=0 -10.5 1.4395090305125509 rpy=0 0 0
- joint Torso_FrontLeg: origin xyz=0 -9.5 1.2277469816650475 rpy=0 0 0 -> xyz=0 -9.5 1.4395090305125509 rpy=0 0 0
- joint Torso_LeftLeg: origin xyz=-0.5 -10 1.2277469816650475 rpy=0 0 0 -> xyz=-0.5 -10 1.4395090305125509 rpy=0 0 0
- joint Torso_RightLeg: origin xyz=0.5 -10 1.2277469816650475 rpy=0 0 0 -> xyz=0.5 -10 1.4395090305125509 rpy=0 0 0

File: bodyFiles/body0-10331.urdf (robot description, URDF)
Before this commit: robot robot, 9 links, 8 joints
Links:
- link BackLeg: geometry collision box size=0.2 0.7745142987190416 0.2; visual box size=0.2 0.7745142987190416 0.2
- link BackLowerLeg: geometry collision box size=0.2 0.2 0.6839409802095587; visual box size=0.2 0.2 0.6839409802095587
- link FrontLeg: geometry collision box size=0.2 1.0659874499963737 0.2; visual box size=0.2 1.0659874499963737 0.2
- link FrontLowerLeg: geometry collision box size=0.2 0.2 0.6549702865211805; visual box size=0.2 0.2 0.6549702865211805
- link LeftLeg: geometry collision box size=0.7553171001181751 0.2 0.2; visual box size=0.7553171001181751 0.2 0.2
- link LeftLowerLeg: geometry collision box size=0.2 0.2 0.5791701536942597; visual box size=0.2 0.2 0.5791701536942597
- link RightLeg: geometry collision box size=0.6634013163947772 0.2 0.2; visual box size=0.6634013163947772 0.2 0.2
- link RightLowerLeg: geometry collision box size=0.2 0.2 1.1981956918077936; visual box size=0.2 0.2 1.1981956918077936
Joints:
- joint BackLeg_BackLowerLeg: origin xyz=0 -0.7002075955727659 0 rpy=0 0 0 -> xyz=0 -0.7745142987190416 0 rpy=0 0 0
- joint FrontLeg_FrontLowerLeg: origin xyz=0 1.0772088781959068 0 rpy=0 0 0 -> xyz=0 1.0659874499963737 0 rpy=0 0 0
- joint LeftLeg_LeftLowerLeg: origin xyz=-0.5315787571536681 0 0 rpy=0 0 0 -> xyz=-0.7553171001181751 0 0 rpy=0 0 0
- joint RightLeg_RightLowerLeg: origin xyz=0.7412517769333762 0 0 rpy=0 0 0 -> xyz=0.6634013163947772 0 0 rpy=0 0 0
- joint Torso_BackLeg: origin xyz=0 -10.5 1.2010222682188858 rpy=0 0 0 -> xyz=0 -10.5 1.1981956918077936 rpy=0 0 0
- joint Torso_FrontLeg: origin xyz=0 -9.5 1.2010222682188858 rpy=0 0 0 -> xyz=0 -9.5 1.1981956918077936 rpy=0 0 0
- joint Torso_LeftLeg: origin xyz=-0.5 -10 1.2010222682188858 rpy=0 0 0 -> xyz=-0.5 -10 1.1981956918077936 rpy=0 0 0
- joint Torso_RightLeg: origin xyz=0.5 -10 1.2010222682188858 rpy=0 0 0 -> xyz=0.5 -10 1.1981956918077936 rpy=0 0 0
