Commit message: collected case3 with weightsFiles

File: bodyFiles/body0-10362.urdf (robot description, URDF)
Before this commit: robot robot, 9 links, 8 joints
Links:
- link BackLeg: geometry collision box size=0.2 1.2690710951925968 0.2; visual box size=0.2 1.2690710951925968 0.2
- link BackLowerLeg: geometry collision box size=0.2 0.2 0.8565328231780543; visual box size=0.2 0.2 0.8565328231780543
- link FrontLeg: geometry collision box size=0.2 0.8717796661084409 0.2; visual box size=0.2 0.8717796661084409 0.2
- link FrontLowerLeg: geometry collision box size=0.2 0.2 0.5387950000953747; visual box size=0.2 0.2 0.5387950000953747
- link LeftLeg: geometry collision box size=1.3179031759780673 0.2 0.2; visual box size=1.3179031759780673 0.2 0.2
- link LeftLowerLeg: geometry collision box size=0.2 0.2 1.449106528386214; visual box size=0.2 0.2 1.449106528386214
- link RightLeg: geometry collision box size=1.4097751841069885 0.2 0.2; visual box size=1.4097751841069885 0.2 0.2
- link RightLowerLeg: geometry collision box size=0.2 0.2 0.6390079087937007; visual box size=0.2 0.2 0.6390079087937007
Joints:
- joint BackLeg_BackLowerLeg: origin xyz=0 -0.6033748038541397 0 rpy=0 0 0 -> xyz=0 -1.2690710951925968 0 rpy=0 0 0
- joint FrontLeg_FrontLowerLeg: origin xyz=0 1.4837873380121374 0 rpy=0 0 0 -> xyz=0 0.8717796661084409 0 rpy=0 0 0
- joint LeftLeg_LeftLowerLeg: origin xyz=-0.7229844176670539 0 0 rpy=0 0 0 -> xyz=-1.3179031759780673 0 0 rpy=0 0 0
- joint RightLeg_RightLowerLeg: origin xyz=0.7176645827522474 0 0 rpy=0 0 0 -> xyz=1.4097751841069885 0 0 rpy=0 0 0
- joint Torso_BackLeg: origin xyz=0 -10.5 1.4837873380121374 rpy=0 0 0 -> xyz=0 -10.5 1.449106528386214 rpy=0 0 0
- joint Torso_FrontLeg: origin xyz=0 -9.5 1.4837873380121374 rpy=0 0 0 -> xyz=0 -9.5 1.449106528386214 rpy=0 0 0
- joint Torso_LeftLeg: origin xyz=-0.5 -10 1.4837873380121374 rpy=0 0 0 -> xyz=-0.5 -10 1.449106528386214 rpy=0 0 0
- joint Torso_RightLeg: origin xyz=0.5 -10 1.4837873380121374 rpy=0 0 0 -> xyz=0.5 -10 1.449106528386214 rpy=0 0 0

File: bodyFiles/body0-10394.urdf (robot description, URDF)
Before this commit: robot robot, 9 links, 8 joints
Links:
- link BackLeg: geometry collision box size=0.2 1.0269781022814473 0.2; visual box size=0.2 1.0269781022814473 0.2
- link BackLowerLeg: geometry collision box size=0.2 0.2 0.9200643347420442; visual box size=0.2 0.2 0.9200643347420442
- link FrontLeg: geometry collision box size=0.2 1.1514338389099348 0.2; visual box size=0.2 1.1514338389099348 0.2
- link FrontLowerLeg: geometry collision box size=0.2 0.2 1.008183460062169; visual box size=0.2 0.2 1.008183460062169
- link LeftLeg: geometry collision box size=0.796694113290188 0.2 0.2; visual box size=0.796694113290188 0.2 0.2
- link LeftLowerLeg: geometry collision box size=0.2 0.2 0.9200699382160368; visual box size=0.2 0.2 0.9200699382160368
- link RightLeg: geometry collision box size=1.4037147040704097 0.2 0.2; visual box size=1.4037147040704097 0.2 0.2
- link RightLowerLeg: geometry collision box size=0.2 0.2 1.4950797808838074; visual box size=0.2 0.2 1.4950797808838074
Joints:
- joint BackLeg_BackLowerLeg: origin xyz=0 -0.7824190101466302 0 rpy=0 0 0 -> xyz=0 -1.0269781022814473 0 rpy=0 0 0
- joint FrontLeg_FrontLowerLeg: origin xyz=0 1.1923372474192695 0 rpy=0 0 0 -> xyz=0 1.1514338389099348 0 rpy=0 0 0
- joint LeftLeg_LeftLowerLeg: origin xyz=-1.1852274405294783 0 0 rpy=0 0 0 -> xyz=-0.796694113290188 0 0 rpy=0 0 0
- joint RightLeg_RightLowerLeg: origin xyz=1.444963820770453 0 0 rpy=0 0 0 -> xyz=1.4037147040704097 0 0 rpy=0 0 0
- joint Torso_BackLeg: origin xyz=0 -10.5 1.444963820770453 rpy=0 0 0 -> xyz=0 -10.5 1.4950797808838074 rpy=0 0 0
- joint Torso_FrontLeg: origin xyz=0 -9.5 1.444963820770453 rpy=0 0 0 -> xyz=0 -9.5 1.4950797808838074 rpy=0 0 0
- joint Torso_LeftLeg: origin xyz=-0.5 -10 1.444963820770453 rpy=0 0 0 -> xyz=-0.5 -10 1.4950797808838074 rpy=0 0 0
- joint Torso_RightLeg: origin xyz=0.5 -10 1.444963820770453 rpy=0 0 0 -> xyz=0.5 -10 1.4950797808838074 rpy=0 0 0

File: bodyFiles/body0-10424.urdf (robot description, URDF)
Before this commit: robot robot, 9 links, 8 joints
Links:
- link BackLeg: geometry collision box size=0.2 0.8644021472373069 0.2; visual box size=0.2 0.8644021472373069 0.2
- link BackLowerLeg: geometry collision box size=0.2 0.2 1.2220934584075214; visual box size=0.2 0.2 1.2220934584075214
- link FrontLeg: geometry collision box size=0.2 1.1211030849978671 0.2; visual box size=0.2 1.1211030849978671 0.2
- link FrontLowerLeg: geometry collision box size=0.2 0.2 0.8802073872028588; visual box size=0.2 0.2 0.8802073872028588
- link LeftLeg: geometry collision box size=0.7251938952527142 0.2 0.2; visual box size=0.7251938952527142 0.2 0.2
- link LeftLowerLeg: geometry collision box size=0.2 0.2 1.1122742439911664; visual box size=0.2 0.2 1.1122742439911664
- link RightLeg: geometry collision box size=0.9849256504285895 0.2 0.2; visual box size=0.9849256504285895 0.2 0.2
- link RightLowerLeg: geometry collision box size=0.2 0.2 1.4473470004136768; visual box size=0.2 0.2 1.4473470004136768
Joints:
- joint BackLeg_BackLowerLeg: origin xyz=0 -0.7716882831634692 0 rpy=0 0 0 -> xyz=0 -0.8644021472373069 0 rpy=0 0 0
- joint FrontLeg_FrontLowerLeg: origin xyz=0 1.2931717314186728 0 rpy=0 0 0 -> xyz=0 1.1211030849978671 0 rpy=0 0 0
- joint LeftLeg_LeftLowerLeg: origin xyz=-1.353904564670244 0 0 rpy=0 0 0 -> xyz=-0.7251938952527142 0 0 rpy=0 0 0
- joint RightLeg_RightLowerLeg: origin xyz=0.8864655784055064 0 0 rpy=0 0 0 -> xyz=0.9849256504285895 0 0 rpy=0 0 0
- joint Torso_BackLeg: origin xyz=0 -10.5 1.353904564670244 rpy=0 0 0 -> xyz=0 -10.5 1.4473470004136768 rpy=0 0 0
- joint Torso_FrontLeg: origin xyz=0 -9.5 1.353904564670244 rpy=0 0 0 -> xyz=0 -9.5 1.4473470004136768 rpy=0 0 0
- joint Torso_LeftLeg: origin xyz=-0.5 -10 1.353904564670244 rpy=0 0 0 -> xyz=-0.5 -10 1.4473470004136768 rpy=0 0 0
- joint Torso_RightLeg: origin xyz=0.5 -10 1.353904564670244 rpy=0 0 0 -> xyz=0.5 -10 1.4473470004136768 rpy=0 0 0

File: bodyFiles/body0-10447.urdf (robot description, URDF)
Before this commit: robot robot, 9 links, 8 joints
Links:
- link BackLeg: geometry collision box size=0.2 0.5429996448635023 0.2; visual box size=0.2 0.5429996448635023 0.2
- link BackLowerLeg: geometry collision box size=0.2 0.2 1.4716846737535185; visual box size=0.2 0.2 1.4716846737535185
- link FrontLeg: geometry collision box size=0.2 1.2545959002799338 0.2; visual box size=0.2 1.2545959002799338 0.2
- link FrontLowerLeg: geometry collision box size=0.2 0.2 1.4912176779919597; visual box size=0.2 0.2 1.4912176779919597
- link LeftLeg: geometry collision box size=0.5822602192512087 0.2 0.2; visual box size=0.5822602192512087 0.2 0.2
- link LeftLowerLeg: geometry collision box size=0.2 0.2 0.9618963803434052; visual box size=0.2 0.2 0.9618963803434052
- link RightLeg: geometry collision box size=0.930238326514406 0.2 0.2; visual box size=0.930238326514406 0.2 0.2
- link RightLowerLeg: geometry collision box size=0.2 0.2 1.0552024488089615; visual box size=0.2 0.2 1.0552024488089615
Joints:
- joint BackLeg_BackLowerLeg: origin xyz=0 -1.0612523145980859 0 rpy=0 0 0 -> xyz=0 -0.5429996448635023 0 rpy=0 0 0
- joint FrontLeg_FrontLowerLeg: origin xyz=0 1.4825473132875935 0 rpy=0 0 0 -> xyz=0 1.2545959002799338 0 rpy=0 0 0
- joint LeftLeg_LeftLowerLeg: origin xyz=-0.5516478145255159 0 0 rpy=0 0 0 -> xyz=-0.5822602192512087 0 0 rpy=0 0 0
- joint RightLeg_RightLowerLeg: origin xyz=1.3539026951956687 0 0 rpy=0 0 0 -> xyz=0.930238326514406 0 0 rpy=0 0 0
- joint Torso_BackLeg: origin xyz=0 -10.5 1.4825473132875935 rpy=0 0 0 -> xyz=0 -10.5 1.4912176779919597 rpy=0 0 0
- joint Torso_FrontLeg: origin xyz=0 -9.5 1.4825473132875935 rpy=0 0 0 -> xyz=0 -9.5 1.4912176779919597 rpy=0 0 0
- joint Torso_LeftLeg: origin xyz=-0.5 -10 1.4825473132875935 rpy=0 0 0 -> xyz=-0.5 -10 1.4912176779919597 rpy=0 0 0
- joint Torso_RightLeg: origin xyz=0.5 -10 1.4825473132875935 rpy=0 0 0 -> xyz=0.5 -10 1.4912176779919597 rpy=0 0 0

File: bodyFiles/body0-1045.urdf (robot description, URDF)
Before this commit: robot robot, 9 links, 8 joints
Links:
- link BackLeg: geometry collision box size=0.2 0.8536753483587342 0.2; visual box size=0.2 0.8536753483587342 0.2
- link BackLowerLeg: geometry collision box size=0.2 0.2 0.5805386252163602; visual box size=0.2 0.2 0.5805386252163602
- link FrontLeg: geometry collision box size=0.2 0.7498333246770145 0.2; visual box size=0.2 0.7498333246770145 0.2
- link FrontLowerLeg: geometry collision box size=0.2 0.2 1.1899121816951004; visual box size=0.2 0.2 1.1899121816951004
- link LeftLeg: geometry collision box size=0.8085696296523127 0.2 0.2; visual box size=0.8085696296523127 0.2 0.2
- link LeftLowerLeg: geometry collision box size=0.2 0.2 1.4442247072316023; visual box size=0.2 0.2 1.4442247072316023
- link RightLeg: geometry collision box size=0.7962190966918885 0.2 0.2; visual box size=0.7962190966918885 0.2 0.2
- link RightLowerLeg: geometry collision box size=0.2 0.2 1.2341114733628014; visual box size=0.2 0.2 1.2341114733628014
Joints:
- joint BackLeg_BackLowerLeg: origin xyz=0 -1.1307522225427786 0 rpy=0 0 0 -> xyz=0 -0.8536753483587342 0 rpy=0 0 0
- joint FrontLeg_FrontLowerLeg: origin xyz=0 0.9839278736502238 0 rpy=0 0 0 -> xyz=0 0.7498333246770145 0 rpy=0 0 0
- joint LeftLeg_LeftLowerLeg: origin xyz=-1.3761938124503004 0 0 rpy=0 0 0 -> xyz=-0.8085696296523127 0 0 rpy=0 0 0
- joint RightLeg_RightLowerLeg: origin xyz=1.0425526728711705 0 0 rpy=0 0 0 -> xyz=0.7962190966918885 0 0 rpy=0 0 0
- joint Torso_BackLeg: origin xyz=0 -10.5 1.3761938124503004 rpy=0 0 0 -> xyz=0 -10.5 1.4442247072316023 rpy=0 0 0
- joint Torso_FrontLeg: origin xyz=0 -9.5 1.3761938124503004 rpy=0 0 0 -> xyz=0 -9.5 1.4442247072316023 rpy=0 0 0
- joint Torso_LeftLeg: origin xyz=-0.5 -10 1.3761938124503004 rpy=0 0 0 -> xyz=-0.5 -10 1.4442247072316023 rpy=0 0 0
- joint Torso_RightLeg: origin xyz=0.5 -10 1.3761938124503004 rpy=0 0 0 -> xyz=0.5 -10 1.4442247072316023 rpy=0 0 0

File: bodyFiles/body0-10480.urdf (robot description, URDF)
Before this commit: robot robot, 9 links, 8 joints
Links:
- link BackLeg: geometry collision box size=0.2 0.9220564474829805 0.2; visual box size=0.2 0.9220564474829805 0.2
- link BackLowerLeg: geometry collision box size=0.2 0.2 1.145270344622431; visual box size=0.2 0.2 1.145270344622431
- link FrontLeg: geometry collision box size=0.2 0.6002367655265101 0.2; visual box size=0.2 0.6002367655265101 0.2
- link FrontLowerLeg: geometry collision box size=0.2 0.2 1.1903347539018982; visual box size=0.2 0.2 1.1903347539018982
- link LeftLeg: geometry collision box size=0.5477831791888442 0.2 0.2; visual box size=0.5477831791888442 0.2 0.2
- link LeftLowerLeg: geometry collision box size=0.2 0.2 1.0613955659236773; visual box size=0.2 0.2 1.0613955659236773
- link RightLeg: geometry collision box size=1.425589055562344 0.2 0.2; visual box size=1.425589055562344 0.2 0.2
- link RightLowerLeg: geometry collision box size=0.2 0.2 1.2806449144271737; visual box size=0.2 0.2 1.2806449144271737
Joints:
- joint BackLeg_BackLowerLeg: origin xyz=0 -0.9546172630647191 0 rpy=0 0 0 -> xyz=0 -0.9220564474829805 0 rpy=0 0 0
- joint FrontLeg_FrontLowerLeg: origin xyz=0 0.8521518254785276 0 rpy=0 0 0 -> xyz=0 0.6002367655265101 0 rpy=0 0 0
- joint LeftLeg_LeftLowerLeg: origin xyz=-0.8236017755843381 0 0 rpy=0 0 0 -> xyz=-0.5477831791888442 0 0 rpy=0 0 0
- joint RightLeg_RightLowerLeg: origin xyz=1.4228384355222459 0 0 rpy=0 0 0 -> xyz=1.425589055562344 0 0 rpy=0 0 0
- joint Torso_BackLeg: origin xyz=0 -10.5 1.4885787718687993 rpy=0 0 0 -> xyz=0 -10.5 1.425589055562344 rpy=0 0 0
- joint Torso_FrontLeg: origin xyz=0 -9.5 1.4885787718687993 rpy=0 0 0 -> xyz=0 -9.5 1.425589055562344 rpy=0 0 0
- joint Torso_LeftLeg: origin xyz=-0.5 -10 1.4885787718687993 rpy=0 0 0 -> xyz=-0.5 -10 1.425589055562344 rpy=0 0 0
- joint Torso_RightLeg: origin xyz=0.5 -10 1.4885787718687993 rpy=0 0 0 -> xyz=0.5 -10 1.425589055562344 rpy=0 0 0

File: bodyFiles/body0-10508.urdf (robot description, URDF)
Before this commit: robot robot, 9 links, 8 joints
Links:
- link BackLeg: geometry collision box size=0.2 0.9140301116351309 0.2; visual box size=0.2 0.9140301116351309 0.2
- link BackLowerLeg: geometry collision box size=0.2 0.2 0.5504991268519592; visual box size=0.2 0.2 0.5504991268519592
- link FrontLeg: geometry collision box size=0.2 0.7613795127695527 0.2; visual box size=0.2 0.7613795127695527 0.2
- link FrontLowerLeg: geometry collision box size=0.2 0.2 0.8749588998145977; visual box size=0.2 0.2 0.8749588998145977
- link LeftLeg: geometry collision box size=1.4245953356455408 0.2 0.2; visual box size=1.4245953356455408 0.2 0.2
- link LeftLowerLeg: geometry collision box size=0.2 0.2 0.7699457337511953; visual box size=0.2 0.2 0.7699457337511953
- link RightLeg: geometry collision box size=0.5265425152097336 0.2 0.2; visual box size=0.5265425152097336 0.2 0.2
- link RightLowerLeg: geometry collision box size=0.2 0.2 1.4413906476868312; visual box size=0.2 0.2 1.4413906476868312
Joints:
- joint BackLeg_BackLowerLeg: origin xyz=0 -1.460200618846577 0 rpy=0 0 0 -> xyz=0 -0.9140301116351309 0 rpy=0 0 0
- joint FrontLeg_FrontLowerLeg: origin xyz=0 1.2382808620445909 0 rpy=0 0 0 -> xyz=0 0.7613795127695527 0 rpy=0 0 0
- joint LeftLeg_LeftLowerLeg: origin xyz=-0.6871499227771116 0 0 rpy=0 0 0 -> xyz=-1.4245953356455408 0 0 rpy=0 0 0
- joint RightLeg_RightLowerLeg: origin xyz=0.9420516402288652 0 0 rpy=0 0 0 -> xyz=0.5265425152097336 0 0 rpy=0 0 0
- joint Torso_BackLeg: origin xyz=0 -10.5 1.4737801018834973 rpy=0 0 0 -> xyz=0 -10.5 1.4413906476868312 rpy=0 0 0
- joint Torso_FrontLeg: origin xyz=0 -9.5 1.4737801018834973 rpy=0 0 0 -> xyz=0 -9.5 1.4413906476868312 rpy=0 0 0
- joint Torso_LeftLeg: origin xyz=-0.5 -10 1.4737801018834973 rpy=0 0 0 -> xyz=-0.5 -10 1.4413906476868312 rpy=0 0 0
- joint Torso_RightLeg: origin xyz=0.5 -10 1.4737801018834973 rpy=0 0 0 -> xyz=0.5 -10 1.4413906476868312 rpy=0 0 0

File: bodyFiles/body0-10531.urdf (robot description, URDF)
Before this commit: robot robot, 9 links, 8 joints
Links:
- link BackLeg: geometry collision box size=0.2 1.2853448348304928 0.2; visual box size=0.2 1.2853448348304928 0.2
- link BackLowerLeg: geometry collision box size=0.2 0.2 1.4080506263020545; visual box size=0.2 0.2 1.4080506263020545
- link FrontLeg: geometry collision box size=0.2 0.877650425720178 0.2; visual box size=0.2 0.877650425720178 0.2
- link FrontLowerLeg: geometry collision box size=0.2 0.2 1.1866766325632845; visual box size=0.2 0.2 1.1866766325632845
- link LeftLeg: geometry collision box size=0.5767882434738305 0.2 0.2; visual box size=0.5767882434738305 0.2 0.2
- link LeftLowerLeg: geometry collision box size=0.2 0.2 0.7816187284325999; visual box size=0.2 0.2 0.7816187284325999
- link RightLeg: geometry collision box size=1.4359985263462707 0.2 0.2; visual box size=1.4359985263462707 0.2 0.2
- link RightLowerLeg: geometry collision box size=0.2 0.2 0.544697078167806; visual box size=0.2 0.2 0.544697078167806
Joints:
- joint BackLeg_BackLowerLeg: origin xyz=0 -1.080926860608923 0 rpy=0 0 0 -> xyz=0 -1.2853448348304928 0 rpy=0 0 0
- joint FrontLeg_FrontLowerLeg: origin xyz=0 0.9472483413143847 0 rpy=0 0 0 -> xyz=0 0.877650425720178 0 rpy=0 0 0
- joint LeftLeg_LeftLowerLeg: origin xyz=-0.6664485089358042 0 0 rpy=0 0 0 -> xyz=-0.5767882434738305 0 0 rpy=0 0 0
- joint RightLeg_RightLowerLeg: origin xyz=1.3988685193963843 0 0 rpy=0 0 0 -> xyz=1.4359985263462707 0 0 rpy=0 0 0
- joint Torso_BackLeg: origin xyz=0 -10.5 1.3988685193963843 rpy=0 0 0 -> xyz=0 -10.5 1.4359985263462707 rpy=0 0 0
- joint Torso_FrontLeg: origin xyz=0 -9.5 1.3988685193963843 rpy=0 0 0 -> xyz=0 -9.5 1.4359985263462707 rpy=0 0 0
- joint Torso_LeftLeg: origin xyz=-0.5 -10 1.3988685193963843 rpy=0 0 0 -> xyz=-0.5 -10 1.4359985263462707 rpy=0 0 0
- joint Torso_RightLeg: origin xyz=0.5 -10 1.3988685193963843 rpy=0 0 0 -> xyz=0.5 -10 1.4359985263462707 rpy=0 0 0

File: bodyFiles/body0-10562.urdf (robot description, URDF)
Before this commit: robot robot, 9 links, 8 joints
Links:
- link BackLeg: geometry collision box size=0.2 0.9160607886758882 0.2; visual box size=0.2 0.9160607886758882 0.2
- link BackLowerLeg: geometry collision box size=0.2 0.2 0.5572105012037089; visual box size=0.2 0.2 0.5572105012037089
- link FrontLeg: geometry collision box size=0.2 1.223298193990448 0.2; visual box size=0.2 1.223298193990448 0.2
- link FrontLowerLeg: geometry collision box size=0.2 0.2 0.8498548886373721; visual box size=0.2 0.2 0.8498548886373721
- link LeftLeg: geometry collision box size=0.7147426213450174 0.2 0.2; visual box size=0.7147426213450174 0.2 0.2
- link LeftLowerLeg: geometry collision box size=0.2 0.2 0.5944998659141228; visual box size=0.2 0.2 0.5944998659141228
- link RightLeg: geometry collision box size=1.3264791032959677 0.2 0.2; visual box size=1.3264791032959677 0.2 0.2
- link RightLowerLeg: geometry collision box size=0.2 0.2 1.0266332107962468; visual box size=0.2 0.2 1.0266332107962468
Joints:
- joint BackLeg_BackLowerLeg: origin xyz=0 -0.9998955385942997 0 rpy=0 0 0 -> xyz=0 -0.9160607886758882 0 rpy=0 0 0
- joint FrontLeg_FrontLowerLeg: origin xyz=0 0.7316272970898129 0 rpy=0 0 0 -> xyz=0 1.223298193990448 0 rpy=0 0 0
- joint LeftLeg_LeftLowerLeg: origin xyz=-1.1995765539765089 0 0 rpy=0 0 0 -> xyz=-0.7147426213450174 0 0 rpy=0 0 0
- joint RightLeg_RightLowerLeg: origin xyz=0.7506791649436788 0 0 rpy=0 0 0 -> xyz=1.3264791032959677 0 0 rpy=0 0 0
- joint Torso_BackLeg: origin xyz=0 -10.5 1.2278047834242742 rpy=0 0 0 -> xyz=0 -10.5 1.3264791032959677 rpy=0 0 0
- joint Torso_FrontLeg: origin xyz=0 -9.5 1.2278047834242742 rpy=0 0 0 -> xyz=0 -9.5 1.3264791032959677 rpy=0 0 0
- joint Torso_LeftLeg: origin xyz=-0.5 -10 1.2278047834242742 rpy=0 0 0 -> xyz=-0.5 -10 1.3264791032959677 rpy=0 0 0
- joint Torso_RightLeg: origin xyz=0.5 -10 1.2278047834242742 rpy=0 0 0 -> xyz=0.5 -10 1.3264791032959677 rpy=0 0 0
