Commit message: case3...30 + 5 + 5 gens

File: bodyFiles/body0-1010.urdf (robot description, URDF)
Before this commit: robot robot, 9 links, 8 joints
Links:
- link BackLeg: geometry collision box size=0.2 0.938975040734509 0.2; visual box size=0.2 0.938975040734509 0.2
- link BackLowerLeg: geometry collision box size=0.2 0.2 1.0633282668784418; visual box size=0.2 0.2 1.0633282668784418
- link FrontLeg: geometry collision box size=0.2 0.647108659411396 0.2; visual box size=0.2 0.647108659411396 0.2
- link FrontLowerLeg: geometry collision box size=0.2 0.2 0.8874216059392438; visual box size=0.2 0.2 0.8874216059392438
- link LeftLeg: geometry collision box size=0.9976720941056783 0.2 0.2; visual box size=0.9976720941056783 0.2 0.2
- link LeftLowerLeg: geometry collision box size=0.2 0.2 1.3849747960183887; visual box size=0.2 0.2 1.3849747960183887
- link RightLeg: geometry collision box size=1.48140314615347 0.2 0.2; visual box size=1.48140314615347 0.2 0.2
- link RightLowerLeg: geometry collision box size=0.2 0.2 1.2860442535083725; visual box size=0.2 0.2 1.2860442535083725
Joints:
- joint BackLeg_BackLowerLeg: origin xyz=0 -0.9220852996555571 0 rpy=0 0 0 -> xyz=0 -0.938975040734509 0 rpy=0 0 0
- joint FrontLeg_FrontLowerLeg: origin xyz=0 0.8407882028193432 0 rpy=0 0 0 -> xyz=0 0.647108659411396 0 rpy=0 0 0
- joint LeftLeg_LeftLowerLeg: origin xyz=-1.025487895197134 0 0 rpy=0 0 0 -> xyz=-0.9976720941056783 0 0 rpy=0 0 0
- joint RightLeg_RightLowerLeg: origin xyz=1.288473352944602 0 0 rpy=0 0 0 -> xyz=1.48140314615347 0 0 rpy=0 0 0
- joint Torso_BackLeg: origin xyz=0 -10.5 1.288473352944602 rpy=0 0 0 -> xyz=0 -10.5 1.48140314615347 rpy=0 0 0
- joint Torso_FrontLeg: origin xyz=0 -9.5 1.288473352944602 rpy=0 0 0 -> xyz=0 -9.5 1.48140314615347 rpy=0 0 0
- joint Torso_LeftLeg: origin xyz=-0.5 -10 1.288473352944602 rpy=0 0 0 -> xyz=-0.5 -10 1.48140314615347 rpy=0 0 0
- joint Torso_RightLeg: origin xyz=0.5 -10 1.288473352944602 rpy=0 0 0 -> xyz=0.5 -10 1.48140314615347 rpy=0 0 0

File: bodyFiles/body0-101034.urdf (robot description, URDF)
Before this commit: robot robot, 9 links, 8 joints
Links:
- link BackLeg: geometry collision box size=0.2 0.6716436271047427 0.2; visual box size=0.2 0.6716436271047427 0.2
- link BackLowerLeg: geometry collision box size=0.2 0.2 0.8702675595261017; visual box size=0.2 0.2 0.8702675595261017
- link FrontLeg: geometry collision box size=0.2 0.8597194956228362 0.2; visual box size=0.2 0.8597194956228362 0.2
- link FrontLowerLeg: geometry collision box size=0.2 0.2 0.6480241679297858; visual box size=0.2 0.2 0.6480241679297858
- link LeftLeg: geometry collision box size=1.450988925512295 0.2 0.2; visual box size=1.450988925512295 0.2 0.2
- link LeftLowerLeg: geometry collision box size=0.2 0.2 1.1591076295443177; visual box size=0.2 0.2 1.1591076295443177
- link RightLeg: geometry collision box size=0.6958736757735828 0.2 0.2; visual box size=0.6958736757735828 0.2 0.2
- link RightLowerLeg: geometry collision box size=0.2 0.2 0.6842472843848938; visual box size=0.2 0.2 0.6842472843848938
Joints:
- joint BackLeg_BackLowerLeg: origin xyz=0 -1.2121639302740672 0 rpy=0 0 0 -> xyz=0 -0.6716436271047427 0 rpy=0 0 0
- joint FrontLeg_FrontLowerLeg: origin xyz=0 0.6059559934242897 0 rpy=0 0 0 -> xyz=0 0.8597194956228362 0 rpy=0 0 0
- joint LeftLeg_LeftLowerLeg: origin xyz=-1.179365430834113 0 0 rpy=0 0 0 -> xyz=-1.450988925512295 0 0 rpy=0 0 0
- joint RightLeg_RightLowerLeg: origin xyz=1.1013902890178153 0 0 rpy=0 0 0 -> xyz=0.6958736757735828 0 0 rpy=0 0 0
- joint Torso_BackLeg: origin xyz=0 -10.5 1.4784620830875828 rpy=0 0 0 -> xyz=0 -10.5 1.450988925512295 rpy=0 0 0
- joint Torso_FrontLeg: origin xyz=0 -9.5 1.4784620830875828 rpy=0 0 0 -> xyz=0 -9.5 1.450988925512295 rpy=0 0 0
- joint Torso_LeftLeg: origin xyz=-0.5 -10 1.4784620830875828 rpy=0 0 0 -> xyz=-0.5 -10 1.450988925512295 rpy=0 0 0
- joint Torso_RightLeg: origin xyz=0.5 -10 1.4784620830875828 rpy=0 0 0 -> xyz=0.5 -10 1.450988925512295 rpy=0 0 0

File: bodyFiles/body0-10104.urdf (robot description, URDF)
Before this commit: robot robot, 9 links, 8 joints
Links:
- link BackLeg: geometry collision box size=0.2 1.1487023117487585 0.2; visual box size=0.2 1.1487023117487585 0.2
- link BackLowerLeg: geometry collision box size=0.2 0.2 1.483143809614299; visual box size=0.2 0.2 1.483143809614299
- link FrontLeg: geometry collision box size=0.2 1.1189057331492467 0.2; visual box size=0.2 1.1189057331492467 0.2
- link FrontLowerLeg: geometry collision box size=0.2 0.2 1.0496727145487017; visual box size=0.2 0.2 1.0496727145487017
- link LeftLeg: geometry collision box size=0.5777070318627731 0.2 0.2; visual box size=0.5777070318627731 0.2 0.2
- link LeftLowerLeg: geometry collision box size=0.2 0.2 1.2018180215368464; visual box size=0.2 0.2 1.2018180215368464
- link RightLeg: geometry collision box size=0.566120334978755 0.2 0.2; visual box size=0.566120334978755 0.2 0.2
- link RightLowerLeg: geometry collision box size=0.2 0.2 1.0796225699023636; visual box size=0.2 0.2 1.0796225699023636
Joints:
- joint BackLeg_BackLowerLeg: origin xyz=0 -1.0721545735055709 0 rpy=0 0 0 -> xyz=0 -1.1487023117487585 0 rpy=0 0 0
- joint FrontLeg_FrontLowerLeg: origin xyz=0 1.1368756145736665 0 rpy=0 0 0 -> xyz=0 1.1189057331492467 0 rpy=0 0 0
- joint LeftLeg_LeftLowerLeg: origin xyz=-0.6711257136467211 0 0 rpy=0 0 0 -> xyz=-0.5777070318627731 0 0 rpy=0 0 0
- joint RightLeg_RightLowerLeg: origin xyz=0.8638017792838052 0 0 rpy=0 0 0 -> xyz=0.566120334978755 0 0 rpy=0 0 0
- joint Torso_BackLeg: origin xyz=0 -10.5 1.3366922788169435 rpy=0 0 0 -> xyz=0 -10.5 1.483143809614299 rpy=0 0 0
- joint Torso_FrontLeg: origin xyz=0 -9.5 1.3366922788169435 rpy=0 0 0 -> xyz=0 -9.5 1.483143809614299 rpy=0 0 0
- joint Torso_LeftLeg: origin xyz=-0.5 -10 1.3366922788169435 rpy=0 0 0 -> xyz=-0.5 -10 1.483143809614299 rpy=0 0 0
- joint Torso_RightLeg: origin xyz=0.5 -10 1.3366922788169435 rpy=0 0 0 -> xyz=0.5 -10 1.483143809614299 rpy=0 0 0

File: bodyFiles/body0-101065.urdf (robot description, URDF)
Before this commit: robot robot, 9 links, 8 joints
Links:
- link BackLeg: geometry collision box size=0.2 0.8063018496814282 0.2; visual box size=0.2 0.8063018496814282 0.2
- link BackLowerLeg: geometry collision box size=0.2 0.2 1.2125614790758719; visual box size=0.2 0.2 1.2125614790758719
- link FrontLeg: geometry collision box size=0.2 0.5173098854993823 0.2; visual box size=0.2 0.5173098854993823 0.2
- link FrontLowerLeg: geometry collision box size=0.2 0.2 0.6870332312183278; visual box size=0.2 0.2 0.6870332312183278
- link LeftLeg: geometry collision box size=1.04036348714792 0.2 0.2; visual box size=1.04036348714792 0.2 0.2
- link LeftLowerLeg: geometry collision box size=0.2 0.2 0.5281735003683462; visual box size=0.2 0.2 0.5281735003683462
- link RightLeg: geometry collision box size=0.9737280623405598 0.2 0.2; visual box size=0.9737280623405598 0.2 0.2
- link RightLowerLeg: geometry collision box size=0.2 0.2 0.8260634052032495; visual box size=0.2 0.2 0.8260634052032495
Joints:
- joint BackLeg_BackLowerLeg: origin xyz=0 -1.2014125987006175 0 rpy=0 0 0 -> xyz=0 -0.8063018496814282 0 rpy=0 0 0
- joint FrontLeg_FrontLowerLeg: origin xyz=0 1.3564532170111852 0 rpy=0 0 0 -> xyz=0 0.5173098854993823 0 rpy=0 0 0
- joint LeftLeg_LeftLowerLeg: origin xyz=-1.1087719306563486 0 0 rpy=0 0 0 -> xyz=-1.04036348714792 0 0 rpy=0 0 0
- joint RightLeg_RightLowerLeg: origin xyz=1.0009863054677388 0 0 rpy=0 0 0 -> xyz=0.9737280623405598 0 0 rpy=0 0 0
- joint Torso_BackLeg: origin xyz=0 -10.5 1.3564532170111852 rpy=0 0 0 -> xyz=0 -10.5 1.2125614790758719 rpy=0 0 0
- joint Torso_FrontLeg: origin xyz=0 -9.5 1.3564532170111852 rpy=0 0 0 -> xyz=0 -9.5 1.2125614790758719 rpy=0 0 0
- joint Torso_LeftLeg: origin xyz=-0.5 -10 1.3564532170111852 rpy=0 0 0 -> xyz=-0.5 -10 1.2125614790758719 rpy=0 0 0
- joint Torso_RightLeg: origin xyz=0.5 -10 1.3564532170111852 rpy=0 0 0 -> xyz=0.5 -10 1.2125614790758719 rpy=0 0 0

File: bodyFiles/body0-10137.urdf (robot description, URDF)
Before this commit: robot robot, 9 links, 8 joints
Links:
- link BackLeg: geometry collision box size=0.2 1.4455804704016542 0.2; visual box size=0.2 1.4455804704016542 0.2
- link BackLowerLeg: geometry collision box size=0.2 0.2 0.524335591985113; visual box size=0.2 0.2 0.524335591985113
- link FrontLeg: geometry collision box size=0.2 0.8113124077355081 0.2; visual box size=0.2 0.8113124077355081 0.2
- link FrontLowerLeg: geometry collision box size=0.2 0.2 1.2050229037877045; visual box size=0.2 0.2 1.2050229037877045
- link LeftLeg: geometry collision box size=0.8366582388235175 0.2 0.2; visual box size=0.8366582388235175 0.2 0.2
- link LeftLowerLeg: geometry collision box size=0.2 0.2 0.6511731260329376; visual box size=0.2 0.2 0.6511731260329376
- link RightLeg: geometry collision box size=0.9952681383275807 0.2 0.2; visual box size=0.9952681383275807 0.2 0.2
- link RightLowerLeg: geometry collision box size=0.2 0.2 0.6402875019758738; visual box size=0.2 0.2 0.6402875019758738
Joints:
- joint BackLeg_BackLowerLeg: origin xyz=0 -0.5594391134313723 0 rpy=0 0 0 -> xyz=0 -1.4455804704016542 0 rpy=0 0 0
- joint FrontLeg_FrontLowerLeg: origin xyz=0 1.0702214467159612 0 rpy=0 0 0 -> xyz=0 0.8113124077355081 0 rpy=0 0 0
- joint LeftLeg_LeftLowerLeg: origin xyz=-1.0258866049401933 0 0 rpy=0 0 0 -> xyz=-0.8366582388235175 0 0 rpy=0 0 0
- joint RightLeg_RightLowerLeg: origin xyz=1.3526570170962389 0 0 rpy=0 0 0 -> xyz=0.9952681383275807 0 0 rpy=0 0 0
- joint Torso_BackLeg: origin xyz=0 -10.5 1.445220661331586 rpy=0 0 0 -> xyz=0 -10.5 1.4455804704016542 rpy=0 0 0
- joint Torso_FrontLeg: origin xyz=0 -9.5 1.445220661331586 rpy=0 0 0 -> xyz=0 -9.5 1.4455804704016542 rpy=0 0 0
- joint Torso_LeftLeg: origin xyz=-0.5 -10 1.445220661331586 rpy=0 0 0 -> xyz=-0.5 -10 1.4455804704016542 rpy=0 0 0
- joint Torso_RightLeg: origin xyz=0.5 -10 1.445220661331586 rpy=0 0 0 -> xyz=0.5 -10 1.4455804704016542 rpy=0 0 0

File: bodyFiles/body0-10168.urdf (robot description, URDF)
Before this commit: robot robot, 9 links, 8 joints
Links:
- link BackLeg: geometry collision box size=0.2 0.7017383725779895 0.2; visual box size=0.2 0.7017383725779895 0.2
- link BackLowerLeg: geometry collision box size=0.2 0.2 1.2548778591480052; visual box size=0.2 0.2 1.2548778591480052
- link FrontLeg: geometry collision box size=0.2 0.5538088899067922 0.2; visual box size=0.2 0.5538088899067922 0.2
- link FrontLowerLeg: geometry collision box size=0.2 0.2 1.2302307504603758; visual box size=0.2 0.2 1.2302307504603758
- link LeftLeg: geometry collision box size=1.3565833921354797 0.2 0.2; visual box size=1.3565833921354797 0.2 0.2
- link LeftLowerLeg: geometry collision box size=0.2 0.2 1.2375465458186556; visual box size=0.2 0.2 1.2375465458186556
- link RightLeg: geometry collision box size=0.7989363977959701 0.2 0.2; visual box size=0.7989363977959701 0.2 0.2
- link RightLowerLeg: geometry collision box size=0.2 0.2 0.6620980371421679; visual box size=0.2 0.2 0.6620980371421679
Joints:
- joint BackLeg_BackLowerLeg: origin xyz=0 -0.9416800575213753 0 rpy=0 0 0 -> xyz=0 -0.7017383725779895 0 rpy=0 0 0
- joint FrontLeg_FrontLowerLeg: origin xyz=0 1.0921333390596577 0 rpy=0 0 0 -> xyz=0 0.5538088899067922 0 rpy=0 0 0
- joint LeftLeg_LeftLowerLeg: origin xyz=-0.995672951487715 0 0 rpy=0 0 0 -> xyz=-1.3565833921354797 0 0 rpy=0 0 0
- joint RightLeg_RightLowerLeg: origin xyz=0.7323130582972708 0 0 rpy=0 0 0 -> xyz=0.7989363977959701 0 0 rpy=0 0 0
- joint Torso_BackLeg: origin xyz=0 -10.5 1.4310011010000352 rpy=0 0 0 -> xyz=0 -10.5 1.3565833921354797 rpy=0 0 0
- joint Torso_FrontLeg: origin xyz=0 -9.5 1.4310011010000352 rpy=0 0 0 -> xyz=0 -9.5 1.3565833921354797 rpy=0 0 0
- joint Torso_LeftLeg: origin xyz=-0.5 -10 1.4310011010000352 rpy=0 0 0 -> xyz=-0.5 -10 1.3565833921354797 rpy=0 0 0
- joint Torso_RightLeg: origin xyz=0.5 -10 1.4310011010000352 rpy=0 0 0 -> xyz=0.5 -10 1.3565833921354797 rpy=0 0 0

File: bodyFiles/body0-10205.urdf (robot description, URDF)
Before this commit: robot robot, 9 links, 8 joints
Links:
- link BackLeg: geometry collision box size=0.2 0.9933306471853152 0.2; visual box size=0.2 0.9933306471853152 0.2
- link BackLowerLeg: geometry collision box size=0.2 0.2 0.5088533334572451; visual box size=0.2 0.2 0.5088533334572451
- link FrontLeg: geometry collision box size=0.2 0.5499424636258314 0.2; visual box size=0.2 0.5499424636258314 0.2
- link FrontLowerLeg: geometry collision box size=0.2 0.2 0.842803966616491; visual box size=0.2 0.2 0.842803966616491
- link LeftLeg: geometry collision box size=1.0228199259811297 0.2 0.2; visual box size=1.0228199259811297 0.2 0.2
- link LeftLowerLeg: geometry collision box size=0.2 0.2 1.4988554417371127; visual box size=0.2 0.2 1.4988554417371127
- link RightLeg: geometry collision box size=0.9048807512886035 0.2 0.2; visual box size=0.9048807512886035 0.2 0.2
- link RightLowerLeg: geometry collision box size=0.2 0.2 0.522323581494751; visual box size=0.2 0.2 0.522323581494751
Joints:
- joint BackLeg_BackLowerLeg: origin xyz=0 -1.0531876928403774 0 rpy=0 0 0 -> xyz=0 -0.9933306471853152 0 rpy=0 0 0
- joint FrontLeg_FrontLowerLeg: origin xyz=0 0.7243964375335676 0 rpy=0 0 0 -> xyz=0 0.5499424636258314 0 rpy=0 0 0
- joint LeftLeg_LeftLowerLeg: origin xyz=-1.418683228986751 0 0 rpy=0 0 0 -> xyz=-1.0228199259811297 0 0 rpy=0 0 0
- joint RightLeg_RightLowerLeg: origin xyz=0.7067867675623617 0 0 rpy=0 0 0 -> xyz=0.9048807512886035 0 0 rpy=0 0 0
- joint Torso_BackLeg: origin xyz=0 -10.5 1.418683228986751 rpy=0 0 0 -> xyz=0 -10.5 1.4988554417371127 rpy=0 0 0
- joint Torso_FrontLeg: origin xyz=0 -9.5 1.418683228986751 rpy=0 0 0 -> xyz=0 -9.5 1.4988554417371127 rpy=0 0 0
- joint Torso_LeftLeg: origin xyz=-0.5 -10 1.418683228986751 rpy=0 0 0 -> xyz=-0.5 -10 1.4988554417371127 rpy=0 0 0
- joint Torso_RightLeg: origin xyz=0.5 -10 1.418683228986751 rpy=0 0 0 -> xyz=0.5 -10 1.4988554417371127 rpy=0 0 0

File: bodyFiles/body0-10238.urdf (robot description, URDF)
Before this commit: robot robot, 9 links, 8 joints
Links:
- link BackLeg: geometry collision box size=0.2 1.2341379048713943 0.2; visual box size=0.2 1.2341379048713943 0.2
- link BackLowerLeg: geometry collision box size=0.2 0.2 1.4009345429051436; visual box size=0.2 0.2 1.4009345429051436
- link FrontLeg: geometry collision box size=0.2 0.7484249942766722 0.2; visual box size=0.2 0.7484249942766722 0.2
- link FrontLowerLeg: geometry collision box size=0.2 0.2 1.18151637325308; visual box size=0.2 0.2 1.18151637325308
- link LeftLeg: geometry collision box size=1.204205843418243 0.2 0.2; visual box size=1.204205843418243 0.2 0.2
- link LeftLowerLeg: geometry collision box size=0.2 0.2 1.0544890202436947; visual box size=0.2 0.2 1.0544890202436947
- link RightLeg: geometry collision box size=1.0608023045334956 0.2 0.2; visual box size=1.0608023045334956 0.2 0.2
- link RightLowerLeg: geometry collision box size=0.2 0.2 1.493990491591033; visual box size=0.2 0.2 1.493990491591033
Joints:
- joint BackLeg_BackLowerLeg: origin xyz=0 -0.8327554538610643 0 rpy=0 0 0 -> xyz=0 -1.2341379048713943 0 rpy=0 0 0
- joint FrontLeg_FrontLowerLeg: origin xyz=0 1.3021422239376534 0 rpy=0 0 0 -> xyz=0 0.7484249942766722 0 rpy=0 0 0
- joint LeftLeg_LeftLowerLeg: origin xyz=-1.0901289197527808 0 0 rpy=0 0 0 -> xyz=-1.204205843418243 0 0 rpy=0 0 0
- joint RightLeg_RightLowerLeg: origin xyz=0.5322753933926542 0 0 rpy=0 0 0 -> xyz=1.0608023045334956 0 0 rpy=0 0 0
- joint Torso_BackLeg: origin xyz=0 -10.5 1.3021422239376534 rpy=0 0 0 -> xyz=0 -10.5 1.493990491591033 rpy=0 0 0
- joint Torso_FrontLeg: origin xyz=0 -9.5 1.3021422239376534 rpy=0 0 0 -> xyz=0 -9.5 1.493990491591033 rpy=0 0 0
- joint Torso_LeftLeg: origin xyz=-0.5 -10 1.3021422239376534 rpy=0 0 0 -> xyz=-0.5 -10 1.493990491591033 rpy=0 0 0
- joint Torso_RightLeg: origin xyz=0.5 -10 1.3021422239376534 rpy=0 0 0 -> xyz=0.5 -10 1.493990491591033 rpy=0 0 0

File: bodyFiles/body0-10270.urdf (robot description, URDF)
Before this commit: robot robot, 9 links, 8 joints
Links:
- link BackLeg: geometry collision box size=0.2 0.8609995470923046 0.2; visual box size=0.2 0.8609995470923046 0.2
- link BackLowerLeg: geometry collision box size=0.2 0.2 0.6016295736197065; visual box size=0.2 0.2 0.6016295736197065
- link FrontLeg: geometry collision box size=0.2 0.6827793631085527 0.2; visual box size=0.2 0.6827793631085527 0.2
- link FrontLowerLeg: geometry collision box size=0.2 0.2 1.0610491926968333; visual box size=0.2 0.2 1.0610491926968333
- link LeftLeg: geometry collision box size=0.8580717514899869 0.2 0.2; visual box size=0.8580717514899869 0.2 0.2
- link LeftLowerLeg: geometry collision box size=0.2 0.2 1.1275540349048545; visual box size=0.2 0.2 1.1275540349048545
- link RightLeg: geometry collision box size=1.2783282423140692 0.2 0.2; visual box size=1.2783282423140692 0.2 0.2
- link RightLowerLeg: geometry collision box size=0.2 0.2 0.9659553705526991; visual box size=0.2 0.2 0.9659553705526991
Joints:
- joint BackLeg_BackLowerLeg: origin xyz=0 -0.9598225911765685 0 rpy=0 0 0 -> xyz=0 -0.8609995470923046 0 rpy=0 0 0
- joint FrontLeg_FrontLowerLeg: origin xyz=0 1.421458590887183 0 rpy=0 0 0 -> xyz=0 0.6827793631085527 0 rpy=0 0 0
- joint LeftLeg_LeftLowerLeg: origin xyz=-0.9243773444531971 0 0 rpy=0 0 0 -> xyz=-0.8580717514899869 0 0 rpy=0 0 0
- joint RightLeg_RightLowerLeg: origin xyz=0.9839797557019082 0 0 rpy=0 0 0 -> xyz=1.2783282423140692 0 0 rpy=0 0 0
- joint Torso_BackLeg: origin xyz=0 -10.5 1.4982976268262127 rpy=0 0 0 -> xyz=0 -10.5 1.2783282423140692 rpy=0 0 0
- joint Torso_FrontLeg: origin xyz=0 -9.5 1.4982976268262127 rpy=0 0 0 -> xyz=0 -9.5 1.2783282423140692 rpy=0 0 0
- joint Torso_LeftLeg: origin xyz=-0.5 -10 1.4982976268262127 rpy=0 0 0 -> xyz=-0.5 -10 1.2783282423140692 rpy=0 0 0
- joint Torso_RightLeg: origin xyz=0.5 -10 1.4982976268262127 rpy=0 0 0 -> xyz=0.5 -10 1.2783282423140692 rpy=0 0 0

File: bodyFiles/body0-10294.urdf (robot description, URDF)
Before this commit: robot robot, 9 links, 8 joints
Links:
- link BackLeg: geometry collision box size=0.2 1.0291908663645837 0.2; visual box size=0.2 1.0291908663645837 0.2
- link BackLowerLeg: geometry collision box size=0.2 0.2 1.4156231048203867; visual box size=0.2 0.2 1.4156231048203867
- link FrontLeg: geometry collision box size=0.2 1.0729360752972548 0.2; visual box size=0.2 1.0729360752972548 0.2
- link FrontLowerLeg: geometry collision box size=0.2 0.2 0.8739276274724795; visual box size=0.2 0.2 0.8739276274724795
- link LeftLeg: geometry collision box size=1.3983166336372341 0.2 0.2; visual box size=1.3983166336372341 0.2 0.2
- link LeftLowerLeg: geometry collision box size=0.2 0.2 1.4090027843401765; visual box size=0.2 0.2 1.4090027843401765
- link RightLeg: geometry collision box size=0.840030584090808 0.2 0.2; visual box size=0.840030584090808 0.2 0.2
- link RightLowerLeg: geometry collision box size=0.2 0.2 0.9059770706500645; visual box size=0.2 0.2 0.9059770706500645
Joints:
- joint BackLeg_BackLowerLeg: origin xyz=0 -1.0938102148376432 0 rpy=0 0 0 -> xyz=0 -1.0291908663645837 0 rpy=0 0 0
- joint FrontLeg_FrontLowerLeg: origin xyz=0 1.2477759250932796 0 rpy=0 0 0 -> xyz=0 1.0729360752972548 0 rpy=0 0 0
- joint LeftLeg_LeftLowerLeg: origin xyz=-1.38056233673465 0 0 rpy=0 0 0 -> xyz=-1.3983166336372341 0 0 rpy=0 0 0
- joint RightLeg_RightLowerLeg: origin xyz=0.5356045092106064 0 0 rpy=0 0 0 -> xyz=0.840030584090808 0 0 rpy=0 0 0
- joint Torso_BackLeg: origin xyz=0 -10.5 1.4395090305125509 rpy=0 0 0 -> xyz=0 -10.5 1.4156231048203867 rpy=0 0 0
- joint Torso_FrontLeg: origin xyz=0 -9.5 1.4395090305125509 rpy=0 0 0 -> xyz=0 -9.5 1.4156231048203867 rpy=0 0 0
- joint Torso_LeftLeg: origin xyz=-0.5 -10 1.4395090305125509 rpy=0 0 0 -> xyz=-0.5 -10 1.4156231048203867 rpy=0 0 0
- joint Torso_RightLeg: origin xyz=0.5 -10 1.4395090305125509 rpy=0 0 0 -> xyz=0.5 -10 1.4156231048203867 rpy=0 0 0

File: bodyFiles/body0-10331.urdf (robot description, URDF)
Before this commit: robot robot, 9 links, 8 joints
Links:
- link BackLeg: geometry collision box size=0.2 0.9768473244800686 0.2; visual box size=0.2 0.9768473244800686 0.2
- link BackLowerLeg: geometry collision box size=0.2 0.2 1.1705736753252864; visual box size=0.2 0.2 1.1705736753252864
- link FrontLeg: geometry collision box size=0.2 0.9115468737011018 0.2; visual box size=0.2 0.9115468737011018 0.2
- link FrontLowerLeg: geometry collision box size=0.2 0.2 0.7959622411435544; visual box size=0.2 0.2 0.7959622411435544
- link LeftLeg: geometry collision box size=0.7254360130415088 0.2 0.2; visual box size=0.7254360130415088 0.2 0.2
- link LeftLowerLeg: geometry collision box size=0.2 0.2 0.5562155662797422; visual box size=0.2 0.2 0.5562155662797422
- link RightLeg: geometry collision box size=0.7375119893455816 0.2 0.2; visual box size=0.7375119893455816 0.2 0.2
- link RightLowerLeg: geometry collision box size=0.2 0.2 1.1620017060156211; visual box size=0.2 0.2 1.1620017060156211
Joints:
- joint BackLeg_BackLowerLeg: origin xyz=0 -0.7745142987190416 0 rpy=0 0 0 -> xyz=0 -0.9768473244800686 0 rpy=0 0 0
- joint FrontLeg_FrontLowerLeg: origin xyz=0 1.0659874499963737 0 rpy=0 0 0 -> xyz=0 0.9115468737011018 0 rpy=0 0 0
- joint LeftLeg_LeftLowerLeg: origin xyz=-0.7553171001181751 0 0 rpy=0 0 0 -> xyz=-0.7254360130415088 0 0 rpy=0 0 0
- joint RightLeg_RightLowerLeg: origin xyz=0.6634013163947772 0 0 rpy=0 0 0 -> xyz=0.7375119893455816 0 0 rpy=0 0 0
- joint Torso_BackLeg: origin xyz=0 -10.5 1.1981956918077936 rpy=0 0 0 -> xyz=0 -10.5 1.1705736753252864 rpy=0 0 0
- joint Torso_FrontLeg: origin xyz=0 -9.5 1.1981956918077936 rpy=0 0 0 -> xyz=0 -9.5 1.1705736753252864 rpy=0 0 0
- joint Torso_LeftLeg: origin xyz=-0.5 -10 1.1981956918077936 rpy=0 0 0 -> xyz=-0.5 -10 1.1705736753252864 rpy=0 0 0
- joint Torso_RightLeg: origin xyz=0.5 -10 1.1981956918077936 rpy=0 0 0 -> xyz=0.5 -10 1.1705736753252864 rpy=0 0 0
