Commit message: case3...30 + 5 + 5 gens

File: bodyFiles/body0-10362.urdf (robot description, URDF)
Before this commit: robot robot, 9 links, 8 joints
Links:
- link BackLeg: geometry collision box size=0.2 1.1880091604116594 0.2; visual box size=0.2 1.1880091604116594 0.2
- link BackLowerLeg: geometry collision box size=0.2 0.2 1.090997954736931; visual box size=0.2 0.2 1.090997954736931
- link FrontLeg: geometry collision box size=0.2 0.5884925214238024 0.2; visual box size=0.2 0.5884925214238024 0.2
- link FrontLowerLeg: geometry collision box size=0.2 0.2 1.0791352180174099; visual box size=0.2 0.2 1.0791352180174099
- link LeftLeg: geometry collision box size=0.9749709917333791 0.2 0.2; visual box size=0.9749709917333791 0.2 0.2
- link LeftLowerLeg: geometry collision box size=0.2 0.2 0.9911931189537365; visual box size=0.2 0.2 0.9911931189537365
- link RightLeg: geometry collision box size=0.852847203483727 0.2 0.2; visual box size=0.852847203483727 0.2 0.2
- link RightLowerLeg: geometry collision box size=0.2 0.2 1.497453426942767; visual box size=0.2 0.2 1.497453426942767
Joints:
- joint BackLeg_BackLowerLeg: origin xyz=0 -1.2690710951925968 0 rpy=0 0 0 -> xyz=0 -1.1880091604116594 0 rpy=0 0 0
- joint FrontLeg_FrontLowerLeg: origin xyz=0 0.8717796661084409 0 rpy=0 0 0 -> xyz=0 0.5884925214238024 0 rpy=0 0 0
- joint LeftLeg_LeftLowerLeg: origin xyz=-1.3179031759780673 0 0 rpy=0 0 0 -> xyz=-0.9749709917333791 0 0 rpy=0 0 0
- joint RightLeg_RightLowerLeg: origin xyz=1.4097751841069885 0 0 rpy=0 0 0 -> xyz=0.852847203483727 0 0 rpy=0 0 0
- joint Torso_BackLeg: origin xyz=0 -10.5 1.449106528386214 rpy=0 0 0 -> xyz=0 -10.5 1.497453426942767 rpy=0 0 0
- joint Torso_FrontLeg: origin xyz=0 -9.5 1.449106528386214 rpy=0 0 0 -> xyz=0 -9.5 1.497453426942767 rpy=0 0 0
- joint Torso_LeftLeg: origin xyz=-0.5 -10 1.449106528386214 rpy=0 0 0 -> xyz=-0.5 -10 1.497453426942767 rpy=0 0 0
- joint Torso_RightLeg: origin xyz=0.5 -10 1.449106528386214 rpy=0 0 0 -> xyz=0.5 -10 1.497453426942767 rpy=0 0 0

File: bodyFiles/body0-10394.urdf (robot description, URDF)
Before this commit: robot robot, 9 links, 8 joints
Links:
- link BackLeg: geometry collision box size=0.2 0.7780762490842805 0.2; visual box size=0.2 0.7780762490842805 0.2
- link BackLowerLeg: geometry collision box size=0.2 0.2 0.5126232578049055; visual box size=0.2 0.2 0.5126232578049055
- link FrontLeg: geometry collision box size=0.2 1.1709503448629313 0.2; visual box size=0.2 1.1709503448629313 0.2
- link FrontLowerLeg: geometry collision box size=0.2 0.2 1.411781124053236; visual box size=0.2 0.2 1.411781124053236
- link LeftLeg: geometry collision box size=1.2988537357417826 0.2 0.2; visual box size=1.2988537357417826 0.2 0.2
- link LeftLowerLeg: geometry collision box size=0.2 0.2 0.510338584631862; visual box size=0.2 0.2 0.510338584631862
- link RightLeg: geometry collision box size=1.1634542180068603 0.2 0.2; visual box size=1.1634542180068603 0.2 0.2
- link RightLowerLeg: geometry collision box size=0.2 0.2 1.1072598695037341; visual box size=0.2 0.2 1.1072598695037341
Joints:
- joint BackLeg_BackLowerLeg: origin xyz=0 -1.0269781022814473 0 rpy=0 0 0 -> xyz=0 -0.7780762490842805 0 rpy=0 0 0
- joint FrontLeg_FrontLowerLeg: origin xyz=0 1.1514338389099348 0 rpy=0 0 0 -> xyz=0 1.1709503448629313 0 rpy=0 0 0
- joint LeftLeg_LeftLowerLeg: origin xyz=-0.796694113290188 0 0 rpy=0 0 0 -> xyz=-1.2988537357417826 0 0 rpy=0 0 0
- joint RightLeg_RightLowerLeg: origin xyz=1.4037147040704097 0 0 rpy=0 0 0 -> xyz=1.1634542180068603 0 0 rpy=0 0 0
- joint Torso_BackLeg: origin xyz=0 -10.5 1.4950797808838074 rpy=0 0 0 -> xyz=0 -10.5 1.411781124053236 rpy=0 0 0
- joint Torso_FrontLeg: origin xyz=0 -9.5 1.4950797808838074 rpy=0 0 0 -> xyz=0 -9.5 1.411781124053236 rpy=0 0 0
- joint Torso_LeftLeg: origin xyz=-0.5 -10 1.4950797808838074 rpy=0 0 0 -> xyz=-0.5 -10 1.411781124053236 rpy=0 0 0
- joint Torso_RightLeg: origin xyz=0.5 -10 1.4950797808838074 rpy=0 0 0 -> xyz=0.5 -10 1.411781124053236 rpy=0 0 0

File: bodyFiles/body0-10424.urdf (robot description, URDF)
Before this commit: robot robot, 9 links, 8 joints
Links:
- link BackLeg: geometry collision box size=0.2 0.5970805739012087 0.2; visual box size=0.2 0.5970805739012087 0.2
- link BackLowerLeg: geometry collision box size=0.2 0.2 1.3010278667987691; visual box size=0.2 0.2 1.3010278667987691
- link FrontLeg: geometry collision box size=0.2 0.5076242801966585 0.2; visual box size=0.2 0.5076242801966585 0.2
- link FrontLowerLeg: geometry collision box size=0.2 0.2 1.1170526757354469; visual box size=0.2 0.2 1.1170526757354469
- link LeftLeg: geometry collision box size=0.6239896656589309 0.2 0.2; visual box size=0.6239896656589309 0.2 0.2
- link LeftLowerLeg: geometry collision box size=0.2 0.2 1.4971888728080764; visual box size=0.2 0.2 1.4971888728080764
- link RightLeg: geometry collision box size=0.6075930639132393 0.2 0.2; visual box size=0.6075930639132393 0.2 0.2
- link RightLowerLeg: geometry collision box size=0.2 0.2 1.1356952245796004; visual box size=0.2 0.2 1.1356952245796004
Joints:
- joint BackLeg_BackLowerLeg: origin xyz=0 -0.8644021472373069 0 rpy=0 0 0 -> xyz=0 -0.5970805739012087 0 rpy=0 0 0
- joint FrontLeg_FrontLowerLeg: origin xyz=0 1.1211030849978671 0 rpy=0 0 0 -> xyz=0 0.5076242801966585 0 rpy=0 0 0
- joint LeftLeg_LeftLowerLeg: origin xyz=-0.7251938952527142 0 0 rpy=0 0 0 -> xyz=-0.6239896656589309 0 0 rpy=0 0 0
- joint RightLeg_RightLowerLeg: origin xyz=0.9849256504285895 0 0 rpy=0 0 0 -> xyz=0.6075930639132393 0 0 rpy=0 0 0
- joint Torso_BackLeg: origin xyz=0 -10.5 1.4473470004136768 rpy=0 0 0 -> xyz=0 -10.5 1.4971888728080764 rpy=0 0 0
- joint Torso_FrontLeg: origin xyz=0 -9.5 1.4473470004136768 rpy=0 0 0 -> xyz=0 -9.5 1.4971888728080764 rpy=0 0 0
- joint Torso_LeftLeg: origin xyz=-0.5 -10 1.4473470004136768 rpy=0 0 0 -> xyz=-0.5 -10 1.4971888728080764 rpy=0 0 0
- joint Torso_RightLeg: origin xyz=0.5 -10 1.4473470004136768 rpy=0 0 0 -> xyz=0.5 -10 1.4971888728080764 rpy=0 0 0

File: bodyFiles/body0-10447.urdf (robot description, URDF)
Before this commit: robot robot, 9 links, 8 joints
Links:
- link BackLeg: geometry collision box size=0.2 0.8955937713285282 0.2; visual box size=0.2 0.8955937713285282 0.2
- link BackLowerLeg: geometry collision box size=0.2 0.2 1.032227536148271; visual box size=0.2 0.2 1.032227536148271
- link FrontLeg: geometry collision box size=0.2 0.8381006876048214 0.2; visual box size=0.2 0.8381006876048214 0.2
- link FrontLowerLeg: geometry collision box size=0.2 0.2 1.1714615503098211; visual box size=0.2 0.2 1.1714615503098211
- link LeftLeg: geometry collision box size=0.8339658600036215 0.2 0.2; visual box size=0.8339658600036215 0.2 0.2
- link LeftLowerLeg: geometry collision box size=0.2 0.2 1.3013562796697673; visual box size=0.2 0.2 1.3013562796697673
- link RightLeg: geometry collision box size=0.6895412746407268 0.2 0.2; visual box size=0.6895412746407268 0.2 0.2
- link RightLowerLeg: geometry collision box size=0.2 0.2 0.7027516895981829; visual box size=0.2 0.2 0.7027516895981829
Joints:
- joint BackLeg_BackLowerLeg: origin xyz=0 -0.5429996448635023 0 rpy=0 0 0 -> xyz=0 -0.8955937713285282 0 rpy=0 0 0
- joint FrontLeg_FrontLowerLeg: origin xyz=0 1.2545959002799338 0 rpy=0 0 0 -> xyz=0 0.8381006876048214 0 rpy=0 0 0
- joint LeftLeg_LeftLowerLeg: origin xyz=-0.5822602192512087 0 0 rpy=0 0 0 -> xyz=-0.8339658600036215 0 0 rpy=0 0 0
- joint RightLeg_RightLowerLeg: origin xyz=0.930238326514406 0 0 rpy=0 0 0 -> xyz=0.6895412746407268 0 0 rpy=0 0 0
- joint Torso_BackLeg: origin xyz=0 -10.5 1.4912176779919597 rpy=0 0 0 -> xyz=0 -10.5 1.3013562796697673 rpy=0 0 0
- joint Torso_FrontLeg: origin xyz=0 -9.5 1.4912176779919597 rpy=0 0 0 -> xyz=0 -9.5 1.3013562796697673 rpy=0 0 0
- joint Torso_LeftLeg: origin xyz=-0.5 -10 1.4912176779919597 rpy=0 0 0 -> xyz=-0.5 -10 1.3013562796697673 rpy=0 0 0
- joint Torso_RightLeg: origin xyz=0.5 -10 1.4912176779919597 rpy=0 0 0 -> xyz=0.5 -10 1.3013562796697673 rpy=0 0 0

File: bodyFiles/body0-1045.urdf (robot description, URDF)
Before this commit: robot robot, 9 links, 8 joints
Links:
- link BackLeg: geometry collision box size=0.2 1.2058596531164543 0.2; visual box size=0.2 1.2058596531164543 0.2
- link BackLowerLeg: geometry collision box size=0.2 0.2 0.6831607372074168; visual box size=0.2 0.2 0.6831607372074168
- link FrontLeg: geometry collision box size=0.2 0.5125941981899634 0.2; visual box size=0.2 0.5125941981899634 0.2
- link FrontLowerLeg: geometry collision box size=0.2 0.2 0.5093762908878443; visual box size=0.2 0.2 0.5093762908878443
- link LeftLeg: geometry collision box size=1.4351909332383728 0.2 0.2; visual box size=1.4351909332383728 0.2 0.2
- link LeftLowerLeg: geometry collision box size=0.2 0.2 1.2081876039163282; visual box size=0.2 0.2 1.2081876039163282
- link RightLeg: geometry collision box size=1.0704962351517895 0.2 0.2; visual box size=1.0704962351517895 0.2 0.2
- link RightLowerLeg: geometry collision box size=0.2 0.2 1.3714079893863038; visual box size=0.2 0.2 1.3714079893863038
Joints:
- joint BackLeg_BackLowerLeg: origin xyz=0 -0.8536753483587342 0 rpy=0 0 0 -> xyz=0 -1.2058596531164543 0 rpy=0 0 0
- joint FrontLeg_FrontLowerLeg: origin xyz=0 0.7498333246770145 0 rpy=0 0 0 -> xyz=0 0.5125941981899634 0 rpy=0 0 0
- joint LeftLeg_LeftLowerLeg: origin xyz=-0.8085696296523127 0 0 rpy=0 0 0 -> xyz=-1.4351909332383728 0 0 rpy=0 0 0
- joint RightLeg_RightLowerLeg: origin xyz=0.7962190966918885 0 0 rpy=0 0 0 -> xyz=1.0704962351517895 0 0 rpy=0 0 0
- joint Torso_BackLeg: origin xyz=0 -10.5 1.4442247072316023 rpy=0 0 0 -> xyz=0 -10.5 1.4351909332383728 rpy=0 0 0
- joint Torso_FrontLeg: origin xyz=0 -9.5 1.4442247072316023 rpy=0 0 0 -> xyz=0 -9.5 1.4351909332383728 rpy=0 0 0
- joint Torso_LeftLeg: origin xyz=-0.5 -10 1.4442247072316023 rpy=0 0 0 -> xyz=-0.5 -10 1.4351909332383728 rpy=0 0 0
- joint Torso_RightLeg: origin xyz=0.5 -10 1.4442247072316023 rpy=0 0 0 -> xyz=0.5 -10 1.4351909332383728 rpy=0 0 0

File: bodyFiles/body0-10480.urdf (robot description, URDF)
Before this commit: robot robot, 9 links, 8 joints
Links:
- link BackLeg: geometry collision box size=0.2 1.2736037105126088 0.2; visual box size=0.2 1.2736037105126088 0.2
- link BackLowerLeg: geometry collision box size=0.2 0.2 1.0731222646765475; visual box size=0.2 0.2 1.0731222646765475
- link FrontLeg: geometry collision box size=0.2 1.0885021428725294 0.2; visual box size=0.2 1.0885021428725294 0.2
- link FrontLowerLeg: geometry collision box size=0.2 0.2 0.8660648641508567; visual box size=0.2 0.2 0.8660648641508567
- link LeftLeg: geometry collision box size=1.4173162651179496 0.2 0.2; visual box size=1.4173162651179496 0.2 0.2
- link LeftLowerLeg: geometry collision box size=0.2 0.2 1.3748371731603544; visual box size=0.2 0.2 1.3748371731603544
- link RightLeg: geometry collision box size=0.9260368634122659 0.2 0.2; visual box size=0.9260368634122659 0.2 0.2
- link RightLowerLeg: geometry collision box size=0.2 0.2 0.6950496057824914; visual box size=0.2 0.2 0.6950496057824914
Joints:
- joint BackLeg_BackLowerLeg: origin xyz=0 -0.9220564474829805 0 rpy=0 0 0 -> xyz=0 -1.2736037105126088 0 rpy=0 0 0
- joint FrontLeg_FrontLowerLeg: origin xyz=0 0.6002367655265101 0 rpy=0 0 0 -> xyz=0 1.0885021428725294 0 rpy=0 0 0
- joint LeftLeg_LeftLowerLeg: origin xyz=-0.5477831791888442 0 0 rpy=0 0 0 -> xyz=-1.4173162651179496 0 0 rpy=0 0 0
- joint RightLeg_RightLowerLeg: origin xyz=1.425589055562344 0 0 rpy=0 0 0 -> xyz=0.9260368634122659 0 0 rpy=0 0 0
- joint Torso_BackLeg: origin xyz=0 -10.5 1.425589055562344 rpy=0 0 0 -> xyz=0 -10.5 1.4173162651179496 rpy=0 0 0
- joint Torso_FrontLeg: origin xyz=0 -9.5 1.425589055562344 rpy=0 0 0 -> xyz=0 -9.5 1.4173162651179496 rpy=0 0 0
- joint Torso_LeftLeg: origin xyz=-0.5 -10 1.425589055562344 rpy=0 0 0 -> xyz=-0.5 -10 1.4173162651179496 rpy=0 0 0
- joint Torso_RightLeg: origin xyz=0.5 -10 1.425589055562344 rpy=0 0 0 -> xyz=0.5 -10 1.4173162651179496 rpy=0 0 0

File: bodyFiles/body0-10508.urdf (robot description, URDF)
Before this commit: robot robot, 9 links, 8 joints
Links:
- link BackLeg: geometry collision box size=0.2 1.2243502635994608 0.2; visual box size=0.2 1.2243502635994608 0.2
- link BackLowerLeg: geometry collision box size=0.2 0.2 0.5950384583623483; visual box size=0.2 0.2 0.5950384583623483
- link FrontLeg: geometry collision box size=0.2 1.3540930668134408 0.2; visual box size=0.2 1.3540930668134408 0.2
- link FrontLowerLeg: geometry collision box size=0.2 0.2 1.4724471929575778; visual box size=0.2 0.2 1.4724471929575778
- link LeftLeg: geometry collision box size=0.8946849357430187 0.2 0.2; visual box size=0.8946849357430187 0.2 0.2
- link LeftLowerLeg: geometry collision box size=0.2 0.2 0.602980625895021; visual box size=0.2 0.2 0.602980625895021
- link RightLeg: geometry collision box size=0.7419205840625641 0.2 0.2; visual box size=0.7419205840625641 0.2 0.2
- link RightLowerLeg: geometry collision box size=0.2 0.2 0.7786234159148689; visual box size=0.2 0.2 0.7786234159148689
Joints:
- joint BackLeg_BackLowerLeg: origin xyz=0 -0.9140301116351309 0 rpy=0 0 0 -> xyz=0 -1.2243502635994608 0 rpy=0 0 0
- joint FrontLeg_FrontLowerLeg: origin xyz=0 0.7613795127695527 0 rpy=0 0 0 -> xyz=0 1.3540930668134408 0 rpy=0 0 0
- joint LeftLeg_LeftLowerLeg: origin xyz=-1.4245953356455408 0 0 rpy=0 0 0 -> xyz=-0.8946849357430187 0 0 rpy=0 0 0
- joint RightLeg_RightLowerLeg: origin xyz=0.5265425152097336 0 0 rpy=0 0 0 -> xyz=0.7419205840625641 0 0 rpy=0 0 0
- joint Torso_BackLeg: origin xyz=0 -10.5 1.4413906476868312 rpy=0 0 0 -> xyz=0 -10.5 1.4724471929575778 rpy=0 0 0
- joint Torso_FrontLeg: origin xyz=0 -9.5 1.4413906476868312 rpy=0 0 0 -> xyz=0 -9.5 1.4724471929575778 rpy=0 0 0
- joint Torso_LeftLeg: origin xyz=-0.5 -10 1.4413906476868312 rpy=0 0 0 -> xyz=-0.5 -10 1.4724471929575778 rpy=0 0 0
- joint Torso_RightLeg: origin xyz=0.5 -10 1.4413906476868312 rpy=0 0 0 -> xyz=0.5 -10 1.4724471929575778 rpy=0 0 0

File: bodyFiles/body0-10531.urdf (robot description, URDF)
Before this commit: robot robot, 9 links, 8 joints
Links:
- link BackLeg: geometry collision box size=0.2 0.8615637872065245 0.2; visual box size=0.2 0.8615637872065245 0.2
- link BackLowerLeg: geometry collision box size=0.2 0.2 0.6000666568360096; visual box size=0.2 0.2 0.6000666568360096
- link FrontLeg: geometry collision box size=0.2 0.6225059208396824 0.2; visual box size=0.2 0.6225059208396824 0.2
- link FrontLowerLeg: geometry collision box size=0.2 0.2 1.3736116731172237; visual box size=0.2 0.2 1.3736116731172237
- link LeftLeg: geometry collision box size=1.0063634030654383 0.2 0.2; visual box size=1.0063634030654383 0.2 0.2
- link LeftLowerLeg: geometry collision box size=0.2 0.2 0.7276149778056845; visual box size=0.2 0.2 0.7276149778056845
- link RightLeg: geometry collision box size=0.8146083503718247 0.2 0.2; visual box size=0.8146083503718247 0.2 0.2
- link RightLowerLeg: geometry collision box size=0.2 0.2 0.572285190667037; visual box size=0.2 0.2 0.572285190667037
Joints:
- joint BackLeg_BackLowerLeg: origin xyz=0 -1.2853448348304928 0 rpy=0 0 0 -> xyz=0 -0.8615637872065245 0 rpy=0 0 0
- joint FrontLeg_FrontLowerLeg: origin xyz=0 0.877650425720178 0 rpy=0 0 0 -> xyz=0 0.6225059208396824 0 rpy=0 0 0
- joint LeftLeg_LeftLowerLeg: origin xyz=-0.5767882434738305 0 0 rpy=0 0 0 -> xyz=-1.0063634030654383 0 0 rpy=0 0 0
- joint RightLeg_RightLowerLeg: origin xyz=1.4359985263462707 0 0 rpy=0 0 0 -> xyz=0.8146083503718247 0 0 rpy=0 0 0
- joint Torso_BackLeg: origin xyz=0 -10.5 1.4359985263462707 rpy=0 0 0 -> xyz=0 -10.5 1.3736116731172237 rpy=0 0 0
- joint Torso_FrontLeg: origin xyz=0 -9.5 1.4359985263462707 rpy=0 0 0 -> xyz=0 -9.5 1.3736116731172237 rpy=0 0 0
- joint Torso_LeftLeg: origin xyz=-0.5 -10 1.4359985263462707 rpy=0 0 0 -> xyz=-0.5 -10 1.3736116731172237 rpy=0 0 0
- joint Torso_RightLeg: origin xyz=0.5 -10 1.4359985263462707 rpy=0 0 0 -> xyz=0.5 -10 1.3736116731172237 rpy=0 0 0

File: bodyFiles/body0-10562.urdf (robot description, URDF)
Before this commit: robot robot, 9 links, 8 joints
Links:
- link BackLeg: geometry collision box size=0.2 1.2954606456154614 0.2; visual box size=0.2 1.2954606456154614 0.2
- link BackLowerLeg: geometry collision box size=0.2 0.2 1.1856968647141826; visual box size=0.2 0.2 1.1856968647141826
- link FrontLeg: geometry collision box size=0.2 1.2037441245638187 0.2; visual box size=0.2 1.2037441245638187 0.2
- link FrontLowerLeg: geometry collision box size=0.2 0.2 0.6614064430416141; visual box size=0.2 0.2 0.6614064430416141
- link LeftLeg: geometry collision box size=1.4505490515564676 0.2 0.2; visual box size=1.4505490515564676 0.2 0.2
- link LeftLowerLeg: geometry collision box size=0.2 0.2 1.1980775754636672; visual box size=0.2 0.2 1.1980775754636672
- link RightLeg: geometry collision box size=0.7353439551113983 0.2 0.2; visual box size=0.7353439551113983 0.2 0.2
- link RightLowerLeg: geometry collision box size=0.2 0.2 1.3454209482136825; visual box size=0.2 0.2 1.3454209482136825
Joints:
- joint BackLeg_BackLowerLeg: origin xyz=0 -0.9160607886758882 0 rpy=0 0 0 -> xyz=0 -1.2954606456154614 0 rpy=0 0 0
- joint FrontLeg_FrontLowerLeg: origin xyz=0 1.223298193990448 0 rpy=0 0 0 -> xyz=0 1.2037441245638187 0 rpy=0 0 0
- joint LeftLeg_LeftLowerLeg: origin xyz=-0.7147426213450174 0 0 rpy=0 0 0 -> xyz=-1.4505490515564676 0 0 rpy=0 0 0
- joint RightLeg_RightLowerLeg: origin xyz=1.3264791032959677 0 0 rpy=0 0 0 -> xyz=0.7353439551113983 0 0 rpy=0 0 0
- joint Torso_BackLeg: origin xyz=0 -10.5 1.3264791032959677 rpy=0 0 0 -> xyz=0 -10.5 1.4505490515564676 rpy=0 0 0
- joint Torso_FrontLeg: origin xyz=0 -9.5 1.3264791032959677 rpy=0 0 0 -> xyz=0 -9.5 1.4505490515564676 rpy=0 0 0
- joint Torso_LeftLeg: origin xyz=-0.5 -10 1.3264791032959677 rpy=0 0 0 -> xyz=-0.5 -10 1.4505490515564676 rpy=0 0 0
- joint Torso_RightLeg: origin xyz=0.5 -10 1.3264791032959677 rpy=0 0 0 -> xyz=0.5 -10 1.4505490515564676 rpy=0 0 0
