Commit message: case3 30 + 10 gens

File: bodyFiles/body0-1010.urdf (robot description, URDF)
Before this commit: robot robot, 9 links, 8 joints
Links:
- link BackLeg: geometry collision box size=0.2 1.4090852278780965 0.2; visual box size=0.2 1.4090852278780965 0.2
- link BackLowerLeg: geometry collision box size=0.2 0.2 0.5677641702463887; visual box size=0.2 0.2 0.5677641702463887
- link FrontLeg: geometry collision box size=0.2 0.9607894874261254 0.2; visual box size=0.2 0.9607894874261254 0.2
- link FrontLowerLeg: geometry collision box size=0.2 0.2 1.0937050618011028; visual box size=0.2 0.2 1.0937050618011028
- link LeftLeg: geometry collision box size=1.0464030274848133 0.2 0.2; visual box size=1.0464030274848133 0.2 0.2
- link LeftLowerLeg: geometry collision box size=0.2 0.2 1.3475738222924507; visual box size=0.2 0.2 1.3475738222924507
- link RightLeg: geometry collision box size=1.3141739622597255 0.2 0.2; visual box size=1.3141739622597255 0.2 0.2
- link RightLowerLeg: geometry collision box size=0.2 0.2 0.9510875617447558; visual box size=0.2 0.2 0.9510875617447558
Joints:
- joint BackLeg_BackLowerLeg: origin xyz=0 -0.938975040734509 0 rpy=0 0 0 -> xyz=0 -1.4090852278780965 0 rpy=0 0 0
- joint FrontLeg_FrontLowerLeg: origin xyz=0 0.647108659411396 0 rpy=0 0 0 -> xyz=0 0.9607894874261254 0 rpy=0 0 0
- joint LeftLeg_LeftLowerLeg: origin xyz=-0.9976720941056783 0 0 rpy=0 0 0 -> xyz=-1.0464030274848133 0 0 rpy=0 0 0
- joint RightLeg_RightLowerLeg: origin xyz=1.48140314615347 0 0 rpy=0 0 0 -> xyz=1.3141739622597255 0 0 rpy=0 0 0
- joint Torso_BackLeg: origin xyz=0 -10.5 1.48140314615347 rpy=0 0 0 -> xyz=0 -10.5 1.4090852278780965 rpy=0 0 0
- joint Torso_FrontLeg: origin xyz=0 -9.5 1.48140314615347 rpy=0 0 0 -> xyz=0 -9.5 1.4090852278780965 rpy=0 0 0
- joint Torso_LeftLeg: origin xyz=-0.5 -10 1.48140314615347 rpy=0 0 0 -> xyz=-0.5 -10 1.4090852278780965 rpy=0 0 0
- joint Torso_RightLeg: origin xyz=0.5 -10 1.48140314615347 rpy=0 0 0 -> xyz=0.5 -10 1.4090852278780965 rpy=0 0 0

File: bodyFiles/body0-101034.urdf (robot description, URDF)
Before this commit: robot robot, 9 links, 8 joints
Links:
- link BackLeg: geometry collision box size=0.2 0.5923778854220229 0.2; visual box size=0.2 0.5923778854220229 0.2
- link BackLowerLeg: geometry collision box size=0.2 0.2 1.4957065423903753; visual box size=0.2 0.2 1.4957065423903753
- link FrontLeg: geometry collision box size=0.2 1.4220381086240987 0.2; visual box size=0.2 1.4220381086240987 0.2
- link FrontLowerLeg: geometry collision box size=0.2 0.2 0.502063193938637; visual box size=0.2 0.2 0.502063193938637
- link LeftLeg: geometry collision box size=0.5985178371821482 0.2 0.2; visual box size=0.5985178371821482 0.2 0.2
- link LeftLowerLeg: geometry collision box size=0.2 0.2 1.394301122010787; visual box size=0.2 0.2 1.394301122010787
- link RightLeg: geometry collision box size=0.7599267928344847 0.2 0.2; visual box size=0.7599267928344847 0.2 0.2
- link RightLowerLeg: geometry collision box size=0.2 0.2 0.6439555894888832; visual box size=0.2 0.2 0.6439555894888832
Joints:
- joint BackLeg_BackLowerLeg: origin xyz=0 -0.6716436271047427 0 rpy=0 0 0 -> xyz=0 -0.5923778854220229 0 rpy=0 0 0
- joint FrontLeg_FrontLowerLeg: origin xyz=0 0.8597194956228362 0 rpy=0 0 0 -> xyz=0 1.4220381086240987 0 rpy=0 0 0
- joint LeftLeg_LeftLowerLeg: origin xyz=-1.450988925512295 0 0 rpy=0 0 0 -> xyz=-0.5985178371821482 0 0 rpy=0 0 0
- joint RightLeg_RightLowerLeg: origin xyz=0.6958736757735828 0 0 rpy=0 0 0 -> xyz=0.7599267928344847 0 0 rpy=0 0 0
- joint Torso_BackLeg: origin xyz=0 -10.5 1.450988925512295 rpy=0 0 0 -> xyz=0 -10.5 1.4957065423903753 rpy=0 0 0
- joint Torso_FrontLeg: origin xyz=0 -9.5 1.450988925512295 rpy=0 0 0 -> xyz=0 -9.5 1.4957065423903753 rpy=0 0 0
- joint Torso_LeftLeg: origin xyz=-0.5 -10 1.450988925512295 rpy=0 0 0 -> xyz=-0.5 -10 1.4957065423903753 rpy=0 0 0
- joint Torso_RightLeg: origin xyz=0.5 -10 1.450988925512295 rpy=0 0 0 -> xyz=0.5 -10 1.4957065423903753 rpy=0 0 0

File: bodyFiles/body0-10104.urdf (robot description, URDF)
Before this commit: robot robot, 9 links, 8 joints
Links:
- link BackLeg: geometry collision box size=0.2 0.5397208110596992 0.2; visual box size=0.2 0.5397208110596992 0.2
- link BackLowerLeg: geometry collision box size=0.2 0.2 0.7095827228493611; visual box size=0.2 0.2 0.7095827228493611
- link FrontLeg: geometry collision box size=0.2 0.6047284848980241 0.2; visual box size=0.2 0.6047284848980241 0.2
- link FrontLowerLeg: geometry collision box size=0.2 0.2 1.26660694190867; visual box size=0.2 0.2 1.26660694190867
- link LeftLeg: geometry collision box size=1.3936995986964509 0.2 0.2; visual box size=1.3936995986964509 0.2 0.2
- link LeftLowerLeg: geometry collision box size=0.2 0.2 1.1482271623562599; visual box size=0.2 0.2 1.1482271623562599
- link RightLeg: geometry collision box size=0.69259729102041 0.2 0.2; visual box size=0.69259729102041 0.2 0.2
- link RightLowerLeg: geometry collision box size=0.2 0.2 1.3433002061966173; visual box size=0.2 0.2 1.3433002061966173
Joints:
- joint BackLeg_BackLowerLeg: origin xyz=0 -1.1487023117487585 0 rpy=0 0 0 -> xyz=0 -0.5397208110596992 0 rpy=0 0 0
- joint FrontLeg_FrontLowerLeg: origin xyz=0 1.1189057331492467 0 rpy=0 0 0 -> xyz=0 0.6047284848980241 0 rpy=0 0 0
- joint LeftLeg_LeftLowerLeg: origin xyz=-0.5777070318627731 0 0 rpy=0 0 0 -> xyz=-1.3936995986964509 0 0 rpy=0 0 0
- joint RightLeg_RightLowerLeg: origin xyz=0.566120334978755 0 0 rpy=0 0 0 -> xyz=0.69259729102041 0 0 rpy=0 0 0
- joint Torso_BackLeg: origin xyz=0 -10.5 1.483143809614299 rpy=0 0 0 -> xyz=0 -10.5 1.3936995986964509 rpy=0 0 0
- joint Torso_FrontLeg: origin xyz=0 -9.5 1.483143809614299 rpy=0 0 0 -> xyz=0 -9.5 1.3936995986964509 rpy=0 0 0
- joint Torso_LeftLeg: origin xyz=-0.5 -10 1.483143809614299 rpy=0 0 0 -> xyz=-0.5 -10 1.3936995986964509 rpy=0 0 0
- joint Torso_RightLeg: origin xyz=0.5 -10 1.483143809614299 rpy=0 0 0 -> xyz=0.5 -10 1.3936995986964509 rpy=0 0 0

File: bodyFiles/body0-101065.urdf (robot description, URDF)
Before this commit: robot robot, 9 links, 8 joints
Links:
- link BackLeg: geometry collision box size=0.2 0.5128842321711606 0.2; visual box size=0.2 0.5128842321711606 0.2
- link BackLowerLeg: geometry collision box size=0.2 0.2 1.4891646916608474; visual box size=0.2 0.2 1.4891646916608474
- link FrontLeg: geometry collision box size=0.2 1.1280303355430767 0.2; visual box size=0.2 1.1280303355430767 0.2
- link FrontLowerLeg: geometry collision box size=0.2 0.2 0.7219977646176983; visual box size=0.2 0.2 0.7219977646176983
- link LeftLeg: geometry collision box size=1.1534798057734803 0.2 0.2; visual box size=1.1534798057734803 0.2 0.2
- link LeftLowerLeg: geometry collision box size=0.2 0.2 0.7295547049851699; visual box size=0.2 0.2 0.7295547049851699
- link RightLeg: geometry collision box size=1.286705025156039 0.2 0.2; visual box size=1.286705025156039 0.2 0.2
- link RightLowerLeg: geometry collision box size=0.2 0.2 1.287057605817445; visual box size=0.2 0.2 1.287057605817445
Joints:
- joint BackLeg_BackLowerLeg: origin xyz=0 -0.8063018496814282 0 rpy=0 0 0 -> xyz=0 -0.5128842321711606 0 rpy=0 0 0
- joint FrontLeg_FrontLowerLeg: origin xyz=0 0.5173098854993823 0 rpy=0 0 0 -> xyz=0 1.1280303355430767 0 rpy=0 0 0
- joint LeftLeg_LeftLowerLeg: origin xyz=-1.04036348714792 0 0 rpy=0 0 0 -> xyz=-1.1534798057734803 0 0 rpy=0 0 0
- joint RightLeg_RightLowerLeg: origin xyz=0.9737280623405598 0 0 rpy=0 0 0 -> xyz=1.286705025156039 0 0 rpy=0 0 0
- joint Torso_BackLeg: origin xyz=0 -10.5 1.2125614790758719 rpy=0 0 0 -> xyz=0 -10.5 1.4891646916608474 rpy=0 0 0
- joint Torso_FrontLeg: origin xyz=0 -9.5 1.2125614790758719 rpy=0 0 0 -> xyz=0 -9.5 1.4891646916608474 rpy=0 0 0
- joint Torso_LeftLeg: origin xyz=-0.5 -10 1.2125614790758719 rpy=0 0 0 -> xyz=-0.5 -10 1.4891646916608474 rpy=0 0 0
- joint Torso_RightLeg: origin xyz=0.5 -10 1.2125614790758719 rpy=0 0 0 -> xyz=0.5 -10 1.4891646916608474 rpy=0 0 0

File: bodyFiles/body0-101158.urdf (robot description, URDF)
Before this commit: robot robot, 9 links, 8 joints
Links:
- link BackLeg: geometry collision box size=0.2 1.467509597836382 0.2; visual box size=0.2 1.467509597836382 0.2
- link BackLowerLeg: geometry collision box size=0.2 0.2 1.3474787632607508; visual box size=0.2 0.2 1.3474787632607508
- link FrontLeg: geometry collision box size=0.2 1.4320073658590102 0.2; visual box size=0.2 1.4320073658590102 0.2
- link FrontLowerLeg: geometry collision box size=0.2 0.2 0.9309322206041079; visual box size=0.2 0.2 0.9309322206041079
- link LeftLeg: geometry collision box size=0.7610877757262116 0.2 0.2; visual box size=0.7610877757262116 0.2 0.2
- link LeftLowerLeg: geometry collision box size=0.2 0.2 1.460768043003967; visual box size=0.2 0.2 1.460768043003967
- link RightLeg: geometry collision box size=1.2821957677281848 0.2 0.2; visual box size=1.2821957677281848 0.2 0.2
- link RightLowerLeg: geometry collision box size=0.2 0.2 0.5187321559279167; visual box size=0.2 0.2 0.5187321559279167
Joints:
- joint BackLeg_BackLowerLeg: origin xyz=0 -0.7260577404979621 0 rpy=0 0 0 -> xyz=0 -1.467509597836382 0 rpy=0 0 0
- joint FrontLeg_FrontLowerLeg: origin xyz=0 0.9275890351528563 0 rpy=0 0 0 -> xyz=0 1.4320073658590102 0 rpy=0 0 0
- joint LeftLeg_LeftLowerLeg: origin xyz=-0.6615502675936074 0 0 rpy=0 0 0 -> xyz=-0.7610877757262116 0 0 rpy=0 0 0
- joint RightLeg_RightLowerLeg: origin xyz=1.0470710222375625 0 0 rpy=0 0 0 -> xyz=1.2821957677281848 0 0 rpy=0 0 0
- joint Torso_BackLeg: origin xyz=0 -10.5 1.4462425419103653 rpy=0 0 0 -> xyz=0 -10.5 1.467509597836382 rpy=0 0 0
- joint Torso_FrontLeg: origin xyz=0 -9.5 1.4462425419103653 rpy=0 0 0 -> xyz=0 -9.5 1.467509597836382 rpy=0 0 0
- joint Torso_LeftLeg: origin xyz=-0.5 -10 1.4462425419103653 rpy=0 0 0 -> xyz=-0.5 -10 1.467509597836382 rpy=0 0 0
- joint Torso_RightLeg: origin xyz=0.5 -10 1.4462425419103653 rpy=0 0 0 -> xyz=0.5 -10 1.467509597836382 rpy=0 0 0

File: bodyFiles/body0-101361.urdf (robot description, URDF)
Before this commit: robot robot, 9 links, 8 joints
Links:
- link BackLeg: geometry collision box size=0.2 1.1358606236461721 0.2; visual box size=0.2 1.1358606236461721 0.2
- link BackLowerLeg: geometry collision box size=0.2 0.2 0.8174986281066574; visual box size=0.2 0.2 0.8174986281066574
- link FrontLeg: geometry collision box size=0.2 1.107033224266101 0.2; visual box size=0.2 1.107033224266101 0.2
- link FrontLowerLeg: geometry collision box size=0.2 0.2 1.3502436642945703; visual box size=0.2 0.2 1.3502436642945703
- link LeftLeg: geometry collision box size=1.0492219968274754 0.2 0.2; visual box size=1.0492219968274754 0.2 0.2
- link LeftLowerLeg: geometry collision box size=0.2 0.2 1.3841511220456795; visual box size=0.2 0.2 1.3841511220456795
- link RightLeg: geometry collision box size=0.9486946183318675 0.2 0.2; visual box size=0.9486946183318675 0.2 0.2
- link RightLowerLeg: geometry collision box size=0.2 0.2 1.1257760242730415; visual box size=0.2 0.2 1.1257760242730415
Joints:
- joint BackLeg_BackLowerLeg: origin xyz=0 -0.7825191924271137 0 rpy=0 0 0 -> xyz=0 -1.1358606236461721 0 rpy=0 0 0
- joint FrontLeg_FrontLowerLeg: origin xyz=0 1.020588646848811 0 rpy=0 0 0 -> xyz=0 1.107033224266101 0 rpy=0 0 0
- joint LeftLeg_LeftLowerLeg: origin xyz=-0.8175369228657552 0 0 rpy=0 0 0 -> xyz=-1.0492219968274754 0 0 rpy=0 0 0
- joint RightLeg_RightLowerLeg: origin xyz=1.3874558360708638 0 0 rpy=0 0 0 -> xyz=0.9486946183318675 0 0 rpy=0 0 0
- joint Torso_BackLeg: origin xyz=0 -10.5 1.3874558360708638 rpy=0 0 0 -> xyz=0 -10.5 1.3841511220456795 rpy=0 0 0
- joint Torso_FrontLeg: origin xyz=0 -9.5 1.3874558360708638 rpy=0 0 0 -> xyz=0 -9.5 1.3841511220456795 rpy=0 0 0
- joint Torso_LeftLeg: origin xyz=-0.5 -10 1.3874558360708638 rpy=0 0 0 -> xyz=-0.5 -10 1.3841511220456795 rpy=0 0 0
- joint Torso_RightLeg: origin xyz=0.5 -10 1.3874558360708638 rpy=0 0 0 -> xyz=0.5 -10 1.3841511220456795 rpy=0 0 0

File: bodyFiles/body0-10137.urdf (robot description, URDF)
Before this commit: robot robot, 9 links, 8 joints
Links:
- link BackLeg: geometry collision box size=0.2 1.4721250780708013 0.2; visual box size=0.2 1.4721250780708013 0.2
- link BackLowerLeg: geometry collision box size=0.2 0.2 1.0121121790725585; visual box size=0.2 0.2 1.0121121790725585
- link FrontLeg: geometry collision box size=0.2 1.0055909513291912 0.2; visual box size=0.2 1.0055909513291912 0.2
- link FrontLowerLeg: geometry collision box size=0.2 0.2 1.4370448076108762; visual box size=0.2 0.2 1.4370448076108762
- link LeftLeg: geometry collision box size=0.6423330482956809 0.2 0.2; visual box size=0.6423330482956809 0.2 0.2
- link LeftLowerLeg: geometry collision box size=0.2 0.2 1.3601895578999847; visual box size=0.2 0.2 1.3601895578999847
- link RightLeg: geometry collision box size=1.4545113997002583 0.2 0.2; visual box size=1.4545113997002583 0.2 0.2
- link RightLowerLeg: geometry collision box size=0.2 0.2 1.4973523409786937; visual box size=0.2 0.2 1.4973523409786937
Joints:
- joint BackLeg_BackLowerLeg: origin xyz=0 -1.4455804704016542 0 rpy=0 0 0 -> xyz=0 -1.4721250780708013 0 rpy=0 0 0
- joint FrontLeg_FrontLowerLeg: origin xyz=0 0.8113124077355081 0 rpy=0 0 0 -> xyz=0 1.0055909513291912 0 rpy=0 0 0
- joint LeftLeg_LeftLowerLeg: origin xyz=-0.8366582388235175 0 0 rpy=0 0 0 -> xyz=-0.6423330482956809 0 0 rpy=0 0 0
- joint RightLeg_RightLowerLeg: origin xyz=0.9952681383275807 0 0 rpy=0 0 0 -> xyz=1.4545113997002583 0 0 rpy=0 0 0
- joint Torso_BackLeg: origin xyz=0 -10.5 1.4455804704016542 rpy=0 0 0 -> xyz=0 -10.5 1.4973523409786937 rpy=0 0 0
- joint Torso_FrontLeg: origin xyz=0 -9.5 1.4455804704016542 rpy=0 0 0 -> xyz=0 -9.5 1.4973523409786937 rpy=0 0 0
- joint Torso_LeftLeg: origin xyz=-0.5 -10 1.4455804704016542 rpy=0 0 0 -> xyz=-0.5 -10 1.4973523409786937 rpy=0 0 0
- joint Torso_RightLeg: origin xyz=0.5 -10 1.4455804704016542 rpy=0 0 0 -> xyz=0.5 -10 1.4973523409786937 rpy=0 0 0

File: bodyFiles/body0-101507.urdf (robot description, URDF)
Before this commit: robot robot, 9 links, 8 joints
Links:
- link BackLeg: geometry collision box size=0.2 0.83717346823166 0.2; visual box size=0.2 0.83717346823166 0.2
- link BackLowerLeg: geometry collision box size=0.2 0.2 1.2183794893748656; visual box size=0.2 0.2 1.2183794893748656
- link FrontLeg: geometry collision box size=0.2 0.5166145327325473 0.2; visual box size=0.2 0.5166145327325473 0.2
- link FrontLowerLeg: geometry collision box size=0.2 0.2 0.9761319026575341; visual box size=0.2 0.2 0.9761319026575341
- link LeftLeg: geometry collision box size=1.2658863999251788 0.2 0.2; visual box size=1.2658863999251788 0.2 0.2
- link LeftLowerLeg: geometry collision box size=0.2 0.2 1.4121944002354039; visual box size=0.2 0.2 1.4121944002354039
- link RightLeg: geometry collision box size=1.0166368745529817 0.2 0.2; visual box size=1.0166368745529817 0.2 0.2
- link RightLowerLeg: geometry collision box size=0.2 0.2 1.4323832132017371; visual box size=0.2 0.2 1.4323832132017371
Joints:
- joint BackLeg_BackLowerLeg: origin xyz=0 -1.0178675090578977 0 rpy=0 0 0 -> xyz=0 -0.83717346823166 0 rpy=0 0 0
- joint FrontLeg_FrontLowerLeg: origin xyz=0 1.461507310665342 0 rpy=0 0 0 -> xyz=0 0.5166145327325473 0 rpy=0 0 0
- joint LeftLeg_LeftLowerLeg: origin xyz=-0.6499727905386965 0 0 rpy=0 0 0 -> xyz=-1.2658863999251788 0 0 rpy=0 0 0
- joint RightLeg_RightLowerLeg: origin xyz=0.8752522170893827 0 0 rpy=0 0 0 -> xyz=1.0166368745529817 0 0 rpy=0 0 0
- joint Torso_BackLeg: origin xyz=0 -10.5 1.461507310665342 rpy=0 0 0 -> xyz=0 -10.5 1.4323832132017371 rpy=0 0 0
- joint Torso_FrontLeg: origin xyz=0 -9.5 1.461507310665342 rpy=0 0 0 -> xyz=0 -9.5 1.4323832132017371 rpy=0 0 0
- joint Torso_LeftLeg: origin xyz=-0.5 -10 1.461507310665342 rpy=0 0 0 -> xyz=-0.5 -10 1.4323832132017371 rpy=0 0 0
- joint Torso_RightLeg: origin xyz=0.5 -10 1.461507310665342 rpy=0 0 0 -> xyz=0.5 -10 1.4323832132017371 rpy=0 0 0

File: bodyFiles/body0-10168.urdf (robot description, URDF)
Before this commit: robot robot, 9 links, 8 joints
Links:
- link BackLeg: geometry collision box size=0.2 0.8957992395330023 0.2; visual box size=0.2 0.8957992395330023 0.2
- link BackLowerLeg: geometry collision box size=0.2 0.2 1.3772509060821092; visual box size=0.2 0.2 1.3772509060821092
- link FrontLeg: geometry collision box size=0.2 0.6213552899976392 0.2; visual box size=0.2 0.6213552899976392 0.2
- link FrontLowerLeg: geometry collision box size=0.2 0.2 1.2390402365981852; visual box size=0.2 0.2 1.2390402365981852
- link LeftLeg: geometry collision box size=0.8750656020765538 0.2 0.2; visual box size=0.8750656020765538 0.2 0.2
- link LeftLowerLeg: geometry collision box size=0.2 0.2 0.9446966138867552; visual box size=0.2 0.2 0.9446966138867552
- link RightLeg: geometry collision box size=0.7330579563271648 0.2 0.2; visual box size=0.7330579563271648 0.2 0.2
- link RightLowerLeg: geometry collision box size=0.2 0.2 1.364114396944021; visual box size=0.2 0.2 1.364114396944021
Joints:
- joint BackLeg_BackLowerLeg: origin xyz=0 -0.7017383725779895 0 rpy=0 0 0 -> xyz=0 -0.8957992395330023 0 rpy=0 0 0
- joint FrontLeg_FrontLowerLeg: origin xyz=0 0.5538088899067922 0 rpy=0 0 0 -> xyz=0 0.6213552899976392 0 rpy=0 0 0
- joint LeftLeg_LeftLowerLeg: origin xyz=-1.3565833921354797 0 0 rpy=0 0 0 -> xyz=-0.8750656020765538 0 0 rpy=0 0 0
- joint RightLeg_RightLowerLeg: origin xyz=0.7989363977959701 0 0 rpy=0 0 0 -> xyz=0.7330579563271648 0 0 rpy=0 0 0
- joint Torso_BackLeg: origin xyz=0 -10.5 1.3565833921354797 rpy=0 0 0 -> xyz=0 -10.5 1.3772509060821092 rpy=0 0 0
- joint Torso_FrontLeg: origin xyz=0 -9.5 1.3565833921354797 rpy=0 0 0 -> xyz=0 -9.5 1.3772509060821092 rpy=0 0 0
- joint Torso_LeftLeg: origin xyz=-0.5 -10 1.3565833921354797 rpy=0 0 0 -> xyz=-0.5 -10 1.3772509060821092 rpy=0 0 0
- joint Torso_RightLeg: origin xyz=0.5 -10 1.3565833921354797 rpy=0 0 0 -> xyz=0.5 -10 1.3772509060821092 rpy=0 0 0

File: bodyFiles/body0-10205.urdf (robot description, URDF)
Before this commit: robot robot, 9 links, 8 joints
Links:
- link BackLeg: geometry collision box size=0.2 1.0152702177774107 0.2; visual box size=0.2 1.0152702177774107 0.2
- link BackLowerLeg: geometry collision box size=0.2 0.2 0.555737645976476; visual box size=0.2 0.2 0.555737645976476
- link FrontLeg: geometry collision box size=0.2 1.1818595440357793 0.2; visual box size=0.2 1.1818595440357793 0.2
- link FrontLowerLeg: geometry collision box size=0.2 0.2 0.5418361047532666; visual box size=0.2 0.2 0.5418361047532666
- link LeftLeg: geometry collision box size=1.1109999044337173 0.2 0.2; visual box size=1.1109999044337173 0.2 0.2
- link LeftLowerLeg: geometry collision box size=0.2 0.2 1.175557828988788; visual box size=0.2 0.2 1.175557828988788
- link RightLeg: geometry collision box size=0.6586882960173703 0.2 0.2; visual box size=0.6586882960173703 0.2 0.2
- link RightLowerLeg: geometry collision box size=0.2 0.2 1.4419235970029254; visual box size=0.2 0.2 1.4419235970029254
Joints:
- joint BackLeg_BackLowerLeg: origin xyz=0 -0.9933306471853152 0 rpy=0 0 0 -> xyz=0 -1.0152702177774107 0 rpy=0 0 0
- joint FrontLeg_FrontLowerLeg: origin xyz=0 0.5499424636258314 0 rpy=0 0 0 -> xyz=0 1.1818595440357793 0 rpy=0 0 0
- joint LeftLeg_LeftLowerLeg: origin xyz=-1.0228199259811297 0 0 rpy=0 0 0 -> xyz=-1.1109999044337173 0 0 rpy=0 0 0
- joint RightLeg_RightLowerLeg: origin xyz=0.9048807512886035 0 0 rpy=0 0 0 -> xyz=0.6586882960173703 0 0 rpy=0 0 0
- joint Torso_BackLeg: origin xyz=0 -10.5 1.4988554417371127 rpy=0 0 0 -> xyz=0 -10.5 1.4419235970029254 rpy=0 0 0
- joint Torso_FrontLeg: origin xyz=0 -9.5 1.4988554417371127 rpy=0 0 0 -> xyz=0 -9.5 1.4419235970029254 rpy=0 0 0
- joint Torso_LeftLeg: origin xyz=-0.5 -10 1.4988554417371127 rpy=0 0 0 -> xyz=-0.5 -10 1.4419235970029254 rpy=0 0 0
- joint Torso_RightLeg: origin xyz=0.5 -10 1.4988554417371127 rpy=0 0 0 -> xyz=0.5 -10 1.4419235970029254 rpy=0 0 0

File: bodyFiles/body0-102061.urdf (robot description, URDF)
Before this commit: robot robot, 9 links, 8 joints
Links:
- link BackLeg: geometry collision box size=0.2 1.021223953385828 0.2; visual box size=0.2 1.021223953385828 0.2
- link BackLowerLeg: geometry collision box size=0.2 0.2 0.8739637697446571; visual box size=0.2 0.2 0.8739637697446571
- link FrontLeg: geometry collision box size=0.2 1.4727453315695498 0.2; visual box size=0.2 1.4727453315695498 0.2
- link FrontLowerLeg: geometry collision box size=0.2 0.2 0.7302804725345728; visual box size=0.2 0.2 0.7302804725345728
- link LeftLeg: geometry collision box size=1.3030705914710816 0.2 0.2; visual box size=1.3030705914710816 0.2 0.2
- link LeftLowerLeg: geometry collision box size=0.2 0.2 1.0579701181823786; visual box size=0.2 0.2 1.0579701181823786
- link RightLeg: geometry collision box size=0.9288627091874215 0.2 0.2; visual box size=0.9288627091874215 0.2 0.2
- link RightLowerLeg: geometry collision box size=0.2 0.2 0.7289616028660652; visual box size=0.2 0.2 0.7289616028660652
Joints:
- joint BackLeg_BackLowerLeg: origin xyz=0 -1.0294916295982948 0 rpy=0 0 0 -> xyz=0 -1.021223953385828 0 rpy=0 0 0
- joint FrontLeg_FrontLowerLeg: origin xyz=0 1.0668902972510146 0 rpy=0 0 0 -> xyz=0 1.4727453315695498 0 rpy=0 0 0
- joint LeftLeg_LeftLowerLeg: origin xyz=-0.8668718581888003 0 0 rpy=0 0 0 -> xyz=-1.3030705914710816 0 0 rpy=0 0 0
- joint RightLeg_RightLowerLeg: origin xyz=1.4041398672435919 0 0 rpy=0 0 0 -> xyz=0.9288627091874215 0 0 rpy=0 0 0
- joint Torso_BackLeg: origin xyz=0 -10.5 1.4041398672435919 rpy=0 0 0 -> xyz=0 -10.5 1.4727453315695498 rpy=0 0 0
- joint Torso_FrontLeg: origin xyz=0 -9.5 1.4041398672435919 rpy=0 0 0 -> xyz=0 -9.5 1.4727453315695498 rpy=0 0 0
- joint Torso_LeftLeg: origin xyz=-0.5 -10 1.4041398672435919 rpy=0 0 0 -> xyz=-0.5 -10 1.4727453315695498 rpy=0 0 0
- joint Torso_RightLeg: origin xyz=0.5 -10 1.4041398672435919 rpy=0 0 0 -> xyz=0.5 -10 1.4727453315695498 rpy=0 0 0
