Commit message: case3 30 + 10 gens

File: bodyFiles/body0-10238.urdf (robot description, URDF)
Before this commit: robot robot, 9 links, 8 joints
Links:
- link BackLeg: geometry collision box size=0.2 1.308238766062125 0.2; visual box size=0.2 1.308238766062125 0.2
- link BackLowerLeg: geometry collision box size=0.2 0.2 1.3355874681841438; visual box size=0.2 0.2 1.3355874681841438
- link FrontLeg: geometry collision box size=0.2 0.5100555829531151 0.2; visual box size=0.2 0.5100555829531151 0.2
- link FrontLowerLeg: geometry collision box size=0.2 0.2 0.5471653771751359; visual box size=0.2 0.2 0.5471653771751359
- link LeftLeg: geometry collision box size=1.2821848322522111 0.2 0.2; visual box size=1.2821848322522111 0.2 0.2
- link LeftLowerLeg: geometry collision box size=0.2 0.2 1.1076503932998958; visual box size=0.2 0.2 1.1076503932998958
- link RightLeg: geometry collision box size=0.5462528743233537 0.2 0.2; visual box size=0.5462528743233537 0.2 0.2
- link RightLowerLeg: geometry collision box size=0.2 0.2 1.2867655255083394; visual box size=0.2 0.2 1.2867655255083394
Joints:
- joint BackLeg_BackLowerLeg: origin xyz=0 -1.2341379048713943 0 rpy=0 0 0 -> xyz=0 -1.308238766062125 0 rpy=0 0 0
- joint FrontLeg_FrontLowerLeg: origin xyz=0 0.7484249942766722 0 rpy=0 0 0 -> xyz=0 0.5100555829531151 0 rpy=0 0 0
- joint LeftLeg_LeftLowerLeg: origin xyz=-1.204205843418243 0 0 rpy=0 0 0 -> xyz=-1.2821848322522111 0 0 rpy=0 0 0
- joint RightLeg_RightLowerLeg: origin xyz=1.0608023045334956 0 0 rpy=0 0 0 -> xyz=0.5462528743233537 0 0 rpy=0 0 0
- joint Torso_BackLeg: origin xyz=0 -10.5 1.493990491591033 rpy=0 0 0 -> xyz=0 -10.5 1.3355874681841438 rpy=0 0 0
- joint Torso_FrontLeg: origin xyz=0 -9.5 1.493990491591033 rpy=0 0 0 -> xyz=0 -9.5 1.3355874681841438 rpy=0 0 0
- joint Torso_LeftLeg: origin xyz=-0.5 -10 1.493990491591033 rpy=0 0 0 -> xyz=-0.5 -10 1.3355874681841438 rpy=0 0 0
- joint Torso_RightLeg: origin xyz=0.5 -10 1.493990491591033 rpy=0 0 0 -> xyz=0.5 -10 1.3355874681841438 rpy=0 0 0

File: bodyFiles/body0-10270.urdf (robot description, URDF)
Before this commit: robot robot, 9 links, 8 joints
Links:
- link BackLeg: geometry collision box size=0.2 1.332736161975493 0.2; visual box size=0.2 1.332736161975493 0.2
- link BackLowerLeg: geometry collision box size=0.2 0.2 0.5123988318545529; visual box size=0.2 0.2 0.5123988318545529
- link FrontLeg: geometry collision box size=0.2 1.373898456266606 0.2; visual box size=0.2 1.373898456266606 0.2
- link FrontLowerLeg: geometry collision box size=0.2 0.2 0.6389972783890574; visual box size=0.2 0.2 0.6389972783890574
- link LeftLeg: geometry collision box size=0.5382098941602057 0.2 0.2; visual box size=0.5382098941602057 0.2 0.2
- link LeftLowerLeg: geometry collision box size=0.2 0.2 0.8063765432481862; visual box size=0.2 0.2 0.8063765432481862
- link RightLeg: geometry collision box size=0.8993537410944455 0.2 0.2; visual box size=0.8993537410944455 0.2 0.2
- link RightLowerLeg: geometry collision box size=0.2 0.2 1.4114263014231248; visual box size=0.2 0.2 1.4114263014231248
Joints:
- joint BackLeg_BackLowerLeg: origin xyz=0 -0.8609995470923046 0 rpy=0 0 0 -> xyz=0 -1.332736161975493 0 rpy=0 0 0
- joint FrontLeg_FrontLowerLeg: origin xyz=0 0.6827793631085527 0 rpy=0 0 0 -> xyz=0 1.373898456266606 0 rpy=0 0 0
- joint LeftLeg_LeftLowerLeg: origin xyz=-0.8580717514899869 0 0 rpy=0 0 0 -> xyz=-0.5382098941602057 0 0 rpy=0 0 0
- joint RightLeg_RightLowerLeg: origin xyz=1.2783282423140692 0 0 rpy=0 0 0 -> xyz=0.8993537410944455 0 0 rpy=0 0 0
- joint Torso_BackLeg: origin xyz=0 -10.5 1.2783282423140692 rpy=0 0 0 -> xyz=0 -10.5 1.4114263014231248 rpy=0 0 0
- joint Torso_FrontLeg: origin xyz=0 -9.5 1.2783282423140692 rpy=0 0 0 -> xyz=0 -9.5 1.4114263014231248 rpy=0 0 0
- joint Torso_LeftLeg: origin xyz=-0.5 -10 1.2783282423140692 rpy=0 0 0 -> xyz=-0.5 -10 1.4114263014231248 rpy=0 0 0
- joint Torso_RightLeg: origin xyz=0.5 -10 1.2783282423140692 rpy=0 0 0 -> xyz=0.5 -10 1.4114263014231248 rpy=0 0 0

File: bodyFiles/body0-102708.urdf (robot description, URDF)
Before this commit: robot robot, 9 links, 8 joints
Links:
- link BackLeg: geometry collision box size=0.2 1.4335609958766153 0.2; visual box size=0.2 1.4335609958766153 0.2
- link BackLowerLeg: geometry collision box size=0.2 0.2 0.8566787068333914; visual box size=0.2 0.2 0.8566787068333914
- link FrontLeg: geometry collision box size=0.2 1.381667962890016 0.2; visual box size=0.2 1.381667962890016 0.2
- link FrontLowerLeg: geometry collision box size=0.2 0.2 0.7016361834653098; visual box size=0.2 0.2 0.7016361834653098
- link LeftLeg: geometry collision box size=1.3659847623481072 0.2 0.2; visual box size=1.3659847623481072 0.2 0.2
- link LeftLowerLeg: geometry collision box size=0.2 0.2 1.2959989269015004; visual box size=0.2 0.2 1.2959989269015004
- link RightLeg: geometry collision box size=1.3715074854191698 0.2 0.2; visual box size=1.3715074854191698 0.2 0.2
- link RightLowerLeg: geometry collision box size=0.2 0.2 1.2114537866511705; visual box size=0.2 0.2 1.2114537866511705
Joints:
- joint BackLeg_BackLowerLeg: origin xyz=0 -1.3856058199664005 0 rpy=0 0 0 -> xyz=0 -1.4335609958766153 0 rpy=0 0 0
- joint FrontLeg_FrontLowerLeg: origin xyz=0 0.5441351922808386 0 rpy=0 0 0 -> xyz=0 1.381667962890016 0 rpy=0 0 0
- joint LeftLeg_LeftLowerLeg: origin xyz=-0.8293725324920873 0 0 rpy=0 0 0 -> xyz=-1.3659847623481072 0 0 rpy=0 0 0
- joint RightLeg_RightLowerLeg: origin xyz=1.3470876417949174 0 0 rpy=0 0 0 -> xyz=1.3715074854191698 0 0 rpy=0 0 0
- joint Torso_BackLeg: origin xyz=0 -10.5 1.3856058199664005 rpy=0 0 0 -> xyz=0 -10.5 1.4335609958766153 rpy=0 0 0
- joint Torso_FrontLeg: origin xyz=0 -9.5 1.3856058199664005 rpy=0 0 0 -> xyz=0 -9.5 1.4335609958766153 rpy=0 0 0
- joint Torso_LeftLeg: origin xyz=-0.5 -10 1.3856058199664005 rpy=0 0 0 -> xyz=-0.5 -10 1.4335609958766153 rpy=0 0 0
- joint Torso_RightLeg: origin xyz=0.5 -10 1.3856058199664005 rpy=0 0 0 -> xyz=0.5 -10 1.4335609958766153 rpy=0 0 0

File: bodyFiles/body0-10294.urdf (robot description, URDF)
Before this commit: robot robot, 9 links, 8 joints
Links:
- link BackLeg: geometry collision box size=0.2 0.8300346621759594 0.2; visual box size=0.2 0.8300346621759594 0.2
- link BackLowerLeg: geometry collision box size=0.2 0.2 1.0922786195381171; visual box size=0.2 0.2 1.0922786195381171
- link FrontLeg: geometry collision box size=0.2 1.0281112088199822 0.2; visual box size=0.2 1.0281112088199822 0.2
- link FrontLowerLeg: geometry collision box size=0.2 0.2 0.9293072599766146; visual box size=0.2 0.2 0.9293072599766146
- link LeftLeg: geometry collision box size=0.9000379161471664 0.2 0.2; visual box size=0.9000379161471664 0.2 0.2
- link LeftLowerLeg: geometry collision box size=0.2 0.2 0.5275607670797866; visual box size=0.2 0.2 0.5275607670797866
- link RightLeg: geometry collision box size=1.2277469816650475 0.2 0.2; visual box size=1.2277469816650475 0.2 0.2
- link RightLowerLeg: geometry collision box size=0.2 0.2 0.9803727244458229; visual box size=0.2 0.2 0.9803727244458229
Joints:
- joint BackLeg_BackLowerLeg: origin xyz=0 -1.0291908663645837 0 rpy=0 0 0 -> xyz=0 -0.8300346621759594 0 rpy=0 0 0
- joint FrontLeg_FrontLowerLeg: origin xyz=0 1.0729360752972548 0 rpy=0 0 0 -> xyz=0 1.0281112088199822 0 rpy=0 0 0
- joint LeftLeg_LeftLowerLeg: origin xyz=-1.3983166336372341 0 0 rpy=0 0 0 -> xyz=-0.9000379161471664 0 0 rpy=0 0 0
- joint RightLeg_RightLowerLeg: origin xyz=0.840030584090808 0 0 rpy=0 0 0 -> xyz=1.2277469816650475 0 0 rpy=0 0 0
- joint Torso_BackLeg: origin xyz=0 -10.5 1.4156231048203867 rpy=0 0 0 -> xyz=0 -10.5 1.2277469816650475 rpy=0 0 0
- joint Torso_FrontLeg: origin xyz=0 -9.5 1.4156231048203867 rpy=0 0 0 -> xyz=0 -9.5 1.2277469816650475 rpy=0 0 0
- joint Torso_LeftLeg: origin xyz=-0.5 -10 1.4156231048203867 rpy=0 0 0 -> xyz=-0.5 -10 1.2277469816650475 rpy=0 0 0
- joint Torso_RightLeg: origin xyz=0.5 -10 1.4156231048203867 rpy=0 0 0 -> xyz=0.5 -10 1.2277469816650475 rpy=0 0 0

File: bodyFiles/body0-10331.urdf (robot description, URDF)
Before this commit: robot robot, 9 links, 8 joints
Links:
- link BackLeg: geometry collision box size=0.2 0.7002075955727659 0.2; visual box size=0.2 0.7002075955727659 0.2
- link BackLowerLeg: geometry collision box size=0.2 0.2 0.762073555131481; visual box size=0.2 0.2 0.762073555131481
- link FrontLeg: geometry collision box size=0.2 1.0772088781959068 0.2; visual box size=0.2 1.0772088781959068 0.2
- link FrontLowerLeg: geometry collision box size=0.2 0.2 0.870625323023213; visual box size=0.2 0.2 0.870625323023213
- link LeftLeg: geometry collision box size=0.5315787571536681 0.2 0.2; visual box size=0.5315787571536681 0.2 0.2
- link LeftLowerLeg: geometry collision box size=0.2 0.2 0.7734390214819538; visual box size=0.2 0.2 0.7734390214819538
- link RightLeg: geometry collision box size=0.7412517769333762 0.2 0.2; visual box size=0.7412517769333762 0.2 0.2
- link RightLowerLeg: geometry collision box size=0.2 0.2 1.2010222682188858; visual box size=0.2 0.2 1.2010222682188858
Joints:
- joint BackLeg_BackLowerLeg: origin xyz=0 -0.9768473244800686 0 rpy=0 0 0 -> xyz=0 -0.7002075955727659 0 rpy=0 0 0
- joint FrontLeg_FrontLowerLeg: origin xyz=0 0.9115468737011018 0 rpy=0 0 0 -> xyz=0 1.0772088781959068 0 rpy=0 0 0
- joint LeftLeg_LeftLowerLeg: origin xyz=-0.7254360130415088 0 0 rpy=0 0 0 -> xyz=-0.5315787571536681 0 0 rpy=0 0 0
- joint RightLeg_RightLowerLeg: origin xyz=0.7375119893455816 0 0 rpy=0 0 0 -> xyz=0.7412517769333762 0 0 rpy=0 0 0
- joint Torso_BackLeg: origin xyz=0 -10.5 1.1705736753252864 rpy=0 0 0 -> xyz=0 -10.5 1.2010222682188858 rpy=0 0 0
- joint Torso_FrontLeg: origin xyz=0 -9.5 1.1705736753252864 rpy=0 0 0 -> xyz=0 -9.5 1.2010222682188858 rpy=0 0 0
- joint Torso_LeftLeg: origin xyz=-0.5 -10 1.1705736753252864 rpy=0 0 0 -> xyz=-0.5 -10 1.2010222682188858 rpy=0 0 0
- joint Torso_RightLeg: origin xyz=0.5 -10 1.1705736753252864 rpy=0 0 0 -> xyz=0.5 -10 1.2010222682188858 rpy=0 0 0

File: bodyFiles/body0-10362.urdf (robot description, URDF)
Before this commit: robot robot, 9 links, 8 joints
Links:
- link BackLeg: geometry collision box size=0.2 0.6033748038541397 0.2; visual box size=0.2 0.6033748038541397 0.2
- link BackLowerLeg: geometry collision box size=0.2 0.2 0.8175419547028236; visual box size=0.2 0.2 0.8175419547028236
- link FrontLeg: geometry collision box size=0.2 1.4837873380121374 0.2; visual box size=0.2 1.4837873380121374 0.2
- link FrontLowerLeg: geometry collision box size=0.2 0.2 1.320190894718561; visual box size=0.2 0.2 1.320190894718561
- link LeftLeg: geometry collision box size=0.7229844176670539 0.2 0.2; visual box size=0.7229844176670539 0.2 0.2
- link LeftLowerLeg: geometry collision box size=0.2 0.2 1.2892878178320046; visual box size=0.2 0.2 1.2892878178320046
- link RightLeg: geometry collision box size=0.7176645827522474 0.2 0.2; visual box size=0.7176645827522474 0.2 0.2
- link RightLowerLeg: geometry collision box size=0.2 0.2 1.1932484372781043; visual box size=0.2 0.2 1.1932484372781043
Joints:
- joint BackLeg_BackLowerLeg: origin xyz=0 -1.1880091604116594 0 rpy=0 0 0 -> xyz=0 -0.6033748038541397 0 rpy=0 0 0
- joint FrontLeg_FrontLowerLeg: origin xyz=0 0.5884925214238024 0 rpy=0 0 0 -> xyz=0 1.4837873380121374 0 rpy=0 0 0
- joint LeftLeg_LeftLowerLeg: origin xyz=-0.9749709917333791 0 0 rpy=0 0 0 -> xyz=-0.7229844176670539 0 0 rpy=0 0 0
- joint RightLeg_RightLowerLeg: origin xyz=0.852847203483727 0 0 rpy=0 0 0 -> xyz=0.7176645827522474 0 0 rpy=0 0 0
- joint Torso_BackLeg: origin xyz=0 -10.5 1.497453426942767 rpy=0 0 0 -> xyz=0 -10.5 1.4837873380121374 rpy=0 0 0
- joint Torso_FrontLeg: origin xyz=0 -9.5 1.497453426942767 rpy=0 0 0 -> xyz=0 -9.5 1.4837873380121374 rpy=0 0 0
- joint Torso_LeftLeg: origin xyz=-0.5 -10 1.497453426942767 rpy=0 0 0 -> xyz=-0.5 -10 1.4837873380121374 rpy=0 0 0
- joint Torso_RightLeg: origin xyz=0.5 -10 1.497453426942767 rpy=0 0 0 -> xyz=0.5 -10 1.4837873380121374 rpy=0 0 0

File: bodyFiles/body0-10394.urdf (robot description, URDF)
Before this commit: robot robot, 9 links, 8 joints
Links:
- link BackLeg: geometry collision box size=0.2 0.7824190101466302 0.2; visual box size=0.2 0.7824190101466302 0.2
- link BackLowerLeg: geometry collision box size=0.2 0.2 0.8946706269061365; visual box size=0.2 0.2 0.8946706269061365
- link FrontLeg: geometry collision box size=0.2 1.1923372474192695 0.2; visual box size=0.2 1.1923372474192695 0.2
- link FrontLowerLeg: geometry collision box size=0.2 0.2 1.0001785781609964; visual box size=0.2 0.2 1.0001785781609964
- link LeftLeg: geometry collision box size=1.1852274405294783 0.2 0.2; visual box size=1.1852274405294783 0.2 0.2
- link LeftLowerLeg: geometry collision box size=0.2 0.2 1.1918591731510202; visual box size=0.2 0.2 1.1918591731510202
- link RightLeg: geometry collision box size=1.444963820770453 0.2 0.2; visual box size=1.444963820770453 0.2 0.2
- link RightLowerLeg: geometry collision box size=0.2 0.2 1.1072558252500837; visual box size=0.2 0.2 1.1072558252500837
Joints:
- joint BackLeg_BackLowerLeg: origin xyz=0 -0.7780762490842805 0 rpy=0 0 0 -> xyz=0 -0.7824190101466302 0 rpy=0 0 0
- joint FrontLeg_FrontLowerLeg: origin xyz=0 1.1709503448629313 0 rpy=0 0 0 -> xyz=0 1.1923372474192695 0 rpy=0 0 0
- joint LeftLeg_LeftLowerLeg: origin xyz=-1.2988537357417826 0 0 rpy=0 0 0 -> xyz=-1.1852274405294783 0 0 rpy=0 0 0
- joint RightLeg_RightLowerLeg: origin xyz=1.1634542180068603 0 0 rpy=0 0 0 -> xyz=1.444963820770453 0 0 rpy=0 0 0
- joint Torso_BackLeg: origin xyz=0 -10.5 1.411781124053236 rpy=0 0 0 -> xyz=0 -10.5 1.444963820770453 rpy=0 0 0
- joint Torso_FrontLeg: origin xyz=0 -9.5 1.411781124053236 rpy=0 0 0 -> xyz=0 -9.5 1.444963820770453 rpy=0 0 0
- joint Torso_LeftLeg: origin xyz=-0.5 -10 1.411781124053236 rpy=0 0 0 -> xyz=-0.5 -10 1.444963820770453 rpy=0 0 0
- joint Torso_RightLeg: origin xyz=0.5 -10 1.411781124053236 rpy=0 0 0 -> xyz=0.5 -10 1.444963820770453 rpy=0 0 0

File: bodyFiles/body0-10424.urdf (robot description, URDF)
Before this commit: robot robot, 9 links, 8 joints
Links:
- link BackLeg: geometry collision box size=0.2 0.7716882831634692 0.2; visual box size=0.2 0.7716882831634692 0.2
- link BackLowerLeg: geometry collision box size=0.2 0.2 0.9564086636781312; visual box size=0.2 0.2 0.9564086636781312
- link FrontLeg: geometry collision box size=0.2 1.2931717314186728 0.2; visual box size=0.2 1.2931717314186728 0.2
- link FrontLowerLeg: geometry collision box size=0.2 0.2 0.8104318169120022; visual box size=0.2 0.2 0.8104318169120022
- link LeftLeg: geometry collision box size=1.353904564670244 0.2 0.2; visual box size=1.353904564670244 0.2 0.2
- link LeftLowerLeg: geometry collision box size=0.2 0.2 0.5056925209366346; visual box size=0.2 0.2 0.5056925209366346
- link RightLeg: geometry collision box size=0.8864655784055064 0.2 0.2; visual box size=0.8864655784055064 0.2 0.2
- link RightLowerLeg: geometry collision box size=0.2 0.2 1.1708454141454985; visual box size=0.2 0.2 1.1708454141454985
Joints:
- joint BackLeg_BackLowerLeg: origin xyz=0 -0.5970805739012087 0 rpy=0 0 0 -> xyz=0 -0.7716882831634692 0 rpy=0 0 0
- joint FrontLeg_FrontLowerLeg: origin xyz=0 0.5076242801966585 0 rpy=0 0 0 -> xyz=0 1.2931717314186728 0 rpy=0 0 0
- joint LeftLeg_LeftLowerLeg: origin xyz=-0.6239896656589309 0 0 rpy=0 0 0 -> xyz=-1.353904564670244 0 0 rpy=0 0 0
- joint RightLeg_RightLowerLeg: origin xyz=0.6075930639132393 0 0 rpy=0 0 0 -> xyz=0.8864655784055064 0 0 rpy=0 0 0
- joint Torso_BackLeg: origin xyz=0 -10.5 1.4971888728080764 rpy=0 0 0 -> xyz=0 -10.5 1.353904564670244 rpy=0 0 0
- joint Torso_FrontLeg: origin xyz=0 -9.5 1.4971888728080764 rpy=0 0 0 -> xyz=0 -9.5 1.353904564670244 rpy=0 0 0
- joint Torso_LeftLeg: origin xyz=-0.5 -10 1.4971888728080764 rpy=0 0 0 -> xyz=-0.5 -10 1.353904564670244 rpy=0 0 0
- joint Torso_RightLeg: origin xyz=0.5 -10 1.4971888728080764 rpy=0 0 0 -> xyz=0.5 -10 1.353904564670244 rpy=0 0 0

File: bodyFiles/body0-10447.urdf (robot description, URDF)
Before this commit: robot robot, 9 links, 8 joints
Links:
- link BackLeg: geometry collision box size=0.2 1.0612523145980859 0.2; visual box size=0.2 1.0612523145980859 0.2
- link BackLowerLeg: geometry collision box size=0.2 0.2 1.0526098156054569; visual box size=0.2 0.2 1.0526098156054569
- link FrontLeg: geometry collision box size=0.2 1.4825473132875935 0.2; visual box size=0.2 1.4825473132875935 0.2
- link FrontLowerLeg: geometry collision box size=0.2 0.2 0.9544126548928862; visual box size=0.2 0.2 0.9544126548928862
- link LeftLeg: geometry collision box size=0.5516478145255159 0.2 0.2; visual box size=0.5516478145255159 0.2 0.2
- link LeftLowerLeg: geometry collision box size=0.2 0.2 1.3122930457294268; visual box size=0.2 0.2 1.3122930457294268
- link RightLeg: geometry collision box size=1.3539026951956687 0.2 0.2; visual box size=1.3539026951956687 0.2 0.2
- link RightLowerLeg: geometry collision box size=0.2 0.2 0.7178937330526155; visual box size=0.2 0.2 0.7178937330526155
Joints:
- joint BackLeg_BackLowerLeg: origin xyz=0 -0.8955937713285282 0 rpy=0 0 0 -> xyz=0 -1.0612523145980859 0 rpy=0 0 0
- joint FrontLeg_FrontLowerLeg: origin xyz=0 0.8381006876048214 0 rpy=0 0 0 -> xyz=0 1.4825473132875935 0 rpy=0 0 0
- joint LeftLeg_LeftLowerLeg: origin xyz=-0.8339658600036215 0 0 rpy=0 0 0 -> xyz=-0.5516478145255159 0 0 rpy=0 0 0
- joint RightLeg_RightLowerLeg: origin xyz=0.6895412746407268 0 0 rpy=0 0 0 -> xyz=1.3539026951956687 0 0 rpy=0 0 0
- joint Torso_BackLeg: origin xyz=0 -10.5 1.3013562796697673 rpy=0 0 0 -> xyz=0 -10.5 1.4825473132875935 rpy=0 0 0
- joint Torso_FrontLeg: origin xyz=0 -9.5 1.3013562796697673 rpy=0 0 0 -> xyz=0 -9.5 1.4825473132875935 rpy=0 0 0
- joint Torso_LeftLeg: origin xyz=-0.5 -10 1.3013562796697673 rpy=0 0 0 -> xyz=-0.5 -10 1.4825473132875935 rpy=0 0 0
- joint Torso_RightLeg: origin xyz=0.5 -10 1.3013562796697673 rpy=0 0 0 -> xyz=0.5 -10 1.4825473132875935 rpy=0 0 0
