Commit message: 40 gens, case3

File: bodyFiles/body0-101461.urdf (robot description, URDF)
Before this commit: robot robot, 9 links, 8 joints
Links:
- link BackLeg: geometry collision box size=0.2 1.256290379959517 0.2; visual box size=0.2 1.256290379959517 0.2
- link BackLowerLeg: geometry collision box size=0.2 0.2 1.29983055795377; visual box size=0.2 0.2 1.29983055795377
- link FrontLeg: geometry collision box size=0.2 1.194318478505912 0.2; visual box size=0.2 1.194318478505912 0.2
- link FrontLowerLeg: geometry collision box size=0.2 0.2 1.3123024128651148; visual box size=0.2 0.2 1.3123024128651148
- link LeftLeg: geometry collision box size=1.1442408422310812 0.2 0.2; visual box size=1.1442408422310812 0.2 0.2
- link LeftLowerLeg: geometry collision box size=0.2 0.2 1.4739001519640096; visual box size=0.2 0.2 1.4739001519640096
- link RightLeg: geometry collision box size=0.7297983158498352 0.2 0.2; visual box size=0.7297983158498352 0.2 0.2
- link RightLowerLeg: geometry collision box size=0.2 0.2 1.3672102855234378; visual box size=0.2 0.2 1.3672102855234378
Joints:
- joint BackLeg_BackLowerLeg: origin xyz=0 -0.635349440316557 0 rpy=0 0 0 -> xyz=0 -1.256290379959517 0 rpy=0 0 0
- joint FrontLeg_FrontLowerLeg: origin xyz=0 1.0020342571753433 0 rpy=0 0 0 -> xyz=0 1.194318478505912 0 rpy=0 0 0
- joint LeftLeg_LeftLowerLeg: origin xyz=-1.1001938302422816 0 0 rpy=0 0 0 -> xyz=-1.1442408422310812 0 0 rpy=0 0 0
- joint RightLeg_RightLowerLeg: origin xyz=1.3000643786854418 0 0 rpy=0 0 0 -> xyz=0.7297983158498352 0 0 rpy=0 0 0
- joint Torso_BackLeg: origin xyz=0 -10.5 1.3085838488192496 rpy=0 0 0 -> xyz=0 -10.5 1.4739001519640096 rpy=0 0 0
- joint Torso_FrontLeg: origin xyz=0 -9.5 1.3085838488192496 rpy=0 0 0 -> xyz=0 -9.5 1.4739001519640096 rpy=0 0 0
- joint Torso_LeftLeg: origin xyz=-0.5 -10 1.3085838488192496 rpy=0 0 0 -> xyz=-0.5 -10 1.4739001519640096 rpy=0 0 0
- joint Torso_RightLeg: origin xyz=0.5 -10 1.3085838488192496 rpy=0 0 0 -> xyz=0.5 -10 1.4739001519640096 rpy=0 0 0

File: bodyFiles/body0-141156.urdf (robot description, URDF)
Before this commit: robot robot, 9 links, 8 joints
Links:
- link BackLeg: geometry collision box size=0.2 1.276135923532396 0.2; visual box size=0.2 1.276135923532396 0.2
- link BackLowerLeg: geometry collision box size=0.2 0.2 0.7245256008057916; visual box size=0.2 0.2 0.7245256008057916
- link FrontLeg: geometry collision box size=0.2 0.5223191996440701 0.2; visual box size=0.2 0.5223191996440701 0.2
- link FrontLowerLeg: geometry collision box size=0.2 0.2 1.4164239340584606; visual box size=0.2 0.2 1.4164239340584606
- link LeftLeg: geometry collision box size=1.254757743529098 0.2 0.2; visual box size=1.254757743529098 0.2 0.2
- link LeftLowerLeg: geometry collision box size=0.2 0.2 0.5721621865960849; visual box size=0.2 0.2 0.5721621865960849
- link RightLeg: geometry collision box size=0.6725535365314553 0.2 0.2; visual box size=0.6725535365314553 0.2 0.2
- link RightLowerLeg: geometry collision box size=0.2 0.2 1.376004320889158; visual box size=0.2 0.2 1.376004320889158
Joints:
- joint BackLeg_BackLowerLeg: origin xyz=0 -0.8062655453653834 0 rpy=0 0 0 -> xyz=0 -1.276135923532396 0 rpy=0 0 0
- joint FrontLeg_FrontLowerLeg: origin xyz=0 1.2016146616545966 0 rpy=0 0 0 -> xyz=0 0.5223191996440701 0 rpy=0 0 0
- joint LeftLeg_LeftLowerLeg: origin xyz=-1.142950279216683 0 0 rpy=0 0 0 -> xyz=-1.254757743529098 0 0 rpy=0 0 0
- joint RightLeg_RightLowerLeg: origin xyz=0.9077452407167629 0 0 rpy=0 0 0 -> xyz=0.6725535365314553 0 0 rpy=0 0 0
- joint Torso_BackLeg: origin xyz=0 -14.5 1.3957969457807038 rpy=0 0 0 -> xyz=0 -14.5 1.4164239340584606 rpy=0 0 0
- joint Torso_FrontLeg: origin xyz=0 -13.5 1.3957969457807038 rpy=0 0 0 -> xyz=0 -13.5 1.4164239340584606 rpy=0 0 0
- joint Torso_LeftLeg: origin xyz=-0.5 -14 1.3957969457807038 rpy=0 0 0 -> xyz=-0.5 -14 1.4164239340584606 rpy=0 0 0
- joint Torso_RightLeg: origin xyz=0.5 -14 1.3957969457807038 rpy=0 0 0 -> xyz=0.5 -14 1.4164239340584606 rpy=0 0 0

File: bodyFiles/body0-181200.urdf (robot description, URDF)
Before this commit: robot robot, 9 links, 8 joints
Links:
- link BackLeg: geometry collision box size=0.2 1.1209992145464955 0.2; visual box size=0.2 1.1209992145464955 0.2
- link BackLowerLeg: geometry collision box size=0.2 0.2 0.633712083231718; visual box size=0.2 0.2 0.633712083231718
- link FrontLeg: geometry collision box size=0.2 0.8096485676193975 0.2; visual box size=0.2 0.8096485676193975 0.2
- link FrontLowerLeg: geometry collision box size=0.2 0.2 1.374008045882197; visual box size=0.2 0.2 1.374008045882197
- link LeftLeg: geometry collision box size=0.8389341950862839 0.2 0.2; visual box size=0.8389341950862839 0.2 0.2
- link LeftLowerLeg: geometry collision box size=0.2 0.2 1.301950222953165; visual box size=0.2 0.2 1.301950222953165
- link RightLeg: geometry collision box size=1.156347451251271 0.2 0.2; visual box size=1.156347451251271 0.2 0.2
- link RightLowerLeg: geometry collision box size=0.2 0.2 0.872083918136901; visual box size=0.2 0.2 0.872083918136901
Joints:
- joint BackLeg_BackLowerLeg: origin xyz=0 -1.379733767253625 0 rpy=0 0 0 -> xyz=0 -1.1209992145464955 0 rpy=0 0 0
- joint FrontLeg_FrontLowerLeg: origin xyz=0 1.3764348528677333 0 rpy=0 0 0 -> xyz=0 0.8096485676193975 0 rpy=0 0 0
- joint LeftLeg_LeftLowerLeg: origin xyz=-1.4135444864081288 0 0 rpy=0 0 0 -> xyz=-0.8389341950862839 0 0 rpy=0 0 0
- joint RightLeg_RightLowerLeg: origin xyz=0.8028471076985344 0 0 rpy=0 0 0 -> xyz=1.156347451251271 0 0 rpy=0 0 0
- joint Torso_BackLeg: origin xyz=0 -18.5 1.4135444864081288 rpy=0 0 0 -> xyz=0 -18.5 1.374008045882197 rpy=0 0 0
- joint Torso_FrontLeg: origin xyz=0 -17.5 1.4135444864081288 rpy=0 0 0 -> xyz=0 -17.5 1.374008045882197 rpy=0 0 0
- joint Torso_LeftLeg: origin xyz=-0.5 -18 1.4135444864081288 rpy=0 0 0 -> xyz=-0.5 -18 1.374008045882197 rpy=0 0 0
- joint Torso_RightLeg: origin xyz=0.5 -18 1.4135444864081288 rpy=0 0 0 -> xyz=0.5 -18 1.374008045882197 rpy=0 0 0

File: bodyFiles/body0-18502.urdf (robot description, URDF)
Before this commit: robot robot, 9 links, 8 joints
Links:
- link BackLeg: geometry collision box size=0.2 0.9474699921212033 0.2; visual box size=0.2 0.9474699921212033 0.2
- link BackLowerLeg: geometry collision box size=0.2 0.2 0.5257976375785741; visual box size=0.2 0.2 0.5257976375785741
- link FrontLeg: geometry collision box size=0.2 1.2577952846465021 0.2; visual box size=0.2 1.2577952846465021 0.2
- link FrontLowerLeg: geometry collision box size=0.2 0.2 1.3963850742271937; visual box size=0.2 0.2 1.3963850742271937
- link LeftLeg: geometry collision box size=0.5797927358417887 0.2 0.2; visual box size=0.5797927358417887 0.2 0.2
- link LeftLowerLeg: geometry collision box size=0.2 0.2 1.1327412860747748; visual box size=0.2 0.2 1.1327412860747748
- link RightLeg: geometry collision box size=1.3733392885213 0.2 0.2; visual box size=1.3733392885213 0.2 0.2
- link RightLowerLeg: geometry collision box size=0.2 0.2 1.1468807179848624; visual box size=0.2 0.2 1.1468807179848624
Joints:
- joint BackLeg_BackLowerLeg: origin xyz=0 -1.4461786418295652 0 rpy=0 0 0 -> xyz=0 -0.9474699921212033 0 rpy=0 0 0
- joint FrontLeg_FrontLowerLeg: origin xyz=0 1.481408787299642 0 rpy=0 0 0 -> xyz=0 1.2577952846465021 0 rpy=0 0 0
- joint LeftLeg_LeftLowerLeg: origin xyz=-1.2635982645108557 0 0 rpy=0 0 0 -> xyz=-0.5797927358417887 0 0 rpy=0 0 0
- joint RightLeg_RightLowerLeg: origin xyz=1.3361653166969232 0 0 rpy=0 0 0 -> xyz=1.3733392885213 0 0 rpy=0 0 0
- joint Torso_BackLeg: origin xyz=0 -18.5 1.481408787299642 rpy=0 0 0 -> xyz=0 -18.5 1.3963850742271937 rpy=0 0 0
- joint Torso_FrontLeg: origin xyz=0 -17.5 1.481408787299642 rpy=0 0 0 -> xyz=0 -17.5 1.3963850742271937 rpy=0 0 0
- joint Torso_LeftLeg: origin xyz=-0.5 -18 1.481408787299642 rpy=0 0 0 -> xyz=-0.5 -18 1.3963850742271937 rpy=0 0 0
- joint Torso_RightLeg: origin xyz=0.5 -18 1.481408787299642 rpy=0 0 0 -> xyz=0.5 -18 1.3963850742271937 rpy=0 0 0

File: bodyFiles/body0-21470.urdf (robot description, URDF)
Before this commit: robot robot, 9 links, 8 joints
Links:
- link BackLeg: geometry collision box size=0.2 1.4554927726374078 0.2; visual box size=0.2 1.4554927726374078 0.2
- link BackLowerLeg: geometry collision box size=0.2 0.2 1.3694434225374028; visual box size=0.2 0.2 1.3694434225374028
- link FrontLeg: geometry collision box size=0.2 0.9530186964514228 0.2; visual box size=0.2 0.9530186964514228 0.2
- link FrontLowerLeg: geometry collision box size=0.2 0.2 0.858278573469119; visual box size=0.2 0.2 0.858278573469119
- link LeftLeg: geometry collision box size=0.6646497517108465 0.2 0.2; visual box size=0.6646497517108465 0.2 0.2
- link LeftLowerLeg: geometry collision box size=0.2 0.2 1.25362895009687; visual box size=0.2 0.2 1.25362895009687
- link RightLeg: geometry collision box size=1.1337428445827296 0.2 0.2; visual box size=1.1337428445827296 0.2 0.2
- link RightLowerLeg: geometry collision box size=0.2 0.2 1.4356201943907347; visual box size=0.2 0.2 1.4356201943907347
Joints:
- joint BackLeg_BackLowerLeg: origin xyz=0 -0.8659680416252934 0 rpy=0 0 0 -> xyz=0 -1.4554927726374078 0 rpy=0 0 0
- joint FrontLeg_FrontLowerLeg: origin xyz=0 0.9790115182328045 0 rpy=0 0 0 -> xyz=0 0.9530186964514228 0 rpy=0 0 0
- joint LeftLeg_LeftLowerLeg: origin xyz=-1.1549901638202265 0 0 rpy=0 0 0 -> xyz=-0.6646497517108465 0 0 rpy=0 0 0
- joint RightLeg_RightLowerLeg: origin xyz=0.8008937238912316 0 0 rpy=0 0 0 -> xyz=1.1337428445827296 0 0 rpy=0 0 0
- joint Torso_BackLeg: origin xyz=0 -2.5 1.4828693895516194 rpy=0 0 0 -> xyz=0 -2.5 1.4554927726374078 rpy=0 0 0
- joint Torso_FrontLeg: origin xyz=0 -1.5 1.4828693895516194 rpy=0 0 0 -> xyz=0 -1.5 1.4554927726374078 rpy=0 0 0
- joint Torso_LeftLeg: origin xyz=-0.5 -2 1.4828693895516194 rpy=0 0 0 -> xyz=-0.5 -2 1.4554927726374078 rpy=0 0 0
- joint Torso_RightLeg: origin xyz=0.5 -2 1.4828693895516194 rpy=0 0 0 -> xyz=0.5 -2 1.4554927726374078 rpy=0 0 0

File: bodyFiles/body0-2370.urdf (robot description, URDF)
Before this commit: robot robot, 9 links, 8 joints
Links:
- link BackLeg: geometry collision box size=0.2 0.5369334449534202 0.2; visual box size=0.2 0.5369334449534202 0.2
- link BackLowerLeg: geometry collision box size=0.2 0.2 1.024014290609204; visual box size=0.2 0.2 1.024014290609204
- link FrontLeg: geometry collision box size=0.2 1.1947985126848213 0.2; visual box size=0.2 1.1947985126848213 0.2
- link FrontLowerLeg: geometry collision box size=0.2 0.2 1.2915961771464792; visual box size=0.2 0.2 1.2915961771464792
- link LeftLeg: geometry collision box size=1.0764112378783537 0.2 0.2; visual box size=1.0764112378783537 0.2 0.2
- link LeftLowerLeg: geometry collision box size=0.2 0.2 0.7329319328712012; visual box size=0.2 0.2 0.7329319328712012
- link RightLeg: geometry collision box size=0.7978552014274994 0.2 0.2; visual box size=0.7978552014274994 0.2 0.2
- link RightLowerLeg: geometry collision box size=0.2 0.2 1.2101339024963815; visual box size=0.2 0.2 1.2101339024963815
Joints:
- joint BackLeg_BackLowerLeg: origin xyz=0 -1.472919263422802 0 rpy=0 0 0 -> xyz=0 -0.5369334449534202 0 rpy=0 0 0
- joint FrontLeg_FrontLowerLeg: origin xyz=0 1.1756043260679614 0 rpy=0 0 0 -> xyz=0 1.1947985126848213 0 rpy=0 0 0
- joint LeftLeg_LeftLowerLeg: origin xyz=-1.2175127091592357 0 0 rpy=0 0 0 -> xyz=-1.0764112378783537 0 0 rpy=0 0 0
- joint RightLeg_RightLowerLeg: origin xyz=1.3849763984130359 0 0 rpy=0 0 0 -> xyz=0.7978552014274994 0 0 rpy=0 0 0
- joint Torso_BackLeg: origin xyz=0 -2.5 1.499105817678516 rpy=0 0 0 -> xyz=0 -2.5 1.2915961771464792 rpy=0 0 0
- joint Torso_FrontLeg: origin xyz=0 -1.5 1.499105817678516 rpy=0 0 0 -> xyz=0 -1.5 1.2915961771464792 rpy=0 0 0
- joint Torso_LeftLeg: origin xyz=-0.5 -2 1.499105817678516 rpy=0 0 0 -> xyz=-0.5 -2 1.2915961771464792 rpy=0 0 0
- joint Torso_RightLeg: origin xyz=0.5 -2 1.499105817678516 rpy=0 0 0 -> xyz=0.5 -2 1.2915961771464792 rpy=0 0 0

File: bodyFiles/body0-61516.urdf (robot description, URDF)
Before this commit: robot robot, 9 links, 8 joints
Links:
- link BackLeg: geometry collision box size=0.2 1.0605863293763655 0.2; visual box size=0.2 1.0605863293763655 0.2
- link BackLowerLeg: geometry collision box size=0.2 0.2 0.7646907463628495; visual box size=0.2 0.2 0.7646907463628495
- link FrontLeg: geometry collision box size=0.2 0.6532258429790402 0.2; visual box size=0.2 0.6532258429790402 0.2
- link FrontLowerLeg: geometry collision box size=0.2 0.2 0.7672307306723557; visual box size=0.2 0.2 0.7672307306723557
- link LeftLeg: geometry collision box size=1.3896704845139833 0.2 0.2; visual box size=1.3896704845139833 0.2 0.2
- link LeftLowerLeg: geometry collision box size=0.2 0.2 0.8581543059353828; visual box size=0.2 0.2 0.8581543059353828
- link RightLeg: geometry collision box size=0.6037375478739105 0.2 0.2; visual box size=0.6037375478739105 0.2 0.2
- link RightLowerLeg: geometry collision box size=0.2 0.2 1.0011485729804481; visual box size=0.2 0.2 1.0011485729804481
Joints:
- joint BackLeg_BackLowerLeg: origin xyz=0 -0.9112695730422359 0 rpy=0 0 0 -> xyz=0 -1.0605863293763655 0 rpy=0 0 0
- joint FrontLeg_FrontLowerLeg: origin xyz=0 1.3575298627472225 0 rpy=0 0 0 -> xyz=0 0.6532258429790402 0 rpy=0 0 0
- joint LeftLeg_LeftLowerLeg: origin xyz=-1.2784107623670409 0 0 rpy=0 0 0 -> xyz=-1.3896704845139833 0 0 rpy=0 0 0
- joint RightLeg_RightLowerLeg: origin xyz=1.4408407642789811 0 0 rpy=0 0 0 -> xyz=0.6037375478739105 0 0 rpy=0 0 0
- joint Torso_BackLeg: origin xyz=0 -6.5 1.4408407642789811 rpy=0 0 0 -> xyz=0 -6.5 1.3896704845139833 rpy=0 0 0
- joint Torso_FrontLeg: origin xyz=0 -5.5 1.4408407642789811 rpy=0 0 0 -> xyz=0 -5.5 1.3896704845139833 rpy=0 0 0
- joint Torso_LeftLeg: origin xyz=-0.5 -6 1.4408407642789811 rpy=0 0 0 -> xyz=-0.5 -6 1.3896704845139833 rpy=0 0 0
- joint Torso_RightLeg: origin xyz=0.5 -6 1.4408407642789811 rpy=0 0 0 -> xyz=0.5 -6 1.3896704845139833 rpy=0 0 0

File: bodyFiles/body0-6367.urdf (robot description, URDF)
Before this commit: robot robot, 9 links, 8 joints
Links:
- link BackLeg: geometry collision box size=0.2 0.5798199071479987 0.2; visual box size=0.2 0.5798199071479987 0.2
- link BackLowerLeg: geometry collision box size=0.2 0.2 0.7224295232076116; visual box size=0.2 0.2 0.7224295232076116
- link FrontLeg: geometry collision box size=0.2 0.5228156591038826 0.2; visual box size=0.2 0.5228156591038826 0.2
- link FrontLowerLeg: geometry collision box size=0.2 0.2 0.5745429068733398; visual box size=0.2 0.2 0.5745429068733398
- link LeftLeg: geometry collision box size=1.1705909165218196 0.2 0.2; visual box size=1.1705909165218196 0.2 0.2
- link LeftLowerLeg: geometry collision box size=0.2 0.2 0.6863412648217606; visual box size=0.2 0.2 0.6863412648217606
- link RightLeg: geometry collision box size=0.5825364590992408 0.2 0.2; visual box size=0.5825364590992408 0.2 0.2
- link RightLowerLeg: geometry collision box size=0.2 0.2 0.9424688347610302; visual box size=0.2 0.2 0.9424688347610302
Joints:
- joint BackLeg_BackLowerLeg: origin xyz=0 -1.0583898059059398 0 rpy=0 0 0 -> xyz=0 -0.5798199071479987 0 rpy=0 0 0
- joint FrontLeg_FrontLowerLeg: origin xyz=0 1.2297562584699147 0 rpy=0 0 0 -> xyz=0 0.5228156591038826 0 rpy=0 0 0
- joint LeftLeg_LeftLowerLeg: origin xyz=-1.1080670416800442 0 0 rpy=0 0 0 -> xyz=-1.1705909165218196 0 0 rpy=0 0 0
- joint RightLeg_RightLowerLeg: origin xyz=1.2531490133544478 0 0 rpy=0 0 0 -> xyz=0.5825364590992408 0 0 rpy=0 0 0
- joint Torso_BackLeg: origin xyz=0 -6.5 1.3559842617857751 rpy=0 0 0 -> xyz=0 -6.5 1.1705909165218196 rpy=0 0 0
- joint Torso_FrontLeg: origin xyz=0 -5.5 1.3559842617857751 rpy=0 0 0 -> xyz=0 -5.5 1.1705909165218196 rpy=0 0 0
- joint Torso_LeftLeg: origin xyz=-0.5 -6 1.3559842617857751 rpy=0 0 0 -> xyz=-0.5 -6 1.1705909165218196 rpy=0 0 0
- joint Torso_RightLeg: origin xyz=0.5 -6 1.3559842617857751 rpy=0 0 0 -> xyz=0.5 -6 1.1705909165218196 rpy=0 0 0

File: bodyFiles/body0-6566.urdf (robot description, URDF)
Before this commit: robot robot, 9 links, 8 joints
Links:
- link BackLeg: geometry collision box size=0.2 0.5144396728177685 0.2; visual box size=0.2 0.5144396728177685 0.2
- link BackLowerLeg: geometry collision box size=0.2 0.2 0.798049802629262; visual box size=0.2 0.2 0.798049802629262
- link FrontLeg: geometry collision box size=0.2 0.5582150408078059 0.2; visual box size=0.2 0.5582150408078059 0.2
- link FrontLowerLeg: geometry collision box size=0.2 0.2 1.45082799476053; visual box size=0.2 0.2 1.45082799476053
- link LeftLeg: geometry collision box size=0.753885115891021 0.2 0.2; visual box size=0.753885115891021 0.2 0.2
- link LeftLowerLeg: geometry collision box size=0.2 0.2 0.6857405285745108; visual box size=0.2 0.2 0.6857405285745108
- link RightLeg: geometry collision box size=0.9054158648925432 0.2 0.2; visual box size=0.9054158648925432 0.2 0.2
- link RightLowerLeg: geometry collision box size=0.2 0.2 0.6935740283354543; visual box size=0.2 0.2 0.6935740283354543
Joints:
- joint BackLeg_BackLowerLeg: origin xyz=0 -1.3643942629705528 0 rpy=0 0 0 -> xyz=0 -0.5144396728177685 0 rpy=0 0 0
- joint FrontLeg_FrontLowerLeg: origin xyz=0 1.2271972724077418 0 rpy=0 0 0 -> xyz=0 0.5582150408078059 0 rpy=0 0 0
- joint LeftLeg_LeftLowerLeg: origin xyz=-0.8292206236305696 0 0 rpy=0 0 0 -> xyz=-0.753885115891021 0 0 rpy=0 0 0
- joint RightLeg_RightLowerLeg: origin xyz=1.4889483958034466 0 0 rpy=0 0 0 -> xyz=0.9054158648925432 0 0 rpy=0 0 0
- joint Torso_BackLeg: origin xyz=0 -6.5 1.4889483958034466 rpy=0 0 0 -> xyz=0 -6.5 1.45082799476053 rpy=0 0 0
- joint Torso_FrontLeg: origin xyz=0 -5.5 1.4889483958034466 rpy=0 0 0 -> xyz=0 -5.5 1.45082799476053 rpy=0 0 0
- joint Torso_LeftLeg: origin xyz=-0.5 -6 1.4889483958034466 rpy=0 0 0 -> xyz=-0.5 -6 1.45082799476053 rpy=0 0 0
- joint Torso_RightLeg: origin xyz=0.5 -6 1.4889483958034466 rpy=0 0 0 -> xyz=0.5 -6 1.45082799476053 rpy=0 0 0

File: bodyFiles/body0101335.urdf (robot description, URDF)
Before this commit: robot robot, 9 links, 8 joints
Links:
- link BackLeg: geometry collision box size=0.2 0.992775167955302 0.2; visual box size=0.2 0.992775167955302 0.2
- link BackLowerLeg: geometry collision box size=0.2 0.2 1.3105326238196064; visual box size=0.2 0.2 1.3105326238196064
- link FrontLeg: geometry collision box size=0.2 0.7293908613481104 0.2; visual box size=0.2 0.7293908613481104 0.2
- link FrontLowerLeg: geometry collision box size=0.2 0.2 1.4729657535058265; visual box size=0.2 0.2 1.4729657535058265
- link LeftLeg: geometry collision box size=0.8356027712493513 0.2 0.2; visual box size=0.8356027712493513 0.2 0.2
- link LeftLowerLeg: geometry collision box size=0.2 0.2 0.5614282405930106; visual box size=0.2 0.2 0.5614282405930106
- link RightLeg: geometry collision box size=0.6154633169471866 0.2 0.2; visual box size=0.6154633169471866 0.2 0.2
- link RightLowerLeg: geometry collision box size=0.2 0.2 1.2912783727853858; visual box size=0.2 0.2 1.2912783727853858
Joints:
- joint BackLeg_BackLowerLeg: origin xyz=0 -0.5592709933916578 0 rpy=0 0 0 -> xyz=0 -0.992775167955302 0 rpy=0 0 0
- joint FrontLeg_FrontLowerLeg: origin xyz=0 0.843227620517826 0 rpy=0 0 0 -> xyz=0 0.7293908613481104 0 rpy=0 0 0
- joint LeftLeg_LeftLowerLeg: origin xyz=-1.127110533185077 0 0 rpy=0 0 0 -> xyz=-0.8356027712493513 0 0 rpy=0 0 0
- joint RightLeg_RightLowerLeg: origin xyz=1.3212408447730442 0 0 rpy=0 0 0 -> xyz=0.6154633169471866 0 0 rpy=0 0 0
- joint Torso_BackLeg: origin xyz=0 9.5 1.3212408447730442 rpy=0 0 0 -> xyz=0 9.5 1.4729657535058265 rpy=0 0 0
- joint Torso_FrontLeg: origin xyz=0 10.5 1.3212408447730442 rpy=0 0 0 -> xyz=0 10.5 1.4729657535058265 rpy=0 0 0
- joint Torso_LeftLeg: origin xyz=-0.5 10 1.3212408447730442 rpy=0 0 0 -> xyz=-0.5 10 1.4729657535058265 rpy=0 0 0
- joint Torso_RightLeg: origin xyz=0.5 10 1.3212408447730442 rpy=0 0 0 -> xyz=0.5 10 1.4729657535058265 rpy=0 0 0

File: bodyFiles/body0101636.urdf (robot description, URDF)
Before this commit: robot robot, 9 links, 8 joints
Links:
- link BackLeg: geometry collision box size=0.2 1.2745956952265147 0.2; visual box size=0.2 1.2745956952265147 0.2
- link BackLowerLeg: geometry collision box size=0.2 0.2 1.022634857705416; visual box size=0.2 0.2 1.022634857705416
- link FrontLeg: geometry collision box size=0.2 0.8487743410138362 0.2; visual box size=0.2 0.8487743410138362 0.2
- link FrontLowerLeg: geometry collision box size=0.2 0.2 1.3702274139747868; visual box size=0.2 0.2 1.3702274139747868
- link LeftLeg: geometry collision box size=0.8125957214951772 0.2 0.2; visual box size=0.8125957214951772 0.2 0.2
- link LeftLowerLeg: geometry collision box size=0.2 0.2 1.3975507875131266; visual box size=0.2 0.2 1.3975507875131266
- link RightLeg: geometry collision box size=0.7127061312216314 0.2 0.2; visual box size=0.7127061312216314 0.2 0.2
- link RightLowerLeg: geometry collision box size=0.2 0.2 1.1423031695423074; visual box size=0.2 0.2 1.1423031695423074
Joints:
- joint BackLeg_BackLowerLeg: origin xyz=0 -0.6050884852636941 0 rpy=0 0 0 -> xyz=0 -1.2745956952265147 0 rpy=0 0 0
- joint FrontLeg_FrontLowerLeg: origin xyz=0 0.9013516387063997 0 rpy=0 0 0 -> xyz=0 0.8487743410138362 0 rpy=0 0 0
- joint LeftLeg_LeftLowerLeg: origin xyz=-0.6564653922654946 0 0 rpy=0 0 0 -> xyz=-0.8125957214951772 0 0 rpy=0 0 0
- joint RightLeg_RightLowerLeg: origin xyz=0.6857427506313392 0 0 rpy=0 0 0 -> xyz=0.7127061312216314 0 0 rpy=0 0 0
- joint Torso_BackLeg: origin xyz=0 9.5 1.4683412743006823 rpy=0 0 0 -> xyz=0 9.5 1.3975507875131266 rpy=0 0 0
- joint Torso_FrontLeg: origin xyz=0 10.5 1.4683412743006823 rpy=0 0 0 -> xyz=0 10.5 1.3975507875131266 rpy=0 0 0
- joint Torso_LeftLeg: origin xyz=-0.5 10 1.4683412743006823 rpy=0 0 0 -> xyz=-0.5 10 1.3975507875131266 rpy=0 0 0
- joint Torso_RightLeg: origin xyz=0.5 10 1.4683412743006823 rpy=0 0 0 -> xyz=0.5 10 1.3975507875131266 rpy=0 0 0
