Commit message: 40 gens, case3

File: bodyFiles/body010435.urdf (robot description, URDF)
Before this commit: robot robot, 9 links, 8 joints
Links:
- link BackLeg: geometry collision box size=0.2 1.3555139704055006 0.2; visual box size=0.2 1.3555139704055006 0.2
- link BackLowerLeg: geometry collision box size=0.2 0.2 1.4145360406510372; visual box size=0.2 0.2 1.4145360406510372
- link FrontLeg: geometry collision box size=0.2 1.2524013357677508 0.2; visual box size=0.2 1.2524013357677508 0.2
- link FrontLowerLeg: geometry collision box size=0.2 0.2 0.6340802718792421; visual box size=0.2 0.2 0.6340802718792421
- link LeftLeg: geometry collision box size=1.445566770752712 0.2 0.2; visual box size=1.445566770752712 0.2 0.2
- link LeftLowerLeg: geometry collision box size=0.2 0.2 1.1261593427957504; visual box size=0.2 0.2 1.1261593427957504
- link RightLeg: geometry collision box size=1.4304131282245236 0.2 0.2; visual box size=1.4304131282245236 0.2 0.2
- link RightLowerLeg: geometry collision box size=0.2 0.2 1.1083781108153834; visual box size=0.2 0.2 1.1083781108153834
Joints:
- joint BackLeg_BackLowerLeg: origin xyz=0 -0.7552608245338704 0 rpy=0 0 0 -> xyz=0 -1.3555139704055006 0 rpy=0 0 0
- joint FrontLeg_FrontLowerLeg: origin xyz=0 0.9647284058348504 0 rpy=0 0 0 -> xyz=0 1.2524013357677508 0 rpy=0 0 0
- joint LeftLeg_LeftLowerLeg: origin xyz=-1.1317530572502335 0 0 rpy=0 0 0 -> xyz=-1.445566770752712 0 0 rpy=0 0 0
- joint RightLeg_RightLowerLeg: origin xyz=1.2693351837293005 0 0 rpy=0 0 0 -> xyz=1.4304131282245236 0 0 rpy=0 0 0
- joint Torso_BackLeg: origin xyz=0 9.5 1.2693351837293005 rpy=0 0 0 -> xyz=0 9.5 1.445566770752712 rpy=0 0 0
- joint Torso_FrontLeg: origin xyz=0 10.5 1.2693351837293005 rpy=0 0 0 -> xyz=0 10.5 1.445566770752712 rpy=0 0 0
- joint Torso_LeftLeg: origin xyz=-0.5 10 1.2693351837293005 rpy=0 0 0 -> xyz=-0.5 10 1.445566770752712 rpy=0 0 0
- joint Torso_RightLeg: origin xyz=0.5 10 1.2693351837293005 rpy=0 0 0 -> xyz=0.5 10 1.445566770752712 rpy=0 0 0

File: bodyFiles/body0181245.urdf (robot description, URDF)
Before this commit: robot robot, 9 links, 8 joints
Links:
- link BackLeg: geometry collision box size=0.2 0.5917323780598515 0.2; visual box size=0.2 0.5917323780598515 0.2
- link BackLowerLeg: geometry collision box size=0.2 0.2 0.803089127044102; visual box size=0.2 0.2 0.803089127044102
- link FrontLeg: geometry collision box size=0.2 1.3910528681600378 0.2; visual box size=0.2 1.3910528681600378 0.2
- link FrontLowerLeg: geometry collision box size=0.2 0.2 1.2132503371445806; visual box size=0.2 0.2 1.2132503371445806
- link LeftLeg: geometry collision box size=0.9982207636909974 0.2 0.2; visual box size=0.9982207636909974 0.2 0.2
- link LeftLowerLeg: geometry collision box size=0.2 0.2 1.3338386266519402; visual box size=0.2 0.2 1.3338386266519402
- link RightLeg: geometry collision box size=1.129380972243177 0.2 0.2; visual box size=1.129380972243177 0.2 0.2
- link RightLowerLeg: geometry collision box size=0.2 0.2 0.766147714444977; visual box size=0.2 0.2 0.766147714444977
Joints:
- joint BackLeg_BackLowerLeg: origin xyz=0 -0.751027328063527 0 rpy=0 0 0 -> xyz=0 -0.5917323780598515 0 rpy=0 0 0
- joint FrontLeg_FrontLowerLeg: origin xyz=0 0.6192109337572642 0 rpy=0 0 0 -> xyz=0 1.3910528681600378 0 rpy=0 0 0
- joint LeftLeg_LeftLowerLeg: origin xyz=-1.176713366282958 0 0 rpy=0 0 0 -> xyz=-0.9982207636909974 0 0 rpy=0 0 0
- joint RightLeg_RightLowerLeg: origin xyz=0.6006190103603357 0 0 rpy=0 0 0 -> xyz=1.129380972243177 0 0 rpy=0 0 0
- joint Torso_BackLeg: origin xyz=0 17.5 1.414148280434802 rpy=0 0 0 -> xyz=0 17.5 1.3910528681600378 rpy=0 0 0
- joint Torso_FrontLeg: origin xyz=0 18.5 1.414148280434802 rpy=0 0 0 -> xyz=0 18.5 1.3910528681600378 rpy=0 0 0
- joint Torso_LeftLeg: origin xyz=-0.5 18 1.414148280434802 rpy=0 0 0 -> xyz=-0.5 18 1.3910528681600378 rpy=0 0 0
- joint Torso_RightLeg: origin xyz=0.5 18 1.414148280434802 rpy=0 0 0 -> xyz=0.5 18 1.3910528681600378 rpy=0 0 0

File: bodyFiles/body021425.urdf (robot description, URDF)
Before this commit: robot robot, 9 links, 8 joints
Links:
- link BackLeg: geometry collision box size=0.2 1.46509168704538 0.2; visual box size=0.2 1.46509168704538 0.2
- link BackLowerLeg: geometry collision box size=0.2 0.2 0.605848415895829; visual box size=0.2 0.2 0.605848415895829
- link FrontLeg: geometry collision box size=0.2 1.0929724823420535 0.2; visual box size=0.2 1.0929724823420535 0.2
- link FrontLowerLeg: geometry collision box size=0.2 0.2 1.0111502781589348; visual box size=0.2 0.2 1.0111502781589348
- link LeftLeg: geometry collision box size=0.8052142609936201 0.2 0.2; visual box size=0.8052142609936201 0.2 0.2
- link LeftLowerLeg: geometry collision box size=0.2 0.2 0.6058270250662229; visual box size=0.2 0.2 0.6058270250662229
- link RightLeg: geometry collision box size=1.4156413861453125 0.2 0.2; visual box size=1.4156413861453125 0.2 0.2
- link RightLowerLeg: geometry collision box size=0.2 0.2 1.2710220104696743; visual box size=0.2 0.2 1.2710220104696743
Joints:
- joint BackLeg_BackLowerLeg: origin xyz=0 -1.1083566014531758 0 rpy=0 0 0 -> xyz=0 -1.46509168704538 0 rpy=0 0 0
- joint FrontLeg_FrontLowerLeg: origin xyz=0 0.7714914812099317 0 rpy=0 0 0 -> xyz=0 1.0929724823420535 0 rpy=0 0 0
- joint LeftLeg_LeftLowerLeg: origin xyz=-0.9253250772692638 0 0 rpy=0 0 0 -> xyz=-0.8052142609936201 0 0 rpy=0 0 0
- joint RightLeg_RightLowerLeg: origin xyz=0.6286699562579648 0 0 rpy=0 0 0 -> xyz=1.4156413861453125 0 0 rpy=0 0 0
- joint Torso_BackLeg: origin xyz=0 1.5 1.3458563555892764 rpy=0 0 0 -> xyz=0 1.5 1.46509168704538 rpy=0 0 0
- joint Torso_FrontLeg: origin xyz=0 2.5 1.3458563555892764 rpy=0 0 0 -> xyz=0 2.5 1.46509168704538 rpy=0 0 0
- joint Torso_LeftLeg: origin xyz=-0.5 2 1.3458563555892764 rpy=0 0 0 -> xyz=-0.5 2 1.46509168704538 rpy=0 0 0
- joint Torso_RightLeg: origin xyz=0.5 2 1.3458563555892764 rpy=0 0 0 -> xyz=0.5 2 1.46509168704538 rpy=0 0 0

File: bodyFiles/body061281.urdf (robot description, URDF)
Before this commit: robot robot, 9 links, 8 joints
Links:
- link BackLeg: geometry collision box size=0.2 1.0330446583052815 0.2; visual box size=0.2 1.0330446583052815 0.2
- link BackLowerLeg: geometry collision box size=0.2 0.2 0.5690190141945223; visual box size=0.2 0.2 0.5690190141945223
- link FrontLeg: geometry collision box size=0.2 0.5657600079182366 0.2; visual box size=0.2 0.5657600079182366 0.2
- link FrontLowerLeg: geometry collision box size=0.2 0.2 1.2254274254168949; visual box size=0.2 0.2 1.2254274254168949
- link LeftLeg: geometry collision box size=1.0233593612651 0.2 0.2; visual box size=1.0233593612651 0.2 0.2
- link LeftLowerLeg: geometry collision box size=0.2 0.2 1.3490533998173775; visual box size=0.2 0.2 1.3490533998173775
- link RightLeg: geometry collision box size=0.5646511496235017 0.2 0.2; visual box size=0.5646511496235017 0.2 0.2
- link RightLowerLeg: geometry collision box size=0.2 0.2 0.8930520370481398; visual box size=0.2 0.2 0.8930520370481398
Joints:
- joint BackLeg_BackLowerLeg: origin xyz=0 -0.7891984576625901 0 rpy=0 0 0 -> xyz=0 -1.0330446583052815 0 rpy=0 0 0
- joint FrontLeg_FrontLowerLeg: origin xyz=0 0.6638071589484359 0 rpy=0 0 0 -> xyz=0 0.5657600079182366 0 rpy=0 0 0
- joint LeftLeg_LeftLowerLeg: origin xyz=-0.7467835410077067 0 0 rpy=0 0 0 -> xyz=-1.0233593612651 0 0 rpy=0 0 0
- joint RightLeg_RightLowerLeg: origin xyz=0.6553662189024642 0 0 rpy=0 0 0 -> xyz=0.5646511496235017 0 0 rpy=0 0 0
- joint Torso_BackLeg: origin xyz=0 5.5 1.3455208894801887 rpy=0 0 0 -> xyz=0 5.5 1.3490533998173775 rpy=0 0 0
- joint Torso_FrontLeg: origin xyz=0 6.5 1.3455208894801887 rpy=0 0 0 -> xyz=0 6.5 1.3490533998173775 rpy=0 0 0
- joint Torso_LeftLeg: origin xyz=-0.5 6 1.3455208894801887 rpy=0 0 0 -> xyz=-0.5 6 1.3490533998173775 rpy=0 0 0
- joint Torso_RightLeg: origin xyz=0.5 6 1.3455208894801887 rpy=0 0 0 -> xyz=0.5 6 1.3490533998173775 rpy=0 0 0

File: bodyFiles/body061630.urdf (robot description, URDF)
Before this commit: robot robot, 9 links, 8 joints
Links:
- link BackLeg: geometry collision box size=0.2 1.0114103570880646 0.2; visual box size=0.2 1.0114103570880646 0.2
- link BackLowerLeg: geometry collision box size=0.2 0.2 1.023430663951915; visual box size=0.2 0.2 1.023430663951915
- link FrontLeg: geometry collision box size=0.2 1.237063495325947 0.2; visual box size=0.2 1.237063495325947 0.2
- link FrontLowerLeg: geometry collision box size=0.2 0.2 1.212247904529126; visual box size=0.2 0.2 1.212247904529126
- link LeftLeg: geometry collision box size=0.6949437588866723 0.2 0.2; visual box size=0.6949437588866723 0.2 0.2
- link LeftLowerLeg: geometry collision box size=0.2 0.2 1.4470517497074544; visual box size=0.2 0.2 1.4470517497074544
- link RightLeg: geometry collision box size=0.8872784358576272 0.2 0.2; visual box size=0.8872784358576272 0.2 0.2
- link RightLowerLeg: geometry collision box size=0.2 0.2 0.7732547897691444; visual box size=0.2 0.2 0.7732547897691444
Joints:
- joint BackLeg_BackLowerLeg: origin xyz=0 -1.4830736258379849 0 rpy=0 0 0 -> xyz=0 -1.0114103570880646 0 rpy=0 0 0
- joint FrontLeg_FrontLowerLeg: origin xyz=0 0.8429328268990222 0 rpy=0 0 0 -> xyz=0 1.237063495325947 0 rpy=0 0 0
- joint LeftLeg_LeftLowerLeg: origin xyz=-0.8828459394628185 0 0 rpy=0 0 0 -> xyz=-0.6949437588866723 0 0 rpy=0 0 0
- joint RightLeg_RightLowerLeg: origin xyz=1.2861848998394274 0 0 rpy=0 0 0 -> xyz=0.8872784358576272 0 0 rpy=0 0 0
- joint Torso_BackLeg: origin xyz=0 5.5 1.4830736258379849 rpy=0 0 0 -> xyz=0 5.5 1.4470517497074544 rpy=0 0 0
- joint Torso_FrontLeg: origin xyz=0 6.5 1.4830736258379849 rpy=0 0 0 -> xyz=0 6.5 1.4470517497074544 rpy=0 0 0
- joint Torso_LeftLeg: origin xyz=-0.5 6 1.4830736258379849 rpy=0 0 0 -> xyz=-0.5 6 1.4470517497074544 rpy=0 0 0
- joint Torso_RightLeg: origin xyz=0.5 6 1.4830736258379849 rpy=0 0 0 -> xyz=0.5 6 1.4470517497074544 rpy=0 0 0

File: bodyFiles/body06184.urdf (robot description, URDF)
Before this commit: robot robot, 9 links, 8 joints
Links:
- link BackLeg: geometry collision box size=0.2 0.8149094513895251 0.2; visual box size=0.2 0.8149094513895251 0.2
- link BackLowerLeg: geometry collision box size=0.2 0.2 1.3566802924524277; visual box size=0.2 0.2 1.3566802924524277
- link FrontLeg: geometry collision box size=0.2 0.594875257635475 0.2; visual box size=0.2 0.594875257635475 0.2
- link FrontLowerLeg: geometry collision box size=0.2 0.2 0.7920783965582919; visual box size=0.2 0.2 0.7920783965582919
- link LeftLeg: geometry collision box size=1.247730312136416 0.2 0.2; visual box size=1.247730312136416 0.2 0.2
- link LeftLowerLeg: geometry collision box size=0.2 0.2 0.7612118489605632; visual box size=0.2 0.2 0.7612118489605632
- link RightLeg: geometry collision box size=0.8993893213652217 0.2 0.2; visual box size=0.8993893213652217 0.2 0.2
- link RightLowerLeg: geometry collision box size=0.2 0.2 1.1624014851878965; visual box size=0.2 0.2 1.1624014851878965
Joints:
- joint BackLeg_BackLowerLeg: origin xyz=0 -1.4941859648316365 0 rpy=0 0 0 -> xyz=0 -0.8149094513895251 0 rpy=0 0 0
- joint FrontLeg_FrontLowerLeg: origin xyz=0 0.5385628661739603 0 rpy=0 0 0 -> xyz=0 0.594875257635475 0 rpy=0 0 0
- joint LeftLeg_LeftLowerLeg: origin xyz=-1.1812678040950995 0 0 rpy=0 0 0 -> xyz=-1.247730312136416 0 0 rpy=0 0 0
- joint RightLeg_RightLowerLeg: origin xyz=0.8584474680511636 0 0 rpy=0 0 0 -> xyz=0.8993893213652217 0 0 rpy=0 0 0
- joint Torso_BackLeg: origin xyz=0 5.5 1.4941859648316365 rpy=0 0 0 -> xyz=0 5.5 1.3566802924524277 rpy=0 0 0
- joint Torso_FrontLeg: origin xyz=0 6.5 1.4941859648316365 rpy=0 0 0 -> xyz=0 6.5 1.3566802924524277 rpy=0 0 0
- joint Torso_LeftLeg: origin xyz=-0.5 6 1.4941859648316365 rpy=0 0 0 -> xyz=-0.5 6 1.3566802924524277 rpy=0 0 0
- joint Torso_RightLeg: origin xyz=0.5 6 1.4941859648316365 rpy=0 0 0 -> xyz=0.5 6 1.3566802924524277 rpy=0 0 0
