Commit message: JAR = .08, Evolved Bots, Case3

File: bodyFiles/body0-10114.urdf (robot description, URDF)
Before this commit: robot robot, 9 links, 8 joints
Links:
- link BackLeg: geometry collision box size=0.2 1.3986528308654131 0.2; visual box size=0.2 1.3986528308654131 0.2
- link BackLowerLeg: geometry collision box size=0.2 0.2 1.1962049880729473; visual box size=0.2 0.2 1.1962049880729473
- link FrontLeg: geometry collision box size=0.2 0.9833286302601155 0.2; visual box size=0.2 0.9833286302601155 0.2
- link FrontLowerLeg: geometry collision box size=0.2 0.2 0.7037253725691722; visual box size=0.2 0.2 0.7037253725691722
- link LeftLeg: geometry collision box size=0.7531311924134694 0.2 0.2; visual box size=0.7531311924134694 0.2 0.2
- link LeftLowerLeg: geometry collision box size=0.2 0.2 0.9947525821100406; visual box size=0.2 0.2 0.9947525821100406
- link RightLeg: geometry collision box size=1.4438664690276446 0.2 0.2; visual box size=1.4438664690276446 0.2 0.2
- link RightLowerLeg: geometry collision box size=0.2 0.2 0.7396352323001707; visual box size=0.2 0.2 0.7396352323001707
Joints:
- joint BackLeg_BackLowerLeg: origin xyz=0 -1.2807905282180767 0 rpy=0 0 0 -> xyz=0 -1.3986528308654131 0 rpy=0 0 0
- joint FrontLeg_FrontLowerLeg: origin xyz=0 1.3154995658616477 0 rpy=0 0 0 -> xyz=0 0.9833286302601155 0 rpy=0 0 0
- joint LeftLeg_LeftLowerLeg: origin xyz=-0.9597455112546808 0 0 rpy=0 0 0 -> xyz=-0.7531311924134694 0 0 rpy=0 0 0
- joint RightLeg_RightLowerLeg: origin xyz=1.4316755727159538 0 0 rpy=0 0 0 -> xyz=1.4438664690276446 0 0 rpy=0 0 0
- joint Torso_BackLeg: origin xyz=0 -10.5 1.4316755727159538 rpy=0 0 0 -> xyz=0 -10.5 1.4438664690276446 rpy=0 0 0
- joint Torso_FrontLeg: origin xyz=0 -9.5 1.4316755727159538 rpy=0 0 0 -> xyz=0 -9.5 1.4438664690276446 rpy=0 0 0
- joint Torso_LeftLeg: origin xyz=-0.5 -10 1.4316755727159538 rpy=0 0 0 -> xyz=-0.5 -10 1.4438664690276446 rpy=0 0 0
- joint Torso_RightLeg: origin xyz=0.5 -10 1.4316755727159538 rpy=0 0 0 -> xyz=0.5 -10 1.4438664690276446 rpy=0 0 0

File: bodyFiles/body0-14206.urdf (robot description, URDF)
Before this commit: robot robot, 9 links, 8 joints
Links:
- link BackLeg: geometry collision box size=0.2 0.8915980484589824 0.2; visual box size=0.2 0.8915980484589824 0.2
- link BackLowerLeg: geometry collision box size=0.2 0.2 0.8018466877463493; visual box size=0.2 0.2 0.8018466877463493
- link FrontLeg: geometry collision box size=0.2 1.0934825241241382 0.2; visual box size=0.2 1.0934825241241382 0.2
- link FrontLowerLeg: geometry collision box size=0.2 0.2 0.6064479083171941; visual box size=0.2 0.2 0.6064479083171941
- link LeftLeg: geometry collision box size=1.4787145598850642 0.2 0.2; visual box size=1.4787145598850642 0.2 0.2
- link LeftLowerLeg: geometry collision box size=0.2 0.2 1.285895677395728; visual box size=0.2 0.2 1.285895677395728
- link RightLeg: geometry collision box size=1.1314506989652435 0.2 0.2; visual box size=1.1314506989652435 0.2 0.2
- link RightLowerLeg: geometry collision box size=0.2 0.2 0.7188382301245332; visual box size=0.2 0.2 0.7188382301245332
Joints:
- joint BackLeg_BackLowerLeg: origin xyz=0 -1.362015909060724 0 rpy=0 0 0 -> xyz=0 -0.8915980484589824 0 rpy=0 0 0
- joint FrontLeg_FrontLowerLeg: origin xyz=0 1.3624452321401437 0 rpy=0 0 0 -> xyz=0 1.0934825241241382 0 rpy=0 0 0
- joint LeftLeg_LeftLowerLeg: origin xyz=-1.4170340393684124 0 0 rpy=0 0 0 -> xyz=-1.4787145598850642 0 0 rpy=0 0 0
- joint RightLeg_RightLowerLeg: origin xyz=1.200685637577722 0 0 rpy=0 0 0 -> xyz=1.1314506989652435 0 0 rpy=0 0 0
- joint Torso_BackLeg: origin xyz=0 -14.5 1.4170340393684124 rpy=0 0 0 -> xyz=0 -14.5 1.4787145598850642 rpy=0 0 0
- joint Torso_FrontLeg: origin xyz=0 -13.5 1.4170340393684124 rpy=0 0 0 -> xyz=0 -13.5 1.4787145598850642 rpy=0 0 0
- joint Torso_LeftLeg: origin xyz=-0.5 -14 1.4170340393684124 rpy=0 0 0 -> xyz=-0.5 -14 1.4787145598850642 rpy=0 0 0
- joint Torso_RightLeg: origin xyz=0.5 -14 1.4170340393684124 rpy=0 0 0 -> xyz=0.5 -14 1.4787145598850642 rpy=0 0 0

File: bodyFiles/body0-180.urdf (robot description, URDF)
Before this commit: robot robot, 9 links, 8 joints
Links:
- link BackLeg: geometry collision box size=0.2 0.7216088284244867 0.2; visual box size=0.2 0.7216088284244867 0.2
- link BackLowerLeg: geometry collision box size=0.2 0.2 1.2408938546638835; visual box size=0.2 0.2 1.2408938546638835
- link FrontLeg: geometry collision box size=0.2 1.0382966005862437 0.2; visual box size=0.2 1.0382966005862437 0.2
- link FrontLowerLeg: geometry collision box size=0.2 0.2 1.3991285688481847; visual box size=0.2 0.2 1.3991285688481847
- link LeftLeg: geometry collision box size=0.8212959562201655 0.2 0.2; visual box size=0.8212959562201655 0.2 0.2
- link LeftLowerLeg: geometry collision box size=0.2 0.2 0.5566565398834636; visual box size=0.2 0.2 0.5566565398834636
- link RightLeg: geometry collision box size=0.5505121554244037 0.2 0.2; visual box size=0.5505121554244037 0.2 0.2
- link RightLowerLeg: geometry collision box size=0.2 0.2 0.7089960495388646; visual box size=0.2 0.2 0.7089960495388646
Joints:
- joint BackLeg_BackLowerLeg: origin xyz=0 -1.4416848487442315 0 rpy=0 0 0 -> xyz=0 -0.7216088284244867 0 rpy=0 0 0
- joint FrontLeg_FrontLowerLeg: origin xyz=0 0.8854684896294055 0 rpy=0 0 0 -> xyz=0 1.0382966005862437 0 rpy=0 0 0
- joint LeftLeg_LeftLowerLeg: origin xyz=-1.4548733393131064 0 0 rpy=0 0 0 -> xyz=-0.8212959562201655 0 0 rpy=0 0 0
- joint RightLeg_RightLowerLeg: origin xyz=0.5927868568892034 0 0 rpy=0 0 0 -> xyz=0.5505121554244037 0 0 rpy=0 0 0
- joint Torso_BackLeg: origin xyz=0 -18.5 1.4548733393131064 rpy=0 0 0 -> xyz=0 -18.5 1.3991285688481847 rpy=0 0 0
- joint Torso_FrontLeg: origin xyz=0 -17.5 1.4548733393131064 rpy=0 0 0 -> xyz=0 -17.5 1.3991285688481847 rpy=0 0 0
- joint Torso_LeftLeg: origin xyz=-0.5 -18 1.4548733393131064 rpy=0 0 0 -> xyz=-0.5 -18 1.3991285688481847 rpy=0 0 0
- joint Torso_RightLeg: origin xyz=0.5 -18 1.4548733393131064 rpy=0 0 0 -> xyz=0.5 -18 1.3991285688481847 rpy=0 0 0

File: bodyFiles/body0-18253.urdf (robot description, URDF)
Before this commit: robot robot, 9 links, 8 joints
Links:
- link BackLeg: geometry collision box size=0.2 1.0119241422170964 0.2; visual box size=0.2 1.0119241422170964 0.2
- link BackLowerLeg: geometry collision box size=0.2 0.2 1.36142129063549; visual box size=0.2 0.2 1.36142129063549
- link FrontLeg: geometry collision box size=0.2 1.1325911809762244 0.2; visual box size=0.2 1.1325911809762244 0.2
- link FrontLowerLeg: geometry collision box size=0.2 0.2 1.4888710760538617; visual box size=0.2 0.2 1.4888710760538617
- link LeftLeg: geometry collision box size=0.5755656843113487 0.2 0.2; visual box size=0.5755656843113487 0.2 0.2
- link LeftLowerLeg: geometry collision box size=0.2 0.2 1.2660532331100929; visual box size=0.2 0.2 1.2660532331100929
- link RightLeg: geometry collision box size=1.3850209586666784 0.2 0.2; visual box size=1.3850209586666784 0.2 0.2
- link RightLowerLeg: geometry collision box size=0.2 0.2 0.5504991636210388; visual box size=0.2 0.2 0.5504991636210388
Joints:
- joint BackLeg_BackLowerLeg: origin xyz=0 -1.4624490802513148 0 rpy=0 0 0 -> xyz=0 -1.0119241422170964 0 rpy=0 0 0
- joint FrontLeg_FrontLowerLeg: origin xyz=0 0.9147762771736269 0 rpy=0 0 0 -> xyz=0 1.1325911809762244 0 rpy=0 0 0
- joint LeftLeg_LeftLowerLeg: origin xyz=-1.4549918295453237 0 0 rpy=0 0 0 -> xyz=-0.5755656843113487 0 0 rpy=0 0 0
- joint RightLeg_RightLowerLeg: origin xyz=0.7428887878284465 0 0 rpy=0 0 0 -> xyz=1.3850209586666784 0 0 rpy=0 0 0
- joint Torso_BackLeg: origin xyz=0 -18.5 1.4747469360797958 rpy=0 0 0 -> xyz=0 -18.5 1.4888710760538617 rpy=0 0 0
- joint Torso_FrontLeg: origin xyz=0 -17.5 1.4747469360797958 rpy=0 0 0 -> xyz=0 -17.5 1.4888710760538617 rpy=0 0 0
- joint Torso_LeftLeg: origin xyz=-0.5 -18 1.4747469360797958 rpy=0 0 0 -> xyz=-0.5 -18 1.4888710760538617 rpy=0 0 0
- joint Torso_RightLeg: origin xyz=0.5 -18 1.4747469360797958 rpy=0 0 0 -> xyz=0.5 -18 1.4888710760538617 rpy=0 0 0

File: bodyFiles/body0-6266.urdf (robot description, URDF)
Before this commit: robot robot, 9 links, 8 joints
Links:
- link BackLeg: geometry collision box size=0.2 0.7525644999652378 0.2; visual box size=0.2 0.7525644999652378 0.2
- link BackLowerLeg: geometry collision box size=0.2 0.2 0.7355169744213452; visual box size=0.2 0.2 0.7355169744213452
- link FrontLeg: geometry collision box size=0.2 0.9058022079767638 0.2; visual box size=0.2 0.9058022079767638 0.2
- link FrontLowerLeg: geometry collision box size=0.2 0.2 0.8788732208274607; visual box size=0.2 0.2 0.8788732208274607
- link LeftLeg: geometry collision box size=1.0431158455101825 0.2 0.2; visual box size=1.0431158455101825 0.2 0.2
- link LeftLowerLeg: geometry collision box size=0.2 0.2 0.5910336637592848; visual box size=0.2 0.2 0.5910336637592848
- link RightLeg: geometry collision box size=1.3937264468783441 0.2 0.2; visual box size=1.3937264468783441 0.2 0.2
- link RightLowerLeg: geometry collision box size=0.2 0.2 0.69559296338694; visual box size=0.2 0.2 0.69559296338694
Joints:
- joint BackLeg_BackLowerLeg: origin xyz=0 -0.8595507882444546 0 rpy=0 0 0 -> xyz=0 -0.7525644999652378 0 rpy=0 0 0
- joint FrontLeg_FrontLowerLeg: origin xyz=0 0.5379255306813561 0 rpy=0 0 0 -> xyz=0 0.9058022079767638 0 rpy=0 0 0
- joint LeftLeg_LeftLowerLeg: origin xyz=-1.4186204498778312 0 0 rpy=0 0 0 -> xyz=-1.0431158455101825 0 0 rpy=0 0 0
- joint RightLeg_RightLowerLeg: origin xyz=1.2998448542730934 0 0 rpy=0 0 0 -> xyz=1.3937264468783441 0 0 rpy=0 0 0
- joint Torso_BackLeg: origin xyz=0 -6.5 1.4186204498778312 rpy=0 0 0 -> xyz=0 -6.5 1.3937264468783441 rpy=0 0 0
- joint Torso_FrontLeg: origin xyz=0 -5.5 1.4186204498778312 rpy=0 0 0 -> xyz=0 -5.5 1.3937264468783441 rpy=0 0 0
- joint Torso_LeftLeg: origin xyz=-0.5 -6 1.4186204498778312 rpy=0 0 0 -> xyz=-0.5 -6 1.3937264468783441 rpy=0 0 0
- joint Torso_RightLeg: origin xyz=0.5 -6 1.4186204498778312 rpy=0 0 0 -> xyz=0.5 -6 1.3937264468783441 rpy=0 0 0

File: bodyFiles/body0-667.urdf (robot description, URDF)
Before this commit: robot robot, 9 links, 8 joints
Links:
- link BackLeg: geometry collision box size=0.2 0.5812503915509525 0.2; visual box size=0.2 0.5812503915509525 0.2
- link BackLowerLeg: geometry collision box size=0.2 0.2 0.679065575421279; visual box size=0.2 0.2 0.679065575421279
- link FrontLeg: geometry collision box size=0.2 0.8391605722313 0.2; visual box size=0.2 0.8391605722313 0.2
- link FrontLowerLeg: geometry collision box size=0.2 0.2 1.215182367319423; visual box size=0.2 0.2 1.215182367319423
- link LeftLeg: geometry collision box size=0.8720294893585898 0.2 0.2; visual box size=0.8720294893585898 0.2 0.2
- link LeftLowerLeg: geometry collision box size=0.2 0.2 1.3687644002426707; visual box size=0.2 0.2 1.3687644002426707
- link RightLeg: geometry collision box size=0.7108473278723345 0.2 0.2; visual box size=0.7108473278723345 0.2 0.2
- link RightLowerLeg: geometry collision box size=0.2 0.2 1.4215280550845968; visual box size=0.2 0.2 1.4215280550845968
Joints:
- joint BackLeg_BackLowerLeg: origin xyz=0 -0.9318887475395646 0 rpy=0 0 0 -> xyz=0 -0.5812503915509525 0 rpy=0 0 0
- joint FrontLeg_FrontLowerLeg: origin xyz=0 1.396648319505197 0 rpy=0 0 0 -> xyz=0 0.8391605722313 0 rpy=0 0 0
- joint LeftLeg_LeftLowerLeg: origin xyz=-1.3834859153232522 0 0 rpy=0 0 0 -> xyz=-0.8720294893585898 0 0 rpy=0 0 0
- joint RightLeg_RightLowerLeg: origin xyz=0.89950990249895 0 0 rpy=0 0 0 -> xyz=0.7108473278723345 0 0 rpy=0 0 0
- joint Torso_BackLeg: origin xyz=0 -6.5 1.396648319505197 rpy=0 0 0 -> xyz=0 -6.5 1.4215280550845968 rpy=0 0 0
- joint Torso_FrontLeg: origin xyz=0 -5.5 1.396648319505197 rpy=0 0 0 -> xyz=0 -5.5 1.4215280550845968 rpy=0 0 0
- joint Torso_LeftLeg: origin xyz=-0.5 -6 1.396648319505197 rpy=0 0 0 -> xyz=-0.5 -6 1.4215280550845968 rpy=0 0 0
- joint Torso_RightLeg: origin xyz=0.5 -6 1.396648319505197 rpy=0 0 0 -> xyz=0.5 -6 1.4215280550845968 rpy=0 0 0

File: bodyFiles/body014140.urdf (robot description, URDF)
Before this commit: robot robot, 9 links, 8 joints
Links:
- link BackLeg: geometry collision box size=0.2 0.9215527234147929 0.2; visual box size=0.2 0.9215527234147929 0.2
- link BackLowerLeg: geometry collision box size=0.2 0.2 1.2027093460783216; visual box size=0.2 0.2 1.2027093460783216
- link FrontLeg: geometry collision box size=0.2 0.8041645284504817 0.2; visual box size=0.2 0.8041645284504817 0.2
- link FrontLowerLeg: geometry collision box size=0.2 0.2 1.4756497557342558; visual box size=0.2 0.2 1.4756497557342558
- link LeftLeg: geometry collision box size=1.2962541716338127 0.2 0.2; visual box size=1.2962541716338127 0.2 0.2
- link LeftLowerLeg: geometry collision box size=0.2 0.2 1.436952884962484; visual box size=0.2 0.2 1.436952884962484
- link RightLeg: geometry collision box size=0.5910487319770273 0.2 0.2; visual box size=0.5910487319770273 0.2 0.2
- link RightLowerLeg: geometry collision box size=0.2 0.2 1.0568743771696216; visual box size=0.2 0.2 1.0568743771696216
Joints:
- joint BackLeg_BackLowerLeg: origin xyz=0 -1.3806478330133518 0 rpy=0 0 0 -> xyz=0 -0.9215527234147929 0 rpy=0 0 0
- joint FrontLeg_FrontLowerLeg: origin xyz=0 1.2835892150021815 0 rpy=0 0 0 -> xyz=0 0.8041645284504817 0 rpy=0 0 0
- joint LeftLeg_LeftLowerLeg: origin xyz=-1.193318774906824 0 0 rpy=0 0 0 -> xyz=-1.2962541716338127 0 0 rpy=0 0 0
- joint RightLeg_RightLowerLeg: origin xyz=1.0071355633326555 0 0 rpy=0 0 0 -> xyz=0.5910487319770273 0 0 rpy=0 0 0
- joint Torso_BackLeg: origin xyz=0 13.5 1.3806478330133518 rpy=0 0 0 -> xyz=0 13.5 1.4756497557342558 rpy=0 0 0
- joint Torso_FrontLeg: origin xyz=0 14.5 1.3806478330133518 rpy=0 0 0 -> xyz=0 14.5 1.4756497557342558 rpy=0 0 0
- joint Torso_LeftLeg: origin xyz=-0.5 14 1.3806478330133518 rpy=0 0 0 -> xyz=-0.5 14 1.4756497557342558 rpy=0 0 0
- joint Torso_RightLeg: origin xyz=0.5 14 1.3806478330133518 rpy=0 0 0 -> xyz=0.5 14 1.4756497557342558 rpy=0 0 0

File: bodyFiles/body02178.urdf (robot description, URDF)
Before this commit: robot robot, 9 links, 8 joints
Links:
- link BackLeg: geometry collision box size=0.2 0.8158354760555248 0.2; visual box size=0.2 0.8158354760555248 0.2
- link BackLowerLeg: geometry collision box size=0.2 0.2 1.1392705642926164; visual box size=0.2 0.2 1.1392705642926164
- link FrontLeg: geometry collision box size=0.2 0.9066212531365069 0.2; visual box size=0.2 0.9066212531365069 0.2
- link FrontLowerLeg: geometry collision box size=0.2 0.2 1.2112113463175516; visual box size=0.2 0.2 1.2112113463175516
- link LeftLeg: geometry collision box size=0.8970745627475432 0.2 0.2; visual box size=0.8970745627475432 0.2 0.2
- link LeftLowerLeg: geometry collision box size=0.2 0.2 1.4251998689341745; visual box size=0.2 0.2 1.4251998689341745
- link RightLeg: geometry collision box size=1.0087622255174375 0.2 0.2; visual box size=1.0087622255174375 0.2 0.2
- link RightLowerLeg: geometry collision box size=0.2 0.2 0.6124417861695092; visual box size=0.2 0.2 0.6124417861695092
Joints:
- joint BackLeg_BackLowerLeg: origin xyz=0 -1.4812548265597278 0 rpy=0 0 0 -> xyz=0 -0.8158354760555248 0 rpy=0 0 0
- joint FrontLeg_FrontLowerLeg: origin xyz=0 1.1579038507711141 0 rpy=0 0 0 -> xyz=0 0.9066212531365069 0 rpy=0 0 0
- joint LeftLeg_LeftLowerLeg: origin xyz=-0.7924353902562836 0 0 rpy=0 0 0 -> xyz=-0.8970745627475432 0 0 rpy=0 0 0
- joint RightLeg_RightLowerLeg: origin xyz=1.1110484003030714 0 0 rpy=0 0 0 -> xyz=1.0087622255174375 0 0 rpy=0 0 0
- joint Torso_BackLeg: origin xyz=0 1.5 1.491774850619921 rpy=0 0 0 -> xyz=0 1.5 1.4251998689341745 rpy=0 0 0
- joint Torso_FrontLeg: origin xyz=0 2.5 1.491774850619921 rpy=0 0 0 -> xyz=0 2.5 1.4251998689341745 rpy=0 0 0
- joint Torso_LeftLeg: origin xyz=-0.5 2 1.491774850619921 rpy=0 0 0 -> xyz=-0.5 2 1.4251998689341745 rpy=0 0 0
- joint Torso_RightLeg: origin xyz=0.5 2 1.491774850619921 rpy=0 0 0 -> xyz=0.5 2 1.4251998689341745 rpy=0 0 0

File: bodyFiles/body0276.urdf (robot description, URDF)
Before this commit: robot robot, 9 links, 8 joints
Links:
- link BackLeg: geometry collision box size=0.2 0.9087990183730742 0.2; visual box size=0.2 0.9087990183730742 0.2
- link BackLowerLeg: geometry collision box size=0.2 0.2 0.9263297306626658; visual box size=0.2 0.2 0.9263297306626658
- link FrontLeg: geometry collision box size=0.2 1.1342439396902275 0.2; visual box size=0.2 1.1342439396902275 0.2
- link FrontLowerLeg: geometry collision box size=0.2 0.2 1.3955203579224116; visual box size=0.2 0.2 1.3955203579224116
- link LeftLeg: geometry collision box size=1.405113720902578 0.2 0.2; visual box size=1.405113720902578 0.2 0.2
- link LeftLowerLeg: geometry collision box size=0.2 0.2 0.6813125923930627; visual box size=0.2 0.2 0.6813125923930627
- link RightLeg: geometry collision box size=0.8889557185163127 0.2 0.2; visual box size=0.8889557185163127 0.2 0.2
- link RightLowerLeg: geometry collision box size=0.2 0.2 1.198532405775017; visual box size=0.2 0.2 1.198532405775017
Joints:
- joint BackLeg_BackLowerLeg: origin xyz=0 -1.3139973579004187 0 rpy=0 0 0 -> xyz=0 -0.9087990183730742 0 rpy=0 0 0
- joint FrontLeg_FrontLowerLeg: origin xyz=0 1.2227074197533292 0 rpy=0 0 0 -> xyz=0 1.1342439396902275 0 rpy=0 0 0
- joint LeftLeg_LeftLowerLeg: origin xyz=-1.3079371690376282 0 0 rpy=0 0 0 -> xyz=-1.405113720902578 0 0 rpy=0 0 0
- joint RightLeg_RightLowerLeg: origin xyz=0.6811595315881341 0 0 rpy=0 0 0 -> xyz=0.8889557185163127 0 0 rpy=0 0 0
- joint Torso_BackLeg: origin xyz=0 1.5 1.338654378451161 rpy=0 0 0 -> xyz=0 1.5 1.405113720902578 rpy=0 0 0
- joint Torso_FrontLeg: origin xyz=0 2.5 1.338654378451161 rpy=0 0 0 -> xyz=0 2.5 1.405113720902578 rpy=0 0 0
- joint Torso_LeftLeg: origin xyz=-0.5 2 1.338654378451161 rpy=0 0 0 -> xyz=-0.5 2 1.405113720902578 rpy=0 0 0
- joint Torso_RightLeg: origin xyz=0.5 2 1.338654378451161 rpy=0 0 0 -> xyz=0.5 2 1.405113720902578 rpy=0 0 0
