Commit message: case3, evolved, JAR = .8

File: bodyFiles/body0-10312.urdf (robot description, URDF)
Before this commit: robot robot, 9 links, 8 joints
Links:
- link BackLeg: geometry collision box size=0.2 0.991524358373082 0.2; visual box size=0.2 0.991524358373082 0.2
- link BackLowerLeg: geometry collision box size=0.2 0.2 1.2066313145207972; visual box size=0.2 0.2 1.2066313145207972
- link FrontLeg: geometry collision box size=0.2 0.6168002532580711 0.2; visual box size=0.2 0.6168002532580711 0.2
- link FrontLowerLeg: geometry collision box size=0.2 0.2 1.2532267314116958; visual box size=0.2 0.2 1.2532267314116958
- link LeftLeg: geometry collision box size=0.6500582235254664 0.2 0.2; visual box size=0.6500582235254664 0.2 0.2
- link LeftLowerLeg: geometry collision box size=0.2 0.2 1.4541558548901798; visual box size=0.2 0.2 1.4541558548901798
- link RightLeg: geometry collision box size=0.9806416868489278 0.2 0.2; visual box size=0.9806416868489278 0.2 0.2
- link RightLowerLeg: geometry collision box size=0.2 0.2 1.1804794067903848; visual box size=0.2 0.2 1.1804794067903848
Joints:
- joint BackLeg_BackLowerLeg: origin xyz=0 -0.6928633997782794 0 rpy=0 0 0 -> xyz=0 -0.991524358373082 0 rpy=0 0 0
- joint FrontLeg_FrontLowerLeg: origin xyz=0 0.6788935042000422 0 rpy=0 0 0 -> xyz=0 0.6168002532580711 0 rpy=0 0 0
- joint LeftLeg_LeftLowerLeg: origin xyz=-0.8228793315569235 0 0 rpy=0 0 0 -> xyz=-0.6500582235254664 0 0 rpy=0 0 0
- joint RightLeg_RightLowerLeg: origin xyz=1.3915215393912113 0 0 rpy=0 0 0 -> xyz=0.9806416868489278 0 0 rpy=0 0 0
- joint Torso_BackLeg: origin xyz=0 -10.5 1.3915215393912113 rpy=0 0 0 -> xyz=0 -10.5 1.4541558548901798 rpy=0 0 0
- joint Torso_FrontLeg: origin xyz=0 -9.5 1.3915215393912113 rpy=0 0 0 -> xyz=0 -9.5 1.4541558548901798 rpy=0 0 0
- joint Torso_LeftLeg: origin xyz=-0.5 -10 1.3915215393912113 rpy=0 0 0 -> xyz=-0.5 -10 1.4541558548901798 rpy=0 0 0
- joint Torso_RightLeg: origin xyz=0.5 -10 1.3915215393912113 rpy=0 0 0 -> xyz=0.5 -10 1.4541558548901798 rpy=0 0 0

File: bodyFiles/body0-180.urdf (robot description, URDF)
Before this commit: robot robot, 9 links, 8 joints
Links:
- link BackLeg: geometry collision box size=0.2 1.12336051075338 0.2; visual box size=0.2 1.12336051075338 0.2
- link BackLowerLeg: geometry collision box size=0.2 0.2 0.6723997472332736; visual box size=0.2 0.2 0.6723997472332736
- link FrontLeg: geometry collision box size=0.2 0.9222473413778454 0.2; visual box size=0.2 0.9222473413778454 0.2
- link FrontLowerLeg: geometry collision box size=0.2 0.2 0.5247631899119634; visual box size=0.2 0.2 0.5247631899119634
- link LeftLeg: geometry collision box size=1.178826621860777 0.2 0.2; visual box size=1.178826621860777 0.2 0.2
- link LeftLowerLeg: geometry collision box size=0.2 0.2 1.2588201230591216; visual box size=0.2 0.2 1.2588201230591216
- link RightLeg: geometry collision box size=0.7396818960740315 0.2 0.2; visual box size=0.7396818960740315 0.2 0.2
- link RightLowerLeg: geometry collision box size=0.2 0.2 1.1435181177952134; visual box size=0.2 0.2 1.1435181177952134
Joints:
- joint BackLeg_BackLowerLeg: origin xyz=0 -0.7216088284244867 0 rpy=0 0 0 -> xyz=0 -1.12336051075338 0 rpy=0 0 0
- joint FrontLeg_FrontLowerLeg: origin xyz=0 1.0382966005862437 0 rpy=0 0 0 -> xyz=0 0.9222473413778454 0 rpy=0 0 0
- joint LeftLeg_LeftLowerLeg: origin xyz=-0.8212959562201655 0 0 rpy=0 0 0 -> xyz=-1.178826621860777 0 0 rpy=0 0 0
- joint RightLeg_RightLowerLeg: origin xyz=0.5505121554244037 0 0 rpy=0 0 0 -> xyz=0.7396818960740315 0 0 rpy=0 0 0
- joint Torso_BackLeg: origin xyz=0 -18.5 1.3991285688481847 rpy=0 0 0 -> xyz=0 -18.5 1.2588201230591216 rpy=0 0 0
- joint Torso_FrontLeg: origin xyz=0 -17.5 1.3991285688481847 rpy=0 0 0 -> xyz=0 -17.5 1.2588201230591216 rpy=0 0 0
- joint Torso_LeftLeg: origin xyz=-0.5 -18 1.3991285688481847 rpy=0 0 0 -> xyz=-0.5 -18 1.2588201230591216 rpy=0 0 0
- joint Torso_RightLeg: origin xyz=0.5 -18 1.3991285688481847 rpy=0 0 0 -> xyz=0.5 -18 1.2588201230591216 rpy=0 0 0

File: bodyFiles/body0-18150.urdf (robot description, URDF)
Before this commit: robot robot, 9 links, 8 joints
Links:
- link BackLeg: geometry collision box size=0.2 0.7375653542138976 0.2; visual box size=0.2 0.7375653542138976 0.2
- link BackLowerLeg: geometry collision box size=0.2 0.2 1.3012943589411679; visual box size=0.2 0.2 1.3012943589411679
- link FrontLeg: geometry collision box size=0.2 0.5962687677792236 0.2; visual box size=0.2 0.5962687677792236 0.2
- link FrontLowerLeg: geometry collision box size=0.2 0.2 0.926592563856005; visual box size=0.2 0.2 0.926592563856005
- link LeftLeg: geometry collision box size=0.9792088011867829 0.2 0.2; visual box size=0.9792088011867829 0.2 0.2
- link LeftLowerLeg: geometry collision box size=0.2 0.2 0.8186854845570453; visual box size=0.2 0.2 0.8186854845570453
- link RightLeg: geometry collision box size=1.0807387410217308 0.2 0.2; visual box size=1.0807387410217308 0.2 0.2
- link RightLowerLeg: geometry collision box size=0.2 0.2 1.3345741633330186; visual box size=0.2 0.2 1.3345741633330186
Joints:
- joint BackLeg_BackLowerLeg: origin xyz=0 -0.6363905603878303 0 rpy=0 0 0 -> xyz=0 -0.7375653542138976 0 rpy=0 0 0
- joint FrontLeg_FrontLowerLeg: origin xyz=0 0.7199065956444131 0 rpy=0 0 0 -> xyz=0 0.5962687677792236 0 rpy=0 0 0
- joint LeftLeg_LeftLowerLeg: origin xyz=-0.8372798789700556 0 0 rpy=0 0 0 -> xyz=-0.9792088011867829 0 0 rpy=0 0 0
- joint RightLeg_RightLowerLeg: origin xyz=0.8266157673145627 0 0 rpy=0 0 0 -> xyz=1.0807387410217308 0 0 rpy=0 0 0
- joint Torso_BackLeg: origin xyz=0 -18.5 1.43814985927939 rpy=0 0 0 -> xyz=0 -18.5 1.3345741633330186 rpy=0 0 0
- joint Torso_FrontLeg: origin xyz=0 -17.5 1.43814985927939 rpy=0 0 0 -> xyz=0 -17.5 1.3345741633330186 rpy=0 0 0
- joint Torso_LeftLeg: origin xyz=-0.5 -18 1.43814985927939 rpy=0 0 0 -> xyz=-0.5 -18 1.3345741633330186 rpy=0 0 0
- joint Torso_RightLeg: origin xyz=0.5 -18 1.43814985927939 rpy=0 0 0 -> xyz=0.5 -18 1.3345741633330186 rpy=0 0 0

File: bodyFiles/body0-18200.urdf (robot description, URDF)
Before this commit: robot robot, 9 links, 8 joints
Links:
- link BackLeg: geometry collision box size=0.2 0.6272607942305353 0.2; visual box size=0.2 0.6272607942305353 0.2
- link BackLowerLeg: geometry collision box size=0.2 0.2 1.374250939663459; visual box size=0.2 0.2 1.374250939663459
- link FrontLeg: geometry collision box size=0.2 1.171127859418643 0.2; visual box size=0.2 1.171127859418643 0.2
- link FrontLowerLeg: geometry collision box size=0.2 0.2 0.7219545950252924; visual box size=0.2 0.2 0.7219545950252924
- link LeftLeg: geometry collision box size=0.8605609894897777 0.2 0.2; visual box size=0.8605609894897777 0.2 0.2
- link LeftLowerLeg: geometry collision box size=0.2 0.2 1.109254276116809; visual box size=0.2 0.2 1.109254276116809
- link RightLeg: geometry collision box size=1.1691054045370626 0.2 0.2; visual box size=1.1691054045370626 0.2 0.2
- link RightLowerLeg: geometry collision box size=0.2 0.2 0.9614078556536175; visual box size=0.2 0.2 0.9614078556536175
Joints:
- joint BackLeg_BackLowerLeg: origin xyz=0 -1.3699046597224105 0 rpy=0 0 0 -> xyz=0 -0.6272607942305353 0 rpy=0 0 0
- joint FrontLeg_FrontLowerLeg: origin xyz=0 0.9901988054003448 0 rpy=0 0 0 -> xyz=0 1.171127859418643 0 rpy=0 0 0
- joint LeftLeg_LeftLowerLeg: origin xyz=-0.7063113382279267 0 0 rpy=0 0 0 -> xyz=-0.8605609894897777 0 0 rpy=0 0 0
- joint RightLeg_RightLowerLeg: origin xyz=1.458410193351785 0 0 rpy=0 0 0 -> xyz=1.1691054045370626 0 0 rpy=0 0 0
- joint Torso_BackLeg: origin xyz=0 -18.5 1.458410193351785 rpy=0 0 0 -> xyz=0 -18.5 1.374250939663459 rpy=0 0 0
- joint Torso_FrontLeg: origin xyz=0 -17.5 1.458410193351785 rpy=0 0 0 -> xyz=0 -17.5 1.374250939663459 rpy=0 0 0
- joint Torso_LeftLeg: origin xyz=-0.5 -18 1.458410193351785 rpy=0 0 0 -> xyz=-0.5 -18 1.374250939663459 rpy=0 0 0
- joint Torso_RightLeg: origin xyz=0.5 -18 1.458410193351785 rpy=0 0 0 -> xyz=0.5 -18 1.374250939663459 rpy=0 0 0

File: bodyFiles/body0-18300.urdf (robot description, URDF)
Before this commit: robot robot, 9 links, 8 joints
Links:
- link BackLeg: geometry collision box size=0.2 0.9099760965401494 0.2; visual box size=0.2 0.9099760965401494 0.2
- link BackLowerLeg: geometry collision box size=0.2 0.2 1.4573194417958022; visual box size=0.2 0.2 1.4573194417958022
- link FrontLeg: geometry collision box size=0.2 1.4235183198212606 0.2; visual box size=0.2 1.4235183198212606 0.2
- link FrontLowerLeg: geometry collision box size=0.2 0.2 0.639727750327235; visual box size=0.2 0.2 0.639727750327235
- link LeftLeg: geometry collision box size=1.1608488939754893 0.2 0.2; visual box size=1.1608488939754893 0.2 0.2
- link LeftLowerLeg: geometry collision box size=0.2 0.2 1.3787014701114462; visual box size=0.2 0.2 1.3787014701114462
- link RightLeg: geometry collision box size=0.9103272621767308 0.2 0.2; visual box size=0.9103272621767308 0.2 0.2
- link RightLowerLeg: geometry collision box size=0.2 0.2 0.6704962666445248; visual box size=0.2 0.2 0.6704962666445248
Joints:
- joint BackLeg_BackLowerLeg: origin xyz=0 -0.9371748523440403 0 rpy=0 0 0 -> xyz=0 -0.9099760965401494 0 rpy=0 0 0
- joint FrontLeg_FrontLowerLeg: origin xyz=0 0.53977573657438 0 rpy=0 0 0 -> xyz=0 1.4235183198212606 0 rpy=0 0 0
- joint LeftLeg_LeftLowerLeg: origin xyz=-1.202055367928415 0 0 rpy=0 0 0 -> xyz=-1.1608488939754893 0 0 rpy=0 0 0
- joint RightLeg_RightLowerLeg: origin xyz=1.4299055779535277 0 0 rpy=0 0 0 -> xyz=0.9103272621767308 0 0 rpy=0 0 0
- joint Torso_BackLeg: origin xyz=0 -18.5 1.4299055779535277 rpy=0 0 0 -> xyz=0 -18.5 1.4573194417958022 rpy=0 0 0
- joint Torso_FrontLeg: origin xyz=0 -17.5 1.4299055779535277 rpy=0 0 0 -> xyz=0 -17.5 1.4573194417958022 rpy=0 0 0
- joint Torso_LeftLeg: origin xyz=-0.5 -18 1.4299055779535277 rpy=0 0 0 -> xyz=-0.5 -18 1.4573194417958022 rpy=0 0 0
- joint Torso_RightLeg: origin xyz=0.5 -18 1.4299055779535277 rpy=0 0 0 -> xyz=0.5 -18 1.4573194417958022 rpy=0 0 0

File: bodyFiles/body0-2124.urdf (robot description, URDF)
Before this commit: robot robot, 9 links, 8 joints
Links:
- link BackLeg: geometry collision box size=0.2 1.2536784090045139 0.2; visual box size=0.2 1.2536784090045139 0.2
- link BackLowerLeg: geometry collision box size=0.2 0.2 0.7089931627316456; visual box size=0.2 0.2 0.7089931627316456
- link FrontLeg: geometry collision box size=0.2 0.8673026036948538 0.2; visual box size=0.2 0.8673026036948538 0.2
- link FrontLowerLeg: geometry collision box size=0.2 0.2 0.792455571209573; visual box size=0.2 0.2 0.792455571209573
- link LeftLeg: geometry collision box size=1.4419352030050478 0.2 0.2; visual box size=1.4419352030050478 0.2 0.2
- link LeftLowerLeg: geometry collision box size=0.2 0.2 0.915711814447169; visual box size=0.2 0.2 0.915711814447169
- link RightLeg: geometry collision box size=0.5401353597104427 0.2 0.2; visual box size=0.5401353597104427 0.2 0.2
- link RightLowerLeg: geometry collision box size=0.2 0.2 0.8494881396364796; visual box size=0.2 0.2 0.8494881396364796
Joints:
- joint BackLeg_BackLowerLeg: origin xyz=0 -0.7219747521155022 0 rpy=0 0 0 -> xyz=0 -1.2536784090045139 0 rpy=0 0 0
- joint FrontLeg_FrontLowerLeg: origin xyz=0 0.748532304770849 0 rpy=0 0 0 -> xyz=0 0.8673026036948538 0 rpy=0 0 0
- joint LeftLeg_LeftLowerLeg: origin xyz=-0.8394507448276499 0 0 rpy=0 0 0 -> xyz=-1.4419352030050478 0 0 rpy=0 0 0
- joint RightLeg_RightLowerLeg: origin xyz=0.7424552258174074 0 0 rpy=0 0 0 -> xyz=0.5401353597104427 0 0 rpy=0 0 0
- joint Torso_BackLeg: origin xyz=0 -2.5 1.4415435498454732 rpy=0 0 0 -> xyz=0 -2.5 1.4419352030050478 rpy=0 0 0
- joint Torso_FrontLeg: origin xyz=0 -1.5 1.4415435498454732 rpy=0 0 0 -> xyz=0 -1.5 1.4419352030050478 rpy=0 0 0
- joint Torso_LeftLeg: origin xyz=-0.5 -2 1.4415435498454732 rpy=0 0 0 -> xyz=-0.5 -2 1.4419352030050478 rpy=0 0 0
- joint Torso_RightLeg: origin xyz=0.5 -2 1.4415435498454732 rpy=0 0 0 -> xyz=0.5 -2 1.4419352030050478 rpy=0 0 0

File: bodyFiles/body0-2324.urdf (robot description, URDF)
Before this commit: robot robot, 9 links, 8 joints
Links:
- link BackLeg: geometry collision box size=0.2 1.0657129852204101 0.2; visual box size=0.2 1.0657129852204101 0.2
- link BackLowerLeg: geometry collision box size=0.2 0.2 0.5229883688366054; visual box size=0.2 0.2 0.5229883688366054
- link FrontLeg: geometry collision box size=0.2 0.8545922112335325 0.2; visual box size=0.2 0.8545922112335325 0.2
- link FrontLowerLeg: geometry collision box size=0.2 0.2 0.9846932605245879; visual box size=0.2 0.2 0.9846932605245879
- link LeftLeg: geometry collision box size=0.5827034826325445 0.2 0.2; visual box size=0.5827034826325445 0.2 0.2
- link LeftLowerLeg: geometry collision box size=0.2 0.2 0.9657203685423629; visual box size=0.2 0.2 0.9657203685423629
- link RightLeg: geometry collision box size=0.6189723941632475 0.2 0.2; visual box size=0.6189723941632475 0.2 0.2
- link RightLowerLeg: geometry collision box size=0.2 0.2 1.0357514438898254; visual box size=0.2 0.2 1.0357514438898254
Joints:
- joint BackLeg_BackLowerLeg: origin xyz=0 -0.6626076648311943 0 rpy=0 0 0 -> xyz=0 -1.0657129852204101 0 rpy=0 0 0
- joint FrontLeg_FrontLowerLeg: origin xyz=0 1.4712402600434258 0 rpy=0 0 0 -> xyz=0 0.8545922112335325 0 rpy=0 0 0
- joint LeftLeg_LeftLowerLeg: origin xyz=-0.9591864853166298 0 0 rpy=0 0 0 -> xyz=-0.5827034826325445 0 0 rpy=0 0 0
- joint RightLeg_RightLowerLeg: origin xyz=1.0805332384465447 0 0 rpy=0 0 0 -> xyz=0.6189723941632475 0 0 rpy=0 0 0
- joint Torso_BackLeg: origin xyz=0 -2.5 1.4712402600434258 rpy=0 0 0 -> xyz=0 -2.5 1.0657129852204101 rpy=0 0 0
- joint Torso_FrontLeg: origin xyz=0 -1.5 1.4712402600434258 rpy=0 0 0 -> xyz=0 -1.5 1.0657129852204101 rpy=0 0 0
- joint Torso_LeftLeg: origin xyz=-0.5 -2 1.4712402600434258 rpy=0 0 0 -> xyz=-0.5 -2 1.0657129852204101 rpy=0 0 0
- joint Torso_RightLeg: origin xyz=0.5 -2 1.4712402600434258 rpy=0 0 0 -> xyz=0.5 -2 1.0657129852204101 rpy=0 0 0

File: bodyFiles/body010337.urdf (robot description, URDF)
Before this commit: robot robot, 9 links, 8 joints
Links:
- link BackLeg: geometry collision box size=0.2 0.7963180811290329 0.2; visual box size=0.2 0.7963180811290329 0.2
- link BackLowerLeg: geometry collision box size=0.2 0.2 1.09566319852139; visual box size=0.2 0.2 1.09566319852139
- link FrontLeg: geometry collision box size=0.2 1.4263490479750178 0.2; visual box size=0.2 1.4263490479750178 0.2
- link FrontLowerLeg: geometry collision box size=0.2 0.2 0.7628526540108704; visual box size=0.2 0.2 0.7628526540108704
- link LeftLeg: geometry collision box size=0.7391764505943964 0.2 0.2; visual box size=0.7391764505943964 0.2 0.2
- link LeftLowerLeg: geometry collision box size=0.2 0.2 0.614198792433788; visual box size=0.2 0.2 0.614198792433788
- link RightLeg: geometry collision box size=0.9077685406984151 0.2 0.2; visual box size=0.9077685406984151 0.2 0.2
- link RightLowerLeg: geometry collision box size=0.2 0.2 1.229821154546142; visual box size=0.2 0.2 1.229821154546142
Joints:
- joint BackLeg_BackLowerLeg: origin xyz=0 -0.8660179758711115 0 rpy=0 0 0 -> xyz=0 -0.7963180811290329 0 rpy=0 0 0
- joint FrontLeg_FrontLowerLeg: origin xyz=0 1.242866717552101 0 rpy=0 0 0 -> xyz=0 1.4263490479750178 0 rpy=0 0 0
- joint LeftLeg_LeftLowerLeg: origin xyz=-0.9739724117827111 0 0 rpy=0 0 0 -> xyz=-0.7391764505943964 0 0 rpy=0 0 0
- joint RightLeg_RightLowerLeg: origin xyz=0.7735373561304516 0 0 rpy=0 0 0 -> xyz=0.9077685406984151 0 0 rpy=0 0 0
- joint Torso_BackLeg: origin xyz=0 9.5 1.4257329239451022 rpy=0 0 0 -> xyz=0 9.5 1.4263490479750178 rpy=0 0 0
- joint Torso_FrontLeg: origin xyz=0 10.5 1.4257329239451022 rpy=0 0 0 -> xyz=0 10.5 1.4263490479750178 rpy=0 0 0
- joint Torso_LeftLeg: origin xyz=-0.5 10 1.4257329239451022 rpy=0 0 0 -> xyz=-0.5 10 1.4263490479750178 rpy=0 0 0
- joint Torso_RightLeg: origin xyz=0.5 10 1.4257329239451022 rpy=0 0 0 -> xyz=0.5 10 1.4263490479750178 rpy=0 0 0

File: bodyFiles/body018199.urdf (robot description, URDF)
Before this commit: robot robot, 9 links, 8 joints
Links:
- link BackLeg: geometry collision box size=0.2 1.0131166021832612 0.2; visual box size=0.2 1.0131166021832612 0.2
- link BackLowerLeg: geometry collision box size=0.2 0.2 1.4143487709057383; visual box size=0.2 0.2 1.4143487709057383
- link FrontLeg: geometry collision box size=0.2 0.900371118286787 0.2; visual box size=0.2 0.900371118286787 0.2
- link FrontLowerLeg: geometry collision box size=0.2 0.2 0.8078843518366375; visual box size=0.2 0.2 0.8078843518366375
- link LeftLeg: geometry collision box size=0.9817348825768154 0.2 0.2; visual box size=0.9817348825768154 0.2 0.2
- link LeftLowerLeg: geometry collision box size=0.2 0.2 1.2039224302270597; visual box size=0.2 0.2 1.2039224302270597
- link RightLeg: geometry collision box size=0.9079894132366894 0.2 0.2; visual box size=0.9079894132366894 0.2 0.2
- link RightLowerLeg: geometry collision box size=0.2 0.2 0.6581529145640315; visual box size=0.2 0.2 0.6581529145640315
Joints:
- joint BackLeg_BackLowerLeg: origin xyz=0 -0.5072447463416918 0 rpy=0 0 0 -> xyz=0 -1.0131166021832612 0 rpy=0 0 0
- joint FrontLeg_FrontLowerLeg: origin xyz=0 1.2925827447519254 0 rpy=0 0 0 -> xyz=0 0.900371118286787 0 rpy=0 0 0
- joint LeftLeg_LeftLowerLeg: origin xyz=-0.9969521589925683 0 0 rpy=0 0 0 -> xyz=-0.9817348825768154 0 0 rpy=0 0 0
- joint RightLeg_RightLowerLeg: origin xyz=0.6702101831103057 0 0 rpy=0 0 0 -> xyz=0.9079894132366894 0 0 rpy=0 0 0
- joint Torso_BackLeg: origin xyz=0 17.5 1.4333492892513857 rpy=0 0 0 -> xyz=0 17.5 1.4143487709057383 rpy=0 0 0
- joint Torso_FrontLeg: origin xyz=0 18.5 1.4333492892513857 rpy=0 0 0 -> xyz=0 18.5 1.4143487709057383 rpy=0 0 0
- joint Torso_LeftLeg: origin xyz=-0.5 18 1.4333492892513857 rpy=0 0 0 -> xyz=-0.5 18 1.4143487709057383 rpy=0 0 0
- joint Torso_RightLeg: origin xyz=0.5 18 1.4333492892513857 rpy=0 0 0 -> xyz=0.5 18 1.4143487709057383 rpy=0 0 0

File: bodyFiles/body018249.urdf (robot description, URDF)
Before this commit: robot robot, 9 links, 8 joints
Links:
- link BackLeg: geometry collision box size=0.2 0.7359762625562544 0.2; visual box size=0.2 0.7359762625562544 0.2
- link BackLowerLeg: geometry collision box size=0.2 0.2 1.3149114289462307; visual box size=0.2 0.2 1.3149114289462307
- link FrontLeg: geometry collision box size=0.2 1.3767759626551916 0.2; visual box size=0.2 1.3767759626551916 0.2
- link FrontLowerLeg: geometry collision box size=0.2 0.2 1.2907846919070236; visual box size=0.2 0.2 1.2907846919070236
- link LeftLeg: geometry collision box size=0.9488718869520614 0.2 0.2; visual box size=0.9488718869520614 0.2 0.2
- link LeftLowerLeg: geometry collision box size=0.2 0.2 1.1841300957246146; visual box size=0.2 0.2 1.1841300957246146
- link RightLeg: geometry collision box size=1.2294096775893029 0.2 0.2; visual box size=1.2294096775893029 0.2 0.2
- link RightLowerLeg: geometry collision box size=0.2 0.2 1.399658204847165; visual box size=0.2 0.2 1.399658204847165
Joints:
- joint BackLeg_BackLowerLeg: origin xyz=0 -0.5370837651599497 0 rpy=0 0 0 -> xyz=0 -0.7359762625562544 0 rpy=0 0 0
- joint FrontLeg_FrontLowerLeg: origin xyz=0 1.4702753783469689 0 rpy=0 0 0 -> xyz=0 1.3767759626551916 0 rpy=0 0 0
- joint LeftLeg_LeftLowerLeg: origin xyz=-1.1578826984166763 0 0 rpy=0 0 0 -> xyz=-0.9488718869520614 0 0 rpy=0 0 0
- joint RightLeg_RightLowerLeg: origin xyz=0.9625990461866641 0 0 rpy=0 0 0 -> xyz=1.2294096775893029 0 0 rpy=0 0 0
- joint Torso_BackLeg: origin xyz=0 17.5 1.4702753783469689 rpy=0 0 0 -> xyz=0 17.5 1.399658204847165 rpy=0 0 0
- joint Torso_FrontLeg: origin xyz=0 18.5 1.4702753783469689 rpy=0 0 0 -> xyz=0 18.5 1.399658204847165 rpy=0 0 0
- joint Torso_LeftLeg: origin xyz=-0.5 18 1.4702753783469689 rpy=0 0 0 -> xyz=-0.5 18 1.399658204847165 rpy=0 0 0
- joint Torso_RightLeg: origin xyz=0.5 18 1.4702753783469689 rpy=0 0 0 -> xyz=0.5 18 1.399658204847165 rpy=0 0 0

File: bodyFiles/body018299.urdf (robot description, URDF)
Before this commit: robot robot, 9 links, 8 joints
Links:
- link BackLeg: geometry collision box size=0.2 1.3563599907891557 0.2; visual box size=0.2 1.3563599907891557 0.2
- link BackLowerLeg: geometry collision box size=0.2 0.2 0.7296996217421776; visual box size=0.2 0.2 0.7296996217421776
- link FrontLeg: geometry collision box size=0.2 0.7175941532726372 0.2; visual box size=0.2 0.7175941532726372 0.2
- link FrontLowerLeg: geometry collision box size=0.2 0.2 0.5413002276874599; visual box size=0.2 0.2 0.5413002276874599
- link LeftLeg: geometry collision box size=1.035536936239799 0.2 0.2; visual box size=1.035536936239799 0.2 0.2
- link LeftLowerLeg: geometry collision box size=0.2 0.2 1.2904757946207503; visual box size=0.2 0.2 1.2904757946207503
- link RightLeg: geometry collision box size=1.1348503026463805 0.2 0.2; visual box size=1.1348503026463805 0.2 0.2
- link RightLowerLeg: geometry collision box size=0.2 0.2 0.7267296259365686; visual box size=0.2 0.2 0.7267296259365686
Joints:
- joint BackLeg_BackLowerLeg: origin xyz=0 -1.1334045029407531 0 rpy=0 0 0 -> xyz=0 -1.3563599907891557 0 rpy=0 0 0
- joint FrontLeg_FrontLowerLeg: origin xyz=0 0.5133325372870038 0 rpy=0 0 0 -> xyz=0 0.7175941532726372 0 rpy=0 0 0
- joint LeftLeg_LeftLowerLeg: origin xyz=-1.0281135399213293 0 0 rpy=0 0 0 -> xyz=-1.035536936239799 0 0 rpy=0 0 0
- joint RightLeg_RightLowerLeg: origin xyz=0.6061793847261452 0 0 rpy=0 0 0 -> xyz=1.1348503026463805 0 0 rpy=0 0 0
- joint Torso_BackLeg: origin xyz=0 17.5 1.2999163970265601 rpy=0 0 0 -> xyz=0 17.5 1.3563599907891557 rpy=0 0 0
- joint Torso_FrontLeg: origin xyz=0 18.5 1.2999163970265601 rpy=0 0 0 -> xyz=0 18.5 1.3563599907891557 rpy=0 0 0
- joint Torso_LeftLeg: origin xyz=-0.5 18 1.2999163970265601 rpy=0 0 0 -> xyz=-0.5 18 1.3563599907891557 rpy=0 0 0
- joint Torso_RightLeg: origin xyz=0.5 18 1.2999163970265601 rpy=0 0 0 -> xyz=0.5 18 1.3563599907891557 rpy=0 0 0
