Commit message: case3, evolved, JAR = .8

File: bodyFiles/body01899.urdf (robot description, URDF)
Before this commit: robot robot, 9 links, 8 joints
Links:
- link BackLeg: geometry collision box size=0.2 1.1428747462871542 0.2; visual box size=0.2 1.1428747462871542 0.2
- link BackLowerLeg: geometry collision box size=0.2 0.2 0.5619202679106461; visual box size=0.2 0.2 0.5619202679106461
- link FrontLeg: geometry collision box size=0.2 0.7835471753316936 0.2; visual box size=0.2 0.7835471753316936 0.2
- link FrontLowerLeg: geometry collision box size=0.2 0.2 0.869868711957066; visual box size=0.2 0.2 0.869868711957066
- link LeftLeg: geometry collision box size=1.278021077855593 0.2 0.2; visual box size=1.278021077855593 0.2 0.2
- link LeftLowerLeg: geometry collision box size=0.2 0.2 0.8432016114962587; visual box size=0.2 0.2 0.8432016114962587
- link RightLeg: geometry collision box size=1.1364776828249128 0.2 0.2; visual box size=1.1364776828249128 0.2 0.2
- link RightLowerLeg: geometry collision box size=0.2 0.2 1.2608510416996626; visual box size=0.2 0.2 1.2608510416996626
Joints:
- joint BackLeg_BackLowerLeg: origin xyz=0 -1.1696788138221441 0 rpy=0 0 0 -> xyz=0 -1.1428747462871542 0 rpy=0 0 0
- joint FrontLeg_FrontLowerLeg: origin xyz=0 1.3327987808227482 0 rpy=0 0 0 -> xyz=0 0.7835471753316936 0 rpy=0 0 0
- joint LeftLeg_LeftLowerLeg: origin xyz=-0.8384067903123168 0 0 rpy=0 0 0 -> xyz=-1.278021077855593 0 0 rpy=0 0 0
- joint RightLeg_RightLowerLeg: origin xyz=1.4153936008184873 0 0 rpy=0 0 0 -> xyz=1.1364776828249128 0 0 rpy=0 0 0
- joint Torso_BackLeg: origin xyz=0 17.5 1.4153936008184873 rpy=0 0 0 -> xyz=0 17.5 1.278021077855593 rpy=0 0 0
- joint Torso_FrontLeg: origin xyz=0 18.5 1.4153936008184873 rpy=0 0 0 -> xyz=0 18.5 1.278021077855593 rpy=0 0 0
- joint Torso_LeftLeg: origin xyz=-0.5 18 1.4153936008184873 rpy=0 0 0 -> xyz=-0.5 18 1.278021077855593 rpy=0 0 0
- joint Torso_RightLeg: origin xyz=0.5 18 1.4153936008184873 rpy=0 0 0 -> xyz=0.5 18 1.278021077855593 rpy=0 0 0
