Commit message: fitness curves: case3

File: bodyFiles/body0-10212.urdf (robot description, URDF)
Before this commit: robot robot, 9 links, 8 joints
Links:
- link BackLeg: geometry collision box size=0.2 0.5716405656859783 0.2; visual box size=0.2 0.5716405656859783 0.2
- link BackLowerLeg: geometry collision box size=0.2 0.2 1.4364559311722929; visual box size=0.2 0.2 1.4364559311722929
- link FrontLeg: geometry collision box size=0.2 1.1416384636998027 0.2; visual box size=0.2 1.1416384636998027 0.2
- link FrontLowerLeg: geometry collision box size=0.2 0.2 1.112710160047987; visual box size=0.2 0.2 1.112710160047987
- link LeftLeg: geometry collision box size=1.315232395041901 0.2 0.2; visual box size=1.315232395041901 0.2 0.2
- link LeftLowerLeg: geometry collision box size=0.2 0.2 0.9549424624476845; visual box size=0.2 0.2 0.9549424624476845
- link RightLeg: geometry collision box size=0.72475274773318 0.2 0.2; visual box size=0.72475274773318 0.2 0.2
- link RightLowerLeg: geometry collision box size=0.2 0.2 1.4300608434281967; visual box size=0.2 0.2 1.4300608434281967
Joints:
- joint BackLeg_BackLowerLeg: origin xyz=0 -1.1328736592006574 0 rpy=0 0 0 -> xyz=0 -0.5716405656859783 0 rpy=0 0 0
- joint FrontLeg_FrontLowerLeg: origin xyz=0 0.5922856923124648 0 rpy=0 0 0 -> xyz=0 1.1416384636998027 0 rpy=0 0 0
- joint LeftLeg_LeftLowerLeg: origin xyz=-0.6016513507269983 0 0 rpy=0 0 0 -> xyz=-1.315232395041901 0 0 rpy=0 0 0
- joint RightLeg_RightLowerLeg: origin xyz=1.497275212257315 0 0 rpy=0 0 0 -> xyz=0.72475274773318 0 0 rpy=0 0 0
- joint Torso_BackLeg: origin xyz=0 -10.5 1.497275212257315 rpy=0 0 0 -> xyz=0 -10.5 1.4364559311722929 rpy=0 0 0
- joint Torso_FrontLeg: origin xyz=0 -9.5 1.497275212257315 rpy=0 0 0 -> xyz=0 -9.5 1.4364559311722929 rpy=0 0 0
- joint Torso_LeftLeg: origin xyz=-0.5 -10 1.497275212257315 rpy=0 0 0 -> xyz=-0.5 -10 1.4364559311722929 rpy=0 0 0
- joint Torso_RightLeg: origin xyz=0.5 -10 1.497275212257315 rpy=0 0 0 -> xyz=0.5 -10 1.4364559311722929 rpy=0 0 0

File: bodyFiles/body0-10264.urdf (robot description, URDF)
Before this commit: robot robot, 9 links, 8 joints
Links:
- link BackLeg: geometry collision box size=0.2 0.5839572593025543 0.2; visual box size=0.2 0.5839572593025543 0.2
- link BackLowerLeg: geometry collision box size=0.2 0.2 0.7097956770575008; visual box size=0.2 0.2 0.7097956770575008
- link FrontLeg: geometry collision box size=0.2 0.7680234228296027 0.2; visual box size=0.2 0.7680234228296027 0.2
- link FrontLowerLeg: geometry collision box size=0.2 0.2 0.6840415724251057; visual box size=0.2 0.2 0.6840415724251057
- link LeftLeg: geometry collision box size=1.3553189618782384 0.2 0.2; visual box size=1.3553189618782384 0.2 0.2
- link LeftLowerLeg: geometry collision box size=0.2 0.2 1.4166341304361718; visual box size=0.2 0.2 1.4166341304361718
- link RightLeg: geometry collision box size=0.6496245170326367 0.2 0.2; visual box size=0.6496245170326367 0.2 0.2
- link RightLowerLeg: geometry collision box size=0.2 0.2 1.302135463666025; visual box size=0.2 0.2 1.302135463666025
Joints:
- joint BackLeg_BackLowerLeg: origin xyz=0 -1.1799286718966355 0 rpy=0 0 0 -> xyz=0 -0.5839572593025543 0 rpy=0 0 0
- joint FrontLeg_FrontLowerLeg: origin xyz=0 0.6835726089300751 0 rpy=0 0 0 -> xyz=0 0.7680234228296027 0 rpy=0 0 0
- joint LeftLeg_LeftLowerLeg: origin xyz=-1.1965982177398158 0 0 rpy=0 0 0 -> xyz=-1.3553189618782384 0 0 rpy=0 0 0
- joint RightLeg_RightLowerLeg: origin xyz=0.5904079879815576 0 0 rpy=0 0 0 -> xyz=0.6496245170326367 0 0 rpy=0 0 0
- joint Torso_BackLeg: origin xyz=0 -10.5 1.4081785379146186 rpy=0 0 0 -> xyz=0 -10.5 1.4166341304361718 rpy=0 0 0
- joint Torso_FrontLeg: origin xyz=0 -9.5 1.4081785379146186 rpy=0 0 0 -> xyz=0 -9.5 1.4166341304361718 rpy=0 0 0
- joint Torso_LeftLeg: origin xyz=-0.5 -10 1.4081785379146186 rpy=0 0 0 -> xyz=-0.5 -10 1.4166341304361718 rpy=0 0 0
- joint Torso_RightLeg: origin xyz=0.5 -10 1.4081785379146186 rpy=0 0 0 -> xyz=0.5 -10 1.4166341304361718 rpy=0 0 0

File: bodyFiles/body0-14105.urdf (robot description, URDF)
Before this commit: robot robot, 9 links, 8 joints
Links:
- link BackLeg: geometry collision box size=0.2 1.4824982324369407 0.2; visual box size=0.2 1.4824982324369407 0.2
- link BackLowerLeg: geometry collision box size=0.2 0.2 0.6517059460823679; visual box size=0.2 0.2 0.6517059460823679
- link FrontLeg: geometry collision box size=0.2 0.7442222444329596 0.2; visual box size=0.2 0.7442222444329596 0.2
- link FrontLowerLeg: geometry collision box size=0.2 0.2 1.302547595159159; visual box size=0.2 0.2 1.302547595159159
- link LeftLeg: geometry collision box size=1.4262657235977612 0.2 0.2; visual box size=1.4262657235977612 0.2 0.2
- link LeftLowerLeg: geometry collision box size=0.2 0.2 1.3581340103516797; visual box size=0.2 0.2 1.3581340103516797
- link RightLeg: geometry collision box size=0.9351719212418178 0.2 0.2; visual box size=0.9351719212418178 0.2 0.2
- link RightLowerLeg: geometry collision box size=0.2 0.2 1.1725155087780492; visual box size=0.2 0.2 1.1725155087780492
Joints:
- joint BackLeg_BackLowerLeg: origin xyz=0 -0.6244105573797067 0 rpy=0 0 0 -> xyz=0 -1.4824982324369407 0 rpy=0 0 0
- joint FrontLeg_FrontLowerLeg: origin xyz=0 0.9336990960276266 0 rpy=0 0 0 -> xyz=0 0.7442222444329596 0 rpy=0 0 0
- joint LeftLeg_LeftLowerLeg: origin xyz=-0.8940361080116215 0 0 rpy=0 0 0 -> xyz=-1.4262657235977612 0 0 rpy=0 0 0
- joint RightLeg_RightLowerLeg: origin xyz=0.5086711115505163 0 0 rpy=0 0 0 -> xyz=0.9351719212418178 0 0 rpy=0 0 0
- joint Torso_BackLeg: origin xyz=0 -14.5 1.467794387271632 rpy=0 0 0 -> xyz=0 -14.5 1.4824982324369407 rpy=0 0 0
- joint Torso_FrontLeg: origin xyz=0 -13.5 1.467794387271632 rpy=0 0 0 -> xyz=0 -13.5 1.4824982324369407 rpy=0 0 0
- joint Torso_LeftLeg: origin xyz=-0.5 -14 1.467794387271632 rpy=0 0 0 -> xyz=-0.5 -14 1.4824982324369407 rpy=0 0 0
- joint Torso_RightLeg: origin xyz=0.5 -14 1.467794387271632 rpy=0 0 0 -> xyz=0.5 -14 1.4824982324369407 rpy=0 0 0

File: bodyFiles/body0-14158.urdf (robot description, URDF)
Before this commit: robot robot, 9 links, 8 joints
Links:
- link BackLeg: geometry collision box size=0.2 1.4181396740390693 0.2; visual box size=0.2 1.4181396740390693 0.2
- link BackLowerLeg: geometry collision box size=0.2 0.2 1.4620517694949406; visual box size=0.2 0.2 1.4620517694949406
- link FrontLeg: geometry collision box size=0.2 0.7157343007311552 0.2; visual box size=0.2 0.7157343007311552 0.2
- link FrontLowerLeg: geometry collision box size=0.2 0.2 1.09740382557678; visual box size=0.2 0.2 1.09740382557678
- link LeftLeg: geometry collision box size=1.4109229457234556 0.2 0.2; visual box size=1.4109229457234556 0.2 0.2
- link LeftLowerLeg: geometry collision box size=0.2 0.2 1.1454245850672171; visual box size=0.2 0.2 1.1454245850672171
- link RightLeg: geometry collision box size=0.5221487732421327 0.2 0.2; visual box size=0.5221487732421327 0.2 0.2
- link RightLowerLeg: geometry collision box size=0.2 0.2 0.5571525400192414; visual box size=0.2 0.2 0.5571525400192414
Joints:
- joint BackLeg_BackLowerLeg: origin xyz=0 -0.9269245998317156 0 rpy=0 0 0 -> xyz=0 -1.4181396740390693 0 rpy=0 0 0
- joint FrontLeg_FrontLowerLeg: origin xyz=0 1.3527254445855363 0 rpy=0 0 0 -> xyz=0 0.7157343007311552 0 rpy=0 0 0
- joint LeftLeg_LeftLowerLeg: origin xyz=-0.7079747078763265 0 0 rpy=0 0 0 -> xyz=-1.4109229457234556 0 0 rpy=0 0 0
- joint RightLeg_RightLowerLeg: origin xyz=0.7718869147496887 0 0 rpy=0 0 0 -> xyz=0.5221487732421327 0 0 rpy=0 0 0
- joint Torso_BackLeg: origin xyz=0 -14.5 1.455236263769434 rpy=0 0 0 -> xyz=0 -14.5 1.4620517694949406 rpy=0 0 0
- joint Torso_FrontLeg: origin xyz=0 -13.5 1.455236263769434 rpy=0 0 0 -> xyz=0 -13.5 1.4620517694949406 rpy=0 0 0
- joint Torso_LeftLeg: origin xyz=-0.5 -14 1.455236263769434 rpy=0 0 0 -> xyz=-0.5 -14 1.4620517694949406 rpy=0 0 0
- joint Torso_RightLeg: origin xyz=0.5 -14 1.455236263769434 rpy=0 0 0 -> xyz=0.5 -14 1.4620517694949406 rpy=0 0 0

File: bodyFiles/body0-14206.urdf (robot description, URDF)
Before this commit: robot robot, 9 links, 8 joints
Links:
- link BackLeg: geometry collision box size=0.2 1.362015909060724 0.2; visual box size=0.2 1.362015909060724 0.2
- link BackLowerLeg: geometry collision box size=0.2 0.2 0.7549351251680259; visual box size=0.2 0.2 0.7549351251680259
- link FrontLeg: geometry collision box size=0.2 1.3624452321401437 0.2; visual box size=0.2 1.3624452321401437 0.2
- link FrontLowerLeg: geometry collision box size=0.2 0.2 1.0798647793870741; visual box size=0.2 0.2 1.0798647793870741
- link LeftLeg: geometry collision box size=1.4170340393684124 0.2 0.2; visual box size=1.4170340393684124 0.2 0.2
- link LeftLowerLeg: geometry collision box size=0.2 0.2 0.8335679874458641; visual box size=0.2 0.2 0.8335679874458641
- link RightLeg: geometry collision box size=1.200685637577722 0.2 0.2; visual box size=1.200685637577722 0.2 0.2
- link RightLowerLeg: geometry collision box size=0.2 0.2 1.2854390810985703; visual box size=0.2 0.2 1.2854390810985703
Joints:
- joint BackLeg_BackLowerLeg: origin xyz=0 -1.1802968418461717 0 rpy=0 0 0 -> xyz=0 -1.362015909060724 0 rpy=0 0 0
- joint FrontLeg_FrontLowerLeg: origin xyz=0 1.4050602433134296 0 rpy=0 0 0 -> xyz=0 1.3624452321401437 0 rpy=0 0 0
- joint LeftLeg_LeftLowerLeg: origin xyz=-0.948118338657177 0 0 rpy=0 0 0 -> xyz=-1.4170340393684124 0 0 rpy=0 0 0
- joint RightLeg_RightLowerLeg: origin xyz=0.7124825147344587 0 0 rpy=0 0 0 -> xyz=1.200685637577722 0 0 rpy=0 0 0
- joint Torso_BackLeg: origin xyz=0 -14.5 1.4050602433134296 rpy=0 0 0 -> xyz=0 -14.5 1.4170340393684124 rpy=0 0 0
- joint Torso_FrontLeg: origin xyz=0 -13.5 1.4050602433134296 rpy=0 0 0 -> xyz=0 -13.5 1.4170340393684124 rpy=0 0 0
- joint Torso_LeftLeg: origin xyz=-0.5 -14 1.4050602433134296 rpy=0 0 0 -> xyz=-0.5 -14 1.4170340393684124 rpy=0 0 0
- joint Torso_RightLeg: origin xyz=0.5 -14 1.4050602433134296 rpy=0 0 0 -> xyz=0.5 -14 1.4170340393684124 rpy=0 0 0

File: bodyFiles/body0-147.urdf (robot description, URDF)
Before this commit: robot robot, 9 links, 8 joints
Links:
- link BackLeg: geometry collision box size=0.2 1.3381989654176427 0.2; visual box size=0.2 1.3381989654176427 0.2
- link BackLowerLeg: geometry collision box size=0.2 0.2 1.3451182272566695; visual box size=0.2 0.2 1.3451182272566695
- link FrontLeg: geometry collision box size=0.2 1.0511840362246518 0.2; visual box size=0.2 1.0511840362246518 0.2
- link FrontLowerLeg: geometry collision box size=0.2 0.2 0.8756446396481777; visual box size=0.2 0.2 0.8756446396481777
- link LeftLeg: geometry collision box size=0.9245033793633056 0.2 0.2; visual box size=0.9245033793633056 0.2 0.2
- link LeftLowerLeg: geometry collision box size=0.2 0.2 0.5377912762163651; visual box size=0.2 0.2 0.5377912762163651
- link RightLeg: geometry collision box size=0.539631711426903 0.2 0.2; visual box size=0.539631711426903 0.2 0.2
- link RightLowerLeg: geometry collision box size=0.2 0.2 0.9555514170136566; visual box size=0.2 0.2 0.9555514170136566
Joints:
- joint BackLeg_BackLowerLeg: origin xyz=0 -0.9177833377187226 0 rpy=0 0 0 -> xyz=0 -1.3381989654176427 0 rpy=0 0 0
- joint FrontLeg_FrontLowerLeg: origin xyz=0 1.0451340662623638 0 rpy=0 0 0 -> xyz=0 1.0511840362246518 0 rpy=0 0 0
- joint LeftLeg_LeftLowerLeg: origin xyz=-0.8960657080860618 0 0 rpy=0 0 0 -> xyz=-0.9245033793633056 0 0 rpy=0 0 0
- joint RightLeg_RightLowerLeg: origin xyz=1.2164589998374267 0 0 rpy=0 0 0 -> xyz=0.539631711426903 0 0 rpy=0 0 0
- joint Torso_BackLeg: origin xyz=0 -14.5 1.2497540097759947 rpy=0 0 0 -> xyz=0 -14.5 1.3451182272566695 rpy=0 0 0
- joint Torso_FrontLeg: origin xyz=0 -13.5 1.2497540097759947 rpy=0 0 0 -> xyz=0 -13.5 1.3451182272566695 rpy=0 0 0
- joint Torso_LeftLeg: origin xyz=-0.5 -14 1.2497540097759947 rpy=0 0 0 -> xyz=-0.5 -14 1.3451182272566695 rpy=0 0 0
- joint Torso_RightLeg: origin xyz=0.5 -14 1.2497540097759947 rpy=0 0 0 -> xyz=0.5 -14 1.3451182272566695 rpy=0 0 0

File: bodyFiles/body0-180.urdf (robot description, URDF)
Before this commit: robot robot, 9 links, 8 joints
Links:
- link BackLeg: geometry collision box size=0.2 1.4416848487442315 0.2; visual box size=0.2 1.4416848487442315 0.2
- link BackLowerLeg: geometry collision box size=0.2 0.2 0.5926069827426426; visual box size=0.2 0.2 0.5926069827426426
- link FrontLeg: geometry collision box size=0.2 0.8854684896294055 0.2; visual box size=0.2 0.8854684896294055 0.2
- link FrontLowerLeg: geometry collision box size=0.2 0.2 0.7340081865595839; visual box size=0.2 0.2 0.7340081865595839
- link LeftLeg: geometry collision box size=1.4548733393131064 0.2 0.2; visual box size=1.4548733393131064 0.2 0.2
- link LeftLowerLeg: geometry collision box size=0.2 0.2 1.1370899113713948; visual box size=0.2 0.2 1.1370899113713948
- link RightLeg: geometry collision box size=0.5927868568892034 0.2 0.2; visual box size=0.5927868568892034 0.2 0.2
- link RightLowerLeg: geometry collision box size=0.2 0.2 1.2714725681784262; visual box size=0.2 0.2 1.2714725681784262
Joints:
- joint BackLeg_BackLowerLeg: origin xyz=0 -1.0102519257024818 0 rpy=0 0 0 -> xyz=0 -1.4416848487442315 0 rpy=0 0 0
- joint FrontLeg_FrontLowerLeg: origin xyz=0 1.3577426099226513 0 rpy=0 0 0 -> xyz=0 0.8854684896294055 0 rpy=0 0 0
- joint LeftLeg_LeftLowerLeg: origin xyz=-1.469806404183906 0 0 rpy=0 0 0 -> xyz=-1.4548733393131064 0 0 rpy=0 0 0
- joint RightLeg_RightLowerLeg: origin xyz=0.5771401235987005 0 0 rpy=0 0 0 -> xyz=0.5927868568892034 0 0 rpy=0 0 0
- joint Torso_BackLeg: origin xyz=0 -18.5 1.469806404183906 rpy=0 0 0 -> xyz=0 -18.5 1.4548733393131064 rpy=0 0 0
- joint Torso_FrontLeg: origin xyz=0 -17.5 1.469806404183906 rpy=0 0 0 -> xyz=0 -17.5 1.4548733393131064 rpy=0 0 0
- joint Torso_LeftLeg: origin xyz=-0.5 -18 1.469806404183906 rpy=0 0 0 -> xyz=-0.5 -18 1.4548733393131064 rpy=0 0 0
- joint Torso_RightLeg: origin xyz=0.5 -18 1.469806404183906 rpy=0 0 0 -> xyz=0.5 -18 1.4548733393131064 rpy=0 0 0

File: bodyFiles/body0-18202.urdf (robot description, URDF)
Before this commit: robot robot, 9 links, 8 joints
Links:
- link BackLeg: geometry collision box size=0.2 0.5817575744833378 0.2; visual box size=0.2 0.5817575744833378 0.2
- link BackLowerLeg: geometry collision box size=0.2 0.2 1.4727943323133559; visual box size=0.2 0.2 1.4727943323133559
- link FrontLeg: geometry collision box size=0.2 1.3795995977453877 0.2; visual box size=0.2 1.3795995977453877 0.2
- link FrontLowerLeg: geometry collision box size=0.2 0.2 0.8290440034075368; visual box size=0.2 0.2 0.8290440034075368
- link LeftLeg: geometry collision box size=1.4708783586952894 0.2 0.2; visual box size=1.4708783586952894 0.2 0.2
- link LeftLowerLeg: geometry collision box size=0.2 0.2 1.040795813955067; visual box size=0.2 0.2 1.040795813955067
- link RightLeg: geometry collision box size=0.6891677293002858 0.2 0.2; visual box size=0.6891677293002858 0.2 0.2
- link RightLowerLeg: geometry collision box size=0.2 0.2 0.9104919626591859; visual box size=0.2 0.2 0.9104919626591859
Joints:
- joint BackLeg_BackLowerLeg: origin xyz=0 -0.542008400323147 0 rpy=0 0 0 -> xyz=0 -0.5817575744833378 0 rpy=0 0 0
- joint FrontLeg_FrontLowerLeg: origin xyz=0 1.149818092886808 0 rpy=0 0 0 -> xyz=0 1.3795995977453877 0 rpy=0 0 0
- joint LeftLeg_LeftLowerLeg: origin xyz=-1.3475194795455145 0 0 rpy=0 0 0 -> xyz=-1.4708783586952894 0 0 rpy=0 0 0
- joint RightLeg_RightLowerLeg: origin xyz=0.8354533459217964 0 0 rpy=0 0 0 -> xyz=0.6891677293002858 0 0 rpy=0 0 0
- joint Torso_BackLeg: origin xyz=0 -18.5 1.3475194795455145 rpy=0 0 0 -> xyz=0 -18.5 1.4727943323133559 rpy=0 0 0
- joint Torso_FrontLeg: origin xyz=0 -17.5 1.3475194795455145 rpy=0 0 0 -> xyz=0 -17.5 1.4727943323133559 rpy=0 0 0
- joint Torso_LeftLeg: origin xyz=-0.5 -18 1.3475194795455145 rpy=0 0 0 -> xyz=-0.5 -18 1.4727943323133559 rpy=0 0 0
- joint Torso_RightLeg: origin xyz=0.5 -18 1.3475194795455145 rpy=0 0 0 -> xyz=0.5 -18 1.4727943323133559 rpy=0 0 0

File: bodyFiles/body0-274.urdf (robot description, URDF)
Before this commit: robot robot, 9 links, 8 joints
Links:
- link BackLeg: geometry collision box size=0.2 1.2813960891099958 0.2; visual box size=0.2 1.2813960891099958 0.2
- link BackLowerLeg: geometry collision box size=0.2 0.2 0.6829853895497167; visual box size=0.2 0.2 0.6829853895497167
- link FrontLeg: geometry collision box size=0.2 0.5918040585608451 0.2; visual box size=0.2 0.5918040585608451 0.2
- link FrontLowerLeg: geometry collision box size=0.2 0.2 0.9722769825585493; visual box size=0.2 0.2 0.9722769825585493
- link LeftLeg: geometry collision box size=1.2816839998979792 0.2 0.2; visual box size=1.2816839998979792 0.2 0.2
- link LeftLowerLeg: geometry collision box size=0.2 0.2 1.3036965519711505; visual box size=0.2 0.2 1.3036965519711505
- link RightLeg: geometry collision box size=0.5665829148187338 0.2 0.2; visual box size=0.5665829148187338 0.2 0.2
- link RightLowerLeg: geometry collision box size=0.2 0.2 1.4484756543563801; visual box size=0.2 0.2 1.4484756543563801
Joints:
- joint BackLeg_BackLowerLeg: origin xyz=0 -0.5737393287595878 0 rpy=0 0 0 -> xyz=0 -1.2813960891099958 0 rpy=0 0 0
- joint FrontLeg_FrontLowerLeg: origin xyz=0 1.352493152096768 0 rpy=0 0 0 -> xyz=0 0.5918040585608451 0 rpy=0 0 0
- joint LeftLeg_LeftLowerLeg: origin xyz=-0.7038323120977741 0 0 rpy=0 0 0 -> xyz=-1.2816839998979792 0 0 rpy=0 0 0
- joint RightLeg_RightLowerLeg: origin xyz=1.067353734726546 0 0 rpy=0 0 0 -> xyz=0.5665829148187338 0 0 rpy=0 0 0
- joint Torso_BackLeg: origin xyz=0 -2.5 1.4938730835966507 rpy=0 0 0 -> xyz=0 -2.5 1.4484756543563801 rpy=0 0 0
- joint Torso_FrontLeg: origin xyz=0 -1.5 1.4938730835966507 rpy=0 0 0 -> xyz=0 -1.5 1.4484756543563801 rpy=0 0 0
- joint Torso_LeftLeg: origin xyz=-0.5 -2 1.4938730835966507 rpy=0 0 0 -> xyz=-0.5 -2 1.4484756543563801 rpy=0 0 0
- joint Torso_RightLeg: origin xyz=0.5 -2 1.4938730835966507 rpy=0 0 0 -> xyz=0.5 -2 1.4484756543563801 rpy=0 0 0

File: bodyFiles/body0-6165.urdf (robot description, URDF)
Before this commit: robot robot, 9 links, 8 joints
Links:
- link BackLeg: geometry collision box size=0.2 0.5141272122165004 0.2; visual box size=0.2 0.5141272122165004 0.2
- link BackLowerLeg: geometry collision box size=0.2 0.2 1.329620909962558; visual box size=0.2 0.2 1.329620909962558
- link FrontLeg: geometry collision box size=0.2 1.4324664106176896 0.2; visual box size=0.2 1.4324664106176896 0.2
- link FrontLowerLeg: geometry collision box size=0.2 0.2 1.435749882462007; visual box size=0.2 0.2 1.435749882462007
- link LeftLeg: geometry collision box size=0.7652915967639768 0.2 0.2; visual box size=0.7652915967639768 0.2 0.2
- link LeftLowerLeg: geometry collision box size=0.2 0.2 0.908065222537727; visual box size=0.2 0.2 0.908065222537727
- link RightLeg: geometry collision box size=1.3666417591604243 0.2 0.2; visual box size=1.3666417591604243 0.2 0.2
- link RightLowerLeg: geometry collision box size=0.2 0.2 0.5787144510964786; visual box size=0.2 0.2 0.5787144510964786
Joints:
- joint BackLeg_BackLowerLeg: origin xyz=0 -1.2858841117544135 0 rpy=0 0 0 -> xyz=0 -0.5141272122165004 0 rpy=0 0 0
- joint FrontLeg_FrontLowerLeg: origin xyz=0 0.8472963441510946 0 rpy=0 0 0 -> xyz=0 1.4324664106176896 0 rpy=0 0 0
- joint LeftLeg_LeftLowerLeg: origin xyz=-1.3505971217698347 0 0 rpy=0 0 0 -> xyz=-0.7652915967639768 0 0 rpy=0 0 0
- joint RightLeg_RightLowerLeg: origin xyz=1.0806489911364483 0 0 rpy=0 0 0 -> xyz=1.3666417591604243 0 0 rpy=0 0 0
- joint Torso_BackLeg: origin xyz=0 -6.5 1.4770041031813115 rpy=0 0 0 -> xyz=0 -6.5 1.435749882462007 rpy=0 0 0
- joint Torso_FrontLeg: origin xyz=0 -5.5 1.4770041031813115 rpy=0 0 0 -> xyz=0 -5.5 1.435749882462007 rpy=0 0 0
- joint Torso_LeftLeg: origin xyz=-0.5 -6 1.4770041031813115 rpy=0 0 0 -> xyz=-0.5 -6 1.435749882462007 rpy=0 0 0
- joint Torso_RightLeg: origin xyz=0.5 -6 1.4770041031813115 rpy=0 0 0 -> xyz=0.5 -6 1.435749882462007 rpy=0 0 0

File: bodyFiles/body0-6266.urdf (robot description, URDF)
Before this commit: robot robot, 9 links, 8 joints
Links:
- link BackLeg: geometry collision box size=0.2 0.8595507882444546 0.2; visual box size=0.2 0.8595507882444546 0.2
- link BackLowerLeg: geometry collision box size=0.2 0.2 1.1683922662455903; visual box size=0.2 0.2 1.1683922662455903
- link FrontLeg: geometry collision box size=0.2 0.5379255306813561 0.2; visual box size=0.2 0.5379255306813561 0.2
- link FrontLowerLeg: geometry collision box size=0.2 0.2 0.8783759490626519; visual box size=0.2 0.2 0.8783759490626519
- link LeftLeg: geometry collision box size=1.4186204498778312 0.2 0.2; visual box size=1.4186204498778312 0.2 0.2
- link LeftLowerLeg: geometry collision box size=0.2 0.2 1.1786353932718705; visual box size=0.2 0.2 1.1786353932718705
- link RightLeg: geometry collision box size=1.2998448542730934 0.2 0.2; visual box size=1.2998448542730934 0.2 0.2
- link RightLowerLeg: geometry collision box size=0.2 0.2 0.8860866676147371; visual box size=0.2 0.2 0.8860866676147371
Joints:
- joint BackLeg_BackLowerLeg: origin xyz=0 -0.8639486246268134 0 rpy=0 0 0 -> xyz=0 -0.8595507882444546 0 rpy=0 0 0
- joint FrontLeg_FrontLowerLeg: origin xyz=0 1.407727054991398 0 rpy=0 0 0 -> xyz=0 0.5379255306813561 0 rpy=0 0 0
- joint LeftLeg_LeftLowerLeg: origin xyz=-0.8528269133719504 0 0 rpy=0 0 0 -> xyz=-1.4186204498778312 0 0 rpy=0 0 0
- joint RightLeg_RightLowerLeg: origin xyz=1.2387426136421218 0 0 rpy=0 0 0 -> xyz=1.2998448542730934 0 0 rpy=0 0 0
- joint Torso_BackLeg: origin xyz=0 -6.5 1.407727054991398 rpy=0 0 0 -> xyz=0 -6.5 1.4186204498778312 rpy=0 0 0
- joint Torso_FrontLeg: origin xyz=0 -5.5 1.407727054991398 rpy=0 0 0 -> xyz=0 -5.5 1.4186204498778312 rpy=0 0 0
- joint Torso_LeftLeg: origin xyz=-0.5 -6 1.407727054991398 rpy=0 0 0 -> xyz=-0.5 -6 1.4186204498778312 rpy=0 0 0
- joint Torso_RightLeg: origin xyz=0.5 -6 1.407727054991398 rpy=0 0 0 -> xyz=0.5 -6 1.4186204498778312 rpy=0 0 0
