Commit message: fitness curves: case3

File: bodyFiles/body010135.urdf (robot description, URDF)
Before this commit: robot robot, 9 links, 8 joints
Links:
- link BackLeg: geometry collision box size=0.2 0.5827568557127135 0.2; visual box size=0.2 0.5827568557127135 0.2
- link BackLowerLeg: geometry collision box size=0.2 0.2 1.2538198379308536; visual box size=0.2 0.2 1.2538198379308536
- link FrontLeg: geometry collision box size=0.2 0.6701278017139972 0.2; visual box size=0.2 0.6701278017139972 0.2
- link FrontLowerLeg: geometry collision box size=0.2 0.2 1.2625107408104577; visual box size=0.2 0.2 1.2625107408104577
- link LeftLeg: geometry collision box size=1.3097098200059154 0.2 0.2; visual box size=1.3097098200059154 0.2 0.2
- link LeftLowerLeg: geometry collision box size=0.2 0.2 1.3555712132045648; visual box size=0.2 0.2 1.3555712132045648
- link RightLeg: geometry collision box size=1.2582296449630626 0.2 0.2; visual box size=1.2582296449630626 0.2 0.2
- link RightLowerLeg: geometry collision box size=0.2 0.2 1.4175662164052043; visual box size=0.2 0.2 1.4175662164052043
Joints:
- joint BackLeg_BackLowerLeg: origin xyz=0 -1.4676977781393128 0 rpy=0 0 0 -> xyz=0 -0.5827568557127135 0 rpy=0 0 0
- joint FrontLeg_FrontLowerLeg: origin xyz=0 0.5376453429613783 0 rpy=0 0 0 -> xyz=0 0.6701278017139972 0 rpy=0 0 0
- joint LeftLeg_LeftLowerLeg: origin xyz=-1.4821481946948682 0 0 rpy=0 0 0 -> xyz=-1.3097098200059154 0 0 rpy=0 0 0
- joint RightLeg_RightLowerLeg: origin xyz=0.858563147945224 0 0 rpy=0 0 0 -> xyz=1.2582296449630626 0 0 rpy=0 0 0
- joint Torso_BackLeg: origin xyz=0 9.5 1.4821481946948682 rpy=0 0 0 -> xyz=0 9.5 1.4175662164052043 rpy=0 0 0
- joint Torso_FrontLeg: origin xyz=0 10.5 1.4821481946948682 rpy=0 0 0 -> xyz=0 10.5 1.4175662164052043 rpy=0 0 0
- joint Torso_LeftLeg: origin xyz=-0.5 10 1.4821481946948682 rpy=0 0 0 -> xyz=-0.5 10 1.4175662164052043 rpy=0 0 0
- joint Torso_RightLeg: origin xyz=0.5 10 1.4821481946948682 rpy=0 0 0 -> xyz=0.5 10 1.4175662164052043 rpy=0 0 0

File: bodyFiles/body01035.urdf (robot description, URDF)
Before this commit: robot robot, 9 links, 8 joints
Links:
- link BackLeg: geometry collision box size=0.2 0.7900673784057026 0.2; visual box size=0.2 0.7900673784057026 0.2
- link BackLowerLeg: geometry collision box size=0.2 0.2 1.4277970682715464; visual box size=0.2 0.2 1.4277970682715464
- link FrontLeg: geometry collision box size=0.2 1.480024572985994 0.2; visual box size=0.2 1.480024572985994 0.2
- link FrontLowerLeg: geometry collision box size=0.2 0.2 1.2709648456282991; visual box size=0.2 0.2 1.2709648456282991
- link LeftLeg: geometry collision box size=0.7121727512689805 0.2 0.2; visual box size=0.7121727512689805 0.2 0.2
- link LeftLowerLeg: geometry collision box size=0.2 0.2 1.3967787983468436; visual box size=0.2 0.2 1.3967787983468436
- link RightLeg: geometry collision box size=1.422569832515354 0.2 0.2; visual box size=1.422569832515354 0.2 0.2
- link RightLowerLeg: geometry collision box size=0.2 0.2 0.9701003508562845; visual box size=0.2 0.2 0.9701003508562845
Joints:
- joint BackLeg_BackLowerLeg: origin xyz=0 -1.4469473166671336 0 rpy=0 0 0 -> xyz=0 -0.7900673784057026 0 rpy=0 0 0
- joint FrontLeg_FrontLowerLeg: origin xyz=0 0.7724969033169515 0 rpy=0 0 0 -> xyz=0 1.480024572985994 0 rpy=0 0 0
- joint LeftLeg_LeftLowerLeg: origin xyz=-0.9112856434262138 0 0 rpy=0 0 0 -> xyz=-0.7121727512689805 0 0 rpy=0 0 0
- joint RightLeg_RightLowerLeg: origin xyz=0.5561682852763828 0 0 rpy=0 0 0 -> xyz=1.422569832515354 0 0 rpy=0 0 0
- joint Torso_BackLeg: origin xyz=0 9.5 1.4922981327498464 rpy=0 0 0 -> xyz=0 9.5 1.480024572985994 rpy=0 0 0
- joint Torso_FrontLeg: origin xyz=0 10.5 1.4922981327498464 rpy=0 0 0 -> xyz=0 10.5 1.480024572985994 rpy=0 0 0
- joint Torso_LeftLeg: origin xyz=-0.5 10 1.4922981327498464 rpy=0 0 0 -> xyz=-0.5 10 1.480024572985994 rpy=0 0 0
- joint Torso_RightLeg: origin xyz=0.5 10 1.4922981327498464 rpy=0 0 0 -> xyz=0.5 10 1.480024572985994 rpy=0 0 0

File: bodyFiles/body01087.urdf (robot description, URDF)
Before this commit: robot robot, 9 links, 8 joints
Links:
- link BackLeg: geometry collision box size=0.2 1.011510062913158 0.2; visual box size=0.2 1.011510062913158 0.2
- link BackLowerLeg: geometry collision box size=0.2 0.2 1.285283290654713; visual box size=0.2 0.2 1.285283290654713
- link FrontLeg: geometry collision box size=0.2 0.9894416798044028 0.2; visual box size=0.2 0.9894416798044028 0.2
- link FrontLowerLeg: geometry collision box size=0.2 0.2 1.1690535445221928; visual box size=0.2 0.2 1.1690535445221928
- link LeftLeg: geometry collision box size=1.1129513129866502 0.2 0.2; visual box size=1.1129513129866502 0.2 0.2
- link LeftLowerLeg: geometry collision box size=0.2 0.2 0.6512315906818162; visual box size=0.2 0.2 0.6512315906818162
- link RightLeg: geometry collision box size=1.3318824226757386 0.2 0.2; visual box size=1.3318824226757386 0.2 0.2
- link RightLowerLeg: geometry collision box size=0.2 0.2 1.355854063546154; visual box size=0.2 0.2 1.355854063546154
Joints:
- joint BackLeg_BackLowerLeg: origin xyz=0 -0.6515595422317949 0 rpy=0 0 0 -> xyz=0 -1.011510062913158 0 rpy=0 0 0
- joint FrontLeg_FrontLowerLeg: origin xyz=0 0.9190235954637531 0 rpy=0 0 0 -> xyz=0 0.9894416798044028 0 rpy=0 0 0
- joint LeftLeg_LeftLowerLeg: origin xyz=-1.3211951788283085 0 0 rpy=0 0 0 -> xyz=-1.1129513129866502 0 0 rpy=0 0 0
- joint RightLeg_RightLowerLeg: origin xyz=0.5107125346546818 0 0 rpy=0 0 0 -> xyz=1.3318824226757386 0 0 rpy=0 0 0
- joint Torso_BackLeg: origin xyz=0 9.5 1.4835274178031361 rpy=0 0 0 -> xyz=0 9.5 1.355854063546154 rpy=0 0 0
- joint Torso_FrontLeg: origin xyz=0 10.5 1.4835274178031361 rpy=0 0 0 -> xyz=0 10.5 1.355854063546154 rpy=0 0 0
- joint Torso_LeftLeg: origin xyz=-0.5 10 1.4835274178031361 rpy=0 0 0 -> xyz=-0.5 10 1.355854063546154 rpy=0 0 0
- joint Torso_RightLeg: origin xyz=0.5 10 1.4835274178031361 rpy=0 0 0 -> xyz=0.5 10 1.355854063546154 rpy=0 0 0

File: bodyFiles/body014192.urdf (robot description, URDF)
Before this commit: robot robot, 9 links, 8 joints
Links:
- link BackLeg: geometry collision box size=0.2 0.9079644376006442 0.2; visual box size=0.2 0.9079644376006442 0.2
- link BackLowerLeg: geometry collision box size=0.2 0.2 0.5004938736404008; visual box size=0.2 0.2 0.5004938736404008
- link FrontLeg: geometry collision box size=0.2 1.2517031746545473 0.2; visual box size=0.2 1.2517031746545473 0.2
- link FrontLowerLeg: geometry collision box size=0.2 0.2 1.228721437344857; visual box size=0.2 0.2 1.228721437344857
- link LeftLeg: geometry collision box size=1.161643296680014 0.2 0.2; visual box size=1.161643296680014 0.2 0.2
- link LeftLowerLeg: geometry collision box size=0.2 0.2 1.242362364098529; visual box size=0.2 0.2 1.242362364098529
- link RightLeg: geometry collision box size=0.6452346987211657 0.2 0.2; visual box size=0.6452346987211657 0.2 0.2
- link RightLowerLeg: geometry collision box size=0.2 0.2 0.5667232896430499; visual box size=0.2 0.2 0.5667232896430499
Joints:
- joint BackLeg_BackLowerLeg: origin xyz=0 -0.8159154641209329 0 rpy=0 0 0 -> xyz=0 -0.9079644376006442 0 rpy=0 0 0
- joint FrontLeg_FrontLowerLeg: origin xyz=0 0.6149771429897862 0 rpy=0 0 0 -> xyz=0 1.2517031746545473 0 rpy=0 0 0
- joint LeftLeg_LeftLowerLeg: origin xyz=-0.5709043179624638 0 0 rpy=0 0 0 -> xyz=-1.161643296680014 0 0 rpy=0 0 0
- joint RightLeg_RightLowerLeg: origin xyz=1.234880449028668 0 0 rpy=0 0 0 -> xyz=0.6452346987211657 0 0 rpy=0 0 0
- joint Torso_BackLeg: origin xyz=0 13.5 1.289229538711671 rpy=0 0 0 -> xyz=0 13.5 1.2517031746545473 rpy=0 0 0
- joint Torso_FrontLeg: origin xyz=0 14.5 1.289229538711671 rpy=0 0 0 -> xyz=0 14.5 1.2517031746545473 rpy=0 0 0
- joint Torso_LeftLeg: origin xyz=-0.5 14 1.289229538711671 rpy=0 0 0 -> xyz=-0.5 14 1.2517031746545473 rpy=0 0 0
- joint Torso_RightLeg: origin xyz=0.5 14 1.289229538711671 rpy=0 0 0 -> xyz=0.5 14 1.2517031746545473 rpy=0 0 0

File: bodyFiles/body01896.urdf (robot description, URDF)
Before this commit: robot robot, 9 links, 8 joints
Links:
- link BackLeg: geometry collision box size=0.2 1.0040441885064466 0.2; visual box size=0.2 1.0040441885064466 0.2
- link BackLowerLeg: geometry collision box size=0.2 0.2 1.2379357933795923; visual box size=0.2 0.2 1.2379357933795923
- link FrontLeg: geometry collision box size=0.2 0.5906025012824483 0.2; visual box size=0.2 0.5906025012824483 0.2
- link FrontLowerLeg: geometry collision box size=0.2 0.2 0.918946768380111; visual box size=0.2 0.2 0.918946768380111
- link LeftLeg: geometry collision box size=1.044226387415327 0.2 0.2; visual box size=1.044226387415327 0.2 0.2
- link LeftLowerLeg: geometry collision box size=0.2 0.2 0.5333031885001225; visual box size=0.2 0.2 0.5333031885001225
- link RightLeg: geometry collision box size=0.9551777236000984 0.2 0.2; visual box size=0.9551777236000984 0.2 0.2
- link RightLowerLeg: geometry collision box size=0.2 0.2 1.4290458543484623; visual box size=0.2 0.2 1.4290458543484623
Joints:
- joint BackLeg_BackLowerLeg: origin xyz=0 -1.4059781176293706 0 rpy=0 0 0 -> xyz=0 -1.0040441885064466 0 rpy=0 0 0
- joint FrontLeg_FrontLowerLeg: origin xyz=0 1.1900593069145433 0 rpy=0 0 0 -> xyz=0 0.5906025012824483 0 rpy=0 0 0
- joint LeftLeg_LeftLowerLeg: origin xyz=-0.5422556486380851 0 0 rpy=0 0 0 -> xyz=-1.044226387415327 0 0 rpy=0 0 0
- joint RightLeg_RightLowerLeg: origin xyz=1.4532113331997771 0 0 rpy=0 0 0 -> xyz=0.9551777236000984 0 0 rpy=0 0 0
- joint Torso_BackLeg: origin xyz=0 17.5 1.4532113331997771 rpy=0 0 0 -> xyz=0 17.5 1.4290458543484623 rpy=0 0 0
- joint Torso_FrontLeg: origin xyz=0 18.5 1.4532113331997771 rpy=0 0 0 -> xyz=0 18.5 1.4290458543484623 rpy=0 0 0
- joint Torso_LeftLeg: origin xyz=-0.5 18 1.4532113331997771 rpy=0 0 0 -> xyz=-0.5 18 1.4290458543484623 rpy=0 0 0
- joint Torso_RightLeg: origin xyz=0.5 18 1.4532113331997771 rpy=0 0 0 -> xyz=0.5 18 1.4290458543484623 rpy=0 0 0

File: bodyFiles/body02226.urdf (robot description, URDF)
Before this commit: robot robot, 9 links, 8 joints
Links:
- link BackLeg: geometry collision box size=0.2 0.9979797008127949 0.2; visual box size=0.2 0.9979797008127949 0.2
- link BackLowerLeg: geometry collision box size=0.2 0.2 0.5161664836763995; visual box size=0.2 0.2 0.5161664836763995
- link FrontLeg: geometry collision box size=0.2 1.0296656455149567 0.2; visual box size=0.2 1.0296656455149567 0.2
- link FrontLowerLeg: geometry collision box size=0.2 0.2 1.2982710547807241; visual box size=0.2 0.2 1.2982710547807241
- link LeftLeg: geometry collision box size=1.1661099064708682 0.2 0.2; visual box size=1.1661099064708682 0.2 0.2
- link LeftLowerLeg: geometry collision box size=0.2 0.2 1.4386443028299576; visual box size=0.2 0.2 1.4386443028299576
- link RightLeg: geometry collision box size=0.6233668332543193 0.2 0.2; visual box size=0.6233668332543193 0.2 0.2
- link RightLowerLeg: geometry collision box size=0.2 0.2 0.6913016736300668; visual box size=0.2 0.2 0.6913016736300668
Joints:
- joint BackLeg_BackLowerLeg: origin xyz=0 -0.7461187442923859 0 rpy=0 0 0 -> xyz=0 -0.9979797008127949 0 rpy=0 0 0
- joint FrontLeg_FrontLowerLeg: origin xyz=0 1.253728260561506 0 rpy=0 0 0 -> xyz=0 1.0296656455149567 0 rpy=0 0 0
- joint LeftLeg_LeftLowerLeg: origin xyz=-1.1813522393790428 0 0 rpy=0 0 0 -> xyz=-1.1661099064708682 0 0 rpy=0 0 0
- joint RightLeg_RightLowerLeg: origin xyz=0.7453426765804821 0 0 rpy=0 0 0 -> xyz=0.6233668332543193 0 0 rpy=0 0 0
- joint Torso_BackLeg: origin xyz=0 1.5 1.253728260561506 rpy=0 0 0 -> xyz=0 1.5 1.4386443028299576 rpy=0 0 0
- joint Torso_FrontLeg: origin xyz=0 2.5 1.253728260561506 rpy=0 0 0 -> xyz=0 2.5 1.4386443028299576 rpy=0 0 0
- joint Torso_LeftLeg: origin xyz=-0.5 2 1.253728260561506 rpy=0 0 0 -> xyz=-0.5 2 1.4386443028299576 rpy=0 0 0
- joint Torso_RightLeg: origin xyz=0.5 2 1.253728260561506 rpy=0 0 0 -> xyz=0.5 2 1.4386443028299576 rpy=0 0 0

File: bodyFiles/body0634.urdf (robot description, URDF)
Before this commit: robot robot, 9 links, 8 joints
Links:
- link BackLeg: geometry collision box size=0.2 0.9020923435702102 0.2; visual box size=0.2 0.9020923435702102 0.2
- link BackLowerLeg: geometry collision box size=0.2 0.2 0.5533084974106074; visual box size=0.2 0.2 0.5533084974106074
- link FrontLeg: geometry collision box size=0.2 0.584263055548962 0.2; visual box size=0.2 0.584263055548962 0.2
- link FrontLowerLeg: geometry collision box size=0.2 0.2 0.8666556061357181; visual box size=0.2 0.2 0.8666556061357181
- link LeftLeg: geometry collision box size=0.6331406808379608 0.2 0.2; visual box size=0.6331406808379608 0.2 0.2
- link LeftLowerLeg: geometry collision box size=0.2 0.2 0.5635366582523826; visual box size=0.2 0.2 0.5635366582523826
- link RightLeg: geometry collision box size=0.6431820278524941 0.2 0.2; visual box size=0.6431820278524941 0.2 0.2
- link RightLowerLeg: geometry collision box size=0.2 0.2 1.247313807623207; visual box size=0.2 0.2 1.247313807623207
Joints:
- joint BackLeg_BackLowerLeg: origin xyz=0 -1.1375656851765201 0 rpy=0 0 0 -> xyz=0 -0.9020923435702102 0 rpy=0 0 0
- joint FrontLeg_FrontLowerLeg: origin xyz=0 0.823500122111556 0 rpy=0 0 0 -> xyz=0 0.584263055548962 0 rpy=0 0 0
- joint LeftLeg_LeftLowerLeg: origin xyz=-0.798545281663112 0 0 rpy=0 0 0 -> xyz=-0.6331406808379608 0 0 rpy=0 0 0
- joint RightLeg_RightLowerLeg: origin xyz=0.6675284490536635 0 0 rpy=0 0 0 -> xyz=0.6431820278524941 0 0 rpy=0 0 0
- joint Torso_BackLeg: origin xyz=0 5.5 1.267093285844465 rpy=0 0 0 -> xyz=0 5.5 1.247313807623207 rpy=0 0 0
- joint Torso_FrontLeg: origin xyz=0 6.5 1.267093285844465 rpy=0 0 0 -> xyz=0 6.5 1.247313807623207 rpy=0 0 0
- joint Torso_LeftLeg: origin xyz=-0.5 6 1.267093285844465 rpy=0 0 0 -> xyz=-0.5 6 1.247313807623207 rpy=0 0 0
- joint Torso_RightLeg: origin xyz=0.5 6 1.267093285844465 rpy=0 0 0 -> xyz=0.5 6 1.247313807623207 rpy=0 0 0
