Commit message: case3, JAR = .8, evolved, more data

File: bodyFiles/body0-10212.urdf (robot description, URDF)
Before this commit: robot robot, 9 links, 8 joints
Links:
- link BackLeg: geometry collision box size=0.2 0.7544787476647049 0.2; visual box size=0.2 0.7544787476647049 0.2
- link BackLowerLeg: geometry collision box size=0.2 0.2 0.6756106064547885; visual box size=0.2 0.2 0.6756106064547885
- link FrontLeg: geometry collision box size=0.2 1.3562958407078756 0.2; visual box size=0.2 1.3562958407078756 0.2
- link FrontLowerLeg: geometry collision box size=0.2 0.2 1.3011606160621363; visual box size=0.2 0.2 1.3011606160621363
- link LeftLeg: geometry collision box size=0.7521750422781276 0.2 0.2; visual box size=0.7521750422781276 0.2 0.2
- link LeftLowerLeg: geometry collision box size=0.2 0.2 0.5014188306432223; visual box size=0.2 0.2 0.5014188306432223
- link RightLeg: geometry collision box size=1.258094567307027 0.2 0.2; visual box size=1.258094567307027 0.2 0.2
- link RightLowerLeg: geometry collision box size=0.2 0.2 0.5570953112225774; visual box size=0.2 0.2 0.5570953112225774
Joints:
- joint BackLeg_BackLowerLeg: origin xyz=0 -1.137143254110991 0 rpy=0 0 0 -> xyz=0 -0.7544787476647049 0 rpy=0 0 0
- joint FrontLeg_FrontLowerLeg: origin xyz=0 0.9489818008380861 0 rpy=0 0 0 -> xyz=0 1.3562958407078756 0 rpy=0 0 0
- joint LeftLeg_LeftLowerLeg: origin xyz=-0.7154521235749964 0 0 rpy=0 0 0 -> xyz=-0.7521750422781276 0 0 rpy=0 0 0
- joint RightLeg_RightLowerLeg: origin xyz=1.0868599443532552 0 0 rpy=0 0 0 -> xyz=1.258094567307027 0 0 rpy=0 0 0
- joint Torso_BackLeg: origin xyz=0 -10.5 1.4092741650626892 rpy=0 0 0 -> xyz=0 -10.5 1.3562958407078756 rpy=0 0 0
- joint Torso_FrontLeg: origin xyz=0 -9.5 1.4092741650626892 rpy=0 0 0 -> xyz=0 -9.5 1.3562958407078756 rpy=0 0 0
- joint Torso_LeftLeg: origin xyz=-0.5 -10 1.4092741650626892 rpy=0 0 0 -> xyz=-0.5 -10 1.3562958407078756 rpy=0 0 0
- joint Torso_RightLeg: origin xyz=0.5 -10 1.4092741650626892 rpy=0 0 0 -> xyz=0.5 -10 1.3562958407078756 rpy=0 0 0

File: bodyFiles/body0-180.urdf (robot description, URDF)
Before this commit: robot robot, 9 links, 8 joints
Links:
- link BackLeg: geometry collision box size=0.2 1.1488897106105662 0.2; visual box size=0.2 1.1488897106105662 0.2
- link BackLowerLeg: geometry collision box size=0.2 0.2 1.2374827543333216; visual box size=0.2 0.2 1.2374827543333216
- link FrontLeg: geometry collision box size=0.2 1.1786962552150047 0.2; visual box size=0.2 1.1786962552150047 0.2
- link FrontLowerLeg: geometry collision box size=0.2 0.2 1.335118991622791; visual box size=0.2 0.2 1.335118991622791
- link LeftLeg: geometry collision box size=1.3393386769251365 0.2 0.2; visual box size=1.3393386769251365 0.2 0.2
- link LeftLowerLeg: geometry collision box size=0.2 0.2 0.8669059490354343; visual box size=0.2 0.2 0.8669059490354343
- link RightLeg: geometry collision box size=0.9705476475038005 0.2 0.2; visual box size=0.9705476475038005 0.2 0.2
- link RightLowerLeg: geometry collision box size=0.2 0.2 0.5722249210980562; visual box size=0.2 0.2 0.5722249210980562
Joints:
- joint BackLeg_BackLowerLeg: origin xyz=0 -1.12336051075338 0 rpy=0 0 0 -> xyz=0 -1.1488897106105662 0 rpy=0 0 0
- joint FrontLeg_FrontLowerLeg: origin xyz=0 0.9222473413778454 0 rpy=0 0 0 -> xyz=0 1.1786962552150047 0 rpy=0 0 0
- joint LeftLeg_LeftLowerLeg: origin xyz=-1.178826621860777 0 0 rpy=0 0 0 -> xyz=-1.3393386769251365 0 0 rpy=0 0 0
- joint RightLeg_RightLowerLeg: origin xyz=0.7396818960740315 0 0 rpy=0 0 0 -> xyz=0.9705476475038005 0 0 rpy=0 0 0
- joint Torso_BackLeg: origin xyz=0 -18.5 1.2588201230591216 rpy=0 0 0 -> xyz=0 -18.5 1.3393386769251365 rpy=0 0 0
- joint Torso_FrontLeg: origin xyz=0 -17.5 1.2588201230591216 rpy=0 0 0 -> xyz=0 -17.5 1.3393386769251365 rpy=0 0 0
- joint Torso_LeftLeg: origin xyz=-0.5 -18 1.2588201230591216 rpy=0 0 0 -> xyz=-0.5 -18 1.3393386769251365 rpy=0 0 0
- joint Torso_RightLeg: origin xyz=0.5 -18 1.2588201230591216 rpy=0 0 0 -> xyz=0.5 -18 1.3393386769251365 rpy=0 0 0

File: bodyFiles/body0-1850.urdf (robot description, URDF)
Before this commit: robot robot, 9 links, 8 joints
Links:
- link BackLeg: geometry collision box size=0.2 0.6896834747009369 0.2; visual box size=0.2 0.6896834747009369 0.2
- link BackLowerLeg: geometry collision box size=0.2 0.2 1.217387833024763; visual box size=0.2 0.2 1.217387833024763
- link FrontLeg: geometry collision box size=0.2 0.5104441251960813 0.2; visual box size=0.2 0.5104441251960813 0.2
- link FrontLowerLeg: geometry collision box size=0.2 0.2 0.7051324832849813; visual box size=0.2 0.2 0.7051324832849813
- link LeftLeg: geometry collision box size=1.4011582543928112 0.2 0.2; visual box size=1.4011582543928112 0.2 0.2
- link LeftLowerLeg: geometry collision box size=0.2 0.2 0.6430918268816207; visual box size=0.2 0.2 0.6430918268816207
- link RightLeg: geometry collision box size=0.7080861404950883 0.2 0.2; visual box size=0.7080861404950883 0.2 0.2
- link RightLowerLeg: geometry collision box size=0.2 0.2 0.8413538488834876; visual box size=0.2 0.2 0.8413538488834876
Joints:
- joint BackLeg_BackLowerLeg: origin xyz=0 -1.2443786580545348 0 rpy=0 0 0 -> xyz=0 -0.6896834747009369 0 rpy=0 0 0
- joint FrontLeg_FrontLowerLeg: origin xyz=0 0.971060486124717 0 rpy=0 0 0 -> xyz=0 0.5104441251960813 0 rpy=0 0 0
- joint LeftLeg_LeftLowerLeg: origin xyz=-0.6092493744343708 0 0 rpy=0 0 0 -> xyz=-1.4011582543928112 0 0 rpy=0 0 0
- joint RightLeg_RightLowerLeg: origin xyz=0.6579086292759486 0 0 rpy=0 0 0 -> xyz=0.7080861404950883 0 0 rpy=0 0 0
- joint Torso_BackLeg: origin xyz=0 -18.5 1.4903281960745018 rpy=0 0 0 -> xyz=0 -18.5 1.4011582543928112 rpy=0 0 0
- joint Torso_FrontLeg: origin xyz=0 -17.5 1.4903281960745018 rpy=0 0 0 -> xyz=0 -17.5 1.4011582543928112 rpy=0 0 0
- joint Torso_LeftLeg: origin xyz=-0.5 -18 1.4903281960745018 rpy=0 0 0 -> xyz=-0.5 -18 1.4011582543928112 rpy=0 0 0
- joint Torso_RightLeg: origin xyz=0.5 -18 1.4903281960745018 rpy=0 0 0 -> xyz=0.5 -18 1.4011582543928112 rpy=0 0 0

File: bodyFiles/body0-2174.urdf (robot description, URDF)
Before this commit: robot robot, 9 links, 8 joints
Links:
- link BackLeg: geometry collision box size=0.2 0.6223352434966839 0.2; visual box size=0.2 0.6223352434966839 0.2
- link BackLowerLeg: geometry collision box size=0.2 0.2 1.2646812161914898; visual box size=0.2 0.2 1.2646812161914898
- link FrontLeg: geometry collision box size=0.2 1.199640261608454 0.2; visual box size=0.2 1.199640261608454 0.2
- link FrontLowerLeg: geometry collision box size=0.2 0.2 0.8038717351722935; visual box size=0.2 0.2 0.8038717351722935
- link LeftLeg: geometry collision box size=1.1418207321112237 0.2 0.2; visual box size=1.1418207321112237 0.2 0.2
- link LeftLowerLeg: geometry collision box size=0.2 0.2 1.4509204395467896; visual box size=0.2 0.2 1.4509204395467896
- link RightLeg: geometry collision box size=0.7960530548399782 0.2 0.2; visual box size=0.7960530548399782 0.2 0.2
- link RightLowerLeg: geometry collision box size=0.2 0.2 0.9673781986622246; visual box size=0.2 0.2 0.9673781986622246
Joints:
- joint BackLeg_BackLowerLeg: origin xyz=0 -0.8774140728607371 0 rpy=0 0 0 -> xyz=0 -0.6223352434966839 0 rpy=0 0 0
- joint FrontLeg_FrontLowerLeg: origin xyz=0 1.1016843496392066 0 rpy=0 0 0 -> xyz=0 1.199640261608454 0 rpy=0 0 0
- joint LeftLeg_LeftLowerLeg: origin xyz=-0.7657705188001657 0 0 rpy=0 0 0 -> xyz=-1.1418207321112237 0 0 rpy=0 0 0
- joint RightLeg_RightLowerLeg: origin xyz=1.4075581093023117 0 0 rpy=0 0 0 -> xyz=0.7960530548399782 0 0 rpy=0 0 0
- joint Torso_BackLeg: origin xyz=0 -2.5 1.4735878742634916 rpy=0 0 0 -> xyz=0 -2.5 1.4509204395467896 rpy=0 0 0
- joint Torso_FrontLeg: origin xyz=0 -1.5 1.4735878742634916 rpy=0 0 0 -> xyz=0 -1.5 1.4509204395467896 rpy=0 0 0
- joint Torso_LeftLeg: origin xyz=-0.5 -2 1.4735878742634916 rpy=0 0 0 -> xyz=-0.5 -2 1.4509204395467896 rpy=0 0 0
- joint Torso_RightLeg: origin xyz=0.5 -2 1.4735878742634916 rpy=0 0 0 -> xyz=0.5 -2 1.4509204395467896 rpy=0 0 0

File: bodyFiles/body010187.urdf (robot description, URDF)
Before this commit: robot robot, 9 links, 8 joints
Links:
- link BackLeg: geometry collision box size=0.2 1.4573064928767707 0.2; visual box size=0.2 1.4573064928767707 0.2
- link BackLowerLeg: geometry collision box size=0.2 0.2 0.9995425273298455; visual box size=0.2 0.2 0.9995425273298455
- link FrontLeg: geometry collision box size=0.2 1.369519263579274 0.2; visual box size=0.2 1.369519263579274 0.2
- link FrontLowerLeg: geometry collision box size=0.2 0.2 1.4011066513539903; visual box size=0.2 0.2 1.4011066513539903
- link LeftLeg: geometry collision box size=1.210366574702932 0.2 0.2; visual box size=1.210366574702932 0.2 0.2
- link LeftLowerLeg: geometry collision box size=0.2 0.2 0.878388104759461; visual box size=0.2 0.2 0.878388104759461
- link RightLeg: geometry collision box size=1.4848370950226515 0.2 0.2; visual box size=1.4848370950226515 0.2 0.2
- link RightLowerLeg: geometry collision box size=0.2 0.2 1.1210631685631274; visual box size=0.2 0.2 1.1210631685631274
Joints:
- joint BackLeg_BackLowerLeg: origin xyz=0 -1.4619009624024075 0 rpy=0 0 0 -> xyz=0 -1.4573064928767707 0 rpy=0 0 0
- joint FrontLeg_FrontLowerLeg: origin xyz=0 0.6077053613842567 0 rpy=0 0 0 -> xyz=0 1.369519263579274 0 rpy=0 0 0
- joint LeftLeg_LeftLowerLeg: origin xyz=-1.2328704132815873 0 0 rpy=0 0 0 -> xyz=-1.210366574702932 0 0 rpy=0 0 0
- joint RightLeg_RightLowerLeg: origin xyz=0.7635452194708969 0 0 rpy=0 0 0 -> xyz=1.4848370950226515 0 0 rpy=0 0 0
- joint Torso_BackLeg: origin xyz=0 9.5 1.4619009624024075 rpy=0 0 0 -> xyz=0 9.5 1.4848370950226515 rpy=0 0 0
- joint Torso_FrontLeg: origin xyz=0 10.5 1.4619009624024075 rpy=0 0 0 -> xyz=0 10.5 1.4848370950226515 rpy=0 0 0
- joint Torso_LeftLeg: origin xyz=-0.5 10 1.4619009624024075 rpy=0 0 0 -> xyz=-0.5 10 1.4848370950226515 rpy=0 0 0
- joint Torso_RightLeg: origin xyz=0.5 10 1.4619009624024075 rpy=0 0 0 -> xyz=0.5 10 1.4848370950226515 rpy=0 0 0

File: bodyFiles/body010287.urdf (robot description, URDF)
Before this commit: robot robot, 9 links, 8 joints
Links:
- link BackLeg: geometry collision box size=0.2 1.3334186669401136 0.2; visual box size=0.2 1.3334186669401136 0.2
- link BackLowerLeg: geometry collision box size=0.2 0.2 0.777639221270847; visual box size=0.2 0.2 0.777639221270847
- link FrontLeg: geometry collision box size=0.2 1.2212484357610243 0.2; visual box size=0.2 1.2212484357610243 0.2
- link FrontLowerLeg: geometry collision box size=0.2 0.2 0.8336036873441685; visual box size=0.2 0.2 0.8336036873441685
- link LeftLeg: geometry collision box size=1.47058184696189 0.2 0.2; visual box size=1.47058184696189 0.2 0.2
- link LeftLowerLeg: geometry collision box size=0.2 0.2 1.2391336194879745; visual box size=0.2 0.2 1.2391336194879745
- link RightLeg: geometry collision box size=1.379597881952324 0.2 0.2; visual box size=1.379597881952324 0.2 0.2
- link RightLowerLeg: geometry collision box size=0.2 0.2 0.7619792781494967; visual box size=0.2 0.2 0.7619792781494967
Joints:
- joint BackLeg_BackLowerLeg: origin xyz=0 -1.2233938698807083 0 rpy=0 0 0 -> xyz=0 -1.3334186669401136 0 rpy=0 0 0
- joint FrontLeg_FrontLowerLeg: origin xyz=0 0.577946302488917 0 rpy=0 0 0 -> xyz=0 1.2212484357610243 0 rpy=0 0 0
- joint LeftLeg_LeftLowerLeg: origin xyz=-0.6867398141269501 0 0 rpy=0 0 0 -> xyz=-1.47058184696189 0 0 rpy=0 0 0
- joint RightLeg_RightLowerLeg: origin xyz=1.3980043405070368 0 0 rpy=0 0 0 -> xyz=1.379597881952324 0 0 rpy=0 0 0
- joint Torso_BackLeg: origin xyz=0 9.5 1.4842514253479475 rpy=0 0 0 -> xyz=0 9.5 1.47058184696189 rpy=0 0 0
- joint Torso_FrontLeg: origin xyz=0 10.5 1.4842514253479475 rpy=0 0 0 -> xyz=0 10.5 1.47058184696189 rpy=0 0 0
- joint Torso_LeftLeg: origin xyz=-0.5 10 1.4842514253479475 rpy=0 0 0 -> xyz=-0.5 10 1.47058184696189 rpy=0 0 0
- joint Torso_RightLeg: origin xyz=0.5 10 1.4842514253479475 rpy=0 0 0 -> xyz=0.5 10 1.47058184696189 rpy=0 0 0

File: bodyFiles/body01087.urdf (robot description, URDF)
Before this commit: robot robot, 9 links, 8 joints
Links:
- link BackLeg: geometry collision box size=0.2 0.6843612362222159 0.2; visual box size=0.2 0.6843612362222159 0.2
- link BackLowerLeg: geometry collision box size=0.2 0.2 0.930852471155635; visual box size=0.2 0.2 0.930852471155635
- link FrontLeg: geometry collision box size=0.2 1.267011817908306 0.2; visual box size=0.2 1.267011817908306 0.2
- link FrontLowerLeg: geometry collision box size=0.2 0.2 1.1843417154865574; visual box size=0.2 0.2 1.1843417154865574
- link LeftLeg: geometry collision box size=0.737704663567613 0.2 0.2; visual box size=0.737704663567613 0.2 0.2
- link LeftLowerLeg: geometry collision box size=0.2 0.2 0.7119999789694573; visual box size=0.2 0.2 0.7119999789694573
- link RightLeg: geometry collision box size=0.9793268894507605 0.2 0.2; visual box size=0.9793268894507605 0.2 0.2
- link RightLowerLeg: geometry collision box size=0.2 0.2 0.6828914139824583; visual box size=0.2 0.2 0.6828914139824583
Joints:
- joint BackLeg_BackLowerLeg: origin xyz=0 -0.6143177802444265 0 rpy=0 0 0 -> xyz=0 -0.6843612362222159 0 rpy=0 0 0
- joint FrontLeg_FrontLowerLeg: origin xyz=0 1.152112154718576 0 rpy=0 0 0 -> xyz=0 1.267011817908306 0 rpy=0 0 0
- joint LeftLeg_LeftLowerLeg: origin xyz=-1.2954792893608984 0 0 rpy=0 0 0 -> xyz=-0.737704663567613 0 0 rpy=0 0 0
- joint RightLeg_RightLowerLeg: origin xyz=0.9849395712801298 0 0 rpy=0 0 0 -> xyz=0.9793268894507605 0 0 rpy=0 0 0
- joint Torso_BackLeg: origin xyz=0 9.5 1.444953310798789 rpy=0 0 0 -> xyz=0 9.5 1.267011817908306 rpy=0 0 0
- joint Torso_FrontLeg: origin xyz=0 10.5 1.444953310798789 rpy=0 0 0 -> xyz=0 10.5 1.267011817908306 rpy=0 0 0
- joint Torso_LeftLeg: origin xyz=-0.5 10 1.444953310798789 rpy=0 0 0 -> xyz=-0.5 10 1.267011817908306 rpy=0 0 0
- joint Torso_RightLeg: origin xyz=0.5 10 1.444953310798789 rpy=0 0 0 -> xyz=0.5 10 1.267011817908306 rpy=0 0 0

File: bodyFiles/body018249.urdf (robot description, URDF)
Before this commit: robot robot, 9 links, 8 joints
Links:
- link BackLeg: geometry collision box size=0.2 0.9367195390882855 0.2; visual box size=0.2 0.9367195390882855 0.2
- link BackLowerLeg: geometry collision box size=0.2 0.2 1.3596980125311244; visual box size=0.2 0.2 1.3596980125311244
- link FrontLeg: geometry collision box size=0.2 0.6365048857184182 0.2; visual box size=0.2 0.6365048857184182 0.2
- link FrontLowerLeg: geometry collision box size=0.2 0.2 0.5682866970459372; visual box size=0.2 0.2 0.5682866970459372
- link LeftLeg: geometry collision box size=1.1917425688314363 0.2 0.2; visual box size=1.1917425688314363 0.2 0.2
- link LeftLowerLeg: geometry collision box size=0.2 0.2 0.8302960264929707; visual box size=0.2 0.2 0.8302960264929707
- link RightLeg: geometry collision box size=0.8772221024504454 0.2 0.2; visual box size=0.8772221024504454 0.2 0.2
- link RightLowerLeg: geometry collision box size=0.2 0.2 1.195706495827296; visual box size=0.2 0.2 1.195706495827296
Joints:
- joint BackLeg_BackLowerLeg: origin xyz=0 -0.7359762625562544 0 rpy=0 0 0 -> xyz=0 -0.9367195390882855 0 rpy=0 0 0
- joint FrontLeg_FrontLowerLeg: origin xyz=0 1.3767759626551916 0 rpy=0 0 0 -> xyz=0 0.6365048857184182 0 rpy=0 0 0
- joint LeftLeg_LeftLowerLeg: origin xyz=-0.9488718869520614 0 0 rpy=0 0 0 -> xyz=-1.1917425688314363 0 0 rpy=0 0 0
- joint RightLeg_RightLowerLeg: origin xyz=1.2294096775893029 0 0 rpy=0 0 0 -> xyz=0.8772221024504454 0 0 rpy=0 0 0
- joint Torso_BackLeg: origin xyz=0 17.5 1.399658204847165 rpy=0 0 0 -> xyz=0 17.5 1.3596980125311244 rpy=0 0 0
- joint Torso_FrontLeg: origin xyz=0 18.5 1.399658204847165 rpy=0 0 0 -> xyz=0 18.5 1.3596980125311244 rpy=0 0 0
- joint Torso_LeftLeg: origin xyz=-0.5 18 1.399658204847165 rpy=0 0 0 -> xyz=-0.5 18 1.3596980125311244 rpy=0 0 0
- joint Torso_RightLeg: origin xyz=0.5 18 1.399658204847165 rpy=0 0 0 -> xyz=0.5 18 1.3596980125311244 rpy=0 0 0

File: bodyFiles/body01849.urdf (robot description, URDF)
Before this commit: robot robot, 9 links, 8 joints
Links:
- link BackLeg: geometry collision box size=0.2 0.816766601371767 0.2; visual box size=0.2 0.816766601371767 0.2
- link BackLowerLeg: geometry collision box size=0.2 0.2 0.6344847925345556; visual box size=0.2 0.2 0.6344847925345556
- link FrontLeg: geometry collision box size=0.2 0.8377179663629899 0.2; visual box size=0.2 0.8377179663629899 0.2
- link FrontLowerLeg: geometry collision box size=0.2 0.2 0.532998462479001; visual box size=0.2 0.2 0.532998462479001
- link LeftLeg: geometry collision box size=1.3787938270767917 0.2 0.2; visual box size=1.3787938270767917 0.2 0.2
- link LeftLowerLeg: geometry collision box size=0.2 0.2 0.853475718570897; visual box size=0.2 0.2 0.853475718570897
- link RightLeg: geometry collision box size=0.865713201405669 0.2 0.2; visual box size=0.865713201405669 0.2 0.2
- link RightLowerLeg: geometry collision box size=0.2 0.2 0.5391011096011749; visual box size=0.2 0.2 0.5391011096011749
Joints:
- joint BackLeg_BackLowerLeg: origin xyz=0 -1.3249581601210654 0 rpy=0 0 0 -> xyz=0 -0.816766601371767 0 rpy=0 0 0
- joint FrontLeg_FrontLowerLeg: origin xyz=0 0.9214726438345228 0 rpy=0 0 0 -> xyz=0 0.8377179663629899 0 rpy=0 0 0
- joint LeftLeg_LeftLowerLeg: origin xyz=-0.9789881096792347 0 0 rpy=0 0 0 -> xyz=-1.3787938270767917 0 0 rpy=0 0 0
- joint RightLeg_RightLowerLeg: origin xyz=0.6227347832677597 0 0 rpy=0 0 0 -> xyz=0.865713201405669 0 0 rpy=0 0 0
- joint Torso_BackLeg: origin xyz=0 17.5 1.3249581601210654 rpy=0 0 0 -> xyz=0 17.5 1.3787938270767917 rpy=0 0 0
- joint Torso_FrontLeg: origin xyz=0 18.5 1.3249581601210654 rpy=0 0 0 -> xyz=0 18.5 1.3787938270767917 rpy=0 0 0
- joint Torso_LeftLeg: origin xyz=-0.5 18 1.3249581601210654 rpy=0 0 0 -> xyz=-0.5 18 1.3787938270767917 rpy=0 0 0
- joint Torso_RightLeg: origin xyz=0.5 18 1.3249581601210654 rpy=0 0 0 -> xyz=0.5 18 1.3787938270767917 rpy=0 0 0

File: bodyFiles/body01899.urdf (robot description, URDF)
Before this commit: robot robot, 9 links, 8 joints
Links:
- link BackLeg: geometry collision box size=0.2 0.8058485628620069 0.2; visual box size=0.2 0.8058485628620069 0.2
- link BackLowerLeg: geometry collision box size=0.2 0.2 0.9795738432070624; visual box size=0.2 0.2 0.9795738432070624
- link FrontLeg: geometry collision box size=0.2 1.4947076369067493 0.2; visual box size=0.2 1.4947076369067493 0.2
- link FrontLowerLeg: geometry collision box size=0.2 0.2 0.8033890715380407; visual box size=0.2 0.2 0.8033890715380407
- link LeftLeg: geometry collision box size=1.4468010698219005 0.2 0.2; visual box size=1.4468010698219005 0.2 0.2
- link LeftLowerLeg: geometry collision box size=0.2 0.2 0.8755315276418723; visual box size=0.2 0.2 0.8755315276418723
- link RightLeg: geometry collision box size=0.7955253963613762 0.2 0.2; visual box size=0.7955253963613762 0.2 0.2
- link RightLowerLeg: geometry collision box size=0.2 0.2 1.395738900144637; visual box size=0.2 0.2 1.395738900144637
Joints:
- joint BackLeg_BackLowerLeg: origin xyz=0 -1.1428747462871542 0 rpy=0 0 0 -> xyz=0 -0.8058485628620069 0 rpy=0 0 0
- joint FrontLeg_FrontLowerLeg: origin xyz=0 0.7835471753316936 0 rpy=0 0 0 -> xyz=0 1.4947076369067493 0 rpy=0 0 0
- joint LeftLeg_LeftLowerLeg: origin xyz=-1.278021077855593 0 0 rpy=0 0 0 -> xyz=-1.4468010698219005 0 0 rpy=0 0 0
- joint RightLeg_RightLowerLeg: origin xyz=1.1364776828249128 0 0 rpy=0 0 0 -> xyz=0.7955253963613762 0 0 rpy=0 0 0
- joint Torso_BackLeg: origin xyz=0 17.5 1.278021077855593 rpy=0 0 0 -> xyz=0 17.5 1.4947076369067493 rpy=0 0 0
- joint Torso_FrontLeg: origin xyz=0 18.5 1.278021077855593 rpy=0 0 0 -> xyz=0 18.5 1.4947076369067493 rpy=0 0 0
- joint Torso_LeftLeg: origin xyz=-0.5 18 1.278021077855593 rpy=0 0 0 -> xyz=-0.5 18 1.4947076369067493 rpy=0 0 0
- joint Torso_RightLeg: origin xyz=0.5 18 1.278021077855593 rpy=0 0 0 -> xyz=0.5 18 1.4947076369067493 rpy=0 0 0

File: bodyFiles/body02175.urdf (robot description, URDF)
Before this commit: robot robot, 9 links, 8 joints
Links:
- link BackLeg: geometry collision box size=0.2 0.6568327086104983 0.2; visual box size=0.2 0.6568327086104983 0.2
- link BackLowerLeg: geometry collision box size=0.2 0.2 0.925955014003568; visual box size=0.2 0.2 0.925955014003568
- link FrontLeg: geometry collision box size=0.2 1.3331710999823192 0.2; visual box size=0.2 1.3331710999823192 0.2
- link FrontLowerLeg: geometry collision box size=0.2 0.2 1.3025127263606247; visual box size=0.2 0.2 1.3025127263606247
- link LeftLeg: geometry collision box size=1.3909423461044175 0.2 0.2; visual box size=1.3909423461044175 0.2 0.2
- link LeftLowerLeg: geometry collision box size=0.2 0.2 1.3032824041057953; visual box size=0.2 0.2 1.3032824041057953
- link RightLeg: geometry collision box size=0.8214751669205668 0.2 0.2; visual box size=0.8214751669205668 0.2 0.2
- link RightLowerLeg: geometry collision box size=0.2 0.2 0.5083445812924121; visual box size=0.2 0.2 0.5083445812924121
Joints:
- joint BackLeg_BackLowerLeg: origin xyz=0 -0.8512009650169191 0 rpy=0 0 0 -> xyz=0 -0.6568327086104983 0 rpy=0 0 0
- joint FrontLeg_FrontLowerLeg: origin xyz=0 0.5352503073565875 0 rpy=0 0 0 -> xyz=0 1.3331710999823192 0 rpy=0 0 0
- joint LeftLeg_LeftLowerLeg: origin xyz=-1.014113294083622 0 0 rpy=0 0 0 -> xyz=-1.3909423461044175 0 0 rpy=0 0 0
- joint RightLeg_RightLowerLeg: origin xyz=0.7630465113271522 0 0 rpy=0 0 0 -> xyz=0.8214751669205668 0 0 rpy=0 0 0
- joint Torso_BackLeg: origin xyz=0 1.5 1.2854280852111803 rpy=0 0 0 -> xyz=0 1.5 1.3909423461044175 rpy=0 0 0
- joint Torso_FrontLeg: origin xyz=0 2.5 1.2854280852111803 rpy=0 0 0 -> xyz=0 2.5 1.3909423461044175 rpy=0 0 0
- joint Torso_LeftLeg: origin xyz=-0.5 2 1.2854280852111803 rpy=0 0 0 -> xyz=-0.5 2 1.3909423461044175 rpy=0 0 0
- joint Torso_RightLeg: origin xyz=0.5 2 1.2854280852111803 rpy=0 0 0 -> xyz=0.5 2 1.3909423461044175 rpy=0 0 0
