Commit message: case3, JAR = .8, evolved, more data

File: bodyFiles/body02325.urdf (robot description, URDF)
Before this commit: robot robot, 9 links, 8 joints
Links:
- link BackLeg: geometry collision box size=0.2 1.475382895464319 0.2; visual box size=0.2 1.475382895464319 0.2
- link BackLowerLeg: geometry collision box size=0.2 0.2 0.6114715952935771; visual box size=0.2 0.2 0.6114715952935771
- link FrontLeg: geometry collision box size=0.2 1.1154859518981348 0.2; visual box size=0.2 1.1154859518981348 0.2
- link FrontLowerLeg: geometry collision box size=0.2 0.2 1.1570878917056242; visual box size=0.2 0.2 1.1570878917056242
- link LeftLeg: geometry collision box size=1.4206066440950833 0.2 0.2; visual box size=1.4206066440950833 0.2 0.2
- link LeftLowerLeg: geometry collision box size=0.2 0.2 0.8054287044305215; visual box size=0.2 0.2 0.8054287044305215
- link RightLeg: geometry collision box size=0.9801766315708486 0.2 0.2; visual box size=0.9801766315708486 0.2 0.2
- link RightLowerLeg: geometry collision box size=0.2 0.2 0.5257524270492625; visual box size=0.2 0.2 0.5257524270492625
Joints:
- joint BackLeg_BackLowerLeg: origin xyz=0 -0.6259617037937549 0 rpy=0 0 0 -> xyz=0 -1.475382895464319 0 rpy=0 0 0
- joint FrontLeg_FrontLowerLeg: origin xyz=0 0.6773832353174731 0 rpy=0 0 0 -> xyz=0 1.1154859518981348 0 rpy=0 0 0
- joint LeftLeg_LeftLowerLeg: origin xyz=-1.0823507909345764 0 0 rpy=0 0 0 -> xyz=-1.4206066440950833 0 0 rpy=0 0 0
- joint RightLeg_RightLowerLeg: origin xyz=1.1697915776232968 0 0 rpy=0 0 0 -> xyz=0.9801766315708486 0 0 rpy=0 0 0
- joint Torso_BackLeg: origin xyz=0 1.5 1.2258518355472399 rpy=0 0 0 -> xyz=0 1.5 1.475382895464319 rpy=0 0 0
- joint Torso_FrontLeg: origin xyz=0 2.5 1.2258518355472399 rpy=0 0 0 -> xyz=0 2.5 1.475382895464319 rpy=0 0 0
- joint Torso_LeftLeg: origin xyz=-0.5 2 1.2258518355472399 rpy=0 0 0 -> xyz=-0.5 2 1.475382895464319 rpy=0 0 0
- joint Torso_RightLeg: origin xyz=0.5 2 1.2258518355472399 rpy=0 0 0 -> xyz=0.5 2 1.475382895464319 rpy=0 0 0
