Commit message: case3, JAR = .8, random, more data

File: bodyFiles/body0-10212.urdf (robot description, URDF)
Before this commit: robot robot, 9 links, 8 joints
Links:
- link BackLeg: geometry collision box size=0.2 0.5108450504362002 0.2; visual box size=0.2 0.5108450504362002 0.2
- link BackLowerLeg: geometry collision box size=0.2 0.2 1.1221777292940882; visual box size=0.2 0.2 1.1221777292940882
- link FrontLeg: geometry collision box size=0.2 1.142206789830654 0.2; visual box size=0.2 1.142206789830654 0.2
- link FrontLowerLeg: geometry collision box size=0.2 0.2 1.2331101142105196; visual box size=0.2 0.2 1.2331101142105196
- link LeftLeg: geometry collision box size=1.0539563091985287 0.2 0.2; visual box size=1.0539563091985287 0.2 0.2
- link LeftLowerLeg: geometry collision box size=0.2 0.2 0.6196800659816518; visual box size=0.2 0.2 0.6196800659816518
- link RightLeg: geometry collision box size=1.3680482613703422 0.2 0.2; visual box size=1.3680482613703422 0.2 0.2
- link RightLowerLeg: geometry collision box size=0.2 0.2 1.4878832536339153; visual box size=0.2 0.2 1.4878832536339153
Joints:
- joint BackLeg_BackLowerLeg: origin xyz=0 -0.7544787476647049 0 rpy=0 0 0 -> xyz=0 -0.5108450504362002 0 rpy=0 0 0
- joint FrontLeg_FrontLowerLeg: origin xyz=0 1.3562958407078756 0 rpy=0 0 0 -> xyz=0 1.142206789830654 0 rpy=0 0 0
- joint LeftLeg_LeftLowerLeg: origin xyz=-0.7521750422781276 0 0 rpy=0 0 0 -> xyz=-1.0539563091985287 0 0 rpy=0 0 0
- joint RightLeg_RightLowerLeg: origin xyz=1.258094567307027 0 0 rpy=0 0 0 -> xyz=1.3680482613703422 0 0 rpy=0 0 0
- joint Torso_BackLeg: origin xyz=0 -10.5 1.3562958407078756 rpy=0 0 0 -> xyz=0 -10.5 1.4878832536339153 rpy=0 0 0
- joint Torso_FrontLeg: origin xyz=0 -9.5 1.3562958407078756 rpy=0 0 0 -> xyz=0 -9.5 1.4878832536339153 rpy=0 0 0
- joint Torso_LeftLeg: origin xyz=-0.5 -10 1.3562958407078756 rpy=0 0 0 -> xyz=-0.5 -10 1.4878832536339153 rpy=0 0 0
- joint Torso_RightLeg: origin xyz=0.5 -10 1.3562958407078756 rpy=0 0 0 -> xyz=0.5 -10 1.4878832536339153 rpy=0 0 0

File: bodyFiles/body0-180.urdf (robot description, URDF)
Before this commit: robot robot, 9 links, 8 joints
Links:
- link BackLeg: geometry collision box size=0.2 1.0797249265584217 0.2; visual box size=0.2 1.0797249265584217 0.2
- link BackLowerLeg: geometry collision box size=0.2 0.2 0.9339877807713444; visual box size=0.2 0.2 0.9339877807713444
- link FrontLeg: geometry collision box size=0.2 1.399540858985737 0.2; visual box size=0.2 1.399540858985737 0.2
- link FrontLowerLeg: geometry collision box size=0.2 0.2 1.3846754345228303; visual box size=0.2 0.2 1.3846754345228303
- link LeftLeg: geometry collision box size=0.7398519106940091 0.2 0.2; visual box size=0.7398519106940091 0.2 0.2
- link LeftLowerLeg: geometry collision box size=0.2 0.2 1.4431833469706774; visual box size=0.2 0.2 1.4431833469706774
- link RightLeg: geometry collision box size=1.4785947681576306 0.2 0.2; visual box size=1.4785947681576306 0.2 0.2
- link RightLowerLeg: geometry collision box size=0.2 0.2 0.9449719084757444; visual box size=0.2 0.2 0.9449719084757444
Joints:
- joint BackLeg_BackLowerLeg: origin xyz=0 -1.1488897106105662 0 rpy=0 0 0 -> xyz=0 -1.0797249265584217 0 rpy=0 0 0
- joint FrontLeg_FrontLowerLeg: origin xyz=0 1.1786962552150047 0 rpy=0 0 0 -> xyz=0 1.399540858985737 0 rpy=0 0 0
- joint LeftLeg_LeftLowerLeg: origin xyz=-1.3393386769251365 0 0 rpy=0 0 0 -> xyz=-0.7398519106940091 0 0 rpy=0 0 0
- joint RightLeg_RightLowerLeg: origin xyz=0.9705476475038005 0 0 rpy=0 0 0 -> xyz=1.4785947681576306 0 0 rpy=0 0 0
- joint Torso_BackLeg: origin xyz=0 -18.5 1.3393386769251365 rpy=0 0 0 -> xyz=0 -18.5 1.4785947681576306 rpy=0 0 0
- joint Torso_FrontLeg: origin xyz=0 -17.5 1.3393386769251365 rpy=0 0 0 -> xyz=0 -17.5 1.4785947681576306 rpy=0 0 0
- joint Torso_LeftLeg: origin xyz=-0.5 -18 1.3393386769251365 rpy=0 0 0 -> xyz=-0.5 -18 1.4785947681576306 rpy=0 0 0
- joint Torso_RightLeg: origin xyz=0.5 -18 1.3393386769251365 rpy=0 0 0 -> xyz=0.5 -18 1.4785947681576306 rpy=0 0 0

File: bodyFiles/body0-1850.urdf (robot description, URDF)
Before this commit: robot robot, 9 links, 8 joints
Links:
- link BackLeg: geometry collision box size=0.2 1.4462693959607282 0.2; visual box size=0.2 1.4462693959607282 0.2
- link BackLowerLeg: geometry collision box size=0.2 0.2 0.8429011462896646; visual box size=0.2 0.2 0.8429011462896646
- link FrontLeg: geometry collision box size=0.2 0.6583965969023619 0.2; visual box size=0.2 0.6583965969023619 0.2
- link FrontLowerLeg: geometry collision box size=0.2 0.2 0.9714019851917849; visual box size=0.2 0.2 0.9714019851917849
- link LeftLeg: geometry collision box size=1.0098103406462045 0.2 0.2; visual box size=1.0098103406462045 0.2 0.2
- link LeftLowerLeg: geometry collision box size=0.2 0.2 1.153889983420095; visual box size=0.2 0.2 1.153889983420095
- link RightLeg: geometry collision box size=1.4265235465428328 0.2 0.2; visual box size=1.4265235465428328 0.2 0.2
- link RightLowerLeg: geometry collision box size=0.2 0.2 0.723778039035265; visual box size=0.2 0.2 0.723778039035265
Joints:
- joint BackLeg_BackLowerLeg: origin xyz=0 -0.6896834747009369 0 rpy=0 0 0 -> xyz=0 -1.4462693959607282 0 rpy=0 0 0
- joint FrontLeg_FrontLowerLeg: origin xyz=0 0.5104441251960813 0 rpy=0 0 0 -> xyz=0 0.6583965969023619 0 rpy=0 0 0
- joint LeftLeg_LeftLowerLeg: origin xyz=-1.4011582543928112 0 0 rpy=0 0 0 -> xyz=-1.0098103406462045 0 0 rpy=0 0 0
- joint RightLeg_RightLowerLeg: origin xyz=0.7080861404950883 0 0 rpy=0 0 0 -> xyz=1.4265235465428328 0 0 rpy=0 0 0
- joint Torso_BackLeg: origin xyz=0 -18.5 1.4011582543928112 rpy=0 0 0 -> xyz=0 -18.5 1.4462693959607282 rpy=0 0 0
- joint Torso_FrontLeg: origin xyz=0 -17.5 1.4011582543928112 rpy=0 0 0 -> xyz=0 -17.5 1.4462693959607282 rpy=0 0 0
- joint Torso_LeftLeg: origin xyz=-0.5 -18 1.4011582543928112 rpy=0 0 0 -> xyz=-0.5 -18 1.4462693959607282 rpy=0 0 0
- joint Torso_RightLeg: origin xyz=0.5 -18 1.4011582543928112 rpy=0 0 0 -> xyz=0.5 -18 1.4462693959607282 rpy=0 0 0

File: bodyFiles/body0-2174.urdf (robot description, URDF)
Before this commit: robot robot, 9 links, 8 joints
Links:
- link BackLeg: geometry collision box size=0.2 1.4835862051664548 0.2; visual box size=0.2 1.4835862051664548 0.2
- link BackLowerLeg: geometry collision box size=0.2 0.2 1.3827197078389015; visual box size=0.2 0.2 1.3827197078389015
- link FrontLeg: geometry collision box size=0.2 0.7005825931715677 0.2; visual box size=0.2 0.7005825931715677 0.2
- link FrontLowerLeg: geometry collision box size=0.2 0.2 0.9706375726563207; visual box size=0.2 0.2 0.9706375726563207
- link LeftLeg: geometry collision box size=1.1190005497938258 0.2 0.2; visual box size=1.1190005497938258 0.2 0.2
- link LeftLowerLeg: geometry collision box size=0.2 0.2 0.8628128227429275; visual box size=0.2 0.2 0.8628128227429275
- link RightLeg: geometry collision box size=1.4206805891975054 0.2 0.2; visual box size=1.4206805891975054 0.2 0.2
- link RightLowerLeg: geometry collision box size=0.2 0.2 1.4041614009037406; visual box size=0.2 0.2 1.4041614009037406
Joints:
- joint BackLeg_BackLowerLeg: origin xyz=0 -0.6223352434966839 0 rpy=0 0 0 -> xyz=0 -1.4835862051664548 0 rpy=0 0 0
- joint FrontLeg_FrontLowerLeg: origin xyz=0 1.199640261608454 0 rpy=0 0 0 -> xyz=0 0.7005825931715677 0 rpy=0 0 0
- joint LeftLeg_LeftLowerLeg: origin xyz=-1.1418207321112237 0 0 rpy=0 0 0 -> xyz=-1.1190005497938258 0 0 rpy=0 0 0
- joint RightLeg_RightLowerLeg: origin xyz=0.7960530548399782 0 0 rpy=0 0 0 -> xyz=1.4206805891975054 0 0 rpy=0 0 0
- joint Torso_BackLeg: origin xyz=0 -2.5 1.4509204395467896 rpy=0 0 0 -> xyz=0 -2.5 1.4835862051664548 rpy=0 0 0
- joint Torso_FrontLeg: origin xyz=0 -1.5 1.4509204395467896 rpy=0 0 0 -> xyz=0 -1.5 1.4835862051664548 rpy=0 0 0
- joint Torso_LeftLeg: origin xyz=-0.5 -2 1.4509204395467896 rpy=0 0 0 -> xyz=-0.5 -2 1.4835862051664548 rpy=0 0 0
- joint Torso_RightLeg: origin xyz=0.5 -2 1.4509204395467896 rpy=0 0 0 -> xyz=0.5 -2 1.4835862051664548 rpy=0 0 0

File: bodyFiles/body010187.urdf (robot description, URDF)
Before this commit: robot robot, 9 links, 8 joints
Links:
- link BackLeg: geometry collision box size=0.2 1.1001499331759268 0.2; visual box size=0.2 1.1001499331759268 0.2
- link BackLowerLeg: geometry collision box size=0.2 0.2 1.0896364390768558; visual box size=0.2 0.2 1.0896364390768558
- link FrontLeg: geometry collision box size=0.2 0.5868569097451182 0.2; visual box size=0.2 0.5868569097451182 0.2
- link FrontLowerLeg: geometry collision box size=0.2 0.2 0.6178183382483949; visual box size=0.2 0.2 0.6178183382483949
- link LeftLeg: geometry collision box size=0.8406268136617657 0.2 0.2; visual box size=0.8406268136617657 0.2 0.2
- link LeftLowerLeg: geometry collision box size=0.2 0.2 1.1614732893589044; visual box size=0.2 0.2 1.1614732893589044
- link RightLeg: geometry collision box size=0.5942498241054437 0.2 0.2; visual box size=0.5942498241054437 0.2 0.2
- link RightLowerLeg: geometry collision box size=0.2 0.2 1.2929640722852382; visual box size=0.2 0.2 1.2929640722852382
Joints:
- joint BackLeg_BackLowerLeg: origin xyz=0 -1.4573064928767707 0 rpy=0 0 0 -> xyz=0 -1.1001499331759268 0 rpy=0 0 0
- joint FrontLeg_FrontLowerLeg: origin xyz=0 1.369519263579274 0 rpy=0 0 0 -> xyz=0 0.5868569097451182 0 rpy=0 0 0
- joint LeftLeg_LeftLowerLeg: origin xyz=-1.210366574702932 0 0 rpy=0 0 0 -> xyz=-0.8406268136617657 0 0 rpy=0 0 0
- joint RightLeg_RightLowerLeg: origin xyz=1.4848370950226515 0 0 rpy=0 0 0 -> xyz=0.5942498241054437 0 0 rpy=0 0 0
- joint Torso_BackLeg: origin xyz=0 9.5 1.4848370950226515 rpy=0 0 0 -> xyz=0 9.5 1.2929640722852382 rpy=0 0 0
- joint Torso_FrontLeg: origin xyz=0 10.5 1.4848370950226515 rpy=0 0 0 -> xyz=0 10.5 1.2929640722852382 rpy=0 0 0
- joint Torso_LeftLeg: origin xyz=-0.5 10 1.4848370950226515 rpy=0 0 0 -> xyz=-0.5 10 1.2929640722852382 rpy=0 0 0
- joint Torso_RightLeg: origin xyz=0.5 10 1.4848370950226515 rpy=0 0 0 -> xyz=0.5 10 1.2929640722852382 rpy=0 0 0

File: bodyFiles/body010287.urdf (robot description, URDF)
Before this commit: robot robot, 9 links, 8 joints
Links:
- link BackLeg: geometry collision box size=0.2 0.6904745025475427 0.2; visual box size=0.2 0.6904745025475427 0.2
- link BackLowerLeg: geometry collision box size=0.2 0.2 0.8478220481754637; visual box size=0.2 0.2 0.8478220481754637
- link FrontLeg: geometry collision box size=0.2 0.7507884875462169 0.2; visual box size=0.2 0.7507884875462169 0.2
- link FrontLowerLeg: geometry collision box size=0.2 0.2 0.8600707446729294; visual box size=0.2 0.2 0.8600707446729294
- link LeftLeg: geometry collision box size=0.6369245541752884 0.2 0.2; visual box size=0.6369245541752884 0.2 0.2
- link LeftLowerLeg: geometry collision box size=0.2 0.2 0.516639732543073; visual box size=0.2 0.2 0.516639732543073
- link RightLeg: geometry collision box size=0.5961682125839739 0.2 0.2; visual box size=0.5961682125839739 0.2 0.2
- link RightLowerLeg: geometry collision box size=0.2 0.2 1.2115705778415056; visual box size=0.2 0.2 1.2115705778415056
Joints:
- joint BackLeg_BackLowerLeg: origin xyz=0 -1.3334186669401136 0 rpy=0 0 0 -> xyz=0 -0.6904745025475427 0 rpy=0 0 0
- joint FrontLeg_FrontLowerLeg: origin xyz=0 1.2212484357610243 0 rpy=0 0 0 -> xyz=0 0.7507884875462169 0 rpy=0 0 0
- joint LeftLeg_LeftLowerLeg: origin xyz=-1.47058184696189 0 0 rpy=0 0 0 -> xyz=-0.6369245541752884 0 0 rpy=0 0 0
- joint RightLeg_RightLowerLeg: origin xyz=1.379597881952324 0 0 rpy=0 0 0 -> xyz=0.5961682125839739 0 0 rpy=0 0 0
- joint Torso_BackLeg: origin xyz=0 9.5 1.47058184696189 rpy=0 0 0 -> xyz=0 9.5 1.2115705778415056 rpy=0 0 0
- joint Torso_FrontLeg: origin xyz=0 10.5 1.47058184696189 rpy=0 0 0 -> xyz=0 10.5 1.2115705778415056 rpy=0 0 0
- joint Torso_LeftLeg: origin xyz=-0.5 10 1.47058184696189 rpy=0 0 0 -> xyz=-0.5 10 1.2115705778415056 rpy=0 0 0
- joint Torso_RightLeg: origin xyz=0.5 10 1.47058184696189 rpy=0 0 0 -> xyz=0.5 10 1.2115705778415056 rpy=0 0 0

File: bodyFiles/body01087.urdf (robot description, URDF)
Before this commit: robot robot, 9 links, 8 joints
Links:
- link BackLeg: geometry collision box size=0.2 0.8885747694958508 0.2; visual box size=0.2 0.8885747694958508 0.2
- link BackLowerLeg: geometry collision box size=0.2 0.2 1.2325628726405151; visual box size=0.2 0.2 1.2325628726405151
- link FrontLeg: geometry collision box size=0.2 1.3611843975971947 0.2; visual box size=0.2 1.3611843975971947 0.2
- link FrontLowerLeg: geometry collision box size=0.2 0.2 0.9620462645930186; visual box size=0.2 0.2 0.9620462645930186
- link LeftLeg: geometry collision box size=1.1834327660740498 0.2 0.2; visual box size=1.1834327660740498 0.2 0.2
- link LeftLowerLeg: geometry collision box size=0.2 0.2 1.2372294855293013; visual box size=0.2 0.2 1.2372294855293013
- link RightLeg: geometry collision box size=0.8116227914684938 0.2 0.2; visual box size=0.8116227914684938 0.2 0.2
- link RightLowerLeg: geometry collision box size=0.2 0.2 0.7506142742756001; visual box size=0.2 0.2 0.7506142742756001
Joints:
- joint BackLeg_BackLowerLeg: origin xyz=0 -0.6843612362222159 0 rpy=0 0 0 -> xyz=0 -0.8885747694958508 0 rpy=0 0 0
- joint FrontLeg_FrontLowerLeg: origin xyz=0 1.267011817908306 0 rpy=0 0 0 -> xyz=0 1.3611843975971947 0 rpy=0 0 0
- joint LeftLeg_LeftLowerLeg: origin xyz=-0.737704663567613 0 0 rpy=0 0 0 -> xyz=-1.1834327660740498 0 0 rpy=0 0 0
- joint RightLeg_RightLowerLeg: origin xyz=0.9793268894507605 0 0 rpy=0 0 0 -> xyz=0.8116227914684938 0 0 rpy=0 0 0
- joint Torso_BackLeg: origin xyz=0 9.5 1.267011817908306 rpy=0 0 0 -> xyz=0 9.5 1.3611843975971947 rpy=0 0 0
- joint Torso_FrontLeg: origin xyz=0 10.5 1.267011817908306 rpy=0 0 0 -> xyz=0 10.5 1.3611843975971947 rpy=0 0 0
- joint Torso_LeftLeg: origin xyz=-0.5 10 1.267011817908306 rpy=0 0 0 -> xyz=-0.5 10 1.3611843975971947 rpy=0 0 0
- joint Torso_RightLeg: origin xyz=0.5 10 1.267011817908306 rpy=0 0 0 -> xyz=0.5 10 1.3611843975971947 rpy=0 0 0

File: bodyFiles/body018249.urdf (robot description, URDF)
Before this commit: robot robot, 9 links, 8 joints
Links:
- link BackLeg: geometry collision box size=0.2 1.0398002398990647 0.2; visual box size=0.2 1.0398002398990647 0.2
- link BackLowerLeg: geometry collision box size=0.2 0.2 0.7991390605318989; visual box size=0.2 0.2 0.7991390605318989
- link FrontLeg: geometry collision box size=0.2 0.8540150976073921 0.2; visual box size=0.2 0.8540150976073921 0.2
- link FrontLowerLeg: geometry collision box size=0.2 0.2 1.1062296246821113; visual box size=0.2 0.2 1.1062296246821113
- link LeftLeg: geometry collision box size=1.4323677892271216 0.2 0.2; visual box size=1.4323677892271216 0.2 0.2
- link LeftLowerLeg: geometry collision box size=0.2 0.2 1.4425504891397218; visual box size=0.2 0.2 1.4425504891397218
- link RightLeg: geometry collision box size=1.4073798853908295 0.2 0.2; visual box size=1.4073798853908295 0.2 0.2
- link RightLowerLeg: geometry collision box size=0.2 0.2 0.6702124096108281; visual box size=0.2 0.2 0.6702124096108281
Joints:
- joint BackLeg_BackLowerLeg: origin xyz=0 -0.9367195390882855 0 rpy=0 0 0 -> xyz=0 -1.0398002398990647 0 rpy=0 0 0
- joint FrontLeg_FrontLowerLeg: origin xyz=0 0.6365048857184182 0 rpy=0 0 0 -> xyz=0 0.8540150976073921 0 rpy=0 0 0
- joint LeftLeg_LeftLowerLeg: origin xyz=-1.1917425688314363 0 0 rpy=0 0 0 -> xyz=-1.4323677892271216 0 0 rpy=0 0 0
- joint RightLeg_RightLowerLeg: origin xyz=0.8772221024504454 0 0 rpy=0 0 0 -> xyz=1.4073798853908295 0 0 rpy=0 0 0
- joint Torso_BackLeg: origin xyz=0 17.5 1.3596980125311244 rpy=0 0 0 -> xyz=0 17.5 1.4425504891397218 rpy=0 0 0
- joint Torso_FrontLeg: origin xyz=0 18.5 1.3596980125311244 rpy=0 0 0 -> xyz=0 18.5 1.4425504891397218 rpy=0 0 0
- joint Torso_LeftLeg: origin xyz=-0.5 18 1.3596980125311244 rpy=0 0 0 -> xyz=-0.5 18 1.4425504891397218 rpy=0 0 0
- joint Torso_RightLeg: origin xyz=0.5 18 1.3596980125311244 rpy=0 0 0 -> xyz=0.5 18 1.4425504891397218 rpy=0 0 0

File: bodyFiles/body01849.urdf (robot description, URDF)
Before this commit: robot robot, 9 links, 8 joints
Links:
- link BackLeg: geometry collision box size=0.2 0.5587067304145726 0.2; visual box size=0.2 0.5587067304145726 0.2
- link BackLowerLeg: geometry collision box size=0.2 0.2 0.8723734256194197; visual box size=0.2 0.2 0.8723734256194197
- link FrontLeg: geometry collision box size=0.2 1.4229184729012392 0.2; visual box size=0.2 1.4229184729012392 0.2
- link FrontLowerLeg: geometry collision box size=0.2 0.2 1.4609118390210631; visual box size=0.2 0.2 1.4609118390210631
- link LeftLeg: geometry collision box size=1.0112399200107363 0.2 0.2; visual box size=1.0112399200107363 0.2 0.2
- link LeftLowerLeg: geometry collision box size=0.2 0.2 1.4695823923026343; visual box size=0.2 0.2 1.4695823923026343
- link RightLeg: geometry collision box size=1.404233666281055 0.2 0.2; visual box size=1.404233666281055 0.2 0.2
- link RightLowerLeg: geometry collision box size=0.2 0.2 1.0427107090477135; visual box size=0.2 0.2 1.0427107090477135
Joints:
- joint BackLeg_BackLowerLeg: origin xyz=0 -0.816766601371767 0 rpy=0 0 0 -> xyz=0 -0.5587067304145726 0 rpy=0 0 0
- joint FrontLeg_FrontLowerLeg: origin xyz=0 0.8377179663629899 0 rpy=0 0 0 -> xyz=0 1.4229184729012392 0 rpy=0 0 0
- joint LeftLeg_LeftLowerLeg: origin xyz=-1.3787938270767917 0 0 rpy=0 0 0 -> xyz=-1.0112399200107363 0 0 rpy=0 0 0
- joint RightLeg_RightLowerLeg: origin xyz=0.865713201405669 0 0 rpy=0 0 0 -> xyz=1.404233666281055 0 0 rpy=0 0 0
- joint Torso_BackLeg: origin xyz=0 17.5 1.3787938270767917 rpy=0 0 0 -> xyz=0 17.5 1.4695823923026343 rpy=0 0 0
- joint Torso_FrontLeg: origin xyz=0 18.5 1.3787938270767917 rpy=0 0 0 -> xyz=0 18.5 1.4695823923026343 rpy=0 0 0
- joint Torso_LeftLeg: origin xyz=-0.5 18 1.3787938270767917 rpy=0 0 0 -> xyz=-0.5 18 1.4695823923026343 rpy=0 0 0
- joint Torso_RightLeg: origin xyz=0.5 18 1.3787938270767917 rpy=0 0 0 -> xyz=0.5 18 1.4695823923026343 rpy=0 0 0

File: bodyFiles/body01899.urdf (robot description, URDF)
Before this commit: robot robot, 9 links, 8 joints
Links:
- link BackLeg: geometry collision box size=0.2 1.2113552187306666 0.2; visual box size=0.2 1.2113552187306666 0.2
- link BackLowerLeg: geometry collision box size=0.2 0.2 1.3041203057180868; visual box size=0.2 0.2 1.3041203057180868
- link FrontLeg: geometry collision box size=0.2 1.0300933826062426 0.2; visual box size=0.2 1.0300933826062426 0.2
- link FrontLowerLeg: geometry collision box size=0.2 0.2 1.430740810839899; visual box size=0.2 0.2 1.430740810839899
- link LeftLeg: geometry collision box size=0.967447753178178 0.2 0.2; visual box size=0.967447753178178 0.2 0.2
- link LeftLowerLeg: geometry collision box size=0.2 0.2 0.6460410685592641; visual box size=0.2 0.2 0.6460410685592641
- link RightLeg: geometry collision box size=1.276419865823108 0.2 0.2; visual box size=1.276419865823108 0.2 0.2
- link RightLowerLeg: geometry collision box size=0.2 0.2 1.0455755606945538; visual box size=0.2 0.2 1.0455755606945538
Joints:
- joint BackLeg_BackLowerLeg: origin xyz=0 -0.8058485628620069 0 rpy=0 0 0 -> xyz=0 -1.2113552187306666 0 rpy=0 0 0
- joint FrontLeg_FrontLowerLeg: origin xyz=0 1.4947076369067493 0 rpy=0 0 0 -> xyz=0 1.0300933826062426 0 rpy=0 0 0
- joint LeftLeg_LeftLowerLeg: origin xyz=-1.4468010698219005 0 0 rpy=0 0 0 -> xyz=-0.967447753178178 0 0 rpy=0 0 0
- joint RightLeg_RightLowerLeg: origin xyz=0.7955253963613762 0 0 rpy=0 0 0 -> xyz=1.276419865823108 0 0 rpy=0 0 0
- joint Torso_BackLeg: origin xyz=0 17.5 1.4947076369067493 rpy=0 0 0 -> xyz=0 17.5 1.430740810839899 rpy=0 0 0
- joint Torso_FrontLeg: origin xyz=0 18.5 1.4947076369067493 rpy=0 0 0 -> xyz=0 18.5 1.430740810839899 rpy=0 0 0
- joint Torso_LeftLeg: origin xyz=-0.5 18 1.4947076369067493 rpy=0 0 0 -> xyz=-0.5 18 1.430740810839899 rpy=0 0 0
- joint Torso_RightLeg: origin xyz=0.5 18 1.4947076369067493 rpy=0 0 0 -> xyz=0.5 18 1.430740810839899 rpy=0 0 0

File: bodyFiles/body02175.urdf (robot description, URDF)
Before this commit: robot robot, 9 links, 8 joints
Links:
- link BackLeg: geometry collision box size=0.2 1.2524600270692137 0.2; visual box size=0.2 1.2524600270692137 0.2
- link BackLowerLeg: geometry collision box size=0.2 0.2 1.3599167773581118; visual box size=0.2 0.2 1.3599167773581118
- link FrontLeg: geometry collision box size=0.2 1.2512331297263817 0.2; visual box size=0.2 1.2512331297263817 0.2
- link FrontLowerLeg: geometry collision box size=0.2 0.2 1.3274107138365552; visual box size=0.2 0.2 1.3274107138365552
- link LeftLeg: geometry collision box size=0.7681553025733237 0.2 0.2; visual box size=0.7681553025733237 0.2 0.2
- link LeftLowerLeg: geometry collision box size=0.2 0.2 1.0529875260252552; visual box size=0.2 0.2 1.0529875260252552
- link RightLeg: geometry collision box size=0.7904153631453081 0.2 0.2; visual box size=0.7904153631453081 0.2 0.2
- link RightLowerLeg: geometry collision box size=0.2 0.2 1.191891141210061; visual box size=0.2 0.2 1.191891141210061
Joints:
- joint BackLeg_BackLowerLeg: origin xyz=0 -0.6568327086104983 0 rpy=0 0 0 -> xyz=0 -1.2524600270692137 0 rpy=0 0 0
- joint FrontLeg_FrontLowerLeg: origin xyz=0 1.3331710999823192 0 rpy=0 0 0 -> xyz=0 1.2512331297263817 0 rpy=0 0 0
- joint LeftLeg_LeftLowerLeg: origin xyz=-1.3909423461044175 0 0 rpy=0 0 0 -> xyz=-0.7681553025733237 0 0 rpy=0 0 0
- joint RightLeg_RightLowerLeg: origin xyz=0.8214751669205668 0 0 rpy=0 0 0 -> xyz=0.7904153631453081 0 0 rpy=0 0 0
- joint Torso_BackLeg: origin xyz=0 1.5 1.3909423461044175 rpy=0 0 0 -> xyz=0 1.5 1.3599167773581118 rpy=0 0 0
- joint Torso_FrontLeg: origin xyz=0 2.5 1.3909423461044175 rpy=0 0 0 -> xyz=0 2.5 1.3599167773581118 rpy=0 0 0
- joint Torso_LeftLeg: origin xyz=-0.5 2 1.3909423461044175 rpy=0 0 0 -> xyz=-0.5 2 1.3599167773581118 rpy=0 0 0
- joint Torso_RightLeg: origin xyz=0.5 2 1.3909423461044175 rpy=0 0 0 -> xyz=0.5 2 1.3599167773581118 rpy=0 0 0
