Commit message: case3, JAR = .8, random, more data

File: bodyFiles/body02325.urdf (robot description, URDF)
Before this commit: robot robot, 9 links, 8 joints
Links:
- link BackLeg: geometry collision box size=0.2 0.9251494804962707 0.2; visual box size=0.2 0.9251494804962707 0.2
- link BackLowerLeg: geometry collision box size=0.2 0.2 1.4905245094204638; visual box size=0.2 0.2 1.4905245094204638
- link FrontLeg: geometry collision box size=0.2 1.387277478554712 0.2; visual box size=0.2 1.387277478554712 0.2
- link FrontLowerLeg: geometry collision box size=0.2 0.2 1.4730556170914175; visual box size=0.2 0.2 1.4730556170914175
- link LeftLeg: geometry collision box size=1.1280221894033664 0.2 0.2; visual box size=1.1280221894033664 0.2 0.2
- link LeftLowerLeg: geometry collision box size=0.2 0.2 1.2287902128823913; visual box size=0.2 0.2 1.2287902128823913
- link RightLeg: geometry collision box size=0.8367264017774663 0.2 0.2; visual box size=0.8367264017774663 0.2 0.2
- link RightLowerLeg: geometry collision box size=0.2 0.2 0.9526337088919351; visual box size=0.2 0.2 0.9526337088919351
Joints:
- joint BackLeg_BackLowerLeg: origin xyz=0 -1.475382895464319 0 rpy=0 0 0 -> xyz=0 -0.9251494804962707 0 rpy=0 0 0
- joint FrontLeg_FrontLowerLeg: origin xyz=0 1.1154859518981348 0 rpy=0 0 0 -> xyz=0 1.387277478554712 0 rpy=0 0 0
- joint LeftLeg_LeftLowerLeg: origin xyz=-1.4206066440950833 0 0 rpy=0 0 0 -> xyz=-1.1280221894033664 0 0 rpy=0 0 0
- joint RightLeg_RightLowerLeg: origin xyz=0.9801766315708486 0 0 rpy=0 0 0 -> xyz=0.8367264017774663 0 0 rpy=0 0 0
- joint Torso_BackLeg: origin xyz=0 1.5 1.475382895464319 rpy=0 0 0 -> xyz=0 1.5 1.4905245094204638 rpy=0 0 0
- joint Torso_FrontLeg: origin xyz=0 2.5 1.475382895464319 rpy=0 0 0 -> xyz=0 2.5 1.4905245094204638 rpy=0 0 0
- joint Torso_LeftLeg: origin xyz=-0.5 2 1.475382895464319 rpy=0 0 0 -> xyz=-0.5 2 1.4905245094204638 rpy=0 0 0
- joint Torso_RightLeg: origin xyz=0.5 2 1.475382895464319 rpy=0 0 0 -> xyz=0.5 2 1.4905245094204638 rpy=0 0 0
