Commit message: jar = 0.8, pop = 5, gens = 40

File: bodyFiles/body0-10112.urdf (robot description, URDF)
Before this commit: robot robot, 9 links, 8 joints
Links:
- link BackLeg: geometry collision box size=0.2 0.7436904594344799 0.2; visual box size=0.2 0.7436904594344799 0.2
- link BackLowerLeg: geometry collision box size=0.2 0.2 0.961534611007083; visual box size=0.2 0.2 0.961534611007083
- link FrontLeg: geometry collision box size=0.2 0.7936679694007732 0.2; visual box size=0.2 0.7936679694007732 0.2
- link FrontLowerLeg: geometry collision box size=0.2 0.2 1.2124746930335046; visual box size=0.2 0.2 1.2124746930335046
- link LeftLeg: geometry collision box size=0.7083018212271307 0.2 0.2; visual box size=0.7083018212271307 0.2 0.2
- link LeftLowerLeg: geometry collision box size=0.2 0.2 0.8286853641591791; visual box size=0.2 0.2 0.8286853641591791
- link RightLeg: geometry collision box size=0.5637536468977369 0.2 0.2; visual box size=0.5637536468977369 0.2 0.2
- link RightLowerLeg: geometry collision box size=0.2 0.2 1.3696585141486146; visual box size=0.2 0.2 1.3696585141486146
Joints:
- joint BackLeg_BackLowerLeg: origin xyz=0 -0.9598723575927692 0 rpy=0 0 0 -> xyz=0 -0.7436904594344799 0 rpy=0 0 0
- joint FrontLeg_FrontLowerLeg: origin xyz=0 1.1817664101154763 0 rpy=0 0 0 -> xyz=0 0.7936679694007732 0 rpy=0 0 0
- joint LeftLeg_LeftLowerLeg: origin xyz=-1.2468517275319715 0 0 rpy=0 0 0 -> xyz=-0.7083018212271307 0 0 rpy=0 0 0
- joint RightLeg_RightLowerLeg: origin xyz=0.5217522699000777 0 0 rpy=0 0 0 -> xyz=0.5637536468977369 0 0 rpy=0 0 0
- joint Torso_BackLeg: origin xyz=0 -10.5 2.2468517275319715 rpy=0 0 0 -> xyz=0 -10.5 2.3696585141486146 rpy=0 0 0
- joint Torso_FrontLeg: origin xyz=0 -9.5 2.2468517275319715 rpy=0 0 0 -> xyz=0 -9.5 2.3696585141486146 rpy=0 0 0
- joint Torso_LeftLeg: origin xyz=-0.5 -10 2.2468517275319715 rpy=0 0 0 -> xyz=-0.5 -10 2.3696585141486146 rpy=0 0 0
- joint Torso_RightLeg: origin xyz=0.5 -10 2.2468517275319715 rpy=0 0 0 -> xyz=0.5 -10 2.3696585141486146 rpy=0 0 0

File: bodyFiles/body0-10162.urdf (robot description, URDF)
Before this commit: robot robot, 9 links, 8 joints
Links:
- link BackLeg: geometry collision box size=0.2 0.6926119499655145 0.2; visual box size=0.2 0.6926119499655145 0.2
- link BackLowerLeg: geometry collision box size=0.2 0.2 1.449492697710856; visual box size=0.2 0.2 1.449492697710856
- link FrontLeg: geometry collision box size=0.2 1.0421665401046902 0.2; visual box size=0.2 1.0421665401046902 0.2
- link FrontLowerLeg: geometry collision box size=0.2 0.2 0.544548680762729; visual box size=0.2 0.2 0.544548680762729
- link LeftLeg: geometry collision box size=0.8485976396591398 0.2 0.2; visual box size=0.8485976396591398 0.2 0.2
- link LeftLowerLeg: geometry collision box size=0.2 0.2 1.1629147311547539; visual box size=0.2 0.2 1.1629147311547539
- link RightLeg: geometry collision box size=1.3994800374326757 0.2 0.2; visual box size=1.3994800374326757 0.2 0.2
- link RightLowerLeg: geometry collision box size=0.2 0.2 1.1048842509953545; visual box size=0.2 0.2 1.1048842509953545
Joints:
- joint BackLeg_BackLowerLeg: origin xyz=0 -0.5814889555343482 0 rpy=0 0 0 -> xyz=0 -0.6926119499655145 0 rpy=0 0 0
- joint FrontLeg_FrontLowerLeg: origin xyz=0 1.084506949126374 0 rpy=0 0 0 -> xyz=0 1.0421665401046902 0 rpy=0 0 0
- joint LeftLeg_LeftLowerLeg: origin xyz=-0.5990102355355081 0 0 rpy=0 0 0 -> xyz=-0.8485976396591398 0 0 rpy=0 0 0
- joint RightLeg_RightLowerLeg: origin xyz=0.9361539523237333 0 0 rpy=0 0 0 -> xyz=1.3994800374326757 0 0 rpy=0 0 0
- joint Torso_BackLeg: origin xyz=0 -10.5 2.465155259336047 rpy=0 0 0 -> xyz=0 -10.5 2.449492697710856 rpy=0 0 0
- joint Torso_FrontLeg: origin xyz=0 -9.5 2.465155259336047 rpy=0 0 0 -> xyz=0 -9.5 2.449492697710856 rpy=0 0 0
- joint Torso_LeftLeg: origin xyz=-0.5 -10 2.465155259336047 rpy=0 0 0 -> xyz=-0.5 -10 2.449492697710856 rpy=0 0 0
- joint Torso_RightLeg: origin xyz=0.5 -10 2.465155259336047 rpy=0 0 0 -> xyz=0.5 -10 2.449492697710856 rpy=0 0 0

File: bodyFiles/body0-10412.urdf (robot description, URDF)
Before this commit: robot robot, 9 links, 8 joints
Links:
- link BackLeg: geometry collision box size=0.2 1.2040624625268155 0.2; visual box size=0.2 1.2040624625268155 0.2
- link BackLowerLeg: geometry collision box size=0.2 0.2 0.6724203058899093; visual box size=0.2 0.2 0.6724203058899093
- link FrontLeg: geometry collision box size=0.2 1.0203989622083107 0.2; visual box size=0.2 1.0203989622083107 0.2
- link FrontLowerLeg: geometry collision box size=0.2 0.2 0.6834914675335809; visual box size=0.2 0.2 0.6834914675335809
- link LeftLeg: geometry collision box size=0.6468667425780166 0.2 0.2; visual box size=0.6468667425780166 0.2 0.2
- link LeftLowerLeg: geometry collision box size=0.2 0.2 1.0363335799091766; visual box size=0.2 0.2 1.0363335799091766
- link RightLeg: geometry collision box size=1.1057460935576167 0.2 0.2; visual box size=1.1057460935576167 0.2 0.2
- link RightLowerLeg: geometry collision box size=0.2 0.2 1.2022660680568984; visual box size=0.2 0.2 1.2022660680568984
Joints:
- joint BackLeg_BackLowerLeg: origin xyz=0 -0.9727942144925528 0 rpy=0 0 0 -> xyz=0 -1.2040624625268155 0 rpy=0 0 0
- joint FrontLeg_FrontLowerLeg: origin xyz=0 0.5493958572773165 0 rpy=0 0 0 -> xyz=0 1.0203989622083107 0 rpy=0 0 0
- joint LeftLeg_LeftLowerLeg: origin xyz=-1.441270103688854 0 0 rpy=0 0 0 -> xyz=-0.6468667425780166 0 0 rpy=0 0 0
- joint RightLeg_RightLowerLeg: origin xyz=1.3502008590163204 0 0 rpy=0 0 0 -> xyz=1.1057460935576167 0 0 rpy=0 0 0
- joint Torso_BackLeg: origin xyz=0 -10.5 2.441270103688854 rpy=0 0 0 -> xyz=0 -10.5 2.2040624625268155 rpy=0 0 0
- joint Torso_FrontLeg: origin xyz=0 -9.5 2.441270103688854 rpy=0 0 0 -> xyz=0 -9.5 2.2040624625268155 rpy=0 0 0
- joint Torso_LeftLeg: origin xyz=-0.5 -10 2.441270103688854 rpy=0 0 0 -> xyz=-0.5 -10 2.2040624625268155 rpy=0 0 0
- joint Torso_RightLeg: origin xyz=0.5 -10 2.441270103688854 rpy=0 0 0 -> xyz=0.5 -10 2.2040624625268155 rpy=0 0 0

File: bodyFiles/body0-14561.urdf (robot description, URDF)
Before this commit: robot robot, 9 links, 8 joints
Links:
- link BackLeg: geometry collision box size=0.2 0.5575082034911842 0.2; visual box size=0.2 0.5575082034911842 0.2
- link BackLowerLeg: geometry collision box size=0.2 0.2 1.457905273847821; visual box size=0.2 0.2 1.457905273847821
- link FrontLeg: geometry collision box size=0.2 1.1820663586434814 0.2; visual box size=0.2 1.1820663586434814 0.2
- link FrontLowerLeg: geometry collision box size=0.2 0.2 0.784357203702586; visual box size=0.2 0.2 0.784357203702586
- link LeftLeg: geometry collision box size=0.8038457900946839 0.2 0.2; visual box size=0.8038457900946839 0.2 0.2
- link LeftLowerLeg: geometry collision box size=0.2 0.2 0.87879653278762; visual box size=0.2 0.2 0.87879653278762
- link RightLeg: geometry collision box size=1.265225731663227 0.2 0.2; visual box size=1.265225731663227 0.2 0.2
- link RightLowerLeg: geometry collision box size=0.2 0.2 1.3800279590361175; visual box size=0.2 0.2 1.3800279590361175
Joints:
- joint BackLeg_BackLowerLeg: origin xyz=0 -1.0637060571203911 0 rpy=0 0 0 -> xyz=0 -0.5575082034911842 0 rpy=0 0 0
- joint FrontLeg_FrontLowerLeg: origin xyz=0 0.6432862057069751 0 rpy=0 0 0 -> xyz=0 1.1820663586434814 0 rpy=0 0 0
- joint LeftLeg_LeftLowerLeg: origin xyz=-0.6448306236020003 0 0 rpy=0 0 0 -> xyz=-0.8038457900946839 0 0 rpy=0 0 0
- joint RightLeg_RightLowerLeg: origin xyz=0.7743318534055684 0 0 rpy=0 0 0 -> xyz=1.265225731663227 0 0 rpy=0 0 0
- joint Torso_BackLeg: origin xyz=0 -14.5 2.4625717531313103 rpy=0 0 0 -> xyz=0 -14.5 2.457905273847821 rpy=0 0 0
- joint Torso_FrontLeg: origin xyz=0 -13.5 2.4625717531313103 rpy=0 0 0 -> xyz=0 -13.5 2.457905273847821 rpy=0 0 0
- joint Torso_LeftLeg: origin xyz=-0.5 -14 2.4625717531313103 rpy=0 0 0 -> xyz=-0.5 -14 2.457905273847821 rpy=0 0 0
- joint Torso_RightLeg: origin xyz=0.5 -14 2.4625717531313103 rpy=0 0 0 -> xyz=0.5 -14 2.457905273847821 rpy=0 0 0

File: bodyFiles/body0-180.urdf (robot description, URDF)
Before this commit: robot robot, 9 links, 8 joints
Links:
- link BackLeg: geometry collision box size=0.2 1.3501152425108363 0.2; visual box size=0.2 1.3501152425108363 0.2
- link BackLowerLeg: geometry collision box size=0.2 0.2 0.9052524711808576; visual box size=0.2 0.2 0.9052524711808576
- link FrontLeg: geometry collision box size=0.2 0.850292401620745 0.2; visual box size=0.2 0.850292401620745 0.2
- link FrontLowerLeg: geometry collision box size=0.2 0.2 0.7759209217001759; visual box size=0.2 0.2 0.7759209217001759
- link LeftLeg: geometry collision box size=0.608751829138665 0.2 0.2; visual box size=0.608751829138665 0.2 0.2
- link LeftLowerLeg: geometry collision box size=0.2 0.2 1.0628278581051511; visual box size=0.2 0.2 1.0628278581051511
- link RightLeg: geometry collision box size=1.381142487977056 0.2 0.2; visual box size=1.381142487977056 0.2 0.2
- link RightLowerLeg: geometry collision box size=0.2 0.2 1.033573573016735; visual box size=0.2 0.2 1.033573573016735
Joints:
- joint BackLeg_BackLowerLeg: origin xyz=0 -0.8597572027470005 0 rpy=0 0 0 -> xyz=0 -1.3501152425108363 0 rpy=0 0 0
- joint FrontLeg_FrontLowerLeg: origin xyz=0 0.9532755602191995 0 rpy=0 0 0 -> xyz=0 0.850292401620745 0 rpy=0 0 0
- joint LeftLeg_LeftLowerLeg: origin xyz=-0.6345145351766656 0 0 rpy=0 0 0 -> xyz=-0.608751829138665 0 0 rpy=0 0 0
- joint RightLeg_RightLowerLeg: origin xyz=1.3475938252467945 0 0 rpy=0 0 0 -> xyz=1.381142487977056 0 0 rpy=0 0 0
- joint Torso_BackLeg: origin xyz=0 -18.5 2.3475938252467943 rpy=0 0 0 -> xyz=0 -18.5 2.3811424879770557 rpy=0 0 0
- joint Torso_FrontLeg: origin xyz=0 -17.5 2.3475938252467943 rpy=0 0 0 -> xyz=0 -17.5 2.3811424879770557 rpy=0 0 0
- joint Torso_LeftLeg: origin xyz=-0.5 -18 2.3475938252467943 rpy=0 0 0 -> xyz=-0.5 -18 2.3811424879770557 rpy=0 0 0
- joint Torso_RightLeg: origin xyz=0.5 -18 2.3475938252467943 rpy=0 0 0 -> xyz=0.5 -18 2.3811424879770557 rpy=0 0 0

File: bodyFiles/body0-18200.urdf (robot description, URDF)
Before this commit: robot robot, 9 links, 8 joints
Links:
- link BackLeg: geometry collision box size=0.2 0.8122961951241093 0.2; visual box size=0.2 0.8122961951241093 0.2
- link BackLowerLeg: geometry collision box size=0.2 0.2 1.4020316226437672; visual box size=0.2 0.2 1.4020316226437672
- link FrontLeg: geometry collision box size=0.2 0.8239326907738544 0.2; visual box size=0.2 0.8239326907738544 0.2
- link FrontLowerLeg: geometry collision box size=0.2 0.2 0.6904918219019818; visual box size=0.2 0.2 0.6904918219019818
- link LeftLeg: geometry collision box size=0.6454467530349345 0.2 0.2; visual box size=0.6454467530349345 0.2 0.2
- link LeftLowerLeg: geometry collision box size=0.2 0.2 1.1292097063501978; visual box size=0.2 0.2 1.1292097063501978
- link RightLeg: geometry collision box size=0.6572985963508875 0.2 0.2; visual box size=0.6572985963508875 0.2 0.2
- link RightLowerLeg: geometry collision box size=0.2 0.2 1.3670476412463546; visual box size=0.2 0.2 1.3670476412463546
Joints:
- joint BackLeg_BackLowerLeg: origin xyz=0 -0.6669465315802477 0 rpy=0 0 0 -> xyz=0 -0.8122961951241093 0 rpy=0 0 0
- joint FrontLeg_FrontLowerLeg: origin xyz=0 0.5299430117891276 0 rpy=0 0 0 -> xyz=0 0.8239326907738544 0 rpy=0 0 0
- joint LeftLeg_LeftLowerLeg: origin xyz=-1.3243116990452042 0 0 rpy=0 0 0 -> xyz=-0.6454467530349345 0 0 rpy=0 0 0
- joint RightLeg_RightLowerLeg: origin xyz=1.142370421067535 0 0 rpy=0 0 0 -> xyz=0.6572985963508875 0 0 rpy=0 0 0
- joint Torso_BackLeg: origin xyz=0 -18.5 2.381222081412949 rpy=0 0 0 -> xyz=0 -18.5 2.4020316226437672 rpy=0 0 0
- joint Torso_FrontLeg: origin xyz=0 -17.5 2.381222081412949 rpy=0 0 0 -> xyz=0 -17.5 2.4020316226437672 rpy=0 0 0
- joint Torso_LeftLeg: origin xyz=-0.5 -18 2.381222081412949 rpy=0 0 0 -> xyz=-0.5 -18 2.4020316226437672 rpy=0 0 0
- joint Torso_RightLeg: origin xyz=0.5 -18 2.381222081412949 rpy=0 0 0 -> xyz=0.5 -18 2.4020316226437672 rpy=0 0 0

File: bodyFiles/body0-1850.urdf (robot description, URDF)
Before this commit: robot robot, 9 links, 8 joints
Links:
- link BackLeg: geometry collision box size=0.2 1.4528197986036369 0.2; visual box size=0.2 1.4528197986036369 0.2
- link BackLowerLeg: geometry collision box size=0.2 0.2 1.2404049026361461; visual box size=0.2 0.2 1.2404049026361461
- link FrontLeg: geometry collision box size=0.2 0.850135580513251 0.2; visual box size=0.2 0.850135580513251 0.2
- link FrontLowerLeg: geometry collision box size=0.2 0.2 1.2274728478400063; visual box size=0.2 0.2 1.2274728478400063
- link LeftLeg: geometry collision box size=0.9462775700684607 0.2 0.2; visual box size=0.9462775700684607 0.2 0.2
- link LeftLowerLeg: geometry collision box size=0.2 0.2 0.529276025042297; visual box size=0.2 0.2 0.529276025042297
- link RightLeg: geometry collision box size=0.6960528672757955 0.2 0.2; visual box size=0.6960528672757955 0.2 0.2
- link RightLowerLeg: geometry collision box size=0.2 0.2 0.5811050544449247; visual box size=0.2 0.2 0.5811050544449247
Joints:
- joint BackLeg_BackLowerLeg: origin xyz=0 -1.0636896472628985 0 rpy=0 0 0 -> xyz=0 -1.4528197986036369 0 rpy=0 0 0
- joint FrontLeg_FrontLowerLeg: origin xyz=0 0.9440397167896779 0 rpy=0 0 0 -> xyz=0 0.850135580513251 0 rpy=0 0 0
- joint LeftLeg_LeftLowerLeg: origin xyz=-0.5222572470246496 0 0 rpy=0 0 0 -> xyz=-0.9462775700684607 0 0 rpy=0 0 0
- joint RightLeg_RightLowerLeg: origin xyz=1.1000427453576238 0 0 rpy=0 0 0 -> xyz=0.6960528672757955 0 0 rpy=0 0 0
- joint Torso_BackLeg: origin xyz=0 -18.5 2.4731842652081153 rpy=0 0 0 -> xyz=0 -18.5 2.452819798603637 rpy=0 0 0
- joint Torso_FrontLeg: origin xyz=0 -17.5 2.4731842652081153 rpy=0 0 0 -> xyz=0 -17.5 2.452819798603637 rpy=0 0 0
- joint Torso_LeftLeg: origin xyz=-0.5 -18 2.4731842652081153 rpy=0 0 0 -> xyz=-0.5 -18 2.452819798603637 rpy=0 0 0
- joint Torso_RightLeg: origin xyz=0.5 -18 2.4731842652081153 rpy=0 0 0 -> xyz=0.5 -18 2.452819798603637 rpy=0 0 0

File: bodyFiles/body0-2224.urdf (robot description, URDF)
Before this commit: robot robot, 9 links, 8 joints
Links:
- link BackLeg: geometry collision box size=0.2 0.6275410930398313 0.2; visual box size=0.2 0.6275410930398313 0.2
- link BackLowerLeg: geometry collision box size=0.2 0.2 1.4785964726072816; visual box size=0.2 0.2 1.4785964726072816
- link FrontLeg: geometry collision box size=0.2 1.0905243515673875 0.2; visual box size=0.2 1.0905243515673875 0.2
- link FrontLowerLeg: geometry collision box size=0.2 0.2 0.9663389194644362; visual box size=0.2 0.2 0.9663389194644362
- link LeftLeg: geometry collision box size=0.5983480330382518 0.2 0.2; visual box size=0.5983480330382518 0.2 0.2
- link LeftLowerLeg: geometry collision box size=0.2 0.2 0.9799617032302482; visual box size=0.2 0.2 0.9799617032302482
- link RightLeg: geometry collision box size=1.4697206381944594 0.2 0.2; visual box size=1.4697206381944594 0.2 0.2
- link RightLowerLeg: geometry collision box size=0.2 0.2 1.0375329945560199; visual box size=0.2 0.2 1.0375329945560199
Joints:
- joint BackLeg_BackLowerLeg: origin xyz=0 -1.2857780160498042 0 rpy=0 0 0 -> xyz=0 -0.6275410930398313 0 rpy=0 0 0
- joint FrontLeg_FrontLowerLeg: origin xyz=0 0.6753063639600841 0 rpy=0 0 0 -> xyz=0 1.0905243515673875 0 rpy=0 0 0
- joint LeftLeg_LeftLowerLeg: origin xyz=-0.5335052558475866 0 0 rpy=0 0 0 -> xyz=-0.5983480330382518 0 0 rpy=0 0 0
- joint RightLeg_RightLowerLeg: origin xyz=1.1939676769413003 0 0 rpy=0 0 0 -> xyz=1.4697206381944594 0 0 rpy=0 0 0
- joint Torso_BackLeg: origin xyz=0 -2.5 2.4505232332676923 rpy=0 0 0 -> xyz=0 -2.5 2.4785964726072818 rpy=0 0 0
- joint Torso_FrontLeg: origin xyz=0 -1.5 2.4505232332676923 rpy=0 0 0 -> xyz=0 -1.5 2.4785964726072818 rpy=0 0 0
- joint Torso_LeftLeg: origin xyz=-0.5 -2 2.4505232332676923 rpy=0 0 0 -> xyz=-0.5 -2 2.4785964726072818 rpy=0 0 0
- joint Torso_RightLeg: origin xyz=0.5 -2 2.4505232332676923 rpy=0 0 0 -> xyz=0.5 -2 2.4785964726072818 rpy=0 0 0

File: bodyFiles/body0-2274.urdf (robot description, URDF)
Before this commit: robot robot, 9 links, 8 joints
Links:
- link BackLeg: geometry collision box size=0.2 0.9165115121577168 0.2; visual box size=0.2 0.9165115121577168 0.2
- link BackLowerLeg: geometry collision box size=0.2 0.2 0.5324262595396168; visual box size=0.2 0.2 0.5324262595396168
- link FrontLeg: geometry collision box size=0.2 1.1710221163306622 0.2; visual box size=0.2 1.1710221163306622 0.2
- link FrontLowerLeg: geometry collision box size=0.2 0.2 0.5127921833469172; visual box size=0.2 0.2 0.5127921833469172
- link LeftLeg: geometry collision box size=0.9113448257611991 0.2 0.2; visual box size=0.9113448257611991 0.2 0.2
- link LeftLowerLeg: geometry collision box size=0.2 0.2 1.1801884690312525; visual box size=0.2 0.2 1.1801884690312525
- link RightLeg: geometry collision box size=0.6994243706095505 0.2 0.2; visual box size=0.6994243706095505 0.2 0.2
- link RightLowerLeg: geometry collision box size=0.2 0.2 0.7438318613477188; visual box size=0.2 0.2 0.7438318613477188
Joints:
- joint BackLeg_BackLowerLeg: origin xyz=0 -0.8723829952652499 0 rpy=0 0 0 -> xyz=0 -0.9165115121577168 0 rpy=0 0 0
- joint FrontLeg_FrontLowerLeg: origin xyz=0 0.9064495925688526 0 rpy=0 0 0 -> xyz=0 1.1710221163306622 0 rpy=0 0 0
- joint LeftLeg_LeftLowerLeg: origin xyz=-0.6953354575086671 0 0 rpy=0 0 0 -> xyz=-0.9113448257611991 0 0 rpy=0 0 0
- joint RightLeg_RightLowerLeg: origin xyz=0.6723421391290116 0 0 rpy=0 0 0 -> xyz=0.6994243706095505 0 0 rpy=0 0 0
- joint Torso_BackLeg: origin xyz=0 -2.5 2.076589849084225 rpy=0 0 0 -> xyz=0 -2.5 2.1801884690312523 rpy=0 0 0
- joint Torso_FrontLeg: origin xyz=0 -1.5 2.076589849084225 rpy=0 0 0 -> xyz=0 -1.5 2.1801884690312523 rpy=0 0 0
- joint Torso_LeftLeg: origin xyz=-0.5 -2 2.076589849084225 rpy=0 0 0 -> xyz=-0.5 -2 2.1801884690312523 rpy=0 0 0
- joint Torso_RightLeg: origin xyz=0.5 -2 2.076589849084225 rpy=0 0 0 -> xyz=0.5 -2 2.1801884690312523 rpy=0 0 0

File: bodyFiles/body010387.urdf (robot description, URDF)
Before this commit: robot robot, 9 links, 8 joints
Links:
- link BackLeg: geometry collision box size=0.2 1.1033159015944358 0.2; visual box size=0.2 1.1033159015944358 0.2
- link BackLowerLeg: geometry collision box size=0.2 0.2 0.6482182333039638; visual box size=0.2 0.2 0.6482182333039638
- link FrontLeg: geometry collision box size=0.2 0.5880392598814125 0.2; visual box size=0.2 0.5880392598814125 0.2
- link FrontLowerLeg: geometry collision box size=0.2 0.2 0.5002306827600588; visual box size=0.2 0.2 0.5002306827600588
- link LeftLeg: geometry collision box size=0.8396561939292551 0.2 0.2; visual box size=0.8396561939292551 0.2 0.2
- link LeftLowerLeg: geometry collision box size=0.2 0.2 0.8677891918174356; visual box size=0.2 0.2 0.8677891918174356
- link RightLeg: geometry collision box size=1.450077969732955 0.2 0.2; visual box size=1.450077969732955 0.2 0.2
- link RightLowerLeg: geometry collision box size=0.2 0.2 0.8806272003361407; visual box size=0.2 0.2 0.8806272003361407
Joints:
- joint BackLeg_BackLowerLeg: origin xyz=0 -1.414228006997345 0 rpy=0 0 0 -> xyz=0 -1.1033159015944358 0 rpy=0 0 0
- joint FrontLeg_FrontLowerLeg: origin xyz=0 0.6562379887170412 0 rpy=0 0 0 -> xyz=0 0.5880392598814125 0 rpy=0 0 0
- joint LeftLeg_LeftLowerLeg: origin xyz=-1.247399448179762 0 0 rpy=0 0 0 -> xyz=-0.8396561939292551 0 0 rpy=0 0 0
- joint RightLeg_RightLowerLeg: origin xyz=0.7930380147555967 0 0 rpy=0 0 0 -> xyz=1.450077969732955 0 0 rpy=0 0 0
- joint Torso_BackLeg: origin xyz=0 9.5 2.414228006997345 rpy=0 0 0 -> xyz=0 9.5 2.450077969732955 rpy=0 0 0
- joint Torso_FrontLeg: origin xyz=0 10.5 2.414228006997345 rpy=0 0 0 -> xyz=0 10.5 2.450077969732955 rpy=0 0 0
- joint Torso_LeftLeg: origin xyz=-0.5 10 2.414228006997345 rpy=0 0 0 -> xyz=-0.5 10 2.450077969732955 rpy=0 0 0
- joint Torso_RightLeg: origin xyz=0.5 10 2.414228006997345 rpy=0 0 0 -> xyz=0.5 10 2.450077969732955 rpy=0 0 0

File: bodyFiles/body01087.urdf (robot description, URDF)
Before this commit: robot robot, 9 links, 8 joints
Links:
- link BackLeg: geometry collision box size=0.2 1.0126031614135762 0.2; visual box size=0.2 1.0126031614135762 0.2
- link BackLowerLeg: geometry collision box size=0.2 0.2 1.0066870513917798; visual box size=0.2 0.2 1.0066870513917798
- link FrontLeg: geometry collision box size=0.2 1.0769892040809688 0.2; visual box size=0.2 1.0769892040809688 0.2
- link FrontLowerLeg: geometry collision box size=0.2 0.2 0.7774215347767971; visual box size=0.2 0.2 0.7774215347767971
- link LeftLeg: geometry collision box size=0.5774183142522672 0.2 0.2; visual box size=0.5774183142522672 0.2 0.2
- link LeftLowerLeg: geometry collision box size=0.2 0.2 0.7643057101166624; visual box size=0.2 0.2 0.7643057101166624
- link RightLeg: geometry collision box size=1.4372214391597158 0.2 0.2; visual box size=1.4372214391597158 0.2 0.2
- link RightLowerLeg: geometry collision box size=0.2 0.2 1.343503315943098; visual box size=0.2 0.2 1.343503315943098
Joints:
- joint BackLeg_BackLowerLeg: origin xyz=0 -1.0357118505124112 0 rpy=0 0 0 -> xyz=0 -1.0126031614135762 0 rpy=0 0 0
- joint FrontLeg_FrontLowerLeg: origin xyz=0 0.7760524460419671 0 rpy=0 0 0 -> xyz=0 1.0769892040809688 0 rpy=0 0 0
- joint LeftLeg_LeftLowerLeg: origin xyz=-1.2582749971916605 0 0 rpy=0 0 0 -> xyz=-0.5774183142522672 0 0 rpy=0 0 0
- joint RightLeg_RightLowerLeg: origin xyz=0.8507664267287971 0 0 rpy=0 0 0 -> xyz=1.4372214391597158 0 0 rpy=0 0 0
- joint Torso_BackLeg: origin xyz=0 9.5 2.2582749971916605 rpy=0 0 0 -> xyz=0 9.5 2.437221439159716 rpy=0 0 0
- joint Torso_FrontLeg: origin xyz=0 10.5 2.2582749971916605 rpy=0 0 0 -> xyz=0 10.5 2.437221439159716 rpy=0 0 0
- joint Torso_LeftLeg: origin xyz=-0.5 10 2.2582749971916605 rpy=0 0 0 -> xyz=-0.5 10 2.437221439159716 rpy=0 0 0
- joint Torso_RightLeg: origin xyz=0.5 10 2.2582749971916605 rpy=0 0 0 -> xyz=0.5 10 2.437221439159716 rpy=0 0 0
