Commit message: jar = 0.8, pop = 5, gens = 40

File: bodyFiles/body014498.urdf (robot description, URDF)
Before this commit: robot robot, 9 links, 8 joints
Links:
- link BackLeg: geometry collision box size=0.2 1.4001491090040425 0.2; visual box size=0.2 1.4001491090040425 0.2
- link BackLowerLeg: geometry collision box size=0.2 0.2 0.8974480035014915; visual box size=0.2 0.2 0.8974480035014915
- link FrontLeg: geometry collision box size=0.2 0.6356698651680014 0.2; visual box size=0.2 0.6356698651680014 0.2
- link FrontLowerLeg: geometry collision box size=0.2 0.2 1.3538806813038822; visual box size=0.2 0.2 1.3538806813038822
- link LeftLeg: geometry collision box size=0.7702939740783916 0.2 0.2; visual box size=0.7702939740783916 0.2 0.2
- link LeftLowerLeg: geometry collision box size=0.2 0.2 1.2012145566002788; visual box size=0.2 0.2 1.2012145566002788
- link RightLeg: geometry collision box size=1.0106123537225804 0.2 0.2; visual box size=1.0106123537225804 0.2 0.2
- link RightLowerLeg: geometry collision box size=0.2 0.2 1.3495386278315225; visual box size=0.2 0.2 1.3495386278315225
Joints:
- joint BackLeg_BackLowerLeg: origin xyz=0 -0.7830307605093939 0 rpy=0 0 0 -> xyz=0 -1.4001491090040425 0 rpy=0 0 0
- joint FrontLeg_FrontLowerLeg: origin xyz=0 1.4413865722217867 0 rpy=0 0 0 -> xyz=0 0.6356698651680014 0 rpy=0 0 0
- joint LeftLeg_LeftLowerLeg: origin xyz=-1.3115465388690732 0 0 rpy=0 0 0 -> xyz=-0.7702939740783916 0 0 rpy=0 0 0
- joint RightLeg_RightLowerLeg: origin xyz=1.2312322989516704 0 0 rpy=0 0 0 -> xyz=1.0106123537225804 0 0 rpy=0 0 0
- joint Torso_BackLeg: origin xyz=0 13.5 2.441386572221787 rpy=0 0 0 -> xyz=0 13.5 2.4001491090040425 rpy=0 0 0
- joint Torso_FrontLeg: origin xyz=0 14.5 2.441386572221787 rpy=0 0 0 -> xyz=0 14.5 2.4001491090040425 rpy=0 0 0
- joint Torso_LeftLeg: origin xyz=-0.5 14 2.441386572221787 rpy=0 0 0 -> xyz=-0.5 14 2.4001491090040425 rpy=0 0 0
- joint Torso_RightLeg: origin xyz=0.5 14 2.441386572221787 rpy=0 0 0 -> xyz=0.5 14 2.4001491090040425 rpy=0 0 0

File: bodyFiles/body02275.urdf (robot description, URDF)
Before this commit: robot robot, 9 links, 8 joints
Links:
- link BackLeg: geometry collision box size=0.2 1.2815908255531452 0.2; visual box size=0.2 1.2815908255531452 0.2
- link BackLowerLeg: geometry collision box size=0.2 0.2 1.4065423468529854; visual box size=0.2 0.2 1.4065423468529854
- link FrontLeg: geometry collision box size=0.2 1.428936326332585 0.2; visual box size=0.2 1.428936326332585 0.2
- link FrontLowerLeg: geometry collision box size=0.2 0.2 1.4462693778162303; visual box size=0.2 0.2 1.4462693778162303
- link LeftLeg: geometry collision box size=1.4757417250322873 0.2 0.2; visual box size=1.4757417250322873 0.2 0.2
- link LeftLowerLeg: geometry collision box size=0.2 0.2 0.872620743085982; visual box size=0.2 0.2 0.872620743085982
- link RightLeg: geometry collision box size=1.2142803973680314 0.2 0.2; visual box size=1.2142803973680314 0.2 0.2
- link RightLowerLeg: geometry collision box size=0.2 0.2 1.074396246923768; visual box size=0.2 0.2 1.074396246923768
Joints:
- joint BackLeg_BackLowerLeg: origin xyz=0 -0.8243719227684694 0 rpy=0 0 0 -> xyz=0 -1.2815908255531452 0 rpy=0 0 0
- joint FrontLeg_FrontLowerLeg: origin xyz=0 1.0988962730114133 0 rpy=0 0 0 -> xyz=0 1.428936326332585 0 rpy=0 0 0
- joint LeftLeg_LeftLowerLeg: origin xyz=-0.9541136227376706 0 0 rpy=0 0 0 -> xyz=-1.4757417250322873 0 0 rpy=0 0 0
- joint RightLeg_RightLowerLeg: origin xyz=1.0091798575059718 0 0 rpy=0 0 0 -> xyz=1.2142803973680314 0 0 rpy=0 0 0
- joint Torso_BackLeg: origin xyz=0 1.5 2.4710299015643464 rpy=0 0 0 -> xyz=0 1.5 2.4757417250322873 rpy=0 0 0
- joint Torso_FrontLeg: origin xyz=0 2.5 2.4710299015643464 rpy=0 0 0 -> xyz=0 2.5 2.4757417250322873 rpy=0 0 0
- joint Torso_LeftLeg: origin xyz=-0.5 2 2.4710299015643464 rpy=0 0 0 -> xyz=-0.5 2 2.4757417250322873 rpy=0 0 0
- joint Torso_RightLeg: origin xyz=0.5 2 2.4710299015643464 rpy=0 0 0 -> xyz=0.5 2 2.4757417250322873 rpy=0 0 0

File: bodyFiles/body02425.urdf (robot description, URDF)
Before this commit: robot robot, 9 links, 8 joints
Links:
- link BackLeg: geometry collision box size=0.2 1.3338966041333544 0.2; visual box size=0.2 1.3338966041333544 0.2
- link BackLowerLeg: geometry collision box size=0.2 0.2 1.3468613491950507; visual box size=0.2 0.2 1.3468613491950507
- link FrontLeg: geometry collision box size=0.2 0.8443755428220826 0.2; visual box size=0.2 0.8443755428220826 0.2
- link FrontLowerLeg: geometry collision box size=0.2 0.2 0.6241245026452616; visual box size=0.2 0.2 0.6241245026452616
- link LeftLeg: geometry collision box size=0.7409173482885808 0.2 0.2; visual box size=0.7409173482885808 0.2 0.2
- link LeftLowerLeg: geometry collision box size=0.2 0.2 1.0049871704054456; visual box size=0.2 0.2 1.0049871704054456
- link RightLeg: geometry collision box size=0.892665465163559 0.2 0.2; visual box size=0.892665465163559 0.2 0.2
- link RightLowerLeg: geometry collision box size=0.2 0.2 0.8151602351236603; visual box size=0.2 0.2 0.8151602351236603
Joints:
- joint BackLeg_BackLowerLeg: origin xyz=0 -1.4929532115175417 0 rpy=0 0 0 -> xyz=0 -1.3338966041333544 0 rpy=0 0 0
- joint FrontLeg_FrontLowerLeg: origin xyz=0 0.5980764302741274 0 rpy=0 0 0 -> xyz=0 0.8443755428220826 0 rpy=0 0 0
- joint LeftLeg_LeftLowerLeg: origin xyz=-0.9805230856708198 0 0 rpy=0 0 0 -> xyz=-0.7409173482885808 0 0 rpy=0 0 0
- joint RightLeg_RightLowerLeg: origin xyz=0.6825034724198578 0 0 rpy=0 0 0 -> xyz=0.892665465163559 0 0 rpy=0 0 0
- joint Torso_BackLeg: origin xyz=0 1.5 2.4929532115175417 rpy=0 0 0 -> xyz=0 1.5 2.3468613491950507 rpy=0 0 0
- joint Torso_FrontLeg: origin xyz=0 2.5 2.4929532115175417 rpy=0 0 0 -> xyz=0 2.5 2.3468613491950507 rpy=0 0 0
- joint Torso_LeftLeg: origin xyz=-0.5 2 2.4929532115175417 rpy=0 0 0 -> xyz=-0.5 2 2.3468613491950507 rpy=0 0 0
- joint Torso_RightLeg: origin xyz=0.5 2 2.4929532115175417 rpy=0 0 0 -> xyz=0.5 2 2.3468613491950507 rpy=0 0 0

File: bodyFiles/body06636.urdf (robot description, URDF)
Before this commit: robot robot, 9 links, 8 joints
Links:
- link BackLeg: geometry collision box size=0.2 1.0393464644506403 0.2; visual box size=0.2 1.0393464644506403 0.2
- link BackLowerLeg: geometry collision box size=0.2 0.2 0.9673042433428715; visual box size=0.2 0.2 0.9673042433428715
- link FrontLeg: geometry collision box size=0.2 0.8661335462955461 0.2; visual box size=0.2 0.8661335462955461 0.2
- link FrontLowerLeg: geometry collision box size=0.2 0.2 1.0851985320659319; visual box size=0.2 0.2 1.0851985320659319
- link LeftLeg: geometry collision box size=1.4947705315083362 0.2 0.2; visual box size=1.4947705315083362 0.2 0.2
- link LeftLowerLeg: geometry collision box size=0.2 0.2 0.9601472322291633; visual box size=0.2 0.2 0.9601472322291633
- link RightLeg: geometry collision box size=1.3984668607574142 0.2 0.2; visual box size=1.3984668607574142 0.2 0.2
- link RightLowerLeg: geometry collision box size=0.2 0.2 1.0680944793580698; visual box size=0.2 0.2 1.0680944793580698
Joints:
- joint BackLeg_BackLowerLeg: origin xyz=0 -0.6850042650122428 0 rpy=0 0 0 -> xyz=0 -1.0393464644506403 0 rpy=0 0 0
- joint FrontLeg_FrontLowerLeg: origin xyz=0 0.7292174944047877 0 rpy=0 0 0 -> xyz=0 0.8661335462955461 0 rpy=0 0 0
- joint LeftLeg_LeftLowerLeg: origin xyz=-1.267216728862134 0 0 rpy=0 0 0 -> xyz=-1.4947705315083362 0 0 rpy=0 0 0
- joint RightLeg_RightLowerLeg: origin xyz=0.7836647516823829 0 0 rpy=0 0 0 -> xyz=1.3984668607574142 0 0 rpy=0 0 0
- joint Torso_BackLeg: origin xyz=0 5.5 2.35672683946511 rpy=0 0 0 -> xyz=0 5.5 2.494770531508336 rpy=0 0 0
- joint Torso_FrontLeg: origin xyz=0 6.5 2.35672683946511 rpy=0 0 0 -> xyz=0 6.5 2.494770531508336 rpy=0 0 0
- joint Torso_LeftLeg: origin xyz=-0.5 6 2.35672683946511 rpy=0 0 0 -> xyz=-0.5 6 2.494770531508336 rpy=0 0 0
- joint Torso_RightLeg: origin xyz=0.5 6 2.35672683946511 rpy=0 0 0 -> xyz=0.5 6 2.494770531508336 rpy=0 0 0
