Commit message: modified phc and soln so continue works

File: bodyFiles/body0-102.urdf (robot description, URDF)
Before this commit: robot robot, 9 links, 8 joints
Links:
- link BackLeg: geometry collision box size=0.2 1.4275749994099776 0.2; visual box size=0.2 1.4275749994099776 0.2
- link BackLowerLeg: geometry collision box size=0.2 0.2 0.5962522582235873; visual box size=0.2 0.2 0.5962522582235873
- link FrontLeg: geometry collision box size=0.2 1.0769079869780585 0.2; visual box size=0.2 1.0769079869780585 0.2
- link FrontLowerLeg: geometry collision box size=0.2 0.2 0.5132560956004169; visual box size=0.2 0.2 0.5132560956004169
- link LeftLeg: geometry collision box size=1.3691600627422513 0.2 0.2; visual box size=1.3691600627422513 0.2 0.2
- link LeftLowerLeg: geometry collision box size=0.2 0.2 1.190456264272874; visual box size=0.2 0.2 1.190456264272874
- link RightLeg: geometry collision box size=0.715110470321962 0.2 0.2; visual box size=0.715110470321962 0.2 0.2
- link RightLowerLeg: geometry collision box size=0.2 0.2 1.2431676217742886; visual box size=0.2 0.2 1.2431676217742886
Joints:
- joint BackLeg_BackLowerLeg: origin xyz=0 -0.795703603921058 0 rpy=0 0 0 -> xyz=0 -1.4275749994099776 0 rpy=0 0 0
- joint FrontLeg_FrontLowerLeg: origin xyz=0 1.1375484563006857 0 rpy=0 0 0 -> xyz=0 1.0769079869780585 0 rpy=0 0 0
- joint LeftLeg_LeftLowerLeg: origin xyz=-1.3575543320552639 0 0 rpy=0 0 0 -> xyz=-1.3691600627422513 0 0 rpy=0 0 0
- joint RightLeg_RightLowerLeg: origin xyz=0.5780501537387961 0 0 rpy=0 0 0 -> xyz=0.715110470321962 0 0 rpy=0 0 0
- joint Torso_BackLeg: origin xyz=0 -18.5 2.3575543320552637 rpy=0 0 0 -> xyz=0 -10.5 2.427574999409978 rpy=0 0 0
- joint Torso_FrontLeg: origin xyz=0 -17.5 2.3575543320552637 rpy=0 0 0 -> xyz=0 -9.5 2.427574999409978 rpy=0 0 0
- joint Torso_LeftLeg: origin xyz=-0.5 -18 2.3575543320552637 rpy=0 0 0 -> xyz=-0.5 -10 2.427574999409978 rpy=0 0 0
- joint Torso_RightLeg: origin xyz=0.5 -18 2.3575543320552637 rpy=0 0 0 -> xyz=0.5 -10 2.427574999409978 rpy=0 0 0

File: bodyFiles/body0-141.urdf (robot description, URDF)
Before this commit: robot robot, 9 links, 8 joints
Links:
- link BackLeg: geometry collision box size=0.2 0.6459125070882793 0.2; visual box size=0.2 0.6459125070882793 0.2
- link BackLowerLeg: geometry collision box size=0.2 0.2 1.2674808844029135; visual box size=0.2 0.2 1.2674808844029135
- link FrontLeg: geometry collision box size=0.2 0.6572399406676798 0.2; visual box size=0.2 0.6572399406676798 0.2
- link FrontLowerLeg: geometry collision box size=0.2 0.2 1.4060061051774984; visual box size=0.2 0.2 1.4060061051774984
- link LeftLeg: geometry collision box size=0.6081438268490993 0.2 0.2; visual box size=0.6081438268490993 0.2 0.2
- link LeftLowerLeg: geometry collision box size=0.2 0.2 0.9220170100692511; visual box size=0.2 0.2 0.9220170100692511
- link RightLeg: geometry collision box size=1.446222544633161 0.2 0.2; visual box size=1.446222544633161 0.2 0.2
- link RightLowerLeg: geometry collision box size=0.2 0.2 1.2774494564463654; visual box size=0.2 0.2 1.2774494564463654
Joints:
- joint BackLeg_BackLowerLeg: origin xyz=0 -0.795703603921058 0 rpy=0 0 0 -> xyz=0 -0.6459125070882793 0 rpy=0 0 0
- joint FrontLeg_FrontLowerLeg: origin xyz=0 1.1375484563006857 0 rpy=0 0 0 -> xyz=0 0.6572399406676798 0 rpy=0 0 0
- joint LeftLeg_LeftLowerLeg: origin xyz=-1.3575543320552639 0 0 rpy=0 0 0 -> xyz=-0.6081438268490993 0 0 rpy=0 0 0
- joint RightLeg_RightLowerLeg: origin xyz=0.5780501537387961 0 0 rpy=0 0 0 -> xyz=1.446222544633161 0 0 rpy=0 0 0
- joint Torso_BackLeg: origin xyz=0 -18.5 2.3575543320552637 rpy=0 0 0 -> xyz=0 -14.5 2.446222544633161 rpy=0 0 0
- joint Torso_FrontLeg: origin xyz=0 -17.5 2.3575543320552637 rpy=0 0 0 -> xyz=0 -13.5 2.446222544633161 rpy=0 0 0
- joint Torso_LeftLeg: origin xyz=-0.5 -18 2.3575543320552637 rpy=0 0 0 -> xyz=-0.5 -14 2.446222544633161 rpy=0 0 0
- joint Torso_RightLeg: origin xyz=0.5 -18 2.3575543320552637 rpy=0 0 0 -> xyz=0.5 -14 2.446222544633161 rpy=0 0 0

File: bodyFiles/body0-184.urdf (robot description, URDF)
Before this commit: robot robot, 9 links, 8 joints
Links:
- link FrontLeg: geometry collision box size=0.2 1.118866894473543 0.2; visual box size=0.2 1.118866894473543 0.2
Joints:
- joint FrontLeg_FrontLowerLeg: origin xyz=0 1.1375484563006857 0 rpy=0 0 0 -> xyz=0 1.118866894473543 0 rpy=0 0 0

File: bodyFiles/body0-67.urdf (robot description, URDF)
Before this commit: robot robot, 9 links, 8 joints
Links:
- link BackLeg: geometry collision box size=0.2 1.470900003764732 0.2; visual box size=0.2 1.470900003764732 0.2
- link BackLowerLeg: geometry collision box size=0.2 0.2 0.7209107242382446; visual box size=0.2 0.2 0.7209107242382446
- link FrontLeg: geometry collision box size=0.2 0.7987276419257794 0.2; visual box size=0.2 0.7987276419257794 0.2
- link FrontLowerLeg: geometry collision box size=0.2 0.2 0.7809903290141487; visual box size=0.2 0.2 0.7809903290141487
- link LeftLeg: geometry collision box size=0.8854507979794787 0.2 0.2; visual box size=0.8854507979794787 0.2 0.2
- link LeftLowerLeg: geometry collision box size=0.2 0.2 0.8560577654859315; visual box size=0.2 0.2 0.8560577654859315
- link RightLeg: geometry collision box size=0.7528540498054029 0.2 0.2; visual box size=0.7528540498054029 0.2 0.2
- link RightLowerLeg: geometry collision box size=0.2 0.2 0.8912302161408768; visual box size=0.2 0.2 0.8912302161408768
Joints:
- joint BackLeg_BackLowerLeg: origin xyz=0 -0.795703603921058 0 rpy=0 0 0 -> xyz=0 -1.470900003764732 0 rpy=0 0 0
- joint FrontLeg_FrontLowerLeg: origin xyz=0 1.1375484563006857 0 rpy=0 0 0 -> xyz=0 0.7987276419257794 0 rpy=0 0 0
- joint LeftLeg_LeftLowerLeg: origin xyz=-1.3575543320552639 0 0 rpy=0 0 0 -> xyz=-0.8854507979794787 0 0 rpy=0 0 0
- joint RightLeg_RightLowerLeg: origin xyz=0.5780501537387961 0 0 rpy=0 0 0 -> xyz=0.7528540498054029 0 0 rpy=0 0 0
- joint Torso_BackLeg: origin xyz=0 -18.5 2.3575543320552637 rpy=0 0 0 -> xyz=0 -6.5 2.470900003764732 rpy=0 0 0
- joint Torso_FrontLeg: origin xyz=0 -17.5 2.3575543320552637 rpy=0 0 0 -> xyz=0 -5.5 2.470900003764732 rpy=0 0 0
- joint Torso_LeftLeg: origin xyz=-0.5 -18 2.3575543320552637 rpy=0 0 0 -> xyz=-0.5 -6 2.470900003764732 rpy=0 0 0
- joint Torso_RightLeg: origin xyz=0.5 -18 2.3575543320552637 rpy=0 0 0 -> xyz=0.5 -6 2.470900003764732 rpy=0 0 0
