Commit message: merged and squashed case3_evolved into case3_ev (which is supposed to become case3_random)

File: bodyFiles/body0-1012.urdf (robot description, URDF)
Before this commit: robot robot, 9 links, 8 joints
Links:
- link BackLeg: geometry collision box size=0.2 0.5211604762115561 0.2; visual box size=0.2 0.5211604762115561 0.2
- link BackLowerLeg: geometry collision box size=0.2 0.2 1.0531570755874742; visual box size=0.2 0.2 1.0531570755874742
- link FrontLeg: geometry collision box size=0.2 0.7186294586990568 0.2; visual box size=0.2 0.7186294586990568 0.2
- link FrontLowerLeg: geometry collision box size=0.2 0.2 0.821621682569965; visual box size=0.2 0.2 0.821621682569965
- link LeftLeg: geometry collision box size=1.149241835706703 0.2 0.2; visual box size=1.149241835706703 0.2 0.2
- link LeftLowerLeg: geometry collision box size=0.2 0.2 0.6586573672315357; visual box size=0.2 0.2 0.6586573672315357
- link RightLeg: geometry collision box size=0.5964605064125298 0.2 0.2; visual box size=0.5964605064125298 0.2 0.2
- link RightLowerLeg: geometry collision box size=0.2 0.2 1.4470909662059057; visual box size=0.2 0.2 1.4470909662059057
Joints:
- joint BackLeg_BackLowerLeg: origin xyz=0 -1.4397175348477087 0 rpy=0 0 0 -> xyz=0 -0.5211604762115561 0 rpy=0 0 0
- joint FrontLeg_FrontLowerLeg: origin xyz=0 1.4653217275796484 0 rpy=0 0 0 -> xyz=0 0.7186294586990568 0 rpy=0 0 0
- joint LeftLeg_LeftLowerLeg: origin xyz=-0.8972519159770695 0 0 rpy=0 0 0 -> xyz=-1.149241835706703 0 0 rpy=0 0 0
- joint RightLeg_RightLowerLeg: origin xyz=1.0660979765455858 0 0 rpy=0 0 0 -> xyz=0.5964605064125298 0 0 rpy=0 0 0
- joint Torso_BackLeg: origin xyz=0 -10.5 2.4653217275796484 rpy=0 0 0 -> xyz=0 -10.5 2.4470909662059057 rpy=0 0 0
- joint Torso_FrontLeg: origin xyz=0 -9.5 2.4653217275796484 rpy=0 0 0 -> xyz=0 -9.5 2.4470909662059057 rpy=0 0 0
- joint Torso_LeftLeg: origin xyz=-0.5 -10 2.4653217275796484 rpy=0 0 0 -> xyz=-0.5 -10 2.4470909662059057 rpy=0 0 0
- joint Torso_RightLeg: origin xyz=0.5 -10 2.4653217275796484 rpy=0 0 0 -> xyz=0.5 -10 2.4470909662059057 rpy=0 0 0

File: bodyFiles/body0-10532.urdf (robot description, URDF)
Before this commit: robot robot, 9 links, 8 joints
Links:
- link BackLeg: geometry collision box size=0.2 1.0313918992716782 0.2; visual box size=0.2 1.0313918992716782 0.2
- link BackLowerLeg: geometry collision box size=0.2 0.2 1.3867676704528455; visual box size=0.2 0.2 1.3867676704528455
- link FrontLeg: geometry collision box size=0.2 0.7761146523712571 0.2; visual box size=0.2 0.7761146523712571 0.2
- link FrontLowerLeg: geometry collision box size=0.2 0.2 1.2718307043054677; visual box size=0.2 0.2 1.2718307043054677
- link LeftLeg: geometry collision box size=1.0664624824195315 0.2 0.2; visual box size=1.0664624824195315 0.2 0.2
- link LeftLowerLeg: geometry collision box size=0.2 0.2 1.2628202510733422; visual box size=0.2 0.2 1.2628202510733422
- link RightLeg: geometry collision box size=1.0142348518451016 0.2 0.2; visual box size=1.0142348518451016 0.2 0.2
- link RightLowerLeg: geometry collision box size=0.2 0.2 1.448035366509675; visual box size=0.2 0.2 1.448035366509675
Joints:
- joint BackLeg_BackLowerLeg: origin xyz=0 -1.3799436598693542 0 rpy=0 0 0 -> xyz=0 -1.0313918992716782 0 rpy=0 0 0
- joint FrontLeg_FrontLowerLeg: origin xyz=0 0.7527127226556776 0 rpy=0 0 0 -> xyz=0 0.7761146523712571 0 rpy=0 0 0
- joint LeftLeg_LeftLowerLeg: origin xyz=-0.7518728600638734 0 0 rpy=0 0 0 -> xyz=-1.0664624824195315 0 0 rpy=0 0 0
- joint RightLeg_RightLowerLeg: origin xyz=1.2310589010482391 0 0 rpy=0 0 0 -> xyz=1.0142348518451016 0 0 rpy=0 0 0
- joint Torso_BackLeg: origin xyz=0 -10.5 2.379943659869354 rpy=0 0 0 -> xyz=0 -10.5 2.448035366509675 rpy=0 0 0
- joint Torso_FrontLeg: origin xyz=0 -9.5 2.379943659869354 rpy=0 0 0 -> xyz=0 -9.5 2.448035366509675 rpy=0 0 0
- joint Torso_LeftLeg: origin xyz=-0.5 -10 2.379943659869354 rpy=0 0 0 -> xyz=-0.5 -10 2.448035366509675 rpy=0 0 0
- joint Torso_RightLeg: origin xyz=0.5 -10 2.379943659869354 rpy=0 0 0 -> xyz=0.5 -10 2.448035366509675 rpy=0 0 0

File: bodyFiles/body0-10642.urdf (robot description, URDF)
Before this commit: robot robot, 9 links, 8 joints
Links:
- link BackLeg: geometry collision box size=0.2 0.8579575214904757 0.2; visual box size=0.2 0.8579575214904757 0.2
- link BackLowerLeg: geometry collision box size=0.2 0.2 0.8216647691256634; visual box size=0.2 0.2 0.8216647691256634
- link FrontLeg: geometry collision box size=0.2 0.8765702169552689 0.2; visual box size=0.2 0.8765702169552689 0.2
- link FrontLowerLeg: geometry collision box size=0.2 0.2 1.260376701567805; visual box size=0.2 0.2 1.260376701567805
- link LeftLeg: geometry collision box size=1.2715606262648378 0.2 0.2; visual box size=1.2715606262648378 0.2 0.2
- link LeftLowerLeg: geometry collision box size=0.2 0.2 1.1936056359199168; visual box size=0.2 0.2 1.1936056359199168
- link RightLeg: geometry collision box size=0.5848937866194583 0.2 0.2; visual box size=0.5848937866194583 0.2 0.2
- link RightLowerLeg: geometry collision box size=0.2 0.2 1.4622677625082332; visual box size=0.2 0.2 1.4622677625082332
Joints:
- joint BackLeg_BackLowerLeg: origin xyz=0 -0.9076176582006167 0 rpy=0 0 0 -> xyz=0 -0.8579575214904757 0 rpy=0 0 0
- joint FrontLeg_FrontLowerLeg: origin xyz=0 0.9099539715874841 0 rpy=0 0 0 -> xyz=0 0.8765702169552689 0 rpy=0 0 0
- joint LeftLeg_LeftLowerLeg: origin xyz=-1.455444051021439 0 0 rpy=0 0 0 -> xyz=-1.2715606262648378 0 0 rpy=0 0 0
- joint RightLeg_RightLowerLeg: origin xyz=0.6560458555626477 0 0 rpy=0 0 0 -> xyz=0.5848937866194583 0 0 rpy=0 0 0
- joint Torso_BackLeg: origin xyz=0 -10.5 2.495693707315572 rpy=0 0 0 -> xyz=0 -10.5 2.462267762508233 rpy=0 0 0
- joint Torso_FrontLeg: origin xyz=0 -9.5 2.495693707315572 rpy=0 0 0 -> xyz=0 -9.5 2.462267762508233 rpy=0 0 0
- joint Torso_LeftLeg: origin xyz=-0.5 -10 2.495693707315572 rpy=0 0 0 -> xyz=-0.5 -10 2.462267762508233 rpy=0 0 0
- joint Torso_RightLeg: origin xyz=0.5 -10 2.495693707315572 rpy=0 0 0 -> xyz=0.5 -10 2.462267762508233 rpy=0 0 0

File: bodyFiles/body0-10692.urdf (robot description, URDF)
Before this commit: robot robot, 9 links, 8 joints
Links:
- link BackLeg: geometry collision box size=0.2 0.660046028348746 0.2; visual box size=0.2 0.660046028348746 0.2
- link BackLowerLeg: geometry collision box size=0.2 0.2 0.5737979061914285; visual box size=0.2 0.2 0.5737979061914285
- link FrontLeg: geometry collision box size=0.2 1.0149170585304728 0.2; visual box size=0.2 1.0149170585304728 0.2
- link FrontLowerLeg: geometry collision box size=0.2 0.2 0.8450214092830298; visual box size=0.2 0.2 0.8450214092830298
- link LeftLeg: geometry collision box size=0.8034617801471663 0.2 0.2; visual box size=0.8034617801471663 0.2 0.2
- link LeftLowerLeg: geometry collision box size=0.2 0.2 1.2213837501659346; visual box size=0.2 0.2 1.2213837501659346
- link RightLeg: geometry collision box size=1.2554648635354746 0.2 0.2; visual box size=1.2554648635354746 0.2 0.2
- link RightLowerLeg: geometry collision box size=0.2 0.2 1.0418806643338494; visual box size=0.2 0.2 1.0418806643338494
Joints:
- joint BackLeg_BackLowerLeg: origin xyz=0 -0.6005223191780467 0 rpy=0 0 0 -> xyz=0 -0.660046028348746 0 rpy=0 0 0
- joint FrontLeg_FrontLowerLeg: origin xyz=0 1.4139441589541153 0 rpy=0 0 0 -> xyz=0 1.0149170585304728 0 rpy=0 0 0
- joint LeftLeg_LeftLowerLeg: origin xyz=-1.4772856639166743 0 0 rpy=0 0 0 -> xyz=-0.8034617801471663 0 0 rpy=0 0 0
- joint RightLeg_RightLowerLeg: origin xyz=1.0328997249961098 0 0 rpy=0 0 0 -> xyz=1.2554648635354746 0 0 rpy=0 0 0
- joint Torso_BackLeg: origin xyz=0 -10.5 2.4772856639166743 rpy=0 0 0 -> xyz=0 -10.5 2.2554648635354746 rpy=0 0 0
- joint Torso_FrontLeg: origin xyz=0 -9.5 2.4772856639166743 rpy=0 0 0 -> xyz=0 -9.5 2.2554648635354746 rpy=0 0 0
- joint Torso_LeftLeg: origin xyz=-0.5 -10 2.4772856639166743 rpy=0 0 0 -> xyz=-0.5 -10 2.2554648635354746 rpy=0 0 0
- joint Torso_RightLeg: origin xyz=0.5 -10 2.4772856639166743 rpy=0 0 0 -> xyz=0.5 -10 2.2554648635354746 rpy=0 0 0

File: bodyFiles/body0-1072.urdf (robot description, URDF)
Before this commit: robot robot, 9 links, 8 joints
Links:
- link BackLeg: geometry collision box size=0.2 0.8110738569355737 0.2; visual box size=0.2 0.8110738569355737 0.2
- link BackLowerLeg: geometry collision box size=0.2 0.2 1.320124641931479; visual box size=0.2 0.2 1.320124641931479
- link FrontLeg: geometry collision box size=0.2 1.0501005398938945 0.2; visual box size=0.2 1.0501005398938945 0.2
- link FrontLowerLeg: geometry collision box size=0.2 0.2 1.4728372311495657; visual box size=0.2 0.2 1.4728372311495657
- link LeftLeg: geometry collision box size=0.6053989318212719 0.2 0.2; visual box size=0.6053989318212719 0.2 0.2
- link LeftLowerLeg: geometry collision box size=0.2 0.2 1.4210917428119976; visual box size=0.2 0.2 1.4210917428119976
- link RightLeg: geometry collision box size=1.3025893237328048 0.2 0.2; visual box size=1.3025893237328048 0.2 0.2
- link RightLowerLeg: geometry collision box size=0.2 0.2 1.3427853767534144; visual box size=0.2 0.2 1.3427853767534144
Joints:
- joint BackLeg_BackLowerLeg: origin xyz=0 -1.4238659350315759 0 rpy=0 0 0 -> xyz=0 -0.8110738569355737 0 rpy=0 0 0
- joint FrontLeg_FrontLowerLeg: origin xyz=0 0.8917251258496538 0 rpy=0 0 0 -> xyz=0 1.0501005398938945 0 rpy=0 0 0
- joint LeftLeg_LeftLowerLeg: origin xyz=-0.993458828553044 0 0 rpy=0 0 0 -> xyz=-0.6053989318212719 0 0 rpy=0 0 0
- joint RightLeg_RightLowerLeg: origin xyz=1.378512496146957 0 0 rpy=0 0 0 -> xyz=1.3025893237328048 0 0 rpy=0 0 0
- joint Torso_BackLeg: origin xyz=0 -10.5 2.423865935031576 rpy=0 0 0 -> xyz=0 -10.5 2.4728372311495654 rpy=0 0 0
- joint Torso_FrontLeg: origin xyz=0 -9.5 2.423865935031576 rpy=0 0 0 -> xyz=0 -9.5 2.4728372311495654 rpy=0 0 0
- joint Torso_LeftLeg: origin xyz=-0.5 -10 2.423865935031576 rpy=0 0 0 -> xyz=-0.5 -10 2.4728372311495654 rpy=0 0 0
- joint Torso_RightLeg: origin xyz=0.5 -10 2.423865935031576 rpy=0 0 0 -> xyz=0.5 -10 2.4728372311495654 rpy=0 0 0

File: bodyFiles/body0-14121.urdf (robot description, URDF)
Before this commit: robot robot, 9 links, 8 joints
Links:
- link BackLeg: geometry collision box size=0.2 0.9931024636824476 0.2; visual box size=0.2 0.9931024636824476 0.2
- link BackLowerLeg: geometry collision box size=0.2 0.2 0.7595307799767398; visual box size=0.2 0.2 0.7595307799767398
- link FrontLeg: geometry collision box size=0.2 1.2145972728683203 0.2; visual box size=0.2 1.2145972728683203 0.2
- link FrontLowerLeg: geometry collision box size=0.2 0.2 1.123672779680599; visual box size=0.2 0.2 1.123672779680599
- link LeftLeg: geometry collision box size=0.9113605189694807 0.2 0.2; visual box size=0.9113605189694807 0.2 0.2
- link LeftLowerLeg: geometry collision box size=0.2 0.2 1.3316137941754234; visual box size=0.2 0.2 1.3316137941754234
- link RightLeg: geometry collision box size=1.2048031813467723 0.2 0.2; visual box size=1.2048031813467723 0.2 0.2
- link RightLowerLeg: geometry collision box size=0.2 0.2 0.803930491742317; visual box size=0.2 0.2 0.803930491742317
Joints:
- joint BackLeg_BackLowerLeg: origin xyz=0 -0.9614048746483048 0 rpy=0 0 0 -> xyz=0 -0.9931024636824476 0 rpy=0 0 0
- joint FrontLeg_FrontLowerLeg: origin xyz=0 1.2180726066434828 0 rpy=0 0 0 -> xyz=0 1.2145972728683203 0 rpy=0 0 0
- joint LeftLeg_LeftLowerLeg: origin xyz=-1.0783437291038556 0 0 rpy=0 0 0 -> xyz=-0.9113605189694807 0 0 rpy=0 0 0
- joint RightLeg_RightLowerLeg: origin xyz=1.4618093856012848 0 0 rpy=0 0 0 -> xyz=1.2048031813467723 0 0 rpy=0 0 0
- joint Torso_BackLeg: origin xyz=0 -14.5 2.467878190590163 rpy=0 0 0 -> xyz=0 -14.5 2.331613794175423 rpy=0 0 0
- joint Torso_FrontLeg: origin xyz=0 -13.5 2.467878190590163 rpy=0 0 0 -> xyz=0 -13.5 2.331613794175423 rpy=0 0 0
- joint Torso_LeftLeg: origin xyz=-0.5 -14 2.467878190590163 rpy=0 0 0 -> xyz=-0.5 -14 2.331613794175423 rpy=0 0 0
- joint Torso_RightLeg: origin xyz=0.5 -14 2.467878190590163 rpy=0 0 0 -> xyz=0.5 -14 2.331613794175423 rpy=0 0 0

File: bodyFiles/body0-14171.urdf (robot description, URDF)
Before this commit: robot robot, 9 links, 8 joints
Links:
- link BackLeg: geometry collision box size=0.2 0.7188865916559471 0.2; visual box size=0.2 0.7188865916559471 0.2
- link BackLowerLeg: geometry collision box size=0.2 0.2 0.6501647069467384; visual box size=0.2 0.2 0.6501647069467384
- link FrontLeg: geometry collision box size=0.2 0.5818023036998935 0.2; visual box size=0.2 0.5818023036998935 0.2
- link FrontLowerLeg: geometry collision box size=0.2 0.2 0.8794407066689257; visual box size=0.2 0.2 0.8794407066689257
- link LeftLeg: geometry collision box size=0.7343021727131351 0.2 0.2; visual box size=0.7343021727131351 0.2 0.2
- link LeftLowerLeg: geometry collision box size=0.2 0.2 0.8601997918957307; visual box size=0.2 0.2 0.8601997918957307
- link RightLeg: geometry collision box size=0.6428421351829458 0.2 0.2; visual box size=0.6428421351829458 0.2 0.2
- link RightLowerLeg: geometry collision box size=0.2 0.2 1.344901986946851; visual box size=0.2 0.2 1.344901986946851
Joints:
- joint BackLeg_BackLowerLeg: origin xyz=0 -0.9927078752235314 0 rpy=0 0 0 -> xyz=0 -0.7188865916559471 0 rpy=0 0 0
- joint FrontLeg_FrontLowerLeg: origin xyz=0 1.3583533353109392 0 rpy=0 0 0 -> xyz=0 0.5818023036998935 0 rpy=0 0 0
- joint LeftLeg_LeftLowerLeg: origin xyz=-0.6391329876710066 0 0 rpy=0 0 0 -> xyz=-0.7343021727131351 0 0 rpy=0 0 0
- joint RightLeg_RightLowerLeg: origin xyz=0.850469261282797 0 0 rpy=0 0 0 -> xyz=0.6428421351829458 0 0 rpy=0 0 0
- joint Torso_BackLeg: origin xyz=0 -14.5 2.493292842547225 rpy=0 0 0 -> xyz=0 -14.5 2.344901986946851 rpy=0 0 0
- joint Torso_FrontLeg: origin xyz=0 -13.5 2.493292842547225 rpy=0 0 0 -> xyz=0 -13.5 2.344901986946851 rpy=0 0 0
- joint Torso_LeftLeg: origin xyz=-0.5 -14 2.493292842547225 rpy=0 0 0 -> xyz=-0.5 -14 2.344901986946851 rpy=0 0 0
- joint Torso_RightLeg: origin xyz=0.5 -14 2.493292842547225 rpy=0 0 0 -> xyz=0.5 -14 2.344901986946851 rpy=0 0 0

File: bodyFiles/body0-14221.urdf (robot description, URDF)
Before this commit: robot robot, 9 links, 8 joints
Links:
- link BackLeg: geometry collision box size=0.2 0.7862080721636425 0.2; visual box size=0.2 0.7862080721636425 0.2
- link BackLowerLeg: geometry collision box size=0.2 0.2 1.4884704257525831; visual box size=0.2 0.2 1.4884704257525831
- link FrontLeg: geometry collision box size=0.2 0.9186741075536171 0.2; visual box size=0.2 0.9186741075536171 0.2
- link FrontLowerLeg: geometry collision box size=0.2 0.2 0.6144233817102301; visual box size=0.2 0.2 0.6144233817102301
- link LeftLeg: geometry collision box size=1.493351461273596 0.2 0.2; visual box size=1.493351461273596 0.2 0.2
- link LeftLowerLeg: geometry collision box size=0.2 0.2 0.6038523089253823; visual box size=0.2 0.2 0.6038523089253823
- link RightLeg: geometry collision box size=1.4252253305969425 0.2 0.2; visual box size=1.4252253305969425 0.2 0.2
- link RightLowerLeg: geometry collision box size=0.2 0.2 1.4729842325239024; visual box size=0.2 0.2 1.4729842325239024
Joints:
- joint BackLeg_BackLowerLeg: origin xyz=0 -0.7288750848284242 0 rpy=0 0 0 -> xyz=0 -0.7862080721636425 0 rpy=0 0 0
- joint FrontLeg_FrontLowerLeg: origin xyz=0 0.7523493098211362 0 rpy=0 0 0 -> xyz=0 0.9186741075536171 0 rpy=0 0 0
- joint LeftLeg_LeftLowerLeg: origin xyz=-1.4051516105707045 0 0 rpy=0 0 0 -> xyz=-1.493351461273596 0 0 rpy=0 0 0
- joint RightLeg_RightLowerLeg: origin xyz=0.972300861393799 0 0 rpy=0 0 0 -> xyz=1.4252253305969425 0 0 rpy=0 0 0
- joint Torso_BackLeg: origin xyz=0 -14.5 2.4051516105707043 rpy=0 0 0 -> xyz=0 -14.5 2.493351461273596 rpy=0 0 0
- joint Torso_FrontLeg: origin xyz=0 -13.5 2.4051516105707043 rpy=0 0 0 -> xyz=0 -13.5 2.493351461273596 rpy=0 0 0
- joint Torso_LeftLeg: origin xyz=-0.5 -14 2.4051516105707043 rpy=0 0 0 -> xyz=-0.5 -14 2.493351461273596 rpy=0 0 0
- joint Torso_RightLeg: origin xyz=0.5 -14 2.4051516105707043 rpy=0 0 0 -> xyz=0.5 -14 2.493351461273596 rpy=0 0 0

File: bodyFiles/body0-14271.urdf (robot description, URDF)
Before this commit: robot robot, 9 links, 8 joints
Links:
- link BackLeg: geometry collision box size=0.2 0.652344904053455 0.2; visual box size=0.2 0.652344904053455 0.2
- link BackLowerLeg: geometry collision box size=0.2 0.2 0.6136296558346088; visual box size=0.2 0.2 0.6136296558346088
- link FrontLeg: geometry collision box size=0.2 0.6842841901934328 0.2; visual box size=0.2 0.6842841901934328 0.2
- link FrontLowerLeg: geometry collision box size=0.2 0.2 1.0480471376170977; visual box size=0.2 0.2 1.0480471376170977
- link LeftLeg: geometry collision box size=0.7345350215974369 0.2 0.2; visual box size=0.7345350215974369 0.2 0.2
- link LeftLowerLeg: geometry collision box size=0.2 0.2 1.062521959932298; visual box size=0.2 0.2 1.062521959932298
- link RightLeg: geometry collision box size=1.1043903493777765 0.2 0.2; visual box size=1.1043903493777765 0.2 0.2
- link RightLowerLeg: geometry collision box size=0.2 0.2 0.5639468586491215; visual box size=0.2 0.2 0.5639468586491215
Joints:
- joint BackLeg_BackLowerLeg: origin xyz=0 -1.013142405906317 0 rpy=0 0 0 -> xyz=0 -0.652344904053455 0 rpy=0 0 0
- joint FrontLeg_FrontLowerLeg: origin xyz=0 0.9481473629820171 0 rpy=0 0 0 -> xyz=0 0.6842841901934328 0 rpy=0 0 0
- joint LeftLeg_LeftLowerLeg: origin xyz=-1.2661206145556674 0 0 rpy=0 0 0 -> xyz=-0.7345350215974369 0 0 rpy=0 0 0
- joint RightLeg_RightLowerLeg: origin xyz=0.5908007815415862 0 0 rpy=0 0 0 -> xyz=1.1043903493777765 0 0 rpy=0 0 0
- joint Torso_BackLeg: origin xyz=0 -14.5 2.2661206145556676 rpy=0 0 0 -> xyz=0 -14.5 2.1043903493777765 rpy=0 0 0
- joint Torso_FrontLeg: origin xyz=0 -13.5 2.2661206145556676 rpy=0 0 0 -> xyz=0 -13.5 2.1043903493777765 rpy=0 0 0
- joint Torso_LeftLeg: origin xyz=-0.5 -14 2.2661206145556676 rpy=0 0 0 -> xyz=-0.5 -14 2.1043903493777765 rpy=0 0 0
- joint Torso_RightLeg: origin xyz=0.5 -14 2.2661206145556676 rpy=0 0 0 -> xyz=0.5 -14 2.1043903493777765 rpy=0 0 0

File: bodyFiles/body0-14321.urdf (robot description, URDF)
Before this commit: robot robot, 9 links, 8 joints
Links:
- link BackLeg: geometry collision box size=0.2 1.4575323398559819 0.2; visual box size=0.2 1.4575323398559819 0.2
- link BackLowerLeg: geometry collision box size=0.2 0.2 1.0117062914238786; visual box size=0.2 0.2 1.0117062914238786
- link FrontLeg: geometry collision box size=0.2 1.2988235486818733 0.2; visual box size=0.2 1.2988235486818733 0.2
- link FrontLowerLeg: geometry collision box size=0.2 0.2 0.7140451846859399; visual box size=0.2 0.2 0.7140451846859399
- link LeftLeg: geometry collision box size=0.6064807096139438 0.2 0.2; visual box size=0.6064807096139438 0.2 0.2
- link LeftLowerLeg: geometry collision box size=0.2 0.2 0.5777350676035573; visual box size=0.2 0.2 0.5777350676035573
- link RightLeg: geometry collision box size=0.6914962503509424 0.2 0.2; visual box size=0.6914962503509424 0.2 0.2
- link RightLowerLeg: geometry collision box size=0.2 0.2 1.367693367433392; visual box size=0.2 0.2 1.367693367433392
Joints:
- joint BackLeg_BackLowerLeg: origin xyz=0 -0.6206113843317199 0 rpy=0 0 0 -> xyz=0 -1.4575323398559819 0 rpy=0 0 0
- joint FrontLeg_FrontLowerLeg: origin xyz=0 1.0682182403897462 0 rpy=0 0 0 -> xyz=0 1.2988235486818733 0 rpy=0 0 0
- joint LeftLeg_LeftLowerLeg: origin xyz=-0.5283464418613886 0 0 rpy=0 0 0 -> xyz=-0.6064807096139438 0 0 rpy=0 0 0
- joint RightLeg_RightLowerLeg: origin xyz=0.9572964137176622 0 0 rpy=0 0 0 -> xyz=0.6914962503509424 0 0 rpy=0 0 0
- joint Torso_BackLeg: origin xyz=0 -14.5 2.3623229181835868 rpy=0 0 0 -> xyz=0 -14.5 2.457532339855982 rpy=0 0 0
- joint Torso_FrontLeg: origin xyz=0 -13.5 2.3623229181835868 rpy=0 0 0 -> xyz=0 -13.5 2.457532339855982 rpy=0 0 0
- joint Torso_LeftLeg: origin xyz=-0.5 -14 2.3623229181835868 rpy=0 0 0 -> xyz=-0.5 -14 2.457532339855982 rpy=0 0 0
- joint Torso_RightLeg: origin xyz=0.5 -14 2.3623229181835868 rpy=0 0 0 -> xyz=0.5 -14 2.457532339855982 rpy=0 0 0

File: bodyFiles/body0-14371.urdf (robot description, URDF)
Before this commit: robot robot, 9 links, 8 joints
Links:
- link BackLeg: geometry collision box size=0.2 1.0980398737823227 0.2; visual box size=0.2 1.0980398737823227 0.2
- link BackLowerLeg: geometry collision box size=0.2 0.2 0.5909569850689194; visual box size=0.2 0.2 0.5909569850689194
- link FrontLeg: geometry collision box size=0.2 1.4028027586663345 0.2; visual box size=0.2 1.4028027586663345 0.2
- link FrontLowerLeg: geometry collision box size=0.2 0.2 1.1281848745811267; visual box size=0.2 0.2 1.1281848745811267
- link LeftLeg: geometry collision box size=1.4949732538946088 0.2 0.2; visual box size=1.4949732538946088 0.2 0.2
- link LeftLowerLeg: geometry collision box size=0.2 0.2 1.3196680038869657; visual box size=0.2 0.2 1.3196680038869657
- link RightLeg: geometry collision box size=1.4483525739106313 0.2 0.2; visual box size=1.4483525739106313 0.2 0.2
- link RightLowerLeg: geometry collision box size=0.2 0.2 0.755013981094839; visual box size=0.2 0.2 0.755013981094839
Joints:
- joint BackLeg_BackLowerLeg: origin xyz=0 -0.7195034559358191 0 rpy=0 0 0 -> xyz=0 -1.0980398737823227 0 rpy=0 0 0
- joint FrontLeg_FrontLowerLeg: origin xyz=0 0.6157298636668674 0 rpy=0 0 0 -> xyz=0 1.4028027586663345 0 rpy=0 0 0
- joint LeftLeg_LeftLowerLeg: origin xyz=-1.3049102615467532 0 0 rpy=0 0 0 -> xyz=-1.4949732538946088 0 0 rpy=0 0 0
- joint RightLeg_RightLowerLeg: origin xyz=1.1300749551989453 0 0 rpy=0 0 0 -> xyz=1.4483525739106313 0 0 rpy=0 0 0
- joint Torso_BackLeg: origin xyz=0 -14.5 2.3414391077423495 rpy=0 0 0 -> xyz=0 -14.5 2.4949732538946088 rpy=0 0 0
- joint Torso_FrontLeg: origin xyz=0 -13.5 2.3414391077423495 rpy=0 0 0 -> xyz=0 -13.5 2.4949732538946088 rpy=0 0 0
- joint Torso_LeftLeg: origin xyz=-0.5 -14 2.3414391077423495 rpy=0 0 0 -> xyz=-0.5 -14 2.4949732538946088 rpy=0 0 0
- joint Torso_RightLeg: origin xyz=0.5 -14 2.3414391077423495 rpy=0 0 0 -> xyz=0.5 -14 2.4949732538946088 rpy=0 0 0
