Commit message: merged and squashed case3_evolved into case3_ev (which is supposed to become case3_random)

File: bodyFiles/body0-14421.urdf (robot description, URDF)
Before this commit: robot robot, 9 links, 8 joints
Links:
- link BackLeg: geometry collision box size=0.2 0.8188954207864741 0.2; visual box size=0.2 0.8188954207864741 0.2
- link BackLowerLeg: geometry collision box size=0.2 0.2 0.6300191081847459; visual box size=0.2 0.2 0.6300191081847459
- link FrontLeg: geometry collision box size=0.2 0.885909684476771 0.2; visual box size=0.2 0.885909684476771 0.2
- link FrontLowerLeg: geometry collision box size=0.2 0.2 0.5186753117552941; visual box size=0.2 0.2 0.5186753117552941
- link LeftLeg: geometry collision box size=1.1696067332464164 0.2 0.2; visual box size=1.1696067332464164 0.2 0.2
- link LeftLowerLeg: geometry collision box size=0.2 0.2 1.425820433870876; visual box size=0.2 0.2 1.425820433870876
- link RightLeg: geometry collision box size=1.1143757421214104 0.2 0.2; visual box size=1.1143757421214104 0.2 0.2
- link RightLowerLeg: geometry collision box size=0.2 0.2 0.8706936995080363; visual box size=0.2 0.2 0.8706936995080363
Joints:
- joint BackLeg_BackLowerLeg: origin xyz=0 -1.3934642014872471 0 rpy=0 0 0 -> xyz=0 -0.8188954207864741 0 rpy=0 0 0
- joint FrontLeg_FrontLowerLeg: origin xyz=0 0.9998651958882552 0 rpy=0 0 0 -> xyz=0 0.885909684476771 0 rpy=0 0 0
- joint LeftLeg_LeftLowerLeg: origin xyz=-1.4688249191888465 0 0 rpy=0 0 0 -> xyz=-1.1696067332464164 0 0 rpy=0 0 0
- joint RightLeg_RightLowerLeg: origin xyz=0.7011184192005129 0 0 rpy=0 0 0 -> xyz=1.1143757421214104 0 0 rpy=0 0 0
- joint Torso_BackLeg: origin xyz=0 -14.5 2.4688249191888465 rpy=0 0 0 -> xyz=0 -14.5 2.425820433870876 rpy=0 0 0
- joint Torso_FrontLeg: origin xyz=0 -13.5 2.4688249191888465 rpy=0 0 0 -> xyz=0 -13.5 2.425820433870876 rpy=0 0 0
- joint Torso_LeftLeg: origin xyz=-0.5 -14 2.4688249191888465 rpy=0 0 0 -> xyz=-0.5 -14 2.425820433870876 rpy=0 0 0
- joint Torso_RightLeg: origin xyz=0.5 -14 2.4688249191888465 rpy=0 0 0 -> xyz=0.5 -14 2.425820433870876 rpy=0 0 0

File: bodyFiles/body0-14471.urdf (robot description, URDF)
Before this commit: robot robot, 9 links, 8 joints
Links:
- link BackLeg: geometry collision box size=0.2 1.0650617074501816 0.2; visual box size=0.2 1.0650617074501816 0.2
- link BackLowerLeg: geometry collision box size=0.2 0.2 1.2417668747511863; visual box size=0.2 0.2 1.2417668747511863
- link FrontLeg: geometry collision box size=0.2 0.9585510460969066 0.2; visual box size=0.2 0.9585510460969066 0.2
- link FrontLowerLeg: geometry collision box size=0.2 0.2 1.0201573798717316; visual box size=0.2 0.2 1.0201573798717316
- link LeftLeg: geometry collision box size=0.7207335194897964 0.2 0.2; visual box size=0.7207335194897964 0.2 0.2
- link LeftLowerLeg: geometry collision box size=0.2 0.2 1.1371163842924985; visual box size=0.2 0.2 1.1371163842924985
- link RightLeg: geometry collision box size=1.2629024629367553 0.2 0.2; visual box size=1.2629024629367553 0.2 0.2
- link RightLowerLeg: geometry collision box size=0.2 0.2 1.204055681712986; visual box size=0.2 0.2 1.204055681712986
Joints:
- joint BackLeg_BackLowerLeg: origin xyz=0 -0.6859083277801145 0 rpy=0 0 0 -> xyz=0 -1.0650617074501816 0 rpy=0 0 0
- joint FrontLeg_FrontLowerLeg: origin xyz=0 0.651112690138383 0 rpy=0 0 0 -> xyz=0 0.9585510460969066 0 rpy=0 0 0
- joint LeftLeg_LeftLowerLeg: origin xyz=-0.9851988963914508 0 0 rpy=0 0 0 -> xyz=-0.7207335194897964 0 0 rpy=0 0 0
- joint RightLeg_RightLowerLeg: origin xyz=1.0247629918182866 0 0 rpy=0 0 0 -> xyz=1.2629024629367553 0 0 rpy=0 0 0
- joint Torso_BackLeg: origin xyz=0 -14.5 2.083558699527514 rpy=0 0 0 -> xyz=0 -14.5 2.262902462936755 rpy=0 0 0
- joint Torso_FrontLeg: origin xyz=0 -13.5 2.083558699527514 rpy=0 0 0 -> xyz=0 -13.5 2.262902462936755 rpy=0 0 0
- joint Torso_LeftLeg: origin xyz=-0.5 -14 2.083558699527514 rpy=0 0 0 -> xyz=-0.5 -14 2.262902462936755 rpy=0 0 0
- joint Torso_RightLeg: origin xyz=0.5 -14 2.083558699527514 rpy=0 0 0 -> xyz=0.5 -14 2.262902462936755 rpy=0 0 0

File: bodyFiles/body0-14581.urdf (robot description, URDF)
Before this commit: robot robot, 9 links, 8 joints
Links:
- link BackLeg: geometry collision box size=0.2 0.7471122312869726 0.2; visual box size=0.2 0.7471122312869726 0.2
- link BackLowerLeg: geometry collision box size=0.2 0.2 1.0901268933269903; visual box size=0.2 0.2 1.0901268933269903
- link FrontLeg: geometry collision box size=0.2 1.4662151618078418 0.2; visual box size=0.2 1.4662151618078418 0.2
- link FrontLowerLeg: geometry collision box size=0.2 0.2 1.2326641460838292; visual box size=0.2 0.2 1.2326641460838292
- link LeftLeg: geometry collision box size=1.417396359815199 0.2 0.2; visual box size=1.417396359815199 0.2 0.2
- link LeftLowerLeg: geometry collision box size=0.2 0.2 0.8667707511471525; visual box size=0.2 0.2 0.8667707511471525
- link RightLeg: geometry collision box size=1.4739953929240328 0.2 0.2; visual box size=1.4739953929240328 0.2 0.2
- link RightLowerLeg: geometry collision box size=0.2 0.2 1.2951122139771245; visual box size=0.2 0.2 1.2951122139771245
Joints:
- joint BackLeg_BackLowerLeg: origin xyz=0 -1.1640470691880238 0 rpy=0 0 0 -> xyz=0 -0.7471122312869726 0 rpy=0 0 0
- joint FrontLeg_FrontLowerLeg: origin xyz=0 0.5625862766779974 0 rpy=0 0 0 -> xyz=0 1.4662151618078418 0 rpy=0 0 0
- joint LeftLeg_LeftLowerLeg: origin xyz=-1.208546895389668 0 0 rpy=0 0 0 -> xyz=-1.417396359815199 0 0 rpy=0 0 0
- joint RightLeg_RightLowerLeg: origin xyz=0.9947954777478099 0 0 rpy=0 0 0 -> xyz=1.4739953929240328 0 0 rpy=0 0 0
- joint Torso_BackLeg: origin xyz=0 -14.5 2.3278274898647333 rpy=0 0 0 -> xyz=0 -14.5 2.473995392924033 rpy=0 0 0
- joint Torso_FrontLeg: origin xyz=0 -13.5 2.3278274898647333 rpy=0 0 0 -> xyz=0 -13.5 2.473995392924033 rpy=0 0 0
- joint Torso_LeftLeg: origin xyz=-0.5 -14 2.3278274898647333 rpy=0 0 0 -> xyz=-0.5 -14 2.473995392924033 rpy=0 0 0
- joint Torso_RightLeg: origin xyz=0.5 -14 2.3278274898647333 rpy=0 0 0 -> xyz=0.5 -14 2.473995392924033 rpy=0 0 0

File: bodyFiles/body0-180.urdf (robot description, URDF)
Before this commit: robot robot, 9 links, 8 joints
Links:
- link BackLeg: geometry collision box size=0.2 1.229704891864707 0.2; visual box size=0.2 1.229704891864707 0.2
- link BackLowerLeg: geometry collision box size=0.2 0.2 0.7015581758862168; visual box size=0.2 0.2 0.7015581758862168
- link FrontLeg: geometry collision box size=0.2 0.9073977077835352 0.2; visual box size=0.2 0.9073977077835352 0.2
- link FrontLowerLeg: geometry collision box size=0.2 0.2 0.6315527899220252; visual box size=0.2 0.2 0.6315527899220252
- link LeftLeg: geometry collision box size=0.8153412143409425 0.2 0.2; visual box size=0.8153412143409425 0.2 0.2
- link LeftLowerLeg: geometry collision box size=0.2 0.2 1.2426320729758753; visual box size=0.2 0.2 1.2426320729758753
- link RightLeg: geometry collision box size=1.4336779769690686 0.2 0.2; visual box size=1.4336779769690686 0.2 0.2
- link RightLowerLeg: geometry collision box size=0.2 0.2 1.1590494011860257; visual box size=0.2 0.2 1.1590494011860257
Joints:
- joint BackLeg_BackLowerLeg: origin xyz=0 -0.8597572027470005 0 rpy=0 0 0 -> xyz=0 -1.229704891864707 0 rpy=0 0 0
- joint FrontLeg_FrontLowerLeg: origin xyz=0 0.9532755602191995 0 rpy=0 0 0 -> xyz=0 0.9073977077835352 0 rpy=0 0 0
- joint LeftLeg_LeftLowerLeg: origin xyz=-0.6345145351766656 0 0 rpy=0 0 0 -> xyz=-0.8153412143409425 0 0 rpy=0 0 0
- joint RightLeg_RightLowerLeg: origin xyz=1.3475938252467945 0 0 rpy=0 0 0 -> xyz=1.4336779769690686 0 0 rpy=0 0 0
- joint Torso_BackLeg: origin xyz=0 -18.5 2.3475938252467943 rpy=0 0 0 -> xyz=0 -18.5 2.4336779769690686 rpy=0 0 0
- joint Torso_FrontLeg: origin xyz=0 -17.5 2.3475938252467943 rpy=0 0 0 -> xyz=0 -17.5 2.4336779769690686 rpy=0 0 0
- joint Torso_LeftLeg: origin xyz=-0.5 -18 2.3475938252467943 rpy=0 0 0 -> xyz=-0.5 -18 2.4336779769690686 rpy=0 0 0
- joint Torso_RightLeg: origin xyz=0.5 -18 2.3475938252467943 rpy=0 0 0 -> xyz=0.5 -18 2.4336779769690686 rpy=0 0 0

File: bodyFiles/body0-18520.urdf (robot description, URDF)
Before this commit: robot robot, 9 links, 8 joints
Links:
- link BackLeg: geometry collision box size=0.2 1.3985535436056145 0.2; visual box size=0.2 1.3985535436056145 0.2
- link BackLowerLeg: geometry collision box size=0.2 0.2 0.5757889699578036; visual box size=0.2 0.2 0.5757889699578036
- link FrontLeg: geometry collision box size=0.2 0.8914463519690072 0.2; visual box size=0.2 0.8914463519690072 0.2
- link FrontLowerLeg: geometry collision box size=0.2 0.2 0.8722634104850099; visual box size=0.2 0.2 0.8722634104850099
- link LeftLeg: geometry collision box size=1.1033983511117864 0.2 0.2; visual box size=1.1033983511117864 0.2 0.2
- link LeftLowerLeg: geometry collision box size=0.2 0.2 0.8897661439941733; visual box size=0.2 0.2 0.8897661439941733
- link RightLeg: geometry collision box size=1.4080226158087221 0.2 0.2; visual box size=1.4080226158087221 0.2 0.2
- link RightLowerLeg: geometry collision box size=0.2 0.2 0.6937936631202338; visual box size=0.2 0.2 0.6937936631202338
Joints:
- joint BackLeg_BackLowerLeg: origin xyz=0 -0.8668675239365025 0 rpy=0 0 0 -> xyz=0 -1.3985535436056145 0 rpy=0 0 0
- joint FrontLeg_FrontLowerLeg: origin xyz=0 1.4947887988763586 0 rpy=0 0 0 -> xyz=0 0.8914463519690072 0 rpy=0 0 0
- joint LeftLeg_LeftLowerLeg: origin xyz=-0.9761800045201299 0 0 rpy=0 0 0 -> xyz=-1.1033983511117864 0 0 rpy=0 0 0
- joint RightLeg_RightLowerLeg: origin xyz=1.00721295930119 0 0 rpy=0 0 0 -> xyz=1.4080226158087221 0 0 rpy=0 0 0
- joint Torso_BackLeg: origin xyz=0 -18.5 2.4947887988763586 rpy=0 0 0 -> xyz=0 -18.5 2.408022615808722 rpy=0 0 0
- joint Torso_FrontLeg: origin xyz=0 -17.5 2.4947887988763586 rpy=0 0 0 -> xyz=0 -17.5 2.408022615808722 rpy=0 0 0
- joint Torso_LeftLeg: origin xyz=-0.5 -18 2.4947887988763586 rpy=0 0 0 -> xyz=-0.5 -18 2.408022615808722 rpy=0 0 0
- joint Torso_RightLeg: origin xyz=0.5 -18 2.4947887988763586 rpy=0 0 0 -> xyz=0.5 -18 2.408022615808722 rpy=0 0 0

File: bodyFiles/body0-1860.urdf (robot description, URDF)
Before this commit: robot robot, 9 links, 8 joints
Links:
- link BackLeg: geometry collision box size=0.2 1.0596229829869874 0.2; visual box size=0.2 1.0596229829869874 0.2
- link BackLowerLeg: geometry collision box size=0.2 0.2 1.17468579754466; visual box size=0.2 0.2 1.17468579754466
- link FrontLeg: geometry collision box size=0.2 0.7898936848975198 0.2; visual box size=0.2 0.7898936848975198 0.2
- link FrontLowerLeg: geometry collision box size=0.2 0.2 0.9086365792178414; visual box size=0.2 0.2 0.9086365792178414
- link LeftLeg: geometry collision box size=1.2975513415202524 0.2 0.2; visual box size=1.2975513415202524 0.2 0.2
- link LeftLowerLeg: geometry collision box size=0.2 0.2 0.873437065566251; visual box size=0.2 0.2 0.873437065566251
- link RightLeg: geometry collision box size=1.4085901177096463 0.2 0.2; visual box size=1.4085901177096463 0.2 0.2
- link RightLowerLeg: geometry collision box size=0.2 0.2 1.3705603816689715; visual box size=0.2 0.2 1.3705603816689715
Joints:
- joint BackLeg_BackLowerLeg: origin xyz=0 -1.474318100220386 0 rpy=0 0 0 -> xyz=0 -1.0596229829869874 0 rpy=0 0 0
- joint FrontLeg_FrontLowerLeg: origin xyz=0 0.5552199265743579 0 rpy=0 0 0 -> xyz=0 0.7898936848975198 0 rpy=0 0 0
- joint LeftLeg_LeftLowerLeg: origin xyz=-1.423641200584335 0 0 rpy=0 0 0 -> xyz=-1.2975513415202524 0 0 rpy=0 0 0
- joint RightLeg_RightLowerLeg: origin xyz=1.3944557864505287 0 0 rpy=0 0 0 -> xyz=1.4085901177096463 0 0 rpy=0 0 0
- joint Torso_BackLeg: origin xyz=0 -18.5 2.474318100220386 rpy=0 0 0 -> xyz=0 -18.5 2.4085901177096463 rpy=0 0 0
- joint Torso_FrontLeg: origin xyz=0 -17.5 2.474318100220386 rpy=0 0 0 -> xyz=0 -17.5 2.4085901177096463 rpy=0 0 0
- joint Torso_LeftLeg: origin xyz=-0.5 -18 2.474318100220386 rpy=0 0 0 -> xyz=-0.5 -18 2.4085901177096463 rpy=0 0 0
- joint Torso_RightLeg: origin xyz=0.5 -18 2.474318100220386 rpy=0 0 0 -> xyz=0.5 -18 2.4085901177096463 rpy=0 0 0

File: bodyFiles/body0-18630.urdf (robot description, URDF)
Before this commit: robot robot, 9 links, 8 joints
Links:
- link BackLeg: geometry collision box size=0.2 1.4236549717849551 0.2; visual box size=0.2 1.4236549717849551 0.2
- link BackLowerLeg: geometry collision box size=0.2 0.2 0.6932606890998145; visual box size=0.2 0.2 0.6932606890998145
- link FrontLeg: geometry collision box size=0.2 1.4851468699411206 0.2; visual box size=0.2 1.4851468699411206 0.2
- link FrontLowerLeg: geometry collision box size=0.2 0.2 0.8739234170807506; visual box size=0.2 0.2 0.8739234170807506
- link LeftLeg: geometry collision box size=1.3879623796278522 0.2 0.2; visual box size=1.3879623796278522 0.2 0.2
- link LeftLowerLeg: geometry collision box size=0.2 0.2 1.3037340208710846; visual box size=0.2 0.2 1.3037340208710846
- link RightLeg: geometry collision box size=1.4264614283046777 0.2 0.2; visual box size=1.4264614283046777 0.2 0.2
- link RightLowerLeg: geometry collision box size=0.2 0.2 1.0096712302654411; visual box size=0.2 0.2 1.0096712302654411
Joints:
- joint BackLeg_BackLowerLeg: origin xyz=0 -1.3763428913254403 0 rpy=0 0 0 -> xyz=0 -1.4236549717849551 0 rpy=0 0 0
- joint FrontLeg_FrontLowerLeg: origin xyz=0 1.1739644338305946 0 rpy=0 0 0 -> xyz=0 1.4851468699411206 0 rpy=0 0 0
- joint LeftLeg_LeftLowerLeg: origin xyz=-1.1866953224236143 0 0 rpy=0 0 0 -> xyz=-1.3879623796278522 0 0 rpy=0 0 0
- joint RightLeg_RightLowerLeg: origin xyz=0.5695502670753783 0 0 rpy=0 0 0 -> xyz=1.4264614283046777 0 0 rpy=0 0 0
- joint Torso_BackLeg: origin xyz=0 -18.5 2.3763428913254403 rpy=0 0 0 -> xyz=0 -18.5 2.4851468699411203 rpy=0 0 0
- joint Torso_FrontLeg: origin xyz=0 -17.5 2.3763428913254403 rpy=0 0 0 -> xyz=0 -17.5 2.4851468699411203 rpy=0 0 0
- joint Torso_LeftLeg: origin xyz=-0.5 -18 2.3763428913254403 rpy=0 0 0 -> xyz=-0.5 -18 2.4851468699411203 rpy=0 0 0
- joint Torso_RightLeg: origin xyz=0.5 -18 2.3763428913254403 rpy=0 0 0 -> xyz=0.5 -18 2.4851468699411203 rpy=0 0 0

File: bodyFiles/body0-18680.urdf (robot description, URDF)
Before this commit: robot robot, 9 links, 8 joints
Links:
- link BackLeg: geometry collision box size=0.2 1.0117388806705545 0.2; visual box size=0.2 1.0117388806705545 0.2
- link BackLowerLeg: geometry collision box size=0.2 0.2 1.0584822376441188; visual box size=0.2 0.2 1.0584822376441188
- link FrontLeg: geometry collision box size=0.2 1.422370990896225 0.2; visual box size=0.2 1.422370990896225 0.2
- link FrontLowerLeg: geometry collision box size=0.2 0.2 1.2221588241860428; visual box size=0.2 0.2 1.2221588241860428
- link LeftLeg: geometry collision box size=0.5008396530104127 0.2 0.2; visual box size=0.5008396530104127 0.2 0.2
- link LeftLowerLeg: geometry collision box size=0.2 0.2 1.3864652605605619; visual box size=0.2 0.2 1.3864652605605619
- link RightLeg: geometry collision box size=1.0786881397525059 0.2 0.2; visual box size=1.0786881397525059 0.2 0.2
- link RightLowerLeg: geometry collision box size=0.2 0.2 1.4261433867290163; visual box size=0.2 0.2 1.4261433867290163
Joints:
- joint BackLeg_BackLowerLeg: origin xyz=0 -0.5143425940636589 0 rpy=0 0 0 -> xyz=0 -1.0117388806705545 0 rpy=0 0 0
- joint FrontLeg_FrontLowerLeg: origin xyz=0 0.6691059866582585 0 rpy=0 0 0 -> xyz=0 1.422370990896225 0 rpy=0 0 0
- joint LeftLeg_LeftLowerLeg: origin xyz=-1.2184912871599018 0 0 rpy=0 0 0 -> xyz=-0.5008396530104127 0 0 rpy=0 0 0
- joint RightLeg_RightLowerLeg: origin xyz=0.9628825169596446 0 0 rpy=0 0 0 -> xyz=1.0786881397525059 0 0 rpy=0 0 0
- joint Torso_BackLeg: origin xyz=0 -18.5 2.4359966706953236 rpy=0 0 0 -> xyz=0 -18.5 2.4261433867290165 rpy=0 0 0
- joint Torso_FrontLeg: origin xyz=0 -17.5 2.4359966706953236 rpy=0 0 0 -> xyz=0 -17.5 2.4261433867290165 rpy=0 0 0
- joint Torso_LeftLeg: origin xyz=-0.5 -18 2.4359966706953236 rpy=0 0 0 -> xyz=-0.5 -18 2.4261433867290165 rpy=0 0 0
- joint Torso_RightLeg: origin xyz=0.5 -18 2.4359966706953236 rpy=0 0 0 -> xyz=0.5 -18 2.4261433867290165 rpy=0 0 0

File: bodyFiles/body0-224.urdf (robot description, URDF)
Before this commit: robot robot, 9 links, 8 joints
Links:
- link BackLeg: geometry collision box size=0.2 0.6981551464305015 0.2; visual box size=0.2 0.6981551464305015 0.2
- link BackLowerLeg: geometry collision box size=0.2 0.2 1.0057591554963912; visual box size=0.2 0.2 1.0057591554963912
- link FrontLeg: geometry collision box size=0.2 1.0912279403210752 0.2; visual box size=0.2 1.0912279403210752 0.2
- link FrontLowerLeg: geometry collision box size=0.2 0.2 1.248685536803225; visual box size=0.2 0.2 1.248685536803225
- link LeftLeg: geometry collision box size=1.0154102468497068 0.2 0.2; visual box size=1.0154102468497068 0.2 0.2
- link LeftLowerLeg: geometry collision box size=0.2 0.2 0.7573571020903066; visual box size=0.2 0.2 0.7573571020903066
- link RightLeg: geometry collision box size=0.513776831045859 0.2 0.2; visual box size=0.513776831045859 0.2 0.2
- link RightLowerLeg: geometry collision box size=0.2 0.2 1.2673845772449435; visual box size=0.2 0.2 1.2673845772449435
Joints:
- joint BackLeg_BackLowerLeg: origin xyz=0 -1.406514952195215 0 rpy=0 0 0 -> xyz=0 -0.6981551464305015 0 rpy=0 0 0
- joint FrontLeg_FrontLowerLeg: origin xyz=0 1.479221720903911 0 rpy=0 0 0 -> xyz=0 1.0912279403210752 0 rpy=0 0 0
- joint LeftLeg_LeftLowerLeg: origin xyz=-0.7248961786671525 0 0 rpy=0 0 0 -> xyz=-1.0154102468497068 0 0 rpy=0 0 0
- joint RightLeg_RightLowerLeg: origin xyz=0.7902856320790941 0 0 rpy=0 0 0 -> xyz=0.513776831045859 0 0 rpy=0 0 0
- joint Torso_BackLeg: origin xyz=0 -2.5 2.4792217209039107 rpy=0 0 0 -> xyz=0 -2.5 2.2673845772449432 rpy=0 0 0
- joint Torso_FrontLeg: origin xyz=0 -1.5 2.4792217209039107 rpy=0 0 0 -> xyz=0 -1.5 2.2673845772449432 rpy=0 0 0
- joint Torso_LeftLeg: origin xyz=-0.5 -2 2.4792217209039107 rpy=0 0 0 -> xyz=-0.5 -2 2.2673845772449432 rpy=0 0 0
- joint Torso_RightLeg: origin xyz=0.5 -2 2.4792217209039107 rpy=0 0 0 -> xyz=0.5 -2 2.2673845772449432 rpy=0 0 0
