Commit message: playback 5x100 evolved

File: bodyFiles/body0-1012.urdf (robot description, URDF)
Before this commit: robot robot, 9 links, 8 joints
Links:
- link BackLeg: geometry collision box size=0.2 1.000075652281187 0.2; visual box size=0.2 1.000075652281187 0.2
- link BackLowerLeg: geometry collision box size=0.2 0.2 1.2055983287087397; visual box size=0.2 0.2 1.2055983287087397
- link FrontLeg: geometry collision box size=0.2 1.3364520286647998 0.2; visual box size=0.2 1.3364520286647998 0.2
- link FrontLowerLeg: geometry collision box size=0.2 0.2 0.7790671571744936; visual box size=0.2 0.2 0.7790671571744936
- link LeftLeg: geometry collision box size=1.0182733586809696 0.2 0.2; visual box size=1.0182733586809696 0.2 0.2
- link LeftLowerLeg: geometry collision box size=0.2 0.2 0.9896659650119696; visual box size=0.2 0.2 0.9896659650119696
- link RightLeg: geometry collision box size=0.7837375337212389 0.2 0.2; visual box size=0.7837375337212389 0.2 0.2
- link RightLowerLeg: geometry collision box size=0.2 0.2 1.4072772113642233; visual box size=0.2 0.2 1.4072772113642233
Joints:
- joint BackLeg_BackLowerLeg: origin xyz=0 -0.5211604762115561 0 rpy=0 0 0 -> xyz=0 -1.000075652281187 0 rpy=0 0 0
- joint FrontLeg_FrontLowerLeg: origin xyz=0 0.7186294586990568 0 rpy=0 0 0 -> xyz=0 1.3364520286647998 0 rpy=0 0 0
- joint LeftLeg_LeftLowerLeg: origin xyz=-1.149241835706703 0 0 rpy=0 0 0 -> xyz=-1.0182733586809696 0 0 rpy=0 0 0
- joint RightLeg_RightLowerLeg: origin xyz=0.5964605064125298 0 0 rpy=0 0 0 -> xyz=0.7837375337212389 0 0 rpy=0 0 0
- joint Torso_BackLeg: origin xyz=0 -10.5 2.4470909662059057 rpy=0 0 0 -> xyz=0 -10.5 2.4072772113642236 rpy=0 0 0
- joint Torso_FrontLeg: origin xyz=0 -9.5 2.4470909662059057 rpy=0 0 0 -> xyz=0 -9.5 2.4072772113642236 rpy=0 0 0
- joint Torso_LeftLeg: origin xyz=-0.5 -10 2.4470909662059057 rpy=0 0 0 -> xyz=-0.5 -10 2.4072772113642236 rpy=0 0 0
- joint Torso_RightLeg: origin xyz=0.5 -10 2.4470909662059057 rpy=0 0 0 -> xyz=0.5 -10 2.4072772113642236 rpy=0 0 0

File: bodyFiles/body0-10532.urdf (robot description, URDF)
Before this commit: robot robot, 9 links, 8 joints
Links:
- link BackLeg: geometry collision box size=0.2 0.6907564543152372 0.2; visual box size=0.2 0.6907564543152372 0.2
- link BackLowerLeg: geometry collision box size=0.2 0.2 1.2336786408862794; visual box size=0.2 0.2 1.2336786408862794
- link FrontLeg: geometry collision box size=0.2 1.0479991399623683 0.2; visual box size=0.2 1.0479991399623683 0.2
- link FrontLowerLeg: geometry collision box size=0.2 0.2 0.8147439714617728; visual box size=0.2 0.2 0.8147439714617728
- link LeftLeg: geometry collision box size=1.1501621350257025 0.2 0.2; visual box size=1.1501621350257025 0.2 0.2
- link LeftLowerLeg: geometry collision box size=0.2 0.2 1.0458698344825856; visual box size=0.2 0.2 1.0458698344825856
- link RightLeg: geometry collision box size=0.9748905071815006 0.2 0.2; visual box size=0.9748905071815006 0.2 0.2
- link RightLowerLeg: geometry collision box size=0.2 0.2 1.2543098329235536; visual box size=0.2 0.2 1.2543098329235536
Joints:
- joint BackLeg_BackLowerLeg: origin xyz=0 -1.0313918992716782 0 rpy=0 0 0 -> xyz=0 -0.6907564543152372 0 rpy=0 0 0
- joint FrontLeg_FrontLowerLeg: origin xyz=0 0.7761146523712571 0 rpy=0 0 0 -> xyz=0 1.0479991399623683 0 rpy=0 0 0
- joint LeftLeg_LeftLowerLeg: origin xyz=-1.0664624824195315 0 0 rpy=0 0 0 -> xyz=-1.1501621350257025 0 0 rpy=0 0 0
- joint RightLeg_RightLowerLeg: origin xyz=1.0142348518451016 0 0 rpy=0 0 0 -> xyz=0.9748905071815006 0 0 rpy=0 0 0
- joint Torso_BackLeg: origin xyz=0 -10.5 2.448035366509675 rpy=0 0 0 -> xyz=0 -10.5 2.2543098329235534 rpy=0 0 0
- joint Torso_FrontLeg: origin xyz=0 -9.5 2.448035366509675 rpy=0 0 0 -> xyz=0 -9.5 2.2543098329235534 rpy=0 0 0
- joint Torso_LeftLeg: origin xyz=-0.5 -10 2.448035366509675 rpy=0 0 0 -> xyz=-0.5 -10 2.2543098329235534 rpy=0 0 0
- joint Torso_RightLeg: origin xyz=0.5 -10 2.448035366509675 rpy=0 0 0 -> xyz=0.5 -10 2.2543098329235534 rpy=0 0 0

File: bodyFiles/body0-10642.urdf (robot description, URDF)
Before this commit: robot robot, 9 links, 8 joints
Links:
- link BackLeg: geometry collision box size=0.2 1.4877981693738322 0.2; visual box size=0.2 1.4877981693738322 0.2
- link BackLowerLeg: geometry collision box size=0.2 0.2 1.271777622294296; visual box size=0.2 0.2 1.271777622294296
- link FrontLeg: geometry collision box size=0.2 0.5979225778299864 0.2; visual box size=0.2 0.5979225778299864 0.2
- link FrontLowerLeg: geometry collision box size=0.2 0.2 1.284142764337735; visual box size=0.2 0.2 1.284142764337735
- link LeftLeg: geometry collision box size=0.9079784043918011 0.2 0.2; visual box size=0.9079784043918011 0.2 0.2
- link LeftLowerLeg: geometry collision box size=0.2 0.2 1.2803684708783596; visual box size=0.2 0.2 1.2803684708783596
- link RightLeg: geometry collision box size=0.839664376198 0.2 0.2; visual box size=0.839664376198 0.2 0.2
- link RightLowerLeg: geometry collision box size=0.2 0.2 1.3726803065743995; visual box size=0.2 0.2 1.3726803065743995
Joints:
- joint BackLeg_BackLowerLeg: origin xyz=0 -0.8579575214904757 0 rpy=0 0 0 -> xyz=0 -1.4877981693738322 0 rpy=0 0 0
- joint FrontLeg_FrontLowerLeg: origin xyz=0 0.8765702169552689 0 rpy=0 0 0 -> xyz=0 0.5979225778299864 0 rpy=0 0 0
- joint LeftLeg_LeftLowerLeg: origin xyz=-1.2715606262648378 0 0 rpy=0 0 0 -> xyz=-0.9079784043918011 0 0 rpy=0 0 0
- joint RightLeg_RightLowerLeg: origin xyz=0.5848937866194583 0 0 rpy=0 0 0 -> xyz=0.839664376198 0 0 rpy=0 0 0
- joint Torso_BackLeg: origin xyz=0 -10.5 2.462267762508233 rpy=0 0 0 -> xyz=0 -10.5 2.487798169373832 rpy=0 0 0
- joint Torso_FrontLeg: origin xyz=0 -9.5 2.462267762508233 rpy=0 0 0 -> xyz=0 -9.5 2.487798169373832 rpy=0 0 0
- joint Torso_LeftLeg: origin xyz=-0.5 -10 2.462267762508233 rpy=0 0 0 -> xyz=-0.5 -10 2.487798169373832 rpy=0 0 0
- joint Torso_RightLeg: origin xyz=0.5 -10 2.462267762508233 rpy=0 0 0 -> xyz=0.5 -10 2.487798169373832 rpy=0 0 0

File: bodyFiles/body0-10692.urdf (robot description, URDF)
Before this commit: robot robot, 9 links, 8 joints
Links:
- link BackLeg: geometry collision box size=0.2 1.0312655504021946 0.2; visual box size=0.2 1.0312655504021946 0.2
- link BackLowerLeg: geometry collision box size=0.2 0.2 1.4152489719298575; visual box size=0.2 0.2 1.4152489719298575
- link FrontLeg: geometry collision box size=0.2 1.2655123208601347 0.2; visual box size=0.2 1.2655123208601347 0.2
- link FrontLowerLeg: geometry collision box size=0.2 0.2 1.1785657774058986; visual box size=0.2 0.2 1.1785657774058986
- link LeftLeg: geometry collision box size=1.1779262348634476 0.2 0.2; visual box size=1.1779262348634476 0.2 0.2
- link LeftLowerLeg: geometry collision box size=0.2 0.2 0.8984527475792041; visual box size=0.2 0.2 0.8984527475792041
- link RightLeg: geometry collision box size=0.7499918915017123 0.2 0.2; visual box size=0.7499918915017123 0.2 0.2
- link RightLowerLeg: geometry collision box size=0.2 0.2 0.7067933091942751; visual box size=0.2 0.2 0.7067933091942751
Joints:
- joint BackLeg_BackLowerLeg: origin xyz=0 -0.660046028348746 0 rpy=0 0 0 -> xyz=0 -1.0312655504021946 0 rpy=0 0 0
- joint FrontLeg_FrontLowerLeg: origin xyz=0 1.0149170585304728 0 rpy=0 0 0 -> xyz=0 1.2655123208601347 0 rpy=0 0 0
- joint LeftLeg_LeftLowerLeg: origin xyz=-0.8034617801471663 0 0 rpy=0 0 0 -> xyz=-1.1779262348634476 0 0 rpy=0 0 0
- joint RightLeg_RightLowerLeg: origin xyz=1.2554648635354746 0 0 rpy=0 0 0 -> xyz=0.7499918915017123 0 0 rpy=0 0 0
- joint Torso_BackLeg: origin xyz=0 -10.5 2.2554648635354746 rpy=0 0 0 -> xyz=0 -10.5 2.4152489719298575 rpy=0 0 0
- joint Torso_FrontLeg: origin xyz=0 -9.5 2.2554648635354746 rpy=0 0 0 -> xyz=0 -9.5 2.4152489719298575 rpy=0 0 0
- joint Torso_LeftLeg: origin xyz=-0.5 -10 2.2554648635354746 rpy=0 0 0 -> xyz=-0.5 -10 2.4152489719298575 rpy=0 0 0
- joint Torso_RightLeg: origin xyz=0.5 -10 2.2554648635354746 rpy=0 0 0 -> xyz=0.5 -10 2.4152489719298575 rpy=0 0 0

File: bodyFiles/body0-1072.urdf (robot description, URDF)
Before this commit: robot robot, 9 links, 8 joints
Links:
- link BackLeg: geometry collision box size=0.2 1.3459979763041854 0.2; visual box size=0.2 1.3459979763041854 0.2
- link BackLowerLeg: geometry collision box size=0.2 0.2 0.9366727326083825; visual box size=0.2 0.2 0.9366727326083825
- link FrontLeg: geometry collision box size=0.2 1.2567033393146096 0.2; visual box size=0.2 1.2567033393146096 0.2
- link FrontLowerLeg: geometry collision box size=0.2 0.2 0.8016929042732136; visual box size=0.2 0.2 0.8016929042732136
- link LeftLeg: geometry collision box size=0.9778446327985183 0.2 0.2; visual box size=0.9778446327985183 0.2 0.2
- link LeftLowerLeg: geometry collision box size=0.2 0.2 0.836065211242257; visual box size=0.2 0.2 0.836065211242257
- link RightLeg: geometry collision box size=1.140889667888854 0.2 0.2; visual box size=1.140889667888854 0.2 0.2
- link RightLowerLeg: geometry collision box size=0.2 0.2 1.4151752478180646; visual box size=0.2 0.2 1.4151752478180646
Joints:
- joint BackLeg_BackLowerLeg: origin xyz=0 -0.8110738569355737 0 rpy=0 0 0 -> xyz=0 -1.3459979763041854 0 rpy=0 0 0
- joint FrontLeg_FrontLowerLeg: origin xyz=0 1.0501005398938945 0 rpy=0 0 0 -> xyz=0 1.2567033393146096 0 rpy=0 0 0
- joint LeftLeg_LeftLowerLeg: origin xyz=-0.6053989318212719 0 0 rpy=0 0 0 -> xyz=-0.9778446327985183 0 0 rpy=0 0 0
- joint RightLeg_RightLowerLeg: origin xyz=1.3025893237328048 0 0 rpy=0 0 0 -> xyz=1.140889667888854 0 0 rpy=0 0 0
- joint Torso_BackLeg: origin xyz=0 -10.5 2.4728372311495654 rpy=0 0 0 -> xyz=0 -10.5 2.4151752478180644 rpy=0 0 0
- joint Torso_FrontLeg: origin xyz=0 -9.5 2.4728372311495654 rpy=0 0 0 -> xyz=0 -9.5 2.4151752478180644 rpy=0 0 0
- joint Torso_LeftLeg: origin xyz=-0.5 -10 2.4728372311495654 rpy=0 0 0 -> xyz=-0.5 -10 2.4151752478180644 rpy=0 0 0
- joint Torso_RightLeg: origin xyz=0.5 -10 2.4728372311495654 rpy=0 0 0 -> xyz=0.5 -10 2.4151752478180644 rpy=0 0 0

File: bodyFiles/body0-14121.urdf (robot description, URDF)
Before this commit: robot robot, 9 links, 8 joints
Links:
- link BackLeg: geometry collision box size=0.2 1.0652409818326523 0.2; visual box size=0.2 1.0652409818326523 0.2
- link BackLowerLeg: geometry collision box size=0.2 0.2 1.278712286632294; visual box size=0.2 0.2 1.278712286632294
- link FrontLeg: geometry collision box size=0.2 1.0511734690408963 0.2; visual box size=0.2 1.0511734690408963 0.2
- link FrontLowerLeg: geometry collision box size=0.2 0.2 0.5958697149841481; visual box size=0.2 0.2 0.5958697149841481
- link LeftLeg: geometry collision box size=1.3617180326887923 0.2 0.2; visual box size=1.3617180326887923 0.2 0.2
- link LeftLowerLeg: geometry collision box size=0.2 0.2 1.281331158947466; visual box size=0.2 0.2 1.281331158947466
- link RightLeg: geometry collision box size=0.9955952884491329 0.2 0.2; visual box size=0.9955952884491329 0.2 0.2
- link RightLowerLeg: geometry collision box size=0.2 0.2 1.1023662261721876; visual box size=0.2 0.2 1.1023662261721876
Joints:
- joint BackLeg_BackLowerLeg: origin xyz=0 -0.9931024636824476 0 rpy=0 0 0 -> xyz=0 -1.0652409818326523 0 rpy=0 0 0
- joint FrontLeg_FrontLowerLeg: origin xyz=0 1.2145972728683203 0 rpy=0 0 0 -> xyz=0 1.0511734690408963 0 rpy=0 0 0
- joint LeftLeg_LeftLowerLeg: origin xyz=-0.9113605189694807 0 0 rpy=0 0 0 -> xyz=-1.3617180326887923 0 0 rpy=0 0 0
- joint RightLeg_RightLowerLeg: origin xyz=1.2048031813467723 0 0 rpy=0 0 0 -> xyz=0.9955952884491329 0 0 rpy=0 0 0
- joint Torso_BackLeg: origin xyz=0 -14.5 2.331613794175423 rpy=0 0 0 -> xyz=0 -14.5 2.3617180326887923 rpy=0 0 0
- joint Torso_FrontLeg: origin xyz=0 -13.5 2.331613794175423 rpy=0 0 0 -> xyz=0 -13.5 2.3617180326887923 rpy=0 0 0
- joint Torso_LeftLeg: origin xyz=-0.5 -14 2.331613794175423 rpy=0 0 0 -> xyz=-0.5 -14 2.3617180326887923 rpy=0 0 0
- joint Torso_RightLeg: origin xyz=0.5 -14 2.331613794175423 rpy=0 0 0 -> xyz=0.5 -14 2.3617180326887923 rpy=0 0 0

File: bodyFiles/body0-14171.urdf (robot description, URDF)
Before this commit: robot robot, 9 links, 8 joints
Links:
- link BackLeg: geometry collision box size=0.2 0.6239027654354744 0.2; visual box size=0.2 0.6239027654354744 0.2
- link BackLowerLeg: geometry collision box size=0.2 0.2 1.4200391507924834; visual box size=0.2 0.2 1.4200391507924834
- link FrontLeg: geometry collision box size=0.2 1.0136973053960494 0.2; visual box size=0.2 1.0136973053960494 0.2
- link FrontLowerLeg: geometry collision box size=0.2 0.2 1.4966910711602066; visual box size=0.2 0.2 1.4966910711602066
- link LeftLeg: geometry collision box size=0.5365875976044888 0.2 0.2; visual box size=0.5365875976044888 0.2 0.2
- link LeftLowerLeg: geometry collision box size=0.2 0.2 1.070818186033937; visual box size=0.2 0.2 1.070818186033937
- link RightLeg: geometry collision box size=1.338063709379228 0.2 0.2; visual box size=1.338063709379228 0.2 0.2
- link RightLowerLeg: geometry collision box size=0.2 0.2 0.894197303710928; visual box size=0.2 0.2 0.894197303710928
Joints:
- joint BackLeg_BackLowerLeg: origin xyz=0 -0.7188865916559471 0 rpy=0 0 0 -> xyz=0 -0.6239027654354744 0 rpy=0 0 0
- joint FrontLeg_FrontLowerLeg: origin xyz=0 0.5818023036998935 0 rpy=0 0 0 -> xyz=0 1.0136973053960494 0 rpy=0 0 0
- joint LeftLeg_LeftLowerLeg: origin xyz=-0.7343021727131351 0 0 rpy=0 0 0 -> xyz=-0.5365875976044888 0 0 rpy=0 0 0
- joint RightLeg_RightLowerLeg: origin xyz=0.6428421351829458 0 0 rpy=0 0 0 -> xyz=1.338063709379228 0 0 rpy=0 0 0
- joint Torso_BackLeg: origin xyz=0 -14.5 2.344901986946851 rpy=0 0 0 -> xyz=0 -14.5 2.496691071160207 rpy=0 0 0
- joint Torso_FrontLeg: origin xyz=0 -13.5 2.344901986946851 rpy=0 0 0 -> xyz=0 -13.5 2.496691071160207 rpy=0 0 0
- joint Torso_LeftLeg: origin xyz=-0.5 -14 2.344901986946851 rpy=0 0 0 -> xyz=-0.5 -14 2.496691071160207 rpy=0 0 0
- joint Torso_RightLeg: origin xyz=0.5 -14 2.344901986946851 rpy=0 0 0 -> xyz=0.5 -14 2.496691071160207 rpy=0 0 0

File: bodyFiles/body0-14221.urdf (robot description, URDF)
Before this commit: robot robot, 9 links, 8 joints
Links:
- link BackLeg: geometry collision box size=0.2 1.2704900398260972 0.2; visual box size=0.2 1.2704900398260972 0.2
- link BackLowerLeg: geometry collision box size=0.2 0.2 1.2734723395100165; visual box size=0.2 0.2 1.2734723395100165
- link FrontLeg: geometry collision box size=0.2 1.2960263433808885 0.2; visual box size=0.2 1.2960263433808885 0.2
- link FrontLowerLeg: geometry collision box size=0.2 0.2 0.6784936325397242; visual box size=0.2 0.2 0.6784936325397242
- link LeftLeg: geometry collision box size=0.764269274544538 0.2 0.2; visual box size=0.764269274544538 0.2 0.2
- link LeftLowerLeg: geometry collision box size=0.2 0.2 1.206003006633976; visual box size=0.2 0.2 1.206003006633976
- link RightLeg: geometry collision box size=0.8983949315857326 0.2 0.2; visual box size=0.8983949315857326 0.2 0.2
- link RightLowerLeg: geometry collision box size=0.2 0.2 1.0821349527214057; visual box size=0.2 0.2 1.0821349527214057
Joints:
- joint BackLeg_BackLowerLeg: origin xyz=0 -0.7862080721636425 0 rpy=0 0 0 -> xyz=0 -1.2704900398260972 0 rpy=0 0 0
- joint FrontLeg_FrontLowerLeg: origin xyz=0 0.9186741075536171 0 rpy=0 0 0 -> xyz=0 1.2960263433808885 0 rpy=0 0 0
- joint LeftLeg_LeftLowerLeg: origin xyz=-1.493351461273596 0 0 rpy=0 0 0 -> xyz=-0.764269274544538 0 0 rpy=0 0 0
- joint RightLeg_RightLowerLeg: origin xyz=1.4252253305969425 0 0 rpy=0 0 0 -> xyz=0.8983949315857326 0 0 rpy=0 0 0
- joint Torso_BackLeg: origin xyz=0 -14.5 2.493351461273596 rpy=0 0 0 -> xyz=0 -14.5 2.2960263433808885 rpy=0 0 0
- joint Torso_FrontLeg: origin xyz=0 -13.5 2.493351461273596 rpy=0 0 0 -> xyz=0 -13.5 2.2960263433808885 rpy=0 0 0
- joint Torso_LeftLeg: origin xyz=-0.5 -14 2.493351461273596 rpy=0 0 0 -> xyz=-0.5 -14 2.2960263433808885 rpy=0 0 0
- joint Torso_RightLeg: origin xyz=0.5 -14 2.493351461273596 rpy=0 0 0 -> xyz=0.5 -14 2.2960263433808885 rpy=0 0 0

File: bodyFiles/body0-14271.urdf (robot description, URDF)
Before this commit: robot robot, 9 links, 8 joints
Links:
- link BackLeg: geometry collision box size=0.2 1.1092272087117718 0.2; visual box size=0.2 1.1092272087117718 0.2
- link BackLowerLeg: geometry collision box size=0.2 0.2 1.0125919254416362; visual box size=0.2 0.2 1.0125919254416362
- link FrontLeg: geometry collision box size=0.2 1.102559074904649 0.2; visual box size=0.2 1.102559074904649 0.2
- link FrontLowerLeg: geometry collision box size=0.2 0.2 0.7755834957699305; visual box size=0.2 0.2 0.7755834957699305
- link LeftLeg: geometry collision box size=1.116753697097894 0.2 0.2; visual box size=1.116753697097894 0.2 0.2
- link LeftLowerLeg: geometry collision box size=0.2 0.2 1.4339109780202441; visual box size=0.2 0.2 1.4339109780202441
- link RightLeg: geometry collision box size=1.2408457616174222 0.2 0.2; visual box size=1.2408457616174222 0.2 0.2
- link RightLowerLeg: geometry collision box size=0.2 0.2 1.486962597087964; visual box size=0.2 0.2 1.486962597087964
Joints:
- joint BackLeg_BackLowerLeg: origin xyz=0 -0.652344904053455 0 rpy=0 0 0 -> xyz=0 -1.1092272087117718 0 rpy=0 0 0
- joint FrontLeg_FrontLowerLeg: origin xyz=0 0.6842841901934328 0 rpy=0 0 0 -> xyz=0 1.102559074904649 0 rpy=0 0 0
- joint LeftLeg_LeftLowerLeg: origin xyz=-0.7345350215974369 0 0 rpy=0 0 0 -> xyz=-1.116753697097894 0 0 rpy=0 0 0
- joint RightLeg_RightLowerLeg: origin xyz=1.1043903493777765 0 0 rpy=0 0 0 -> xyz=1.2408457616174222 0 0 rpy=0 0 0
- joint Torso_BackLeg: origin xyz=0 -14.5 2.1043903493777765 rpy=0 0 0 -> xyz=0 -14.5 2.486962597087964 rpy=0 0 0
- joint Torso_FrontLeg: origin xyz=0 -13.5 2.1043903493777765 rpy=0 0 0 -> xyz=0 -13.5 2.486962597087964 rpy=0 0 0
- joint Torso_LeftLeg: origin xyz=-0.5 -14 2.1043903493777765 rpy=0 0 0 -> xyz=-0.5 -14 2.486962597087964 rpy=0 0 0
- joint Torso_RightLeg: origin xyz=0.5 -14 2.1043903493777765 rpy=0 0 0 -> xyz=0.5 -14 2.486962597087964 rpy=0 0 0

File: bodyFiles/body0-14321.urdf (robot description, URDF)
Before this commit: robot robot, 9 links, 8 joints
Links:
- link BackLeg: geometry collision box size=0.2 0.7494180307358763 0.2; visual box size=0.2 0.7494180307358763 0.2
- link BackLowerLeg: geometry collision box size=0.2 0.2 0.8614233847765977; visual box size=0.2 0.2 0.8614233847765977
- link FrontLeg: geometry collision box size=0.2 0.8451704150979913 0.2; visual box size=0.2 0.8451704150979913 0.2
- link FrontLowerLeg: geometry collision box size=0.2 0.2 0.5517909709564389; visual box size=0.2 0.2 0.5517909709564389
- link LeftLeg: geometry collision box size=0.8618228484796303 0.2 0.2; visual box size=0.8618228484796303 0.2 0.2
- link LeftLowerLeg: geometry collision box size=0.2 0.2 1.3138110626928419; visual box size=0.2 0.2 1.3138110626928419
- link RightLeg: geometry collision box size=1.176375372664793 0.2 0.2; visual box size=1.176375372664793 0.2 0.2
- link RightLowerLeg: geometry collision box size=0.2 0.2 1.0715341349501206; visual box size=0.2 0.2 1.0715341349501206
Joints:
- joint BackLeg_BackLowerLeg: origin xyz=0 -1.4575323398559819 0 rpy=0 0 0 -> xyz=0 -0.7494180307358763 0 rpy=0 0 0
- joint FrontLeg_FrontLowerLeg: origin xyz=0 1.2988235486818733 0 rpy=0 0 0 -> xyz=0 0.8451704150979913 0 rpy=0 0 0
- joint LeftLeg_LeftLowerLeg: origin xyz=-0.6064807096139438 0 0 rpy=0 0 0 -> xyz=-0.8618228484796303 0 0 rpy=0 0 0
- joint RightLeg_RightLowerLeg: origin xyz=0.6914962503509424 0 0 rpy=0 0 0 -> xyz=1.176375372664793 0 0 rpy=0 0 0
- joint Torso_BackLeg: origin xyz=0 -14.5 2.457532339855982 rpy=0 0 0 -> xyz=0 -14.5 2.313811062692842 rpy=0 0 0
- joint Torso_FrontLeg: origin xyz=0 -13.5 2.457532339855982 rpy=0 0 0 -> xyz=0 -13.5 2.313811062692842 rpy=0 0 0
- joint Torso_LeftLeg: origin xyz=-0.5 -14 2.457532339855982 rpy=0 0 0 -> xyz=-0.5 -14 2.313811062692842 rpy=0 0 0
- joint Torso_RightLeg: origin xyz=0.5 -14 2.457532339855982 rpy=0 0 0 -> xyz=0.5 -14 2.313811062692842 rpy=0 0 0

File: bodyFiles/body0-14371.urdf (robot description, URDF)
Before this commit: robot robot, 9 links, 8 joints
Links:
- link BackLeg: geometry collision box size=0.2 0.6865351724641189 0.2; visual box size=0.2 0.6865351724641189 0.2
- link BackLowerLeg: geometry collision box size=0.2 0.2 1.2817574551932562; visual box size=0.2 0.2 1.2817574551932562
- link FrontLeg: geometry collision box size=0.2 0.5088308287026956 0.2; visual box size=0.2 0.5088308287026956 0.2
- link FrontLowerLeg: geometry collision box size=0.2 0.2 1.4898776944154046; visual box size=0.2 0.2 1.4898776944154046
- link LeftLeg: geometry collision box size=1.132811997045073 0.2 0.2; visual box size=1.132811997045073 0.2 0.2
- link LeftLowerLeg: geometry collision box size=0.2 0.2 1.484886492157167; visual box size=0.2 0.2 1.484886492157167
- link RightLeg: geometry collision box size=0.7763365185488067 0.2 0.2; visual box size=0.7763365185488067 0.2 0.2
- link RightLowerLeg: geometry collision box size=0.2 0.2 0.917696090112766; visual box size=0.2 0.2 0.917696090112766
Joints:
- joint BackLeg_BackLowerLeg: origin xyz=0 -1.0980398737823227 0 rpy=0 0 0 -> xyz=0 -0.6865351724641189 0 rpy=0 0 0
- joint FrontLeg_FrontLowerLeg: origin xyz=0 1.4028027586663345 0 rpy=0 0 0 -> xyz=0 0.5088308287026956 0 rpy=0 0 0
- joint LeftLeg_LeftLowerLeg: origin xyz=-1.4949732538946088 0 0 rpy=0 0 0 -> xyz=-1.132811997045073 0 0 rpy=0 0 0
- joint RightLeg_RightLowerLeg: origin xyz=1.4483525739106313 0 0 rpy=0 0 0 -> xyz=0.7763365185488067 0 0 rpy=0 0 0
- joint Torso_BackLeg: origin xyz=0 -14.5 2.4949732538946088 rpy=0 0 0 -> xyz=0 -14.5 2.4898776944154046 rpy=0 0 0
- joint Torso_FrontLeg: origin xyz=0 -13.5 2.4949732538946088 rpy=0 0 0 -> xyz=0 -13.5 2.4898776944154046 rpy=0 0 0
- joint Torso_LeftLeg: origin xyz=-0.5 -14 2.4949732538946088 rpy=0 0 0 -> xyz=-0.5 -14 2.4898776944154046 rpy=0 0 0
- joint Torso_RightLeg: origin xyz=0.5 -14 2.4949732538946088 rpy=0 0 0 -> xyz=0.5 -14 2.4898776944154046 rpy=0 0 0
