Commit message: playback 5x100 evolved

File: bodyFiles/body0-14421.urdf (robot description, URDF)
Before this commit: robot robot, 9 links, 8 joints
Links:
- link BackLeg: geometry collision box size=0.2 0.86786583055541 0.2; visual box size=0.2 0.86786583055541 0.2
- link BackLowerLeg: geometry collision box size=0.2 0.2 1.3143309191756534; visual box size=0.2 0.2 1.3143309191756534
- link FrontLeg: geometry collision box size=0.2 1.4098084430331101 0.2; visual box size=0.2 1.4098084430331101 0.2
- link FrontLowerLeg: geometry collision box size=0.2 0.2 1.2410521701111092; visual box size=0.2 0.2 1.2410521701111092
- link LeftLeg: geometry collision box size=0.5270491602320612 0.2 0.2; visual box size=0.5270491602320612 0.2 0.2
- link LeftLowerLeg: geometry collision box size=0.2 0.2 1.283801323539627; visual box size=0.2 0.2 1.283801323539627
- link RightLeg: geometry collision box size=1.2535408743421492 0.2 0.2; visual box size=1.2535408743421492 0.2 0.2
- link RightLowerLeg: geometry collision box size=0.2 0.2 0.675112711650654; visual box size=0.2 0.2 0.675112711650654
Joints:
- joint BackLeg_BackLowerLeg: origin xyz=0 -0.8188954207864741 0 rpy=0 0 0 -> xyz=0 -0.86786583055541 0 rpy=0 0 0
- joint FrontLeg_FrontLowerLeg: origin xyz=0 0.885909684476771 0 rpy=0 0 0 -> xyz=0 1.4098084430331101 0 rpy=0 0 0
- joint LeftLeg_LeftLowerLeg: origin xyz=-1.1696067332464164 0 0 rpy=0 0 0 -> xyz=-0.5270491602320612 0 0 rpy=0 0 0
- joint RightLeg_RightLowerLeg: origin xyz=1.1143757421214104 0 0 rpy=0 0 0 -> xyz=1.2535408743421492 0 0 rpy=0 0 0
- joint Torso_BackLeg: origin xyz=0 -14.5 2.425820433870876 rpy=0 0 0 -> xyz=0 -14.5 2.40980844303311 rpy=0 0 0
- joint Torso_FrontLeg: origin xyz=0 -13.5 2.425820433870876 rpy=0 0 0 -> xyz=0 -13.5 2.40980844303311 rpy=0 0 0
- joint Torso_LeftLeg: origin xyz=-0.5 -14 2.425820433870876 rpy=0 0 0 -> xyz=-0.5 -14 2.40980844303311 rpy=0 0 0
- joint Torso_RightLeg: origin xyz=0.5 -14 2.425820433870876 rpy=0 0 0 -> xyz=0.5 -14 2.40980844303311 rpy=0 0 0

File: bodyFiles/body0-14471.urdf (robot description, URDF)
Before this commit: robot robot, 9 links, 8 joints
Links:
- link BackLeg: geometry collision box size=0.2 0.6394982186203166 0.2; visual box size=0.2 0.6394982186203166 0.2
- link BackLowerLeg: geometry collision box size=0.2 0.2 0.8566318589802251; visual box size=0.2 0.2 0.8566318589802251
- link FrontLeg: geometry collision box size=0.2 1.0073973512176075 0.2; visual box size=0.2 1.0073973512176075 0.2
- link FrontLowerLeg: geometry collision box size=0.2 0.2 0.6367408532358336; visual box size=0.2 0.2 0.6367408532358336
- link LeftLeg: geometry collision box size=0.9401852167650583 0.2 0.2; visual box size=0.9401852167650583 0.2 0.2
- link LeftLowerLeg: geometry collision box size=0.2 0.2 1.231006608005167; visual box size=0.2 0.2 1.231006608005167
- link RightLeg: geometry collision box size=1.1756528444315464 0.2 0.2; visual box size=1.1756528444315464 0.2 0.2
- link RightLowerLeg: geometry collision box size=0.2 0.2 1.2562717128128391; visual box size=0.2 0.2 1.2562717128128391
Joints:
- joint BackLeg_BackLowerLeg: origin xyz=0 -1.0650617074501816 0 rpy=0 0 0 -> xyz=0 -0.6394982186203166 0 rpy=0 0 0
- joint FrontLeg_FrontLowerLeg: origin xyz=0 0.9585510460969066 0 rpy=0 0 0 -> xyz=0 1.0073973512176075 0 rpy=0 0 0
- joint LeftLeg_LeftLowerLeg: origin xyz=-0.7207335194897964 0 0 rpy=0 0 0 -> xyz=-0.9401852167650583 0 0 rpy=0 0 0
- joint RightLeg_RightLowerLeg: origin xyz=1.2629024629367553 0 0 rpy=0 0 0 -> xyz=1.1756528444315464 0 0 rpy=0 0 0
- joint Torso_BackLeg: origin xyz=0 -14.5 2.262902462936755 rpy=0 0 0 -> xyz=0 -14.5 2.256271712812839 rpy=0 0 0
- joint Torso_FrontLeg: origin xyz=0 -13.5 2.262902462936755 rpy=0 0 0 -> xyz=0 -13.5 2.256271712812839 rpy=0 0 0
- joint Torso_LeftLeg: origin xyz=-0.5 -14 2.262902462936755 rpy=0 0 0 -> xyz=-0.5 -14 2.256271712812839 rpy=0 0 0
- joint Torso_RightLeg: origin xyz=0.5 -14 2.262902462936755 rpy=0 0 0 -> xyz=0.5 -14 2.256271712812839 rpy=0 0 0

File: bodyFiles/body0-14581.urdf (robot description, URDF)
Before this commit: robot robot, 9 links, 8 joints
Links:
- link BackLeg: geometry collision box size=0.2 1.3970104942589818 0.2; visual box size=0.2 1.3970104942589818 0.2
- link BackLowerLeg: geometry collision box size=0.2 0.2 1.3514406268973422; visual box size=0.2 0.2 1.3514406268973422
- link FrontLeg: geometry collision box size=0.2 1.4291352851530719 0.2; visual box size=0.2 1.4291352851530719 0.2
- link FrontLowerLeg: geometry collision box size=0.2 0.2 0.9627144657339924; visual box size=0.2 0.2 0.9627144657339924
- link LeftLeg: geometry collision box size=1.142038966082247 0.2 0.2; visual box size=1.142038966082247 0.2 0.2
- link LeftLowerLeg: geometry collision box size=0.2 0.2 1.3991371017861511; visual box size=0.2 0.2 1.3991371017861511
- link RightLeg: geometry collision box size=0.8202913257848955 0.2 0.2; visual box size=0.8202913257848955 0.2 0.2
- link RightLowerLeg: geometry collision box size=0.2 0.2 0.7739325611435525; visual box size=0.2 0.2 0.7739325611435525
Joints:
- joint BackLeg_BackLowerLeg: origin xyz=0 -0.7471122312869726 0 rpy=0 0 0 -> xyz=0 -1.3970104942589818 0 rpy=0 0 0
- joint FrontLeg_FrontLowerLeg: origin xyz=0 1.4662151618078418 0 rpy=0 0 0 -> xyz=0 1.4291352851530719 0 rpy=0 0 0
- joint LeftLeg_LeftLowerLeg: origin xyz=-1.417396359815199 0 0 rpy=0 0 0 -> xyz=-1.142038966082247 0 0 rpy=0 0 0
- joint RightLeg_RightLowerLeg: origin xyz=1.4739953929240328 0 0 rpy=0 0 0 -> xyz=0.8202913257848955 0 0 rpy=0 0 0
- joint Torso_BackLeg: origin xyz=0 -14.5 2.473995392924033 rpy=0 0 0 -> xyz=0 -14.5 2.429135285153072 rpy=0 0 0
- joint Torso_FrontLeg: origin xyz=0 -13.5 2.473995392924033 rpy=0 0 0 -> xyz=0 -13.5 2.429135285153072 rpy=0 0 0
- joint Torso_LeftLeg: origin xyz=-0.5 -14 2.473995392924033 rpy=0 0 0 -> xyz=-0.5 -14 2.429135285153072 rpy=0 0 0
- joint Torso_RightLeg: origin xyz=0.5 -14 2.473995392924033 rpy=0 0 0 -> xyz=0.5 -14 2.429135285153072 rpy=0 0 0

File: bodyFiles/body0-180.urdf (robot description, URDF)
Before this commit: robot robot, 9 links, 8 joints
Links:
- link BackLeg: geometry collision box size=0.2 1.340944195731549 0.2; visual box size=0.2 1.340944195731549 0.2
- link BackLowerLeg: geometry collision box size=0.2 0.2 0.8581108891102676; visual box size=0.2 0.2 0.8581108891102676
- link FrontLeg: geometry collision box size=0.2 1.1237734662792427 0.2; visual box size=0.2 1.1237734662792427 0.2
- link FrontLowerLeg: geometry collision box size=0.2 0.2 1.0227231198950482; visual box size=0.2 0.2 1.0227231198950482
- link LeftLeg: geometry collision box size=1.0609147724614933 0.2 0.2; visual box size=1.0609147724614933 0.2 0.2
- link LeftLowerLeg: geometry collision box size=0.2 0.2 1.107858631574879; visual box size=0.2 0.2 1.107858631574879
- link RightLeg: geometry collision box size=1.1097387162991441 0.2 0.2; visual box size=1.1097387162991441 0.2 0.2
- link RightLowerLeg: geometry collision box size=0.2 0.2 0.52248219469437; visual box size=0.2 0.2 0.52248219469437
Joints:
- joint BackLeg_BackLowerLeg: origin xyz=0 -1.229704891864707 0 rpy=0 0 0 -> xyz=0 -1.340944195731549 0 rpy=0 0 0
- joint FrontLeg_FrontLowerLeg: origin xyz=0 0.9073977077835352 0 rpy=0 0 0 -> xyz=0 1.1237734662792427 0 rpy=0 0 0
- joint LeftLeg_LeftLowerLeg: origin xyz=-0.8153412143409425 0 0 rpy=0 0 0 -> xyz=-1.0609147724614933 0 0 rpy=0 0 0
- joint RightLeg_RightLowerLeg: origin xyz=1.4336779769690686 0 0 rpy=0 0 0 -> xyz=1.1097387162991441 0 0 rpy=0 0 0
- joint Torso_BackLeg: origin xyz=0 -18.5 2.4336779769690686 rpy=0 0 0 -> xyz=0 -18.5 2.340944195731549 rpy=0 0 0
- joint Torso_FrontLeg: origin xyz=0 -17.5 2.4336779769690686 rpy=0 0 0 -> xyz=0 -17.5 2.340944195731549 rpy=0 0 0
- joint Torso_LeftLeg: origin xyz=-0.5 -18 2.4336779769690686 rpy=0 0 0 -> xyz=-0.5 -18 2.340944195731549 rpy=0 0 0
- joint Torso_RightLeg: origin xyz=0.5 -18 2.4336779769690686 rpy=0 0 0 -> xyz=0.5 -18 2.340944195731549 rpy=0 0 0

File: bodyFiles/body0-18520.urdf (robot description, URDF)
Before this commit: robot robot, 9 links, 8 joints
Links:
- link BackLeg: geometry collision box size=0.2 0.5581370648682562 0.2; visual box size=0.2 0.5581370648682562 0.2
- link BackLowerLeg: geometry collision box size=0.2 0.2 0.7740620998868041; visual box size=0.2 0.2 0.7740620998868041
- link FrontLeg: geometry collision box size=0.2 1.040317222978512 0.2; visual box size=0.2 1.040317222978512 0.2
- link FrontLowerLeg: geometry collision box size=0.2 0.2 1.484893877882087; visual box size=0.2 0.2 1.484893877882087
- link LeftLeg: geometry collision box size=0.7549614411153641 0.2 0.2; visual box size=0.7549614411153641 0.2 0.2
- link LeftLowerLeg: geometry collision box size=0.2 0.2 0.8683330780679536; visual box size=0.2 0.2 0.8683330780679536
- link RightLeg: geometry collision box size=1.0367219497118059 0.2 0.2; visual box size=1.0367219497118059 0.2 0.2
- link RightLowerLeg: geometry collision box size=0.2 0.2 1.1954735911496956; visual box size=0.2 0.2 1.1954735911496956
Joints:
- joint BackLeg_BackLowerLeg: origin xyz=0 -1.3985535436056145 0 rpy=0 0 0 -> xyz=0 -0.5581370648682562 0 rpy=0 0 0
- joint FrontLeg_FrontLowerLeg: origin xyz=0 0.8914463519690072 0 rpy=0 0 0 -> xyz=0 1.040317222978512 0 rpy=0 0 0
- joint LeftLeg_LeftLowerLeg: origin xyz=-1.1033983511117864 0 0 rpy=0 0 0 -> xyz=-0.7549614411153641 0 0 rpy=0 0 0
- joint RightLeg_RightLowerLeg: origin xyz=1.4080226158087221 0 0 rpy=0 0 0 -> xyz=1.0367219497118059 0 0 rpy=0 0 0
- joint Torso_BackLeg: origin xyz=0 -18.5 2.408022615808722 rpy=0 0 0 -> xyz=0 -18.5 2.484893877882087 rpy=0 0 0
- joint Torso_FrontLeg: origin xyz=0 -17.5 2.408022615808722 rpy=0 0 0 -> xyz=0 -17.5 2.484893877882087 rpy=0 0 0
- joint Torso_LeftLeg: origin xyz=-0.5 -18 2.408022615808722 rpy=0 0 0 -> xyz=-0.5 -18 2.484893877882087 rpy=0 0 0
- joint Torso_RightLeg: origin xyz=0.5 -18 2.408022615808722 rpy=0 0 0 -> xyz=0.5 -18 2.484893877882087 rpy=0 0 0

File: bodyFiles/body0-1860.urdf (robot description, URDF)
Before this commit: robot robot, 9 links, 8 joints
Links:
- link BackLeg: geometry collision box size=0.2 1.3021301803183265 0.2; visual box size=0.2 1.3021301803183265 0.2
- link BackLowerLeg: geometry collision box size=0.2 0.2 1.0717178281669122; visual box size=0.2 0.2 1.0717178281669122
- link FrontLeg: geometry collision box size=0.2 0.953380288441899 0.2; visual box size=0.2 0.953380288441899 0.2
- link FrontLowerLeg: geometry collision box size=0.2 0.2 0.7127244152616129; visual box size=0.2 0.2 0.7127244152616129
- link LeftLeg: geometry collision box size=0.6405611310351442 0.2 0.2; visual box size=0.6405611310351442 0.2 0.2
- link LeftLowerLeg: geometry collision box size=0.2 0.2 1.0624442105237961; visual box size=0.2 0.2 1.0624442105237961
- link RightLeg: geometry collision box size=0.7878093503674571 0.2 0.2; visual box size=0.7878093503674571 0.2 0.2
- link RightLowerLeg: geometry collision box size=0.2 0.2 0.8883381582752118; visual box size=0.2 0.2 0.8883381582752118
Joints:
- joint BackLeg_BackLowerLeg: origin xyz=0 -1.0596229829869874 0 rpy=0 0 0 -> xyz=0 -1.3021301803183265 0 rpy=0 0 0
- joint FrontLeg_FrontLowerLeg: origin xyz=0 0.7898936848975198 0 rpy=0 0 0 -> xyz=0 0.953380288441899 0 rpy=0 0 0
- joint LeftLeg_LeftLowerLeg: origin xyz=-1.2975513415202524 0 0 rpy=0 0 0 -> xyz=-0.6405611310351442 0 0 rpy=0 0 0
- joint RightLeg_RightLowerLeg: origin xyz=1.4085901177096463 0 0 rpy=0 0 0 -> xyz=0.7878093503674571 0 0 rpy=0 0 0
- joint Torso_BackLeg: origin xyz=0 -18.5 2.4085901177096463 rpy=0 0 0 -> xyz=0 -18.5 2.3021301803183265 rpy=0 0 0
- joint Torso_FrontLeg: origin xyz=0 -17.5 2.4085901177096463 rpy=0 0 0 -> xyz=0 -17.5 2.3021301803183265 rpy=0 0 0
- joint Torso_LeftLeg: origin xyz=-0.5 -18 2.4085901177096463 rpy=0 0 0 -> xyz=-0.5 -18 2.3021301803183265 rpy=0 0 0
- joint Torso_RightLeg: origin xyz=0.5 -18 2.4085901177096463 rpy=0 0 0 -> xyz=0.5 -18 2.3021301803183265 rpy=0 0 0

File: bodyFiles/body0-18630.urdf (robot description, URDF)
Before this commit: robot robot, 9 links, 8 joints
Links:
- link BackLeg: geometry collision box size=0.2 1.157379973445601 0.2; visual box size=0.2 1.157379973445601 0.2
- link BackLowerLeg: geometry collision box size=0.2 0.2 1.4329572338361702; visual box size=0.2 0.2 1.4329572338361702
- link FrontLeg: geometry collision box size=0.2 1.178697896522813 0.2; visual box size=0.2 1.178697896522813 0.2
- link FrontLowerLeg: geometry collision box size=0.2 0.2 0.755449435440359; visual box size=0.2 0.2 0.755449435440359
- link LeftLeg: geometry collision box size=1.4381731088254877 0.2 0.2; visual box size=1.4381731088254877 0.2 0.2
- link LeftLowerLeg: geometry collision box size=0.2 0.2 1.1504416682951455; visual box size=0.2 0.2 1.1504416682951455
- link RightLeg: geometry collision box size=0.8204793490386969 0.2 0.2; visual box size=0.8204793490386969 0.2 0.2
- link RightLowerLeg: geometry collision box size=0.2 0.2 0.8233792087499808; visual box size=0.2 0.2 0.8233792087499808
Joints:
- joint BackLeg_BackLowerLeg: origin xyz=0 -1.4236549717849551 0 rpy=0 0 0 -> xyz=0 -1.157379973445601 0 rpy=0 0 0
- joint FrontLeg_FrontLowerLeg: origin xyz=0 1.4851468699411206 0 rpy=0 0 0 -> xyz=0 1.178697896522813 0 rpy=0 0 0
- joint LeftLeg_LeftLowerLeg: origin xyz=-1.3879623796278522 0 0 rpy=0 0 0 -> xyz=-1.4381731088254877 0 0 rpy=0 0 0
- joint RightLeg_RightLowerLeg: origin xyz=1.4264614283046777 0 0 rpy=0 0 0 -> xyz=0.8204793490386969 0 0 rpy=0 0 0
- joint Torso_BackLeg: origin xyz=0 -18.5 2.4851468699411203 rpy=0 0 0 -> xyz=0 -18.5 2.4381731088254877 rpy=0 0 0
- joint Torso_FrontLeg: origin xyz=0 -17.5 2.4851468699411203 rpy=0 0 0 -> xyz=0 -17.5 2.4381731088254877 rpy=0 0 0
- joint Torso_LeftLeg: origin xyz=-0.5 -18 2.4851468699411203 rpy=0 0 0 -> xyz=-0.5 -18 2.4381731088254877 rpy=0 0 0
- joint Torso_RightLeg: origin xyz=0.5 -18 2.4851468699411203 rpy=0 0 0 -> xyz=0.5 -18 2.4381731088254877 rpy=0 0 0

File: bodyFiles/body0-18680.urdf (robot description, URDF)
Before this commit: robot robot, 9 links, 8 joints
Links:
- link BackLeg: geometry collision box size=0.2 1.0976424797501383 0.2; visual box size=0.2 1.0976424797501383 0.2
- link BackLowerLeg: geometry collision box size=0.2 0.2 0.6164073053087291; visual box size=0.2 0.2 0.6164073053087291
- link FrontLeg: geometry collision box size=0.2 0.8345997144433448 0.2; visual box size=0.2 0.8345997144433448 0.2
- link FrontLowerLeg: geometry collision box size=0.2 0.2 1.4713944755964687; visual box size=0.2 0.2 1.4713944755964687
- link LeftLeg: geometry collision box size=0.9317117747576366 0.2 0.2; visual box size=0.9317117747576366 0.2 0.2
- link LeftLowerLeg: geometry collision box size=0.2 0.2 0.9149110870177265; visual box size=0.2 0.2 0.9149110870177265
- link RightLeg: geometry collision box size=0.9818281985216422 0.2 0.2; visual box size=0.9818281985216422 0.2 0.2
- link RightLowerLeg: geometry collision box size=0.2 0.2 0.8033707430809901; visual box size=0.2 0.2 0.8033707430809901
Joints:
- joint BackLeg_BackLowerLeg: origin xyz=0 -1.0117388806705545 0 rpy=0 0 0 -> xyz=0 -1.0976424797501383 0 rpy=0 0 0
- joint FrontLeg_FrontLowerLeg: origin xyz=0 1.422370990896225 0 rpy=0 0 0 -> xyz=0 0.8345997144433448 0 rpy=0 0 0
- joint LeftLeg_LeftLowerLeg: origin xyz=-0.5008396530104127 0 0 rpy=0 0 0 -> xyz=-0.9317117747576366 0 0 rpy=0 0 0
- joint RightLeg_RightLowerLeg: origin xyz=1.0786881397525059 0 0 rpy=0 0 0 -> xyz=0.9818281985216422 0 0 rpy=0 0 0
- joint Torso_BackLeg: origin xyz=0 -18.5 2.4261433867290165 rpy=0 0 0 -> xyz=0 -18.5 2.471394475596469 rpy=0 0 0
- joint Torso_FrontLeg: origin xyz=0 -17.5 2.4261433867290165 rpy=0 0 0 -> xyz=0 -17.5 2.471394475596469 rpy=0 0 0
- joint Torso_LeftLeg: origin xyz=-0.5 -18 2.4261433867290165 rpy=0 0 0 -> xyz=-0.5 -18 2.471394475596469 rpy=0 0 0
- joint Torso_RightLeg: origin xyz=0.5 -18 2.4261433867290165 rpy=0 0 0 -> xyz=0.5 -18 2.471394475596469 rpy=0 0 0

File: bodyFiles/body0-224.urdf (robot description, URDF)
Before this commit: robot robot, 9 links, 8 joints
Links:
- link BackLeg: geometry collision box size=0.2 1.2655370333528126 0.2; visual box size=0.2 1.2655370333528126 0.2
- link BackLowerLeg: geometry collision box size=0.2 0.2 1.0108434707685399; visual box size=0.2 0.2 1.0108434707685399
- link FrontLeg: geometry collision box size=0.2 1.4851242315113928 0.2; visual box size=0.2 1.4851242315113928 0.2
- link FrontLowerLeg: geometry collision box size=0.2 0.2 1.0571248389885948; visual box size=0.2 0.2 1.0571248389885948
- link LeftLeg: geometry collision box size=1.4883854093460287 0.2 0.2; visual box size=1.4883854093460287 0.2 0.2
- link LeftLowerLeg: geometry collision box size=0.2 0.2 0.93246230443729; visual box size=0.2 0.2 0.93246230443729
- link RightLeg: geometry collision box size=0.6606462674809893 0.2 0.2; visual box size=0.6606462674809893 0.2 0.2
- link RightLowerLeg: geometry collision box size=0.2 0.2 0.516277554870642; visual box size=0.2 0.2 0.516277554870642
Joints:
- joint BackLeg_BackLowerLeg: origin xyz=0 -0.6981551464305015 0 rpy=0 0 0 -> xyz=0 -1.2655370333528126 0 rpy=0 0 0
- joint FrontLeg_FrontLowerLeg: origin xyz=0 1.0912279403210752 0 rpy=0 0 0 -> xyz=0 1.4851242315113928 0 rpy=0 0 0
- joint LeftLeg_LeftLowerLeg: origin xyz=-1.0154102468497068 0 0 rpy=0 0 0 -> xyz=-1.4883854093460287 0 0 rpy=0 0 0
- joint RightLeg_RightLowerLeg: origin xyz=0.513776831045859 0 0 rpy=0 0 0 -> xyz=0.6606462674809893 0 0 rpy=0 0 0
- joint Torso_BackLeg: origin xyz=0 -2.5 2.2673845772449432 rpy=0 0 0 -> xyz=0 -2.5 2.4883854093460287 rpy=0 0 0
- joint Torso_FrontLeg: origin xyz=0 -1.5 2.2673845772449432 rpy=0 0 0 -> xyz=0 -1.5 2.4883854093460287 rpy=0 0 0
- joint Torso_LeftLeg: origin xyz=-0.5 -2 2.2673845772449432 rpy=0 0 0 -> xyz=-0.5 -2 2.4883854093460287 rpy=0 0 0
- joint Torso_RightLeg: origin xyz=0.5 -2 2.2673845772449432 rpy=0 0 0 -> xyz=0.5 -2 2.4883854093460287 rpy=0 0 0
