Commit message: case3, evolved, 10x150

File: bodyFiles/body0-101220.urdf (robot description, URDF)
Before this commit: robot robot, 9 links, 8 joints
Links:
- link BackLeg: geometry collision box size=0.2 0.5319504317329907 0.2; visual box size=0.2 0.5319504317329907 0.2
- link BackLowerLeg: geometry collision box size=0.2 0.2 1.2363435169310943; visual box size=0.2 0.2 1.2363435169310943
- link FrontLeg: geometry collision box size=0.2 1.0967030027841895 0.2; visual box size=0.2 1.0967030027841895 0.2
- link FrontLowerLeg: geometry collision box size=0.2 0.2 0.891336453308446; visual box size=0.2 0.2 0.891336453308446
- link LeftLeg: geometry collision box size=1.37018610665484 0.2 0.2; visual box size=1.37018610665484 0.2 0.2
- link LeftLowerLeg: geometry collision box size=0.2 0.2 1.4631543418720718; visual box size=0.2 0.2 1.4631543418720718
- link RightLeg: geometry collision box size=0.8547951829408119 0.2 0.2; visual box size=0.8547951829408119 0.2 0.2
- link RightLowerLeg: geometry collision box size=0.2 0.2 0.77067122503419; visual box size=0.2 0.2 0.77067122503419
Joints:
- joint BackLeg_BackLowerLeg: origin xyz=0 -0.9634056824232704 0 rpy=0 0 0 -> xyz=0 -0.5319504317329907 0 rpy=0 0 0
- joint FrontLeg_FrontLowerLeg: origin xyz=0 1.2616044261612818 0 rpy=0 0 0 -> xyz=0 1.0967030027841895 0 rpy=0 0 0
- joint LeftLeg_LeftLowerLeg: origin xyz=-0.8973007387681753 0 0 rpy=0 0 0 -> xyz=-1.37018610665484 0 0 rpy=0 0 0
- joint RightLeg_RightLowerLeg: origin xyz=1.1336304960327461 0 0 rpy=0 0 0 -> xyz=0.8547951829408119 0 0 rpy=0 0 0
- joint Torso_BackLeg: origin xyz=0 -10.5 2.470275760387215 rpy=0 0 0 -> xyz=0 -10.5 2.463154341872072 rpy=0 0 0
- joint Torso_FrontLeg: origin xyz=0 -9.5 2.470275760387215 rpy=0 0 0 -> xyz=0 -9.5 2.463154341872072 rpy=0 0 0
- joint Torso_LeftLeg: origin xyz=-0.5 -10 2.470275760387215 rpy=0 0 0 -> xyz=-0.5 -10 2.463154341872072 rpy=0 0 0
- joint Torso_RightLeg: origin xyz=0.5 -10 2.470275760387215 rpy=0 0 0 -> xyz=0.5 -10 2.463154341872072 rpy=0 0 0

File: bodyFiles/body0-101221.urdf (robot description, URDF)
Before this commit: robot robot, 9 links, 8 joints
Links:
- link BackLeg: geometry collision box size=0.2 1.2615450667995303 0.2; visual box size=0.2 1.2615450667995303 0.2
- link BackLowerLeg: geometry collision box size=0.2 0.2 0.6279667564308582; visual box size=0.2 0.2 0.6279667564308582
- link FrontLeg: geometry collision box size=0.2 0.9208821093372731 0.2; visual box size=0.2 0.9208821093372731 0.2
- link FrontLowerLeg: geometry collision box size=0.2 0.2 0.5602889686321292; visual box size=0.2 0.2 0.5602889686321292
- link LeftLeg: geometry collision box size=1.0308440947075734 0.2 0.2; visual box size=1.0308440947075734 0.2 0.2
- link LeftLowerLeg: geometry collision box size=0.2 0.2 1.3697931402738905; visual box size=0.2 0.2 1.3697931402738905
- link RightLeg: geometry collision box size=0.7018855525732339 0.2 0.2; visual box size=0.7018855525732339 0.2 0.2
- link RightLowerLeg: geometry collision box size=0.2 0.2 0.8267530217022542; visual box size=0.2 0.2 0.8267530217022542
Joints:
- joint BackLeg_BackLowerLeg: origin xyz=0 -1.2787372480532082 0 rpy=0 0 0 -> xyz=0 -1.2615450667995303 0 rpy=0 0 0
- joint FrontLeg_FrontLowerLeg: origin xyz=0 0.7248992845758848 0 rpy=0 0 0 -> xyz=0 0.9208821093372731 0 rpy=0 0 0
- joint LeftLeg_LeftLowerLeg: origin xyz=-1.4148755452167712 0 0 rpy=0 0 0 -> xyz=-1.0308440947075734 0 0 rpy=0 0 0
- joint RightLeg_RightLowerLeg: origin xyz=1.4058197769234801 0 0 rpy=0 0 0 -> xyz=0.7018855525732339 0 0 rpy=0 0 0
- joint Torso_BackLeg: origin xyz=0 -10.5 2.414875545216771 rpy=0 0 0 -> xyz=0 -10.5 2.3697931402738908 rpy=0 0 0
- joint Torso_FrontLeg: origin xyz=0 -9.5 2.414875545216771 rpy=0 0 0 -> xyz=0 -9.5 2.3697931402738908 rpy=0 0 0
- joint Torso_LeftLeg: origin xyz=-0.5 -10 2.414875545216771 rpy=0 0 0 -> xyz=-0.5 -10 2.3697931402738908 rpy=0 0 0
- joint Torso_RightLeg: origin xyz=0.5 -10 2.414875545216771 rpy=0 0 0 -> xyz=0.5 -10 2.3697931402738908 rpy=0 0 0

File: bodyFiles/body0-101222.urdf (robot description, URDF)
Before this commit: robot robot, 9 links, 8 joints
Links:
- link BackLeg: geometry collision box size=0.2 1.1300570620353552 0.2; visual box size=0.2 1.1300570620353552 0.2
- link BackLowerLeg: geometry collision box size=0.2 0.2 1.0789875688296682; visual box size=0.2 0.2 1.0789875688296682
- link FrontLeg: geometry collision box size=0.2 1.4946458272871215 0.2; visual box size=0.2 1.4946458272871215 0.2
- link FrontLowerLeg: geometry collision box size=0.2 0.2 1.198484545839814; visual box size=0.2 0.2 1.198484545839814
- link LeftLeg: geometry collision box size=1.4114465782604853 0.2 0.2; visual box size=1.4114465782604853 0.2 0.2
- link LeftLowerLeg: geometry collision box size=0.2 0.2 0.7339191349360232; visual box size=0.2 0.2 0.7339191349360232
- link RightLeg: geometry collision box size=0.6300668997311585 0.2 0.2; visual box size=0.6300668997311585 0.2 0.2
- link RightLowerLeg: geometry collision box size=0.2 0.2 0.6363055052720059; visual box size=0.2 0.2 0.6363055052720059
Joints:
- joint BackLeg_BackLowerLeg: origin xyz=0 -1.0513224798598846 0 rpy=0 0 0 -> xyz=0 -1.1300570620353552 0 rpy=0 0 0
- joint FrontLeg_FrontLowerLeg: origin xyz=0 0.9022731237195615 0 rpy=0 0 0 -> xyz=0 1.4946458272871215 0 rpy=0 0 0
- joint LeftLeg_LeftLowerLeg: origin xyz=-1.0695733922789499 0 0 rpy=0 0 0 -> xyz=-1.4114465782604853 0 0 rpy=0 0 0
- joint RightLeg_RightLowerLeg: origin xyz=0.6823607390342061 0 0 rpy=0 0 0 -> xyz=0.6300668997311585 0 0 rpy=0 0 0
- joint Torso_BackLeg: origin xyz=0 -10.5 2.489847873316184 rpy=0 0 0 -> xyz=0 -10.5 2.4946458272871217 rpy=0 0 0
- joint Torso_FrontLeg: origin xyz=0 -9.5 2.489847873316184 rpy=0 0 0 -> xyz=0 -9.5 2.4946458272871217 rpy=0 0 0
- joint Torso_LeftLeg: origin xyz=-0.5 -10 2.489847873316184 rpy=0 0 0 -> xyz=-0.5 -10 2.4946458272871217 rpy=0 0 0
- joint Torso_RightLeg: origin xyz=0.5 -10 2.489847873316184 rpy=0 0 0 -> xyz=0.5 -10 2.4946458272871217 rpy=0 0 0

File: bodyFiles/body0-101223.urdf (robot description, URDF)
Before this commit: robot robot, 9 links, 8 joints
Links:
- link BackLeg: geometry collision box size=0.2 0.7092841340128183 0.2; visual box size=0.2 0.7092841340128183 0.2
- link BackLowerLeg: geometry collision box size=0.2 0.2 0.6315301844332378; visual box size=0.2 0.2 0.6315301844332378
- link FrontLeg: geometry collision box size=0.2 0.6045592151359729 0.2; visual box size=0.2 0.6045592151359729 0.2
- link FrontLowerLeg: geometry collision box size=0.2 0.2 0.6868005772632474; visual box size=0.2 0.2 0.6868005772632474
- link LeftLeg: geometry collision box size=0.8707483065181584 0.2 0.2; visual box size=0.8707483065181584 0.2 0.2
- link LeftLowerLeg: geometry collision box size=0.2 0.2 0.8108554890456957; visual box size=0.2 0.2 0.8108554890456957
- link RightLeg: geometry collision box size=1.230380471594311 0.2 0.2; visual box size=1.230380471594311 0.2 0.2
- link RightLowerLeg: geometry collision box size=0.2 0.2 1.1021533254437472; visual box size=0.2 0.2 1.1021533254437472
Joints:
- joint BackLeg_BackLowerLeg: origin xyz=0 -0.5305876398828367 0 rpy=0 0 0 -> xyz=0 -0.7092841340128183 0 rpy=0 0 0
- joint FrontLeg_FrontLowerLeg: origin xyz=0 1.3810393046623277 0 rpy=0 0 0 -> xyz=0 0.6045592151359729 0 rpy=0 0 0
- joint LeftLeg_LeftLowerLeg: origin xyz=-1.2148601472229932 0 0 rpy=0 0 0 -> xyz=-0.8707483065181584 0 0 rpy=0 0 0
- joint RightLeg_RightLowerLeg: origin xyz=1.1988217250685125 0 0 rpy=0 0 0 -> xyz=1.230380471594311 0 0 rpy=0 0 0
- joint Torso_BackLeg: origin xyz=0 -10.5 2.402193527314842 rpy=0 0 0 -> xyz=0 -10.5 2.230380471594311 rpy=0 0 0
- joint Torso_FrontLeg: origin xyz=0 -9.5 2.402193527314842 rpy=0 0 0 -> xyz=0 -9.5 2.230380471594311 rpy=0 0 0
- joint Torso_LeftLeg: origin xyz=-0.5 -10 2.402193527314842 rpy=0 0 0 -> xyz=-0.5 -10 2.230380471594311 rpy=0 0 0
- joint Torso_RightLeg: origin xyz=0.5 -10 2.402193527314842 rpy=0 0 0 -> xyz=0.5 -10 2.230380471594311 rpy=0 0 0

File: bodyFiles/body0-101224.urdf (robot description, URDF)
Before this commit: robot robot, 9 links, 8 joints
Links:
- link BackLeg: geometry collision box size=0.2 0.7369367117439393 0.2; visual box size=0.2 0.7369367117439393 0.2
- link BackLowerLeg: geometry collision box size=0.2 0.2 1.4814881132637254; visual box size=0.2 0.2 1.4814881132637254
- link FrontLeg: geometry collision box size=0.2 0.699169794391177 0.2; visual box size=0.2 0.699169794391177 0.2
- link FrontLowerLeg: geometry collision box size=0.2 0.2 0.5661738984114714; visual box size=0.2 0.2 0.5661738984114714
- link LeftLeg: geometry collision box size=0.9869828657956574 0.2 0.2; visual box size=0.9869828657956574 0.2 0.2
- link LeftLowerLeg: geometry collision box size=0.2 0.2 1.121424593458817; visual box size=0.2 0.2 1.121424593458817
- link RightLeg: geometry collision box size=1.2992691657009452 0.2 0.2; visual box size=1.2992691657009452 0.2 0.2
- link RightLowerLeg: geometry collision box size=0.2 0.2 0.6128584729302271; visual box size=0.2 0.2 0.6128584729302271
Joints:
- joint BackLeg_BackLowerLeg: origin xyz=0 -1.0609350742151928 0 rpy=0 0 0 -> xyz=0 -0.7369367117439393 0 rpy=0 0 0
- joint FrontLeg_FrontLowerLeg: origin xyz=0 1.0912389744993027 0 rpy=0 0 0 -> xyz=0 0.699169794391177 0 rpy=0 0 0
- joint LeftLeg_LeftLowerLeg: origin xyz=-1.1768169104675992 0 0 rpy=0 0 0 -> xyz=-0.9869828657956574 0 0 rpy=0 0 0
- joint RightLeg_RightLowerLeg: origin xyz=0.6299889901898353 0 0 rpy=0 0 0 -> xyz=1.2992691657009452 0 0 rpy=0 0 0
- joint Torso_BackLeg: origin xyz=0 -10.5 2.3970167507091795 rpy=0 0 0 -> xyz=0 -10.5 2.481488113263725 rpy=0 0 0
- joint Torso_FrontLeg: origin xyz=0 -9.5 2.3970167507091795 rpy=0 0 0 -> xyz=0 -9.5 2.481488113263725 rpy=0 0 0
- joint Torso_LeftLeg: origin xyz=-0.5 -10 2.3970167507091795 rpy=0 0 0 -> xyz=-0.5 -10 2.481488113263725 rpy=0 0 0
- joint Torso_RightLeg: origin xyz=0.5 -10 2.3970167507091795 rpy=0 0 0 -> xyz=0.5 -10 2.481488113263725 rpy=0 0 0

File: bodyFiles/body0-101225.urdf (robot description, URDF)
Before this commit: robot robot, 9 links, 8 joints
Links:
- link BackLeg: geometry collision box size=0.2 1.3106162794241678 0.2; visual box size=0.2 1.3106162794241678 0.2
- link BackLowerLeg: geometry collision box size=0.2 0.2 0.9101029162952421; visual box size=0.2 0.2 0.9101029162952421
- link FrontLeg: geometry collision box size=0.2 0.5176719549085717 0.2; visual box size=0.2 0.5176719549085717 0.2
- link FrontLowerLeg: geometry collision box size=0.2 0.2 1.3984851219337906; visual box size=0.2 0.2 1.3984851219337906
- link LeftLeg: geometry collision box size=0.7512600520016638 0.2 0.2; visual box size=0.7512600520016638 0.2 0.2
- link LeftLowerLeg: geometry collision box size=0.2 0.2 0.5328659890037727; visual box size=0.2 0.2 0.5328659890037727
- link RightLeg: geometry collision box size=0.9272595191419802 0.2 0.2; visual box size=0.9272595191419802 0.2 0.2
- link RightLowerLeg: geometry collision box size=0.2 0.2 0.726123515785933; visual box size=0.2 0.2 0.726123515785933
Joints:
- joint BackLeg_BackLowerLeg: origin xyz=0 -0.9975504527501676 0 rpy=0 0 0 -> xyz=0 -1.3106162794241678 0 rpy=0 0 0
- joint FrontLeg_FrontLowerLeg: origin xyz=0 0.833245534502029 0 rpy=0 0 0 -> xyz=0 0.5176719549085717 0 rpy=0 0 0
- joint LeftLeg_LeftLowerLeg: origin xyz=-1.1762087555097593 0 0 rpy=0 0 0 -> xyz=-0.7512600520016638 0 0 rpy=0 0 0
- joint RightLeg_RightLowerLeg: origin xyz=1.1897326663716146 0 0 rpy=0 0 0 -> xyz=0.9272595191419802 0 0 rpy=0 0 0
- joint Torso_BackLeg: origin xyz=0 -10.5 2.2849939923049765 rpy=0 0 0 -> xyz=0 -10.5 2.3984851219337906 rpy=0 0 0
- joint Torso_FrontLeg: origin xyz=0 -9.5 2.2849939923049765 rpy=0 0 0 -> xyz=0 -9.5 2.3984851219337906 rpy=0 0 0
- joint Torso_LeftLeg: origin xyz=-0.5 -10 2.2849939923049765 rpy=0 0 0 -> xyz=-0.5 -10 2.3984851219337906 rpy=0 0 0
- joint Torso_RightLeg: origin xyz=0.5 -10 2.2849939923049765 rpy=0 0 0 -> xyz=0.5 -10 2.3984851219337906 rpy=0 0 0

File: bodyFiles/body0-101226.urdf (robot description, URDF)
Before this commit: robot robot, 9 links, 8 joints
Links:
- link BackLeg: geometry collision box size=0.2 0.6733950959127997 0.2; visual box size=0.2 0.6733950959127997 0.2
- link BackLowerLeg: geometry collision box size=0.2 0.2 1.4442259692049406; visual box size=0.2 0.2 1.4442259692049406
- link FrontLeg: geometry collision box size=0.2 0.6344444327887053 0.2; visual box size=0.2 0.6344444327887053 0.2
- link FrontLowerLeg: geometry collision box size=0.2 0.2 1.4649190969603816; visual box size=0.2 0.2 1.4649190969603816
- link LeftLeg: geometry collision box size=0.8273558227674042 0.2 0.2; visual box size=0.8273558227674042 0.2 0.2
- link LeftLowerLeg: geometry collision box size=0.2 0.2 0.6311152999052582; visual box size=0.2 0.2 0.6311152999052582
- link RightLeg: geometry collision box size=0.7931195654173978 0.2 0.2; visual box size=0.7931195654173978 0.2 0.2
- link RightLowerLeg: geometry collision box size=0.2 0.2 1.2126181000241956; visual box size=0.2 0.2 1.2126181000241956
Joints:
- joint BackLeg_BackLowerLeg: origin xyz=0 -0.5647732602450478 0 rpy=0 0 0 -> xyz=0 -0.6733950959127997 0 rpy=0 0 0
- joint FrontLeg_FrontLowerLeg: origin xyz=0 0.6887457995164751 0 rpy=0 0 0 -> xyz=0 0.6344444327887053 0 rpy=0 0 0
- joint LeftLeg_LeftLowerLeg: origin xyz=-1.0678388667924343 0 0 rpy=0 0 0 -> xyz=-0.8273558227674042 0 0 rpy=0 0 0
- joint RightLeg_RightLowerLeg: origin xyz=1.4085591974689873 0 0 rpy=0 0 0 -> xyz=0.7931195654173978 0 0 rpy=0 0 0
- joint Torso_BackLeg: origin xyz=0 -10.5 2.4085591974689873 rpy=0 0 0 -> xyz=0 -10.5 2.4649190969603816 rpy=0 0 0
- joint Torso_FrontLeg: origin xyz=0 -9.5 2.4085591974689873 rpy=0 0 0 -> xyz=0 -9.5 2.4649190969603816 rpy=0 0 0
- joint Torso_LeftLeg: origin xyz=-0.5 -10 2.4085591974689873 rpy=0 0 0 -> xyz=-0.5 -10 2.4649190969603816 rpy=0 0 0
- joint Torso_RightLeg: origin xyz=0.5 -10 2.4085591974689873 rpy=0 0 0 -> xyz=0.5 -10 2.4649190969603816 rpy=0 0 0

File: bodyFiles/body0-101227.urdf (robot description, URDF)
Before this commit: robot robot, 9 links, 8 joints
Links:
- link BackLeg: geometry collision box size=0.2 0.73865046718386 0.2; visual box size=0.2 0.73865046718386 0.2
- link BackLowerLeg: geometry collision box size=0.2 0.2 0.5633226301906208; visual box size=0.2 0.2 0.5633226301906208
- link FrontLeg: geometry collision box size=0.2 0.8829230013939459 0.2; visual box size=0.2 0.8829230013939459 0.2
- link FrontLowerLeg: geometry collision box size=0.2 0.2 1.4392640182898457; visual box size=0.2 0.2 1.4392640182898457
- link LeftLeg: geometry collision box size=1.4284590890708544 0.2 0.2; visual box size=1.4284590890708544 0.2 0.2
- link LeftLowerLeg: geometry collision box size=0.2 0.2 0.7414726443376278; visual box size=0.2 0.2 0.7414726443376278
- link RightLeg: geometry collision box size=0.8841688126826049 0.2 0.2; visual box size=0.8841688126826049 0.2 0.2
- link RightLowerLeg: geometry collision box size=0.2 0.2 1.1660903744778914; visual box size=0.2 0.2 1.1660903744778914
Joints:
- joint BackLeg_BackLowerLeg: origin xyz=0 -1.044365544155216 0 rpy=0 0 0 -> xyz=0 -0.73865046718386 0 rpy=0 0 0
- joint FrontLeg_FrontLowerLeg: origin xyz=0 0.9443381134230567 0 rpy=0 0 0 -> xyz=0 0.8829230013939459 0 rpy=0 0 0
- joint LeftLeg_LeftLowerLeg: origin xyz=-0.5165584146983927 0 0 rpy=0 0 0 -> xyz=-1.4284590890708544 0 0 rpy=0 0 0
- joint RightLeg_RightLowerLeg: origin xyz=1.4657355241669738 0 0 rpy=0 0 0 -> xyz=0.8841688126826049 0 0 rpy=0 0 0
- joint Torso_BackLeg: origin xyz=0 -10.5 2.465735524166974 rpy=0 0 0 -> xyz=0 -10.5 2.4392640182898457 rpy=0 0 0
- joint Torso_FrontLeg: origin xyz=0 -9.5 2.465735524166974 rpy=0 0 0 -> xyz=0 -9.5 2.4392640182898457 rpy=0 0 0
- joint Torso_LeftLeg: origin xyz=-0.5 -10 2.465735524166974 rpy=0 0 0 -> xyz=-0.5 -10 2.4392640182898457 rpy=0 0 0
- joint Torso_RightLeg: origin xyz=0.5 -10 2.465735524166974 rpy=0 0 0 -> xyz=0.5 -10 2.4392640182898457 rpy=0 0 0

File: bodyFiles/body0-101228.urdf (robot description, URDF)
Before this commit: robot robot, 9 links, 8 joints
Links:
- link BackLeg: geometry collision box size=0.2 1.2746716875793291 0.2; visual box size=0.2 1.2746716875793291 0.2
- link BackLowerLeg: geometry collision box size=0.2 0.2 0.903381360223909; visual box size=0.2 0.2 0.903381360223909
- link FrontLeg: geometry collision box size=0.2 0.7802676061103565 0.2; visual box size=0.2 0.7802676061103565 0.2
- link FrontLowerLeg: geometry collision box size=0.2 0.2 0.908409201333066; visual box size=0.2 0.2 0.908409201333066
- link LeftLeg: geometry collision box size=0.616431621882398 0.2 0.2; visual box size=0.616431621882398 0.2 0.2
- link LeftLowerLeg: geometry collision box size=0.2 0.2 0.9262154735299474; visual box size=0.2 0.2 0.9262154735299474
- link RightLeg: geometry collision box size=0.9241297677041921 0.2 0.2; visual box size=0.9241297677041921 0.2 0.2
- link RightLowerLeg: geometry collision box size=0.2 0.2 1.0744679360397442; visual box size=0.2 0.2 1.0744679360397442
Joints:
- joint BackLeg_BackLowerLeg: origin xyz=0 -0.7028029173552196 0 rpy=0 0 0 -> xyz=0 -1.2746716875793291 0 rpy=0 0 0
- joint FrontLeg_FrontLowerLeg: origin xyz=0 1.4562255474108898 0 rpy=0 0 0 -> xyz=0 0.7802676061103565 0 rpy=0 0 0
- joint LeftLeg_LeftLowerLeg: origin xyz=-0.9797844408941506 0 0 rpy=0 0 0 -> xyz=-0.616431621882398 0 0 rpy=0 0 0
- joint RightLeg_RightLowerLeg: origin xyz=1.2171833202753661 0 0 rpy=0 0 0 -> xyz=0.9241297677041921 0 0 rpy=0 0 0
- joint Torso_BackLeg: origin xyz=0 -10.5 2.45622554741089 rpy=0 0 0 -> xyz=0 -10.5 2.274671687579329 rpy=0 0 0
- joint Torso_FrontLeg: origin xyz=0 -9.5 2.45622554741089 rpy=0 0 0 -> xyz=0 -9.5 2.274671687579329 rpy=0 0 0
- joint Torso_LeftLeg: origin xyz=-0.5 -10 2.45622554741089 rpy=0 0 0 -> xyz=-0.5 -10 2.274671687579329 rpy=0 0 0
- joint Torso_RightLeg: origin xyz=0.5 -10 2.45622554741089 rpy=0 0 0 -> xyz=0.5 -10 2.274671687579329 rpy=0 0 0

File: bodyFiles/body0-101229.urdf (robot description, URDF)
Before this commit: robot robot, 9 links, 8 joints
Links:
- link BackLeg: geometry collision box size=0.2 0.9855002917032472 0.2; visual box size=0.2 0.9855002917032472 0.2
- link BackLowerLeg: geometry collision box size=0.2 0.2 0.5919986573424911; visual box size=0.2 0.2 0.5919986573424911
- link FrontLeg: geometry collision box size=0.2 0.5608903452803458 0.2; visual box size=0.2 0.5608903452803458 0.2
- link FrontLowerLeg: geometry collision box size=0.2 0.2 1.362747464684447; visual box size=0.2 0.2 1.362747464684447
- link LeftLeg: geometry collision box size=0.7768700035668051 0.2 0.2; visual box size=0.7768700035668051 0.2 0.2
- link LeftLowerLeg: geometry collision box size=0.2 0.2 0.5039598619178167; visual box size=0.2 0.2 0.5039598619178167
- link RightLeg: geometry collision box size=1.0668544202653525 0.2 0.2; visual box size=1.0668544202653525 0.2 0.2
- link RightLowerLeg: geometry collision box size=0.2 0.2 1.0997105545964745; visual box size=0.2 0.2 1.0997105545964745
Joints:
- joint BackLeg_BackLowerLeg: origin xyz=0 -1.458125278515697 0 rpy=0 0 0 -> xyz=0 -0.9855002917032472 0 rpy=0 0 0
- joint FrontLeg_FrontLowerLeg: origin xyz=0 0.8535308973062438 0 rpy=0 0 0 -> xyz=0 0.5608903452803458 0 rpy=0 0 0
- joint LeftLeg_LeftLowerLeg: origin xyz=-0.9597653668014496 0 0 rpy=0 0 0 -> xyz=-0.7768700035668051 0 0 rpy=0 0 0
- joint RightLeg_RightLowerLeg: origin xyz=0.8110716525716972 0 0 rpy=0 0 0 -> xyz=1.0668544202653525 0 0 rpy=0 0 0
- joint Torso_BackLeg: origin xyz=0 -10.5 2.458125278515697 rpy=0 0 0 -> xyz=0 -10.5 2.362747464684447 rpy=0 0 0
- joint Torso_FrontLeg: origin xyz=0 -9.5 2.458125278515697 rpy=0 0 0 -> xyz=0 -9.5 2.362747464684447 rpy=0 0 0
- joint Torso_LeftLeg: origin xyz=-0.5 -10 2.458125278515697 rpy=0 0 0 -> xyz=-0.5 -10 2.362747464684447 rpy=0 0 0
- joint Torso_RightLeg: origin xyz=0.5 -10 2.458125278515697 rpy=0 0 0 -> xyz=0.5 -10 2.362747464684447 rpy=0 0 0

File: bodyFiles/body0-10125.urdf (robot description, URDF)
Before this commit: robot robot, 9 links, 8 joints
Links:
- link BackLeg: geometry collision box size=0.2 0.609786825554618 0.2; visual box size=0.2 0.609786825554618 0.2
- link BackLowerLeg: geometry collision box size=0.2 0.2 0.986609032410476; visual box size=0.2 0.2 0.986609032410476
- link FrontLeg: geometry collision box size=0.2 1.4861288029812885 0.2; visual box size=0.2 1.4861288029812885 0.2
- link FrontLowerLeg: geometry collision box size=0.2 0.2 1.1882266398724575; visual box size=0.2 0.2 1.1882266398724575
- link LeftLeg: geometry collision box size=1.3309546714460625 0.2 0.2; visual box size=1.3309546714460625 0.2 0.2
- link LeftLowerLeg: geometry collision box size=0.2 0.2 1.3815215887193846; visual box size=0.2 0.2 1.3815215887193846
- link RightLeg: geometry collision box size=1.0537015044209377 0.2 0.2; visual box size=1.0537015044209377 0.2 0.2
- link RightLowerLeg: geometry collision box size=0.2 0.2 1.4690908661149475; visual box size=0.2 0.2 1.4690908661149475
Joints:
- joint BackLeg_BackLowerLeg: origin xyz=0 -1.4085034630559505 0 rpy=0 0 0 -> xyz=0 -0.609786825554618 0 rpy=0 0 0
- joint FrontLeg_FrontLowerLeg: origin xyz=0 0.6388316790857079 0 rpy=0 0 0 -> xyz=0 1.4861288029812885 0 rpy=0 0 0
- joint LeftLeg_LeftLowerLeg: origin xyz=-1.104167301358808 0 0 rpy=0 0 0 -> xyz=-1.3309546714460625 0 0 rpy=0 0 0
- joint RightLeg_RightLowerLeg: origin xyz=1.0667327408513774 0 0 rpy=0 0 0 -> xyz=1.0537015044209377 0 0 rpy=0 0 0
- joint Torso_BackLeg: origin xyz=0 -10.5 2.4085034630559505 rpy=0 0 0 -> xyz=0 -10.5 2.4861288029812885 rpy=0 0 0
- joint Torso_FrontLeg: origin xyz=0 -9.5 2.4085034630559505 rpy=0 0 0 -> xyz=0 -9.5 2.4861288029812885 rpy=0 0 0
- joint Torso_LeftLeg: origin xyz=-0.5 -10 2.4085034630559505 rpy=0 0 0 -> xyz=-0.5 -10 2.4861288029812885 rpy=0 0 0
- joint Torso_RightLeg: origin xyz=0.5 -10 2.4085034630559505 rpy=0 0 0 -> xyz=0.5 -10 2.4861288029812885 rpy=0 0 0
