Commit message: case3, evolved, 10x150

File: bodyFiles/body0-10126.urdf (robot description, URDF)
Before this commit: robot robot, 9 links, 8 joints
Links:
- link BackLeg: geometry collision box size=0.2 1.42345159481419 0.2; visual box size=0.2 1.42345159481419 0.2
- link BackLowerLeg: geometry collision box size=0.2 0.2 0.519226082738684; visual box size=0.2 0.2 0.519226082738684
- link FrontLeg: geometry collision box size=0.2 0.8736736825875894 0.2; visual box size=0.2 0.8736736825875894 0.2
- link FrontLowerLeg: geometry collision box size=0.2 0.2 0.8083254070960556; visual box size=0.2 0.2 0.8083254070960556
- link LeftLeg: geometry collision box size=1.0366499476566151 0.2 0.2; visual box size=1.0366499476566151 0.2 0.2
- link LeftLowerLeg: geometry collision box size=0.2 0.2 1.4535651226226105; visual box size=0.2 0.2 1.4535651226226105
- link RightLeg: geometry collision box size=0.6888624712668237 0.2 0.2; visual box size=0.6888624712668237 0.2 0.2
- link RightLowerLeg: geometry collision box size=0.2 0.2 0.6341396582685329; visual box size=0.2 0.2 0.6341396582685329
Joints:
- joint BackLeg_BackLowerLeg: origin xyz=0 -0.9084466639368907 0 rpy=0 0 0 -> xyz=0 -1.42345159481419 0 rpy=0 0 0
- joint FrontLeg_FrontLowerLeg: origin xyz=0 1.4321861028609582 0 rpy=0 0 0 -> xyz=0 0.8736736825875894 0 rpy=0 0 0
- joint LeftLeg_LeftLowerLeg: origin xyz=-0.5804368903267044 0 0 rpy=0 0 0 -> xyz=-1.0366499476566151 0 0 rpy=0 0 0
- joint RightLeg_RightLowerLeg: origin xyz=0.6190818040337186 0 0 rpy=0 0 0 -> xyz=0.6888624712668237 0 0 rpy=0 0 0
- joint Torso_BackLeg: origin xyz=0 -10.5 2.432186102860958 rpy=0 0 0 -> xyz=0 -10.5 2.4535651226226105 rpy=0 0 0
- joint Torso_FrontLeg: origin xyz=0 -9.5 2.432186102860958 rpy=0 0 0 -> xyz=0 -9.5 2.4535651226226105 rpy=0 0 0
- joint Torso_LeftLeg: origin xyz=-0.5 -10 2.432186102860958 rpy=0 0 0 -> xyz=-0.5 -10 2.4535651226226105 rpy=0 0 0
- joint Torso_RightLeg: origin xyz=0.5 -10 2.432186102860958 rpy=0 0 0 -> xyz=0.5 -10 2.4535651226226105 rpy=0 0 0

File: bodyFiles/body0-10127.urdf (robot description, URDF)
Before this commit: robot robot, 9 links, 8 joints
Links:
- link BackLeg: geometry collision box size=0.2 1.3129529809095177 0.2; visual box size=0.2 1.3129529809095177 0.2
- link BackLowerLeg: geometry collision box size=0.2 0.2 1.469086512366397; visual box size=0.2 0.2 1.469086512366397
- link FrontLeg: geometry collision box size=0.2 0.8594821042948787 0.2; visual box size=0.2 0.8594821042948787 0.2
- link FrontLowerLeg: geometry collision box size=0.2 0.2 1.229019889385727; visual box size=0.2 0.2 1.229019889385727
- link LeftLeg: geometry collision box size=1.3814286359986827 0.2 0.2; visual box size=1.3814286359986827 0.2 0.2
- link LeftLowerLeg: geometry collision box size=0.2 0.2 1.12024757080131; visual box size=0.2 0.2 1.12024757080131
- link RightLeg: geometry collision box size=1.49040277364801 0.2 0.2; visual box size=1.49040277364801 0.2 0.2
- link RightLowerLeg: geometry collision box size=0.2 0.2 1.3258756904339455; visual box size=0.2 0.2 1.3258756904339455
Joints:
- joint BackLeg_BackLowerLeg: origin xyz=0 -0.7185866790359823 0 rpy=0 0 0 -> xyz=0 -1.3129529809095177 0 rpy=0 0 0
- joint FrontLeg_FrontLowerLeg: origin xyz=0 1.0350156322439577 0 rpy=0 0 0 -> xyz=0 0.8594821042948787 0 rpy=0 0 0
- joint LeftLeg_LeftLowerLeg: origin xyz=-0.8243930382640302 0 0 rpy=0 0 0 -> xyz=-1.3814286359986827 0 0 rpy=0 0 0
- joint RightLeg_RightLowerLeg: origin xyz=1.0780934310539885 0 0 rpy=0 0 0 -> xyz=1.49040277364801 0 0 rpy=0 0 0
- joint Torso_BackLeg: origin xyz=0 -10.5 2.36008895373363 rpy=0 0 0 -> xyz=0 -10.5 2.49040277364801 rpy=0 0 0
- joint Torso_FrontLeg: origin xyz=0 -9.5 2.36008895373363 rpy=0 0 0 -> xyz=0 -9.5 2.49040277364801 rpy=0 0 0
- joint Torso_LeftLeg: origin xyz=-0.5 -10 2.36008895373363 rpy=0 0 0 -> xyz=-0.5 -10 2.49040277364801 rpy=0 0 0
- joint Torso_RightLeg: origin xyz=0.5 -10 2.36008895373363 rpy=0 0 0 -> xyz=0.5 -10 2.49040277364801 rpy=0 0 0

File: bodyFiles/body0-10128.urdf (robot description, URDF)
Before this commit: robot robot, 9 links, 8 joints
Links:
- link BackLeg: geometry collision box size=0.2 1.2104899923721488 0.2; visual box size=0.2 1.2104899923721488 0.2
- link BackLowerLeg: geometry collision box size=0.2 0.2 1.0612026054886776; visual box size=0.2 0.2 1.0612026054886776
- link FrontLeg: geometry collision box size=0.2 1.3916068592686766 0.2; visual box size=0.2 1.3916068592686766 0.2
- link FrontLowerLeg: geometry collision box size=0.2 0.2 0.872155645405973; visual box size=0.2 0.2 0.872155645405973
- link LeftLeg: geometry collision box size=1.3893191100707347 0.2 0.2; visual box size=1.3893191100707347 0.2 0.2
- link LeftLowerLeg: geometry collision box size=0.2 0.2 0.6361771849974347; visual box size=0.2 0.2 0.6361771849974347
- link RightLeg: geometry collision box size=0.9306905741829308 0.2 0.2; visual box size=0.9306905741829308 0.2 0.2
- link RightLowerLeg: geometry collision box size=0.2 0.2 0.8290929356007722; visual box size=0.2 0.2 0.8290929356007722
Joints:
- joint BackLeg_BackLowerLeg: origin xyz=0 -0.7016210151163151 0 rpy=0 0 0 -> xyz=0 -1.2104899923721488 0 rpy=0 0 0
- joint FrontLeg_FrontLowerLeg: origin xyz=0 1.20763075853496 0 rpy=0 0 0 -> xyz=0 1.3916068592686766 0 rpy=0 0 0
- joint LeftLeg_LeftLowerLeg: origin xyz=-1.265756587488485 0 0 rpy=0 0 0 -> xyz=-1.3893191100707347 0 0 rpy=0 0 0
- joint RightLeg_RightLowerLeg: origin xyz=0.7406515714792306 0 0 rpy=0 0 0 -> xyz=0.9306905741829308 0 0 rpy=0 0 0
- joint Torso_BackLeg: origin xyz=0 -10.5 2.265756587488485 rpy=0 0 0 -> xyz=0 -10.5 2.3916068592686766 rpy=0 0 0
- joint Torso_FrontLeg: origin xyz=0 -9.5 2.265756587488485 rpy=0 0 0 -> xyz=0 -9.5 2.3916068592686766 rpy=0 0 0
- joint Torso_LeftLeg: origin xyz=-0.5 -10 2.265756587488485 rpy=0 0 0 -> xyz=-0.5 -10 2.3916068592686766 rpy=0 0 0
- joint Torso_RightLeg: origin xyz=0.5 -10 2.265756587488485 rpy=0 0 0 -> xyz=0.5 -10 2.3916068592686766 rpy=0 0 0

File: bodyFiles/body0-10129.urdf (robot description, URDF)
Before this commit: robot robot, 9 links, 8 joints
Links:
- link BackLeg: geometry collision box size=0.2 1.1453664085423574 0.2; visual box size=0.2 1.1453664085423574 0.2
- link BackLowerLeg: geometry collision box size=0.2 0.2 0.8488163816490376; visual box size=0.2 0.2 0.8488163816490376
- link FrontLeg: geometry collision box size=0.2 0.5030743484205691 0.2; visual box size=0.2 0.5030743484205691 0.2
- link FrontLowerLeg: geometry collision box size=0.2 0.2 0.6106034794433042; visual box size=0.2 0.2 0.6106034794433042
- link LeftLeg: geometry collision box size=0.7580096634272554 0.2 0.2; visual box size=0.7580096634272554 0.2 0.2
- link LeftLowerLeg: geometry collision box size=0.2 0.2 1.227492072325079; visual box size=0.2 0.2 1.227492072325079
- link RightLeg: geometry collision box size=1.016526405397173 0.2 0.2; visual box size=1.016526405397173 0.2 0.2
- link RightLowerLeg: geometry collision box size=0.2 0.2 0.6405699818357363; visual box size=0.2 0.2 0.6405699818357363
Joints:
- joint BackLeg_BackLowerLeg: origin xyz=0 -0.58814393377418 0 rpy=0 0 0 -> xyz=0 -1.1453664085423574 0 rpy=0 0 0
- joint FrontLeg_FrontLowerLeg: origin xyz=0 1.2334742282715867 0 rpy=0 0 0 -> xyz=0 0.5030743484205691 0 rpy=0 0 0
- joint LeftLeg_LeftLowerLeg: origin xyz=-1.0679719066896636 0 0 rpy=0 0 0 -> xyz=-0.7580096634272554 0 0 rpy=0 0 0
- joint RightLeg_RightLowerLeg: origin xyz=1.1370240302908223 0 0 rpy=0 0 0 -> xyz=1.016526405397173 0 0 rpy=0 0 0
- joint Torso_BackLeg: origin xyz=0 -10.5 2.253356861654022 rpy=0 0 0 -> xyz=0 -10.5 2.227492072325079 rpy=0 0 0
- joint Torso_FrontLeg: origin xyz=0 -9.5 2.253356861654022 rpy=0 0 0 -> xyz=0 -9.5 2.227492072325079 rpy=0 0 0
- joint Torso_LeftLeg: origin xyz=-0.5 -10 2.253356861654022 rpy=0 0 0 -> xyz=-0.5 -10 2.227492072325079 rpy=0 0 0
- joint Torso_RightLeg: origin xyz=0.5 -10 2.253356861654022 rpy=0 0 0 -> xyz=0.5 -10 2.227492072325079 rpy=0 0 0

File: bodyFiles/body0-101325.urdf (robot description, URDF)
Before this commit: robot robot, 9 links, 8 joints
Links:
- link BackLeg: geometry collision box size=0.2 1.1580560165054838 0.2; visual box size=0.2 1.1580560165054838 0.2
- link BackLowerLeg: geometry collision box size=0.2 0.2 0.8140455819382587; visual box size=0.2 0.2 0.8140455819382587
- link FrontLeg: geometry collision box size=0.2 1.3134163021476137 0.2; visual box size=0.2 1.3134163021476137 0.2
- link FrontLowerLeg: geometry collision box size=0.2 0.2 1.3580758910224535; visual box size=0.2 0.2 1.3580758910224535
- link LeftLeg: geometry collision box size=0.5734970562215963 0.2 0.2; visual box size=0.5734970562215963 0.2 0.2
- link LeftLowerLeg: geometry collision box size=0.2 0.2 1.0583448554919777; visual box size=0.2 0.2 1.0583448554919777
- link RightLeg: geometry collision box size=0.6154627212618355 0.2 0.2; visual box size=0.6154627212618355 0.2 0.2
- link RightLowerLeg: geometry collision box size=0.2 0.2 0.8240061136266689; visual box size=0.2 0.2 0.8240061136266689
Joints:
- joint BackLeg_BackLowerLeg: origin xyz=0 -0.571310813279803 0 rpy=0 0 0 -> xyz=0 -1.1580560165054838 0 rpy=0 0 0
- joint FrontLeg_FrontLowerLeg: origin xyz=0 1.1704514315758092 0 rpy=0 0 0 -> xyz=0 1.3134163021476137 0 rpy=0 0 0
- joint LeftLeg_LeftLowerLeg: origin xyz=-0.8850688507738395 0 0 rpy=0 0 0 -> xyz=-0.5734970562215963 0 0 rpy=0 0 0
- joint RightLeg_RightLowerLeg: origin xyz=0.8436740138928163 0 0 rpy=0 0 0 -> xyz=0.6154627212618355 0 0 rpy=0 0 0
- joint Torso_BackLeg: origin xyz=0 -10.5 2.331563269706439 rpy=0 0 0 -> xyz=0 -10.5 2.3580758910224535 rpy=0 0 0
- joint Torso_FrontLeg: origin xyz=0 -9.5 2.331563269706439 rpy=0 0 0 -> xyz=0 -9.5 2.3580758910224535 rpy=0 0 0
- joint Torso_LeftLeg: origin xyz=-0.5 -10 2.331563269706439 rpy=0 0 0 -> xyz=-0.5 -10 2.3580758910224535 rpy=0 0 0
- joint Torso_RightLeg: origin xyz=0.5 -10 2.331563269706439 rpy=0 0 0 -> xyz=0.5 -10 2.3580758910224535 rpy=0 0 0

File: bodyFiles/body0-101326.urdf (robot description, URDF)
Before this commit: robot robot, 9 links, 8 joints
Links:
- link BackLeg: geometry collision box size=0.2 1.014023370752437 0.2; visual box size=0.2 1.014023370752437 0.2
- link BackLowerLeg: geometry collision box size=0.2 0.2 1.4241500037782309; visual box size=0.2 0.2 1.4241500037782309
- link FrontLeg: geometry collision box size=0.2 1.2303089113716923 0.2; visual box size=0.2 1.2303089113716923 0.2
- link FrontLowerLeg: geometry collision box size=0.2 0.2 1.1938369526458485; visual box size=0.2 0.2 1.1938369526458485
- link LeftLeg: geometry collision box size=0.541925385655425 0.2 0.2; visual box size=0.541925385655425 0.2 0.2
- link LeftLowerLeg: geometry collision box size=0.2 0.2 1.2113797113528775; visual box size=0.2 0.2 1.2113797113528775
- link RightLeg: geometry collision box size=1.0810640723265537 0.2 0.2; visual box size=1.0810640723265537 0.2 0.2
- link RightLowerLeg: geometry collision box size=0.2 0.2 0.8382497759611245; visual box size=0.2 0.2 0.8382497759611245
Joints:
- joint BackLeg_BackLowerLeg: origin xyz=0 -0.603034689297907 0 rpy=0 0 0 -> xyz=0 -1.014023370752437 0 rpy=0 0 0
- joint FrontLeg_FrontLowerLeg: origin xyz=0 1.4645864173143939 0 rpy=0 0 0 -> xyz=0 1.2303089113716923 0 rpy=0 0 0
- joint LeftLeg_LeftLowerLeg: origin xyz=-0.5965199326330171 0 0 rpy=0 0 0 -> xyz=-0.541925385655425 0 0 rpy=0 0 0
- joint RightLeg_RightLowerLeg: origin xyz=1.1823675613878586 0 0 rpy=0 0 0 -> xyz=1.0810640723265537 0 0 rpy=0 0 0
- joint Torso_BackLeg: origin xyz=0 -10.5 2.464586417314394 rpy=0 0 0 -> xyz=0 -10.5 2.424150003778231 rpy=0 0 0
- joint Torso_FrontLeg: origin xyz=0 -9.5 2.464586417314394 rpy=0 0 0 -> xyz=0 -9.5 2.424150003778231 rpy=0 0 0
- joint Torso_LeftLeg: origin xyz=-0.5 -10 2.464586417314394 rpy=0 0 0 -> xyz=-0.5 -10 2.424150003778231 rpy=0 0 0
- joint Torso_RightLeg: origin xyz=0.5 -10 2.464586417314394 rpy=0 0 0 -> xyz=0.5 -10 2.424150003778231 rpy=0 0 0

File: bodyFiles/body0-101327.urdf (robot description, URDF)
Before this commit: robot robot, 9 links, 8 joints
Links:
- link BackLeg: geometry collision box size=0.2 1.472194925191054 0.2; visual box size=0.2 1.472194925191054 0.2
- link BackLowerLeg: geometry collision box size=0.2 0.2 1.1483931697541858; visual box size=0.2 0.2 1.1483931697541858
- link FrontLeg: geometry collision box size=0.2 0.6899866587806156 0.2; visual box size=0.2 0.6899866587806156 0.2
- link FrontLowerLeg: geometry collision box size=0.2 0.2 1.067427110792916; visual box size=0.2 0.2 1.067427110792916
- link LeftLeg: geometry collision box size=0.6901475322984767 0.2 0.2; visual box size=0.6901475322984767 0.2 0.2
- link LeftLowerLeg: geometry collision box size=0.2 0.2 0.5442663350188159; visual box size=0.2 0.2 0.5442663350188159
- link RightLeg: geometry collision box size=1.1662313818007284 0.2 0.2; visual box size=1.1662313818007284 0.2 0.2
- link RightLowerLeg: geometry collision box size=0.2 0.2 0.8328543094956986; visual box size=0.2 0.2 0.8328543094956986
Joints:
- joint BackLeg_BackLowerLeg: origin xyz=0 -0.9740449102132307 0 rpy=0 0 0 -> xyz=0 -1.472194925191054 0 rpy=0 0 0
- joint FrontLeg_FrontLowerLeg: origin xyz=0 0.8141015844223752 0 rpy=0 0 0 -> xyz=0 0.6899866587806156 0 rpy=0 0 0
- joint LeftLeg_LeftLowerLeg: origin xyz=-1.1619082144353765 0 0 rpy=0 0 0 -> xyz=-0.6901475322984767 0 0 rpy=0 0 0
- joint RightLeg_RightLowerLeg: origin xyz=1.186578899952159 0 0 rpy=0 0 0 -> xyz=1.1662313818007284 0 0 rpy=0 0 0
- joint Torso_BackLeg: origin xyz=0 -10.5 2.277152957293625 rpy=0 0 0 -> xyz=0 -10.5 2.472194925191054 rpy=0 0 0
- joint Torso_FrontLeg: origin xyz=0 -9.5 2.277152957293625 rpy=0 0 0 -> xyz=0 -9.5 2.472194925191054 rpy=0 0 0
- joint Torso_LeftLeg: origin xyz=-0.5 -10 2.277152957293625 rpy=0 0 0 -> xyz=-0.5 -10 2.472194925191054 rpy=0 0 0
- joint Torso_RightLeg: origin xyz=0.5 -10 2.277152957293625 rpy=0 0 0 -> xyz=0.5 -10 2.472194925191054 rpy=0 0 0

File: bodyFiles/body0-101328.urdf (robot description, URDF)
Before this commit: robot robot, 9 links, 8 joints
Links:
- link BackLeg: geometry collision box size=0.2 1.0781300760432826 0.2; visual box size=0.2 1.0781300760432826 0.2
- link BackLowerLeg: geometry collision box size=0.2 0.2 1.44463101777879; visual box size=0.2 0.2 1.44463101777879
- link FrontLeg: geometry collision box size=0.2 0.8774946852034108 0.2; visual box size=0.2 0.8774946852034108 0.2
- link FrontLowerLeg: geometry collision box size=0.2 0.2 1.1429964425339905; visual box size=0.2 0.2 1.1429964425339905
- link LeftLeg: geometry collision box size=1.2157153424961706 0.2 0.2; visual box size=1.2157153424961706 0.2 0.2
- link LeftLowerLeg: geometry collision box size=0.2 0.2 0.6575112123960158; visual box size=0.2 0.2 0.6575112123960158
- link RightLeg: geometry collision box size=0.9751934513707929 0.2 0.2; visual box size=0.9751934513707929 0.2 0.2
- link RightLowerLeg: geometry collision box size=0.2 0.2 0.8854801517107219; visual box size=0.2 0.2 0.8854801517107219
Joints:
- joint BackLeg_BackLowerLeg: origin xyz=0 -0.8306986107901135 0 rpy=0 0 0 -> xyz=0 -1.0781300760432826 0 rpy=0 0 0
- joint FrontLeg_FrontLowerLeg: origin xyz=0 0.5532550568675532 0 rpy=0 0 0 -> xyz=0 0.8774946852034108 0 rpy=0 0 0
- joint LeftLeg_LeftLowerLeg: origin xyz=-0.5906123255764437 0 0 rpy=0 0 0 -> xyz=-1.2157153424961706 0 0 rpy=0 0 0
- joint RightLeg_RightLowerLeg: origin xyz=1.132680183636532 0 0 rpy=0 0 0 -> xyz=0.9751934513707929 0 0 rpy=0 0 0
- joint Torso_BackLeg: origin xyz=0 -10.5 2.1690354764122066 rpy=0 0 0 -> xyz=0 -10.5 2.44463101777879 rpy=0 0 0
- joint Torso_FrontLeg: origin xyz=0 -9.5 2.1690354764122066 rpy=0 0 0 -> xyz=0 -9.5 2.44463101777879 rpy=0 0 0
- joint Torso_LeftLeg: origin xyz=-0.5 -10 2.1690354764122066 rpy=0 0 0 -> xyz=-0.5 -10 2.44463101777879 rpy=0 0 0
- joint Torso_RightLeg: origin xyz=0.5 -10 2.1690354764122066 rpy=0 0 0 -> xyz=0.5 -10 2.44463101777879 rpy=0 0 0

File: bodyFiles/body0-101329.urdf (robot description, URDF)
Before this commit: robot robot, 9 links, 8 joints
Links:
- link BackLeg: geometry collision box size=0.2 0.6443169364596457 0.2; visual box size=0.2 0.6443169364596457 0.2
- link BackLowerLeg: geometry collision box size=0.2 0.2 1.4496587814732576; visual box size=0.2 0.2 1.4496587814732576
- link FrontLeg: geometry collision box size=0.2 0.5028913235030448 0.2; visual box size=0.2 0.5028913235030448 0.2
- link FrontLowerLeg: geometry collision box size=0.2 0.2 1.3087190957341903; visual box size=0.2 0.2 1.3087190957341903
- link LeftLeg: geometry collision box size=1.3561872870652816 0.2 0.2; visual box size=1.3561872870652816 0.2 0.2
- link LeftLowerLeg: geometry collision box size=0.2 0.2 1.2245213980280392; visual box size=0.2 0.2 1.2245213980280392
- link RightLeg: geometry collision box size=1.3434251052237387 0.2 0.2; visual box size=1.3434251052237387 0.2 0.2
- link RightLowerLeg: geometry collision box size=0.2 0.2 0.7661265614431194; visual box size=0.2 0.2 0.7661265614431194
Joints:
- joint BackLeg_BackLowerLeg: origin xyz=0 -0.7667332486961986 0 rpy=0 0 0 -> xyz=0 -0.6443169364596457 0 rpy=0 0 0
- joint FrontLeg_FrontLowerLeg: origin xyz=0 0.63038818501925 0 rpy=0 0 0 -> xyz=0 0.5028913235030448 0 rpy=0 0 0
- joint LeftLeg_LeftLowerLeg: origin xyz=-1.337354085682243 0 0 rpy=0 0 0 -> xyz=-1.3561872870652816 0 0 rpy=0 0 0
- joint RightLeg_RightLowerLeg: origin xyz=1.4414700349107048 0 0 rpy=0 0 0 -> xyz=1.3434251052237387 0 0 rpy=0 0 0
- joint Torso_BackLeg: origin xyz=0 -10.5 2.441470034910705 rpy=0 0 0 -> xyz=0 -10.5 2.4496587814732576 rpy=0 0 0
- joint Torso_FrontLeg: origin xyz=0 -9.5 2.441470034910705 rpy=0 0 0 -> xyz=0 -9.5 2.4496587814732576 rpy=0 0 0
- joint Torso_LeftLeg: origin xyz=-0.5 -10 2.441470034910705 rpy=0 0 0 -> xyz=-0.5 -10 2.4496587814732576 rpy=0 0 0
- joint Torso_RightLeg: origin xyz=0.5 -10 2.441470034910705 rpy=0 0 0 -> xyz=0.5 -10 2.4496587814732576 rpy=0 0 0
