Commit message: collected 350 of 1/6 cubes, now ready for dynamic obstacles by bot position

File: bodyFiles/body0-104720.urdf (robot description, URDF)
Before this commit: robot robot, 9 links, 8 joints
Links:
- link BackLeg: geometry collision box size=0.2 0.651406957225098 0.2; visual box size=0.2 0.651406957225098 0.2
- link BackLowerLeg: geometry collision box size=0.2 0.2 1.2094204711841778; visual box size=0.2 0.2 1.2094204711841778
- link FrontLeg: geometry collision box size=0.2 1.4611055652395875 0.2; visual box size=0.2 1.4611055652395875 0.2
- link FrontLowerLeg: geometry collision box size=0.2 0.2 0.7564108089344633; visual box size=0.2 0.2 0.7564108089344633
- link LeftLeg: geometry collision box size=0.6396264718140404 0.2 0.2; visual box size=0.6396264718140404 0.2 0.2
- link LeftLowerLeg: geometry collision box size=0.2 0.2 1.3501120896474368; visual box size=0.2 0.2 1.3501120896474368
- link RightLeg: geometry collision box size=0.5892754979227791 0.2 0.2; visual box size=0.5892754979227791 0.2 0.2
- link RightLowerLeg: geometry collision box size=0.2 0.2 0.6807952581950769; visual box size=0.2 0.2 0.6807952581950769
Joints:
- joint BackLeg_BackLowerLeg: origin xyz=0 -0.7531634734977798 0 rpy=0 0 0 -> xyz=0 -0.651406957225098 0 rpy=0 0 0
- joint FrontLeg_FrontLowerLeg: origin xyz=0 1.0148634449820504 0 rpy=0 0 0 -> xyz=0 1.4611055652395875 0 rpy=0 0 0
- joint LeftLeg_LeftLowerLeg: origin xyz=-1.4946719545145792 0 0 rpy=0 0 0 -> xyz=-0.6396264718140404 0 0 rpy=0 0 0
- joint RightLeg_RightLowerLeg: origin xyz=1.2359569597034996 0 0 rpy=0 0 0 -> xyz=0.5892754979227791 0 0 rpy=0 0 0
- joint Torso_BackLeg: origin xyz=0 -10.5 2.4946719545145792 rpy=0 0 0 -> xyz=0 -10.5 2.4611055652395875 rpy=0 0 0
- joint Torso_FrontLeg: origin xyz=0 -9.5 2.4946719545145792 rpy=0 0 0 -> xyz=0 -9.5 2.4611055652395875 rpy=0 0 0
- joint Torso_LeftLeg: origin xyz=-0.5 -10 2.4946719545145792 rpy=0 0 0 -> xyz=-0.5 -10 2.4611055652395875 rpy=0 0 0
- joint Torso_RightLeg: origin xyz=0.5 -10 2.4946719545145792 rpy=0 0 0 -> xyz=0.5 -10 2.4611055652395875 rpy=0 0 0

File: bodyFiles/body0-104721.urdf (robot description, URDF)
Before this commit: robot robot, 9 links, 8 joints
Links:
- link BackLeg: geometry collision box size=0.2 1.2039723182951416 0.2; visual box size=0.2 1.2039723182951416 0.2
- link BackLowerLeg: geometry collision box size=0.2 0.2 1.2745096288727753; visual box size=0.2 0.2 1.2745096288727753
- link FrontLeg: geometry collision box size=0.2 0.6224204186522945 0.2; visual box size=0.2 0.6224204186522945 0.2
- link FrontLowerLeg: geometry collision box size=0.2 0.2 1.279846640916624; visual box size=0.2 0.2 1.279846640916624
- link LeftLeg: geometry collision box size=1.006574714371144 0.2 0.2; visual box size=1.006574714371144 0.2 0.2
- link LeftLowerLeg: geometry collision box size=0.2 0.2 1.0169969604115532; visual box size=0.2 0.2 1.0169969604115532
- link RightLeg: geometry collision box size=1.1747069632613754 0.2 0.2; visual box size=1.1747069632613754 0.2 0.2
- link RightLowerLeg: geometry collision box size=0.2 0.2 0.9292500789040081; visual box size=0.2 0.2 0.9292500789040081
Joints:
- joint BackLeg_BackLowerLeg: origin xyz=0 -0.6915975629296751 0 rpy=0 0 0 -> xyz=0 -1.2039723182951416 0 rpy=0 0 0
- joint FrontLeg_FrontLowerLeg: origin xyz=0 1.321580157710295 0 rpy=0 0 0 -> xyz=0 0.6224204186522945 0 rpy=0 0 0
- joint LeftLeg_LeftLowerLeg: origin xyz=-0.8886528432550819 0 0 rpy=0 0 0 -> xyz=-1.006574714371144 0 0 rpy=0 0 0
- joint RightLeg_RightLowerLeg: origin xyz=1.473784300626987 0 0 rpy=0 0 0 -> xyz=1.1747069632613754 0 0 rpy=0 0 0
- joint Torso_BackLeg: origin xyz=0 -10.5 2.4863578587671546 rpy=0 0 0 -> xyz=0 -10.5 2.279846640916624 rpy=0 0 0
- joint Torso_FrontLeg: origin xyz=0 -9.5 2.4863578587671546 rpy=0 0 0 -> xyz=0 -9.5 2.279846640916624 rpy=0 0 0
- joint Torso_LeftLeg: origin xyz=-0.5 -10 2.4863578587671546 rpy=0 0 0 -> xyz=-0.5 -10 2.279846640916624 rpy=0 0 0
- joint Torso_RightLeg: origin xyz=0.5 -10 2.4863578587671546 rpy=0 0 0 -> xyz=0.5 -10 2.279846640916624 rpy=0 0 0

File: bodyFiles/body0-104722.urdf (robot description, URDF)
Before this commit: robot robot, 9 links, 8 joints
Links:
- link BackLeg: geometry collision box size=0.2 1.3558421582412494 0.2; visual box size=0.2 1.3558421582412494 0.2
- link BackLowerLeg: geometry collision box size=0.2 0.2 1.0869046603798882; visual box size=0.2 0.2 1.0869046603798882
- link FrontLeg: geometry collision box size=0.2 0.6235161814786055 0.2; visual box size=0.2 0.6235161814786055 0.2
- link FrontLowerLeg: geometry collision box size=0.2 0.2 1.4169000142290349; visual box size=0.2 0.2 1.4169000142290349
- link LeftLeg: geometry collision box size=0.7047249069622904 0.2 0.2; visual box size=0.7047249069622904 0.2 0.2
- link LeftLowerLeg: geometry collision box size=0.2 0.2 1.4467892557340831; visual box size=0.2 0.2 1.4467892557340831
- link RightLeg: geometry collision box size=0.6986855312873005 0.2 0.2; visual box size=0.6986855312873005 0.2 0.2
- link RightLowerLeg: geometry collision box size=0.2 0.2 0.6171128116903652; visual box size=0.2 0.2 0.6171128116903652
Joints:
- joint BackLeg_BackLowerLeg: origin xyz=0 -1.4564628467743415 0 rpy=0 0 0 -> xyz=0 -1.3558421582412494 0 rpy=0 0 0
- joint FrontLeg_FrontLowerLeg: origin xyz=0 1.1720719892170521 0 rpy=0 0 0 -> xyz=0 0.6235161814786055 0 rpy=0 0 0
- joint LeftLeg_LeftLowerLeg: origin xyz=-0.8486400546228385 0 0 rpy=0 0 0 -> xyz=-0.7047249069622904 0 0 rpy=0 0 0
- joint RightLeg_RightLowerLeg: origin xyz=1.3798198914825308 0 0 rpy=0 0 0 -> xyz=0.6986855312873005 0 0 rpy=0 0 0
- joint Torso_BackLeg: origin xyz=0 -10.5 2.4951661703818226 rpy=0 0 0 -> xyz=0 -10.5 2.446789255734083 rpy=0 0 0
- joint Torso_FrontLeg: origin xyz=0 -9.5 2.4951661703818226 rpy=0 0 0 -> xyz=0 -9.5 2.446789255734083 rpy=0 0 0
- joint Torso_LeftLeg: origin xyz=-0.5 -10 2.4951661703818226 rpy=0 0 0 -> xyz=-0.5 -10 2.446789255734083 rpy=0 0 0
- joint Torso_RightLeg: origin xyz=0.5 -10 2.4951661703818226 rpy=0 0 0 -> xyz=0.5 -10 2.446789255734083 rpy=0 0 0

File: bodyFiles/body0-104723.urdf (robot description, URDF)
Before this commit: robot robot, 9 links, 8 joints
Links:
- link BackLeg: geometry collision box size=0.2 0.9656288759511134 0.2; visual box size=0.2 0.9656288759511134 0.2
- link BackLowerLeg: geometry collision box size=0.2 0.2 1.4289572450206172; visual box size=0.2 0.2 1.4289572450206172
- link FrontLeg: geometry collision box size=0.2 1.3513197768216596 0.2; visual box size=0.2 1.3513197768216596 0.2
- link FrontLowerLeg: geometry collision box size=0.2 0.2 1.0317267773416599; visual box size=0.2 0.2 1.0317267773416599
- link LeftLeg: geometry collision box size=1.4459891778912666 0.2 0.2; visual box size=1.4459891778912666 0.2 0.2
- link LeftLowerLeg: geometry collision box size=0.2 0.2 1.0580396703592303; visual box size=0.2 0.2 1.0580396703592303
- link RightLeg: geometry collision box size=1.489934815534482 0.2 0.2; visual box size=1.489934815534482 0.2 0.2
- link RightLowerLeg: geometry collision box size=0.2 0.2 1.1343466320209008; visual box size=0.2 0.2 1.1343466320209008
Joints:
- joint BackLeg_BackLowerLeg: origin xyz=0 -0.6413510946624721 0 rpy=0 0 0 -> xyz=0 -0.9656288759511134 0 rpy=0 0 0
- joint FrontLeg_FrontLowerLeg: origin xyz=0 0.5708769166801878 0 rpy=0 0 0 -> xyz=0 1.3513197768216596 0 rpy=0 0 0
- joint LeftLeg_LeftLowerLeg: origin xyz=-1.0816679442475499 0 0 rpy=0 0 0 -> xyz=-1.4459891778912666 0 0 rpy=0 0 0
- joint RightLeg_RightLowerLeg: origin xyz=1.442815242120386 0 0 rpy=0 0 0 -> xyz=1.489934815534482 0 0 rpy=0 0 0
- joint Torso_BackLeg: origin xyz=0 -10.5 2.442815242120386 rpy=0 0 0 -> xyz=0 -10.5 2.489934815534482 rpy=0 0 0
- joint Torso_FrontLeg: origin xyz=0 -9.5 2.442815242120386 rpy=0 0 0 -> xyz=0 -9.5 2.489934815534482 rpy=0 0 0
- joint Torso_LeftLeg: origin xyz=-0.5 -10 2.442815242120386 rpy=0 0 0 -> xyz=-0.5 -10 2.489934815534482 rpy=0 0 0
- joint Torso_RightLeg: origin xyz=0.5 -10 2.442815242120386 rpy=0 0 0 -> xyz=0.5 -10 2.489934815534482 rpy=0 0 0

File: bodyFiles/body0-104724.urdf (robot description, URDF)
Before this commit: robot robot, 9 links, 8 joints
Links:
- link BackLeg: geometry collision box size=0.2 1.0828114420745811 0.2; visual box size=0.2 1.0828114420745811 0.2
- link BackLowerLeg: geometry collision box size=0.2 0.2 1.0261802853846307; visual box size=0.2 0.2 1.0261802853846307
- link FrontLeg: geometry collision box size=0.2 0.5587865989925322 0.2; visual box size=0.2 0.5587865989925322 0.2
- link FrontLowerLeg: geometry collision box size=0.2 0.2 0.8368517265323504; visual box size=0.2 0.2 0.8368517265323504
- link LeftLeg: geometry collision box size=1.4643060018114897 0.2 0.2; visual box size=1.4643060018114897 0.2 0.2
- link LeftLowerLeg: geometry collision box size=0.2 0.2 1.1009268405726882; visual box size=0.2 0.2 1.1009268405726882
- link RightLeg: geometry collision box size=0.8425705139290934 0.2 0.2; visual box size=0.8425705139290934 0.2 0.2
- link RightLowerLeg: geometry collision box size=0.2 0.2 0.5633251354925279; visual box size=0.2 0.2 0.5633251354925279
Joints:
- joint BackLeg_BackLowerLeg: origin xyz=0 -1.2431393133371262 0 rpy=0 0 0 -> xyz=0 -1.0828114420745811 0 rpy=0 0 0
- joint FrontLeg_FrontLowerLeg: origin xyz=0 1.22446273513027 0 rpy=0 0 0 -> xyz=0 0.5587865989925322 0 rpy=0 0 0
- joint LeftLeg_LeftLowerLeg: origin xyz=-0.7014766865676275 0 0 rpy=0 0 0 -> xyz=-1.4643060018114897 0 0 rpy=0 0 0
- joint RightLeg_RightLowerLeg: origin xyz=0.6403650042314872 0 0 rpy=0 0 0 -> xyz=0.8425705139290934 0 0 rpy=0 0 0
- joint Torso_BackLeg: origin xyz=0 -10.5 2.2896844113671806 rpy=0 0 0 -> xyz=0 -10.5 2.4643060018114897 rpy=0 0 0
- joint Torso_FrontLeg: origin xyz=0 -9.5 2.2896844113671806 rpy=0 0 0 -> xyz=0 -9.5 2.4643060018114897 rpy=0 0 0
- joint Torso_LeftLeg: origin xyz=-0.5 -10 2.2896844113671806 rpy=0 0 0 -> xyz=-0.5 -10 2.4643060018114897 rpy=0 0 0
- joint Torso_RightLeg: origin xyz=0.5 -10 2.2896844113671806 rpy=0 0 0 -> xyz=0.5 -10 2.4643060018114897 rpy=0 0 0

File: bodyFiles/body0-104725.urdf (robot description, URDF)
Before this commit: robot robot, 9 links, 8 joints
Links:
- link BackLeg: geometry collision box size=0.2 0.9376163449621246 0.2; visual box size=0.2 0.9376163449621246 0.2
- link BackLowerLeg: geometry collision box size=0.2 0.2 0.8758172378368125; visual box size=0.2 0.2 0.8758172378368125
- link FrontLeg: geometry collision box size=0.2 0.7233407878970094 0.2; visual box size=0.2 0.7233407878970094 0.2
- link FrontLowerLeg: geometry collision box size=0.2 0.2 1.1972731137801984; visual box size=0.2 0.2 1.1972731137801984
- link LeftLeg: geometry collision box size=0.8681765039501625 0.2 0.2; visual box size=0.8681765039501625 0.2 0.2
- link LeftLowerLeg: geometry collision box size=0.2 0.2 0.6183753351064977; visual box size=0.2 0.2 0.6183753351064977
- link RightLeg: geometry collision box size=0.7066556040456669 0.2 0.2; visual box size=0.7066556040456669 0.2 0.2
- link RightLowerLeg: geometry collision box size=0.2 0.2 1.4393485866628066; visual box size=0.2 0.2 1.4393485866628066
Joints:
- joint BackLeg_BackLowerLeg: origin xyz=0 -0.5238095343161759 0 rpy=0 0 0 -> xyz=0 -0.9376163449621246 0 rpy=0 0 0
- joint FrontLeg_FrontLowerLeg: origin xyz=0 1.0144008218177532 0 rpy=0 0 0 -> xyz=0 0.7233407878970094 0 rpy=0 0 0
- joint LeftLeg_LeftLowerLeg: origin xyz=-0.6113171697096333 0 0 rpy=0 0 0 -> xyz=-0.8681765039501625 0 0 rpy=0 0 0
- joint RightLeg_RightLowerLeg: origin xyz=1.4827940543201321 0 0 rpy=0 0 0 -> xyz=0.7066556040456669 0 0 rpy=0 0 0
- joint Torso_BackLeg: origin xyz=0 -10.5 2.482794054320132 rpy=0 0 0 -> xyz=0 -10.5 2.4393485866628066 rpy=0 0 0
- joint Torso_FrontLeg: origin xyz=0 -9.5 2.482794054320132 rpy=0 0 0 -> xyz=0 -9.5 2.4393485866628066 rpy=0 0 0
- joint Torso_LeftLeg: origin xyz=-0.5 -10 2.482794054320132 rpy=0 0 0 -> xyz=-0.5 -10 2.4393485866628066 rpy=0 0 0
- joint Torso_RightLeg: origin xyz=0.5 -10 2.482794054320132 rpy=0 0 0 -> xyz=0.5 -10 2.4393485866628066 rpy=0 0 0

File: bodyFiles/body0-104726.urdf (robot description, URDF)
Before this commit: robot robot, 9 links, 8 joints
Links:
- link BackLeg: geometry collision box size=0.2 1.3564523351081297 0.2; visual box size=0.2 1.3564523351081297 0.2
- link BackLowerLeg: geometry collision box size=0.2 0.2 0.7803610385671702; visual box size=0.2 0.2 0.7803610385671702
- link FrontLeg: geometry collision box size=0.2 0.7729272772059502 0.2; visual box size=0.2 0.7729272772059502 0.2
- link FrontLowerLeg: geometry collision box size=0.2 0.2 1.0290311001115002; visual box size=0.2 0.2 1.0290311001115002
- link LeftLeg: geometry collision box size=0.5597736479084287 0.2 0.2; visual box size=0.5597736479084287 0.2 0.2
- link LeftLowerLeg: geometry collision box size=0.2 0.2 0.6490164892004525; visual box size=0.2 0.2 0.6490164892004525
- link RightLeg: geometry collision box size=1.1538590103813027 0.2 0.2; visual box size=1.1538590103813027 0.2 0.2
- link RightLowerLeg: geometry collision box size=0.2 0.2 0.72467819702255; visual box size=0.2 0.2 0.72467819702255
Joints:
- joint BackLeg_BackLowerLeg: origin xyz=0 -0.6778380807495019 0 rpy=0 0 0 -> xyz=0 -1.3564523351081297 0 rpy=0 0 0
- joint FrontLeg_FrontLowerLeg: origin xyz=0 1.0868795103846622 0 rpy=0 0 0 -> xyz=0 0.7729272772059502 0 rpy=0 0 0
- joint LeftLeg_LeftLowerLeg: origin xyz=-0.9821047454141695 0 0 rpy=0 0 0 -> xyz=-0.5597736479084287 0 0 rpy=0 0 0
- joint RightLeg_RightLowerLeg: origin xyz=0.8955455191673162 0 0 rpy=0 0 0 -> xyz=1.1538590103813027 0 0 rpy=0 0 0
- joint Torso_BackLeg: origin xyz=0 -10.5 2.2137520042306247 rpy=0 0 0 -> xyz=0 -10.5 2.3564523351081297 rpy=0 0 0
- joint Torso_FrontLeg: origin xyz=0 -9.5 2.2137520042306247 rpy=0 0 0 -> xyz=0 -9.5 2.3564523351081297 rpy=0 0 0
- joint Torso_LeftLeg: origin xyz=-0.5 -10 2.2137520042306247 rpy=0 0 0 -> xyz=-0.5 -10 2.3564523351081297 rpy=0 0 0
- joint Torso_RightLeg: origin xyz=0.5 -10 2.2137520042306247 rpy=0 0 0 -> xyz=0.5 -10 2.3564523351081297 rpy=0 0 0

File: bodyFiles/body0-104727.urdf (robot description, URDF)
Before this commit: robot robot, 9 links, 8 joints
Links:
- link BackLeg: geometry collision box size=0.2 0.9283286710994529 0.2; visual box size=0.2 0.9283286710994529 0.2
- link BackLowerLeg: geometry collision box size=0.2 0.2 0.8033444580515934; visual box size=0.2 0.2 0.8033444580515934
- link FrontLeg: geometry collision box size=0.2 1.4214153367317348 0.2; visual box size=0.2 1.4214153367317348 0.2
- link FrontLowerLeg: geometry collision box size=0.2 0.2 1.4471785144646105; visual box size=0.2 0.2 1.4471785144646105
- link LeftLeg: geometry collision box size=0.5245064284268757 0.2 0.2; visual box size=0.5245064284268757 0.2 0.2
- link LeftLowerLeg: geometry collision box size=0.2 0.2 0.8927143317327341; visual box size=0.2 0.2 0.8927143317327341
- link RightLeg: geometry collision box size=1.1971491040977829 0.2 0.2; visual box size=1.1971491040977829 0.2 0.2
- link RightLowerLeg: geometry collision box size=0.2 0.2 0.754562545497727; visual box size=0.2 0.2 0.754562545497727
Joints:
- joint BackLeg_BackLowerLeg: origin xyz=0 -0.9102875294206811 0 rpy=0 0 0 -> xyz=0 -0.9283286710994529 0 rpy=0 0 0
- joint FrontLeg_FrontLowerLeg: origin xyz=0 0.5725188796674602 0 rpy=0 0 0 -> xyz=0 1.4214153367317348 0 rpy=0 0 0
- joint LeftLeg_LeftLowerLeg: origin xyz=-1.1553952024259786 0 0 rpy=0 0 0 -> xyz=-0.5245064284268757 0 0 rpy=0 0 0
- joint RightLeg_RightLowerLeg: origin xyz=1.056459742392605 0 0 rpy=0 0 0 -> xyz=1.1971491040977829 0 0 rpy=0 0 0
- joint Torso_BackLeg: origin xyz=0 -10.5 2.446475767359834 rpy=0 0 0 -> xyz=0 -10.5 2.4471785144646105 rpy=0 0 0
- joint Torso_FrontLeg: origin xyz=0 -9.5 2.446475767359834 rpy=0 0 0 -> xyz=0 -9.5 2.4471785144646105 rpy=0 0 0
- joint Torso_LeftLeg: origin xyz=-0.5 -10 2.446475767359834 rpy=0 0 0 -> xyz=-0.5 -10 2.4471785144646105 rpy=0 0 0
- joint Torso_RightLeg: origin xyz=0.5 -10 2.446475767359834 rpy=0 0 0 -> xyz=0.5 -10 2.4471785144646105 rpy=0 0 0

File: bodyFiles/body0-104728.urdf (robot description, URDF)
Before this commit: robot robot, 9 links, 8 joints
Links:
- link BackLeg: geometry collision box size=0.2 0.566065690293851 0.2; visual box size=0.2 0.566065690293851 0.2
- link BackLowerLeg: geometry collision box size=0.2 0.2 1.0356941859781088; visual box size=0.2 0.2 1.0356941859781088
- link FrontLeg: geometry collision box size=0.2 1.4629581616879686 0.2; visual box size=0.2 1.4629581616879686 0.2
- link FrontLowerLeg: geometry collision box size=0.2 0.2 1.0865813502186614; visual box size=0.2 0.2 1.0865813502186614
- link LeftLeg: geometry collision box size=1.4573936017112998 0.2 0.2; visual box size=1.4573936017112998 0.2 0.2
- link LeftLowerLeg: geometry collision box size=0.2 0.2 1.218824275525035; visual box size=0.2 0.2 1.218824275525035
- link RightLeg: geometry collision box size=0.8196217884845067 0.2 0.2; visual box size=0.8196217884845067 0.2 0.2
- link RightLowerLeg: geometry collision box size=0.2 0.2 1.2986507220158765; visual box size=0.2 0.2 1.2986507220158765
Joints:
- joint BackLeg_BackLowerLeg: origin xyz=0 -1.4196123446808278 0 rpy=0 0 0 -> xyz=0 -0.566065690293851 0 rpy=0 0 0
- joint FrontLeg_FrontLowerLeg: origin xyz=0 0.9677886154218 0 rpy=0 0 0 -> xyz=0 1.4629581616879686 0 rpy=0 0 0
- joint LeftLeg_LeftLowerLeg: origin xyz=-0.669522054470305 0 0 rpy=0 0 0 -> xyz=-1.4573936017112998 0 0 rpy=0 0 0
- joint RightLeg_RightLowerLeg: origin xyz=0.6237679943916898 0 0 rpy=0 0 0 -> xyz=0.8196217884845067 0 0 rpy=0 0 0
- joint Torso_BackLeg: origin xyz=0 -10.5 2.4196123446808278 rpy=0 0 0 -> xyz=0 -10.5 2.4629581616879683 rpy=0 0 0
- joint Torso_FrontLeg: origin xyz=0 -9.5 2.4196123446808278 rpy=0 0 0 -> xyz=0 -9.5 2.4629581616879683 rpy=0 0 0
- joint Torso_LeftLeg: origin xyz=-0.5 -10 2.4196123446808278 rpy=0 0 0 -> xyz=-0.5 -10 2.4629581616879683 rpy=0 0 0
- joint Torso_RightLeg: origin xyz=0.5 -10 2.4196123446808278 rpy=0 0 0 -> xyz=0.5 -10 2.4629581616879683 rpy=0 0 0

File: bodyFiles/body0-104729.urdf (robot description, URDF)
Before this commit: robot robot, 9 links, 8 joints
Links:
- link BackLeg: geometry collision box size=0.2 0.7677521087624102 0.2; visual box size=0.2 0.7677521087624102 0.2
- link BackLowerLeg: geometry collision box size=0.2 0.2 1.033126887281187; visual box size=0.2 0.2 1.033126887281187
- link FrontLeg: geometry collision box size=0.2 0.5516954694486 0.2; visual box size=0.2 0.5516954694486 0.2
- link FrontLowerLeg: geometry collision box size=0.2 0.2 1.4403458930318447; visual box size=0.2 0.2 1.4403458930318447
- link LeftLeg: geometry collision box size=1.1068438098360065 0.2 0.2; visual box size=1.1068438098360065 0.2 0.2
- link LeftLowerLeg: geometry collision box size=0.2 0.2 0.8873352308761197; visual box size=0.2 0.2 0.8873352308761197
- link RightLeg: geometry collision box size=1.4744096996049523 0.2 0.2; visual box size=1.4744096996049523 0.2 0.2
- link RightLowerLeg: geometry collision box size=0.2 0.2 1.1479347197442749; visual box size=0.2 0.2 1.1479347197442749
Joints:
- joint BackLeg_BackLowerLeg: origin xyz=0 -1.2219842298495667 0 rpy=0 0 0 -> xyz=0 -0.7677521087624102 0 rpy=0 0 0
- joint FrontLeg_FrontLowerLeg: origin xyz=0 0.8865777307973665 0 rpy=0 0 0 -> xyz=0 0.5516954694486 0 rpy=0 0 0
- joint LeftLeg_LeftLowerLeg: origin xyz=-0.9366333200761993 0 0 rpy=0 0 0 -> xyz=-1.1068438098360065 0 0 rpy=0 0 0
- joint RightLeg_RightLowerLeg: origin xyz=0.9586964996755069 0 0 rpy=0 0 0 -> xyz=1.4744096996049523 0 0 rpy=0 0 0
- joint Torso_BackLeg: origin xyz=0 -10.5 2.221984229849567 rpy=0 0 0 -> xyz=0 -10.5 2.4744096996049523 rpy=0 0 0
- joint Torso_FrontLeg: origin xyz=0 -9.5 2.221984229849567 rpy=0 0 0 -> xyz=0 -9.5 2.4744096996049523 rpy=0 0 0
- joint Torso_LeftLeg: origin xyz=-0.5 -10 2.221984229849567 rpy=0 0 0 -> xyz=-0.5 -10 2.4744096996049523 rpy=0 0 0
- joint Torso_RightLeg: origin xyz=0.5 -10 2.221984229849567 rpy=0 0 0 -> xyz=0.5 -10 2.4744096996049523 rpy=0 0 0
